Commit message: Add ring

File: kuroko_description/xacro/physics/default_gazebo_params.xacro (robot description, xacro)
@@ -43,3 +43,9 @@
 		</gazebo>
 	</xacro:macro>
+	<xacro:macro name="preserve_fixed_joint" params="joint_name">
+		<gazebo reference="${joint_name}">
+			<disableFixedJointLumping>true</disableFixedJointLumping>
+			<preserveFixedJoint>true</preserveFixedJoint>
+		</gazebo>
+	</xacro:macro>
 </robot>

File: kuroko_description/xacro/roboone_ring/large_ring.xacro (robot description, xacro)
@@ -3,5 +3,5 @@
 	<xacro:include filename="./large_ring.gazebo" />
 	<xacro:macro name="large_ring">
-		<link name="large_ring_link0">
+		<link name="ring_link">
 			<collision>
 				<origin xyz="0 0 -0.97" rpy="0 0 0" />

File: kuroko_description/xacro/roboone_ring/small_ring.xacro (robot description, xacro)
@@ -3,5 +3,5 @@
 	<xacro:include filename="./small_ring.gazebo" />
 	<xacro:macro name="small_ring">
-		<link name="small_ring_link0">
+		<link name="ring_link">
 			<collision>
 				<origin xyz="0 0 -0.97" rpy="0 0 0" />

Commit message: Edit joint stiffness

File: kuroko_description/xacro/physics/default_gazebo_params.xacro (robot description, xacro)
@@ -40,5 +40,16 @@
 	<xacro:macro name="implicit_joint" params="joint_name">
 		<gazebo reference="${joint_name}">
-			<implicitSpringDamper>1</implicitSpringDamper>
+			<physics>
+				<ode>
+					<implicit_spring_damper>1</implicit_spring_damper>
+					<cfm_damping>0</cfm_damping>
+					<cfm>1e-7</cfm>
+					<erp>0.8</erp>
+					<limit>
+						<cfm>1e-7</cfm>
+						<erp>0.8</erp>
+					</limit>
+				</ode>
+			</physics>
 		</gazebo>
 	</xacro:macro>

File: kuroko_description/xacro/physics/gazebo_passive_joint.xacro (robot description, xacro)
@@ -24,4 +24,6 @@
 						<implicit_spring_damper>1</implicit_spring_damper>
 						<cfm_damping>0</cfm_damping>
+						<cfm>1e-7</cfm>
+						<erp>0.8</erp>
 						<limit>
 							<cfm>1e-7</cfm>
