Commit message: Change joint name waist -> chest

File: kuroko_description/xacro/kuroko/parts/body.xacro (robot description, xacro)
@@ -15,5 +15,5 @@
     </link>
     <!-- Joint1 -->
-    <joint name="waist" type="revolute">
+    <joint name="chest" type="revolute">
       <parent link="waist_link"/>
       <child link="chest_link"/>
