Commit message: add leg

File: kuroko_description/xacro/kuroko/parts/leg_r.xacro (robot description, xacro)
@@ -62,5 +62,5 @@
 			<parent link="thigh_r_01" />
 			<child link="thigh_r_03" />
-			<origin xyz="-0.015 -0.02925 -0.0305" rpy="0 0 0" />
+			<origin xyz="-0.0185 -0.02925 -0.0305" rpy="0 0 0" />
 			<axis xyz="0 1 0" />
 			<limit effort="1000.0" lower="-3.1" upper="3.1" velocity="10.0" />
@@ -81,9 +81,9 @@
 			<parent link="thigh_r_01" />
 			<child link="thigh_r_04" />
-			<origin xyz="-0.015 -0.02925 -0.0305" rpy="0 0 0" />
+			<origin xyz="-0.0185 -0.02925 -0.0305" rpy="0 0 0" />
 			<axis xyz="0 1 0" />
 			<limit effort="1000.0" lower="-3.1" upper="3.1" velocity="10.0" />
 			<dynamics damping="0.0" friction="0.0" />
-			<mimic joint="thigh_r_02_joint" multiplier="1" offset="0"/>
+			<mimic joint="thigh_r_02_joint" multiplier="1" offset="0" />
 		</joint>
 		<link name="thigh_r_04">
@@ -97,4 +97,52 @@
 			<xacro:box_inertial xyz="0 0 -0.05" rpy="0 0 0" size="0.014 0.0345 0.114" mass="0.011" />
 		</link>
+		<joint name="thigh_r_05_mimic_joint" type="revolute">
+			<parent link="thigh_r_03" />
+			<child link="thigh_r_05_mimic" />
+			<origin xyz="0 0 -0.03" rpy="0 0 0" />
+			<axis xyz="0 1 0" />
+			<limit effort="1000.0" lower="-3.1" upper="3.1" velocity="10.0" />
+			<dynamics damping="0.0" friction="0.0" />
+			<mimic joint="thigh_r_03_joint" multiplier="-1" offset="0" />
+		</joint>
+		<link name="thigh_r_05_mimic" />
+		<joint name="thigh_r_05_joint" type="revolute">
+			<parent link="thigh_r_05_mimic" />
+			<child link="thigh_r_05" />
+			<origin xyz="0 0 0" rpy="0 0 0" />
+			<axis xyz="0 1 0" />
+			<limit effort="1000.0" lower="-3.1" upper="3.1" velocity="10.0" />
+			<dynamics damping="0.0" friction="0.0" />
+			<mimic joint="thigh_r_02_joint" multiplier="1" offset="0" />
+		</joint>
+		<link name="thigh_r_05">
+			<visual>
+				<origin xyz="0 0 0" rpy="0 0 0" />
+				<geometry>
+					<mesh filename="package://kuroko_description/meshes/kuroko/obj/thigh_r_05.obj" />
+				</geometry>
+			</visual>
+			<xacro:box_collision xyz="0 0 -0.05" rpy="0 0 0" size="0.014 0.0285 0.114" />
+			<xacro:box_inertial xyz="0 0 -0.05" rpy="0 0 0" size="0.014 0.0285 0.114" mass="0.011" />
+		</link>
+		<joint name="knee_r_joint" type="revolute">
+			<parent link="thigh_r_02" />
+			<child link="knee_r" />
+			<origin xyz="0 0 -0.1" rpy="0 0 0" />
+			<axis xyz="0 1 0" />
+			<limit effort="1000.0" lower="-3.1" upper="3.1" velocity="10.0" />
+			<dynamics damping="0.0" friction="0.0" />
+			<mimic joint="thigh_r_02_joint" multiplier="-1" offset="0" />
+		</joint>
+		<link name="knee_r">
+			<visual>
+				<origin xyz="0 0 0" rpy="0 0 0" />
+				<geometry>
+					<mesh filename="package://kuroko_description/meshes/kuroko/obj/knee_r.obj" />
+				</geometry>
+			</visual>
+			<xacro:box_collision xyz="-0.01675 0 0" rpy="0 0 0" size="0.0475 0.0505 0.014" />
+			<xacro:box_inertial xyz="-0.01675 0 0" rpy="0 0 0" size="0.0475 0.0505 0.014" mass="0.0054" />
+		</link>
 	</xacro:macro>
 </robot>

Commit message: Fix params

File: kuroko_description/xacro/kuroko/parts/leg_r.xacro (robot description, xacro)
@@ -132,5 +132,5 @@
 			</joint>
 			<xacro:gazebo_poassive_joint name="thigh_r_05_loop" xyz="-0.00765471 0 -0.02897777"
-				parent="leg_r_02" child="thigh_r_05"/>
+				parent="leg_r_02" child="thigh_r_05" />
 		</xacro:if>
 		<link name="thigh_r_05">

File: kuroko_description/xacro/physics/default_gazebo_params.xacro (robot description, xacro)
@@ -3,5 +3,5 @@
 	<xacro:macro name="default_motor_transmission" params="joint_name gazebo_hw_interface">
 		<gazebo reference="${joint_name}">
-  		    <implicitSpringDamper>1</implicitSpringDamper>
+			<implicitSpringDamper>1</implicitSpringDamper>
 		</gazebo>
 		<transmission name="${joint_name}_trans">
@@ -20,5 +20,5 @@
 				</xacro:if>
 				<xacro:if value="${gazebo_hw_interface=='position'}">
-                    <hardwareInterface>hardware_interface/PositionJointInterface</hardwareInterface>
+					<hardwareInterface>hardware_interface/PositionJointInterface</hardwareInterface>
 				</xacro:if>
 				<mechanicalReduction>1</mechanicalReduction>
@@ -38,7 +38,7 @@
 		</gazebo>
 	</xacro:macro>
-	<xacro:macro name="default_passive_joint" params="joint_name">
+	<xacro:macro name="implicit_joint" params="joint_name">
 		<gazebo reference="${joint_name}">
-  		    <implicitSpringDamper>1</implicitSpringDamper>
+			<implicitSpringDamper>1</implicitSpringDamper>
 		</gazebo>
 	</xacro:macro>

Commit message: Update right leg joint tree

File: kuroko_description/xacro/kuroko/parts/leg_r.xacro (robot description, xacro)
@@ -41,4 +41,23 @@
         mass="0.478"/>
     </link>
+    <joint name="shin_r_active" type="revolute">
+      <parent link="hip_r_pitch_link"/>
+      <child link="shin_r_active_link"/>
+      <origin xyz="-0.0185 -0.02925 -0.0305" rpy="0 1.047197551 0"/>
+      <axis xyz="0 1 0"/>
+      <limit effort="8.9" lower="-1.8588" upper="0.4974" velocity="6.9"/>
+      <dynamics damping="1.29" friction="0.0"/>
+    </joint>
+    <link name="shin_r_active_link">
+      <visual>
+        <origin xyz="0 0 0" rpy="0 0 0"/>
+        <geometry>
+          <mesh filename="package://kuroko_description/meshes/kuroko/obj/shin_r_active.obj"/>
+        </geometry>
+      </visual>
+      <xacro:box_collision xyz="-0.004745 0 -0.015" rpy="0 0 0" size="0.02349 0.0445 0.044"/>
+      <xacro:box_inertial xyz="-0.004745 0 -0.015" rpy="0 0 0" size="0.02349 0.0445 0.044"
+        mass="0.008"/>
+    </link>
     <joint name="thigh_r_active" type="revolute">
       <parent link="hip_r_pitch_link"/>
@@ -46,6 +65,6 @@
       <origin xyz="0.015 -0.02925 -0.0305" rpy="0 -0.785398163 0"/>
       <axis xyz="0 1 0"/>
-      <limit effort="1000.0" lower="-0.4974" upper="1.8588" velocity="10.0"/>
-      <dynamics damping="0.0" friction="0.0"/>
+      <limit effort="8.9" lower="-0.4974" upper="1.8588" velocity="6.9"/>
+      <dynamics damping="1.29" friction="0.0"/>
     </joint>
     <link name="thigh_r_active_link">
@@ -59,22 +78,44 @@
       <xacro:box_inertial xyz="0 0 -0.05" rpy="0 0 0" size="0.014 0.0445 0.114" mass="0.012"/>
     </link>
-    <joint name="shin_r_active" type="revolute">
-      <parent link="hip_r_pitch_link"/>
-      <child link="shin_r_active_link"/>
-      <origin xyz="-0.0185 -0.02925 -0.0305" rpy="0 1.047197551 0"/>
-      <axis xyz="0 1 0"/>
-      <limit effort="1000.0" lower="-1.8588" upper="0.4974" velocity="10.0"/>
-      <dynamics damping="0.0" friction="0.0"/>
-    </joint>
-    <link name="shin_r_active_link">
-      <visual>
-        <origin xyz="0 0 0" rpy="0 0 0"/>
-        <geometry>
-          <mesh filename="package://kuroko_description/meshes/kuroko/obj/shin_r_active.obj"/>
-        </geometry>
-      </visual>
-      <xacro:box_collision xyz="-0.004745 0 -0.015" rpy="0 0 0" size="0.02349 0.0445 0.044"/>
-      <xacro:box_inertial xyz="-0.004745 0 -0.015" rpy="0 0 0" size="0.02349 0.0445 0.044"
-        mass="0.008"/>
+    <xacro:unless value="$(arg gazebo)">
+      <joint name="shin_r_front_mimic" type="revolute">
+        <parent link="thigh_r_active_link"/>
+        <child link="shin_r_front_mimic_link"/>
+        <origin xyz="0 0 -0.1" rpy="0 0.785398163 0"/>
+        <axis xyz="0 1 0"/>
+        <limit effort="0" lower="-3.1416" upper="3.1416" velocity="1000"/>
+        <dynamics damping="0.0" friction="0.0"/>
+        <mimic joint="thigh_r_active" multiplier="-1" offset="0"/>
+      </joint>
+      <link name="shin_r_front_mimic_link"/>
+      <joint name="shin_r_front_passive" type="revolute">
+        <parent link="shin_r_front_mimic_link"/>
+        <child link="shin_r_front_passive_link"/>
+        <origin xyz="0 0 0" rpy="0 0.785398163 0"/>
+        <axis xyz="0 1 0"/>
+        <limit effort="0" lower="-3.1416" upper="3.1416" velocity="1000"/>
+        <dynamics damping="0.0" friction="0.0"/>
+        <mimic joint="shin_r_active" multiplier="1" offset="0"/>
+      </joint>
+    </xacro:unless>
+    <xacro:if value="$(arg gazebo)">
+      <joint name="shin_r_front_passive" type="revolute">
+        <parent link="thigh_r_active_link"/>
+        <child link="shin_r_front_passive_link"/>
+        <origin xyz="0 0 -0.1" rpy="0 1.570796327 0"/>
+        <axis xyz="0 1 0"/>
+        <limit effort="0" lower="-1.570796327" upper="0.9948" velocity="1000.0"/>
+        <dynamics damping="0.0" friction="0.0"/>
+      </joint>
+    </xacro:if>
+    <link name="shin_r_front_passive_link">
+      <visual>
+        <origin xyz="0 0 0" rpy="0 0 0"/>
+        <geometry>
+          <mesh filename="package://kuroko_description/meshes/kuroko/obj/shin_r_front_passive.obj"/>
+        </geometry>
+      </visual>
+      <xacro:box_collision xyz="0 0 -0.05" rpy="0 0 0" size="0.014 0.0385 0.114"/>
+      <xacro:box_inertial xyz="0 0 -0.05" rpy="0 0 0" size="0.014 0.0385 0.114" mass="0.013"/>
     </link>
     <joint name="thigh_r_middle_passive" type="revolute">
@@ -83,12 +124,8 @@
       <origin xyz="-0.0185 -0.02925 -0.0305" rpy="0 -0.785398163 0"/>
       <axis xyz="0 1 0"/>
-      <limit effort="1000.0" lower="-3.1" upper="3.1" velocity="10.0"/>
-      <dynamics damping="0.0" friction="0.0"/>
+      <limit effort="0" lower="-0.4974" upper="1.8588" velocity="1000"/>
+      <dynamics damping="0" friction="0"/>
       <mimic joint="thigh_r_active" multiplier="1" offset="0"/>
     </joint>
-    <xacro:if value="$(arg gazebo)">
-      <xacro:gazebo_poassive_joint name="thigh_r_middle_passive_loop" xyz="-0.0335 0 0"
-        parent="knee_r_passive_link" child="thigh_r_middle_passive_link"/>
-    </xacro:if>
     <link name="thigh_r_middle_passive_link">
       <visual>
@@ -102,96 +139,33 @@
     </link>
     <xacro:unless value="$(arg gazebo)">
-      <joint name="thigh_r_rear_passive_mimic" type="revolute">
-        <parent link="shin_r_active_link"/>
-        <child link="thigh_r_rear_passive_mimic_link"/>
-        <origin xyz="0 0 -0.03" rpy="0 -1.832597551 0"/>
-        <axis xyz="0 1 0"/>
-        <limit effort="1000.0" lower="-3.1" upper="3.1" velocity="10.0"/>
-        <dynamics damping="0.0" friction="0.0"/>
-        <mimic joint="shin_r_active" multiplier="-1" offset="0"/>
-      </joint>
-      <link name="thigh_r_rear_passive_mimic_link"/>
-      <joint name="thigh_r_rear_passive" type="revolute">
-        <parent link="thigh_r_rear_passive_mimic_link"/>
-        <child link="thigh_r_rear_passive_link"/>
-        <origin xyz="0 0 0" rpy="0 0 0"/>
-        <axis xyz="0 1 0"/>
-        <limit effort="1000.0" lower="-3.1" upper="3.1" velocity="10.0"/>
-        <dynamics damping="0.0" friction="0.0"/>
-        <mimic joint="thigh_r_active" multiplier="1" offset="0"/>
+      <joint name="shin_r_rear_mimic" type="revolute">
+        <parent link="thigh_r_middle_passive_link"/>
+        <child link="shin_r_rear_mimic_link"/>
+        <origin xyz="0 0 -0.1" rpy="0 0.785398163 0"/>
+        <axis xyz="0 1 0"/>
+        <limit effort="0" lower="-3.1416" upper="3.1416" velocity="1000"/>
+        <dynamics damping="0.0" friction="0.0"/>
+        <mimic joint="thigh_r_active" multiplier="-1" offset="0"/>
+      </joint>
+      <link name="shin_r_rear_mimic_link"/>
+      <joint name="shin_r_rear_passive" type="revolute">
+        <parent link="shin_r_rear_mimic_link"/>
+        <child link="shin_r_rear_passive_link"/>
+        <origin xyz="0 0 0" rpy="0 0.785398163 0"/>
+        <axis xyz="0 1 0"/>
+        <limit effort="0" lower="-3.1416" upper="3.1416" velocity="1000"/>
+        <dynamics damping="0.0" friction="0.0"/>
+        <mimic joint="shin_r_active" multiplier="1" offset="0"/>
       </joint>
     </xacro:unless>
     <xacro:if value="$(arg gazebo)">
-      <joint name="thigh_r_rear_passive" type="revolute">
-        <parent link="shin_r_active_link"/>
-        <child link="thigh_r_rear_passive_link"/>
-        <origin xyz="0 0 -0.03" rpy="0 -1.832597551 0"/>
-        <axis xyz="0 1 0"/>
-        <limit effort="1000.0" lower="-0.9948" upper="1.5708" velocity="10.0"/>
-        <dynamics damping="0.0" friction="0.0"/>
-      </joint>
-      <xacro:gazebo_poassive_joint name="thigh_r_rear_passive_loop" xyz="-0.00765471 0 -0.02897777"
-        parent="shin_r_rear_passive_link" child="thigh_r_rear_passive_link"/>
-    </xacro:if>
-    <link name="thigh_r_rear_passive_link">
-      <visual>
-        <origin xyz="0 0 0" rpy="0 0 0"/>
-        <geometry>
-          <mesh filename="package://kuroko_description/meshes/kuroko/obj/thigh_r_rear_passive.obj"/>
-        </geometry>
-      </visual>
-      <xacro:box_collision xyz="0 0 -0.05" rpy="0 0 0" size="0.014 0.0285 0.114"/>
-      <xacro:box_inertial xyz="0 0 -0.05" rpy="0 0 0" size="0.014 0.0285 0.114" mass="0.011"/>
-    </link>
-    <joint name="knee_r_passive" type="revolute">
-      <parent link="thigh_r_active_link"/>
-      <child link="knee_r_passive_link"/>
-      <origin xyz="0 0 -0.1" rpy="0 0.785398163 0"/>
-      <axis xyz="0 1 0"/>
-      <limit effort="1000.0" lower="-1.8588" upper="0.4974" velocity="10.0"/>
-      <dynamics damping="0.0" friction="0.0"/>
-      <mimic joint="thigh_r_active" multiplier="-1" offset="0"/>
-    </joint>
-    <link name="knee_r_passive_link">
-      <visual>
-        <origin xyz="0 0 0" rpy="0 0 0"/>
-        <geometry>
-          <mesh filename="package://kuroko_description/meshes/kuroko/obj/knee_r_passive.obj"/>
-        </geometry>
-      </visual>
-      <xacro:box_collision xyz="-0.01675 0 0" rpy="0 0 0" size="0.0475 0.0505 0.014"/>
-      <xacro:box_inertial xyz="-0.01675 0 0" rpy="0 0 0" size="0.0475 0.0505 0.014" mass="0.007"/>
-    </link>
-    <joint name="shin_r_front_passive" type="revolute">
-      <parent link="knee_r_passive_link"/>
-      <child link="shin_r_front_passive_link"/>
-      <origin xyz="0 0 0" rpy="0 0.785398163 0"/>
-      <axis xyz="0 1 0"/>
-      <limit effort="1000.0" lower="-1.8588" upper="0.4974" velocity="10.0"/>
-      <dynamics damping="0.0" friction="0.0"/>
-      <mimic joint="shin_r_active" multiplier="1" offset="0"/>
-    </joint>
-    <link name="shin_r_front_passive_link">
-      <visual>
-        <origin xyz="0 0 0" rpy="0 0 0"/>
-        <geometry>
-          <mesh filename="package://kuroko_description/meshes/kuroko/obj/shin_r_front_passive.obj"/>
-        </geometry>
-      </visual>
-      <xacro:box_collision xyz="0 0 -0.05" rpy="0 0 0" size="0.014 0.0385 0.114"/>
-      <xacro:box_inertial xyz="0 0 -0.05" rpy="0 0 0" size="0.014 0.0385 0.114" mass="0.013"/>
-    </link>
-    <joint name="shin_r_rear_passive" type="revolute">
-      <parent link="knee_r_passive_link"/>
-      <child link="shin_r_rear_passive_link"/>
-      <origin xyz="-0.0335 0 0" rpy="0 0.785398163 0"/>
-      <axis xyz="0 1 0"/>
-      <limit effort="1000.0" lower="-1.8588" upper="0.4974" velocity="10.0"/>
-      <dynamics damping="0.0" friction="0.0"/>
-      <mimic joint="shin_r_active" multiplier="1" offset="0"/>
-    </joint>
-    <xacro:if value="$(arg gazebo)">
-      <xacro:gazebo_poassive_joint name="shin_r_rear_passive_loop" xyz="-0.0335 0 0"
-        parent="ankle_r_pitch_passive_link" child="shin_r_rear_passive_link"/>
+      <joint name="shin_r_rear_passive" type="revolute">
+        <parent link="thigh_r_middle_passive_link"/>
+        <child link="shin_r_rear_passive_link"/>
+        <origin xyz="0 0 -0.1" rpy="0 1.570796327 0"/>
+        <axis xyz="0 1 0"/>
+        <limit effort="0" lower="-1.570796327" upper="0.9948" velocity="1000.0"/>
+        <dynamics damping="0.0" friction="0.0"/>
+      </joint>
     </xacro:if>
     <link name="shin_r_rear_passive_link">
@@ -205,28 +179,100 @@
       <xacro:box_inertial xyz="0 0 -0.05" rpy="0 0 0" size="0.014 0.0445 0.114" mass="0.016"/>
     </link>
-    <joint name="ankle_r_pitch_passive" type="revolute">
-      <parent link="shin_r_front_passive_link"/>
-      <child link="ankle_r_pitch_passive_link"/>
+    <joint name="knee_r_rear_passive" type="revolute">
+      <parent link="shin_r_rear_passive_link"/>
+      <child link="knee_r_passive_link"/>
+      <origin xyz="0 0 0" rpy="0 -0.785398164 0"/>
+      <axis xyz="0 1 0"/>
+      <limit effort="0" lower="-3.141592654" upper="3.141592654" velocity="1000.0"/>
+      <dynamics damping="0.0" friction="0.0"/>
+      <mimic joint="shin_r_active" multiplier="-1" offset="0"/>
+    </joint>
+    <link name="knee_r_passive_link">
+      <visual>
+        <origin xyz="0.0335 0 0" rpy="0 0 0"/>
+        <geometry>
+          <mesh filename="package://kuroko_description/meshes/kuroko/obj/knee_r_passive.obj"/>
+        </geometry>
+      </visual>
+      <xacro:box_collision xyz="0.01675 0 0" rpy="0 0 0" size="0.0475 0.0505 0.014"/>
+      <xacro:box_inertial xyz="0.01675 0 0" rpy="0 0 0" size="0.0475 0.0505 0.014" mass="0.007"/>
+    </link>
+    <xacro:if value="$(arg gazebo)">
+      <xacro:gazebo_poassive_joint name="knee_r_front_passive_loop" xyz="0.0335 0 0"
+        parent="knee_r_passive_link" child="thigh_r_active_link" axis="0 1 0" lower="-1.8588" upper="0.4974"/>
+    </xacro:if>
+    <xacro:unless value="$(arg gazebo)">
+      <joint name="thigh_r_rear_mimic" type="revolute">
+        <parent link="shin_r_rear_passive_link"/>
+        <child link="thigh_r_rear_mimic_link"/>
+        <origin xyz="-0.00776457 0 -0.0289778" rpy="0 -0.785398163 0"/>
+        <axis xyz="0 1 0"/>
+        <limit effort="0" lower="-3.1416" upper="3.1416" velocity="1000"/>
+        <dynamics damping="0.0" friction="0.0"/>
+        <mimic joint="thigh_r_active" multiplier="1" offset="0"/>
+      </joint>
+      <link name="thigh_r_rear_mimic_link"/>
+      <joint name="thigh_r_rear_passive" type="revolute">
+        <parent link="thigh_r_rear_mimic_link"/>
+        <child link="thigh_r_rear_passive_link"/>
+        <origin xyz="0 0 0" rpy="0 -0.785398163 0"/>
+        <axis xyz="0 1 0"/>
+        <limit effort="0" lower="-3.1416" upper="3.1416" velocity="1000"/>
+        <dynamics damping="0.0" friction="0.0"/>
+        <mimic joint="shin_r_active" multiplier="-1" offset="0"/>
+      </joint>
+    </xacro:unless>
+    <xacro:if value="$(arg gazebo)">
+      <joint name="thigh_r_rear_passive" type="revolute">
+        <parent link="shin_r_rear_passive_link"/>
+        <child link="thigh_r_rear_passive_link"/>
+        <origin xyz="-0.00776457 0 -0.0289778" rpy="0 -1.570796327 0"/>
+        <axis xyz="0 1 0"/>
+        <limit effort="0" lower="-0.9948" upper="1.570796327" velocity="1000.0"/>
+        <dynamics damping="0.0" friction="0.0"/>
+      </joint>
+    </xacro:if>
+    <link name="thigh_r_rear_passive_link">
+      <visual>
+        <origin xyz="0 0 0.1" rpy="0 0 0"/>
+        <geometry>
+          <mesh filename="package://kuroko_description/meshes/kuroko/obj/thigh_r_rear_passive.obj"/>
+        </geometry>
+      </visual>
+      <xacro:box_collision xyz="0 0 0.05" rpy="0 0 0" size="0.014 0.0285 0.114"/>
+      <xacro:box_inertial xyz="0 0 0.05" rpy="0 0 0" size="0.014 0.0285 0.114" mass="0.011"/>
+    </link>
+    <xacro:if value="$(arg gazebo)">
+      <xacro:gazebo_poassive_joint name="thigh_r_rear_passive_loop" xyz="0 0 0.1" rpy="0 1.832597551 0"
+        parent="thigh_r_rear_passive_link" child="shin_r_active_link" axis="0 1 0"/>
+    </xacro:if>
+    <joint name="ankle_r_rear_passive" type="revolute">
+      <parent link="shin_r_rear_passive_link"/>
+      <child link="ankle_r_rear_passive_link"/>
       <origin xyz="0 0 -0.1" rpy="0 -0.785398163 0"/>
       <axis xyz="0 1 0"/>
-      <limit effort="1000.0" lower="-0.4974" upper="1.8588" velocity="10.0"/>
+      <limit effort="0" lower="-0.4974" upper="1.8588" velocity="1000.0"/>
       <dynamics damping="0.0" friction="0.0"/>
       <mimic joint="shin_r_active" multiplier="-1" offset="0"/>
     </joint>
-    <link name="ankle_r_pitch_passive_link">
-      <visual>
-        <origin xyz="0 0 0" rpy="0 0 0"/>
+    <link name="ankle_r_rear_passive_link">
+      <visual>
+        <origin xyz="0.0335 0 0" rpy="0 0 0"/>
         <geometry>
           <mesh filename="package://kuroko_description/meshes/kuroko/obj/ankle_r_pitch_passive.obj"/>
         </geometry>
       </visual>
-      <xacro:box_collision xyz="-0.0285 0 -0.013" rpy="0 0 0" size="0.0855 0.0325 0.0465"/>
-      <xacro:box_inertial xyz="-0.0285 0 -0.013" rpy="0 0 0" size="0.0855 0.0325 0.0465"
+      <xacro:box_collision xyz="0.005 0 -0.013" rpy="0 0 0" size="0.0855 0.0325 0.0465"/>
+      <xacro:box_inertial xyz="0.005 0 -0.013" rpy="0 0 0" size="0.0855 0.0325 0.0465"
         mass="0.104"/>
     </link>
+    <xacro:if value="$(arg gazebo)">
+      <xacro:gazebo_poassive_joint name="ankle_r_front_passive_loop" xyz="0.0335 0 0" rpy="0 -0.785398163 0"
+        parent="ankle_r_rear_passive_link" child="shin_r_front_passive_link" axis="0 1 0"/>
+    </xacro:if>
     <joint name="ankle_r_roll" type="revolute">
-      <parent link="ankle_r_pitch_passive_link"/>
+      <parent link="ankle_r_rear_passive_link"/>
       <child link="ankle_r_roll_link"/>
-      <origin xyz="-0.015 0 -0.027" rpy="0 0 0"/>
+      <origin xyz="0.0185 0 -0.027" rpy="0 0 0"/>
       <axis xyz="1 0 0"/>
       <limit effort="1000.0" lower="-0.3704" upper="1.5708" velocity="10.0"/>
