Commit message: Fix directions and limits

File: kuroko_description/xacro/kuroko/parts/arm_l.xacro (robot description, xacro)
@@ -26,5 +26,5 @@
 			<origin xyz="0 0.028 0" rpy="0 0 0" />
 			<axis xyz="-1 0 0" />
-			<limit effort="1000.0" lower="-3.1" upper="3.1" velocity="10.0" />
+			<limit effort="1000.0" lower="-2.0071" upper="1.0472" velocity="10.0" />
 			<dynamics damping="0.0" friction="0.0" />
 		</joint>
@@ -43,6 +43,6 @@
 			<child link="scissor_lf" />
 			<origin xyz="0 0.0265 -0.0545" rpy="0 0 0" />
-			<axis xyz="0 1 0" />
-			<limit effort="1000.0" lower="-3.1" upper="3.1" velocity="10.0" />
+			<axis xyz="0 -1 0" />
+			<limit effort="1000.0" lower="-2.6180" upper="2.6180" velocity="10.0" />
 			<dynamics damping="0.0" friction="0.0" />
 		</joint>
@@ -62,6 +62,6 @@
 			<child link="scissor_lr" />
 			<origin xyz="0 0.0265 -0.0545" rpy="0 0 0" />
-			<axis xyz="0 -1 0" />
-			<limit effort="1000.0" lower="-3.1" upper="3.1" velocity="10.0" />
+			<axis xyz="0 1 0" />
+			<limit effort="1000.0" lower="-2.6180" upper="2.6180" velocity="10.0" />
 			<dynamics damping="0.0" friction="0.0" />
 		</joint>

File: kuroko_description/xacro/kuroko/parts/arm_r.xacro (robot description, xacro)
@@ -26,5 +26,5 @@
 			<origin xyz="0 -0.028 0" rpy="0 0 0" />
 			<axis xyz="-1 0 0" />
-			<limit effort="1000.0" lower="-3.1" upper="3.1" velocity="10.0" />
+			<limit effort="1000.0" lower="-1.0472" upper="2.0071" velocity="10.0" />
 			<dynamics damping="0.0" friction="0.0" />
 		</joint>
@@ -44,6 +44,6 @@
 			<child link="scissor_rf" />
 			<origin xyz="0 -0.0265 -0.0545" rpy="0 0 0" />
-			<axis xyz="0 -1 0" />
-			<limit effort="1000.0" lower="-3.1" upper="3.1" velocity="10.0" />
+			<axis xyz="0 1 0" />
+			<limit effort="1000.0" lower="-2.6180" upper="2.6180" velocity="10.0" />
 			<dynamics damping="0.0" friction="0.0" />
 		</joint>
@@ -63,6 +63,6 @@
 			<child link="scissor_rr" />
 			<origin xyz="0 -0.0265 -0.0545" rpy="0 0 0" />
-			<axis xyz="0 1 0" />
-			<limit effort="1000.0" lower="-3.1" upper="3.1" velocity="10.0" />
+			<axis xyz="0 -1 0" />
+			<limit effort="1000.0" lower="-2.6180" upper="2.6180" velocity="10.0" />
 			<dynamics damping="0.0" friction="0.0" />
 		</joint>

File: kuroko_description/xacro/kuroko/parts/leg_r.xacro (robot description, xacro)
@@ -8,5 +8,5 @@
 			<origin xyz="0.00125 0 -0.08425" rpy="0 0 0" />
 			<axis xyz="1 0 0" />
-			<limit effort="1000.0" lower="-3.1" upper="3.1" velocity="10.0" />
+			<limit effort="1000.0" lower="-0.5550" upper="1.8640" velocity="10.0" />
 			<dynamics damping="0.0" friction="0.0" />
 		</joint>
@@ -46,5 +46,5 @@
 			<origin xyz="0.015 -0.02925 -0.0305" rpy="0 -0.785398163 0" />
 			<axis xyz="0 1 0" />
-			<limit effort="1000.0" lower="-3.1" upper="3.1" velocity="10.0" />
+			<limit effort="1000.0" lower="-0.4974" upper="1.8588" velocity="10.0" />
 			<dynamics damping="0.0" friction="0.0" />
 		</joint>
@@ -64,5 +64,5 @@
 			<origin xyz="-0.0185 -0.02925 -0.0305" rpy="0 1.047197551 0" />
 			<axis xyz="0 1 0" />
-			<limit effort="1000.0" lower="-3.1" upper="3.1" velocity="10.0" />
+			<limit effort="1000.0" lower="-1.8588" upper="0.4974" velocity="10.0" />
 			<dynamics damping="0.0" friction="0.0" />
 		</joint>
@@ -89,5 +89,5 @@
 		<xacro:if value="$(arg gazebo)">
 			<xacro:gazebo_poassive_joint name="thigh_r_04_loop" xyz="-0.0335 0 0"
-				parent="knee_r" child="thigh_r_04" />
+				parent="knee_r" child="thigh_r_04" lower="-1.8588" upper="0.4974" />
 		</xacro:if>
 		<link name="thigh_r_04">
@@ -128,9 +128,9 @@
 				<origin xyz="0 0 -0.03" rpy="0 -1.832597551 0" />
 				<axis xyz="0 1 0" />
-				<limit effort="1000.0" lower="-3.1" upper="3.1" velocity="10.0" />
+				<limit effort="1000.0" lower="-0.7767" upper="1.5708" velocity="10.0" />
 				<dynamics damping="0.0" friction="0.0" />
 			</joint>
 			<xacro:gazebo_poassive_joint name="thigh_r_05_loop" xyz="-0.00765471 0 -0.02897777"
-				parent="leg_r_02" child="thigh_r_05" />
+				parent="leg_r_02" child="thigh_r_05"/>
 		</xacro:if>
 		<link name="thigh_r_05">
@@ -149,5 +149,5 @@
 			<origin xyz="0 0 -0.1" rpy="0 0.785398163 0" />
 			<axis xyz="0 1 0" />
-			<limit effort="1000.0" lower="-3.1" upper="3.1" velocity="10.0" />
+			<limit effort="1000.0" lower="-1.8588" upper="0.4974" velocity="10.0" />
 			<dynamics damping="0.0" friction="0.0" />
 			<mimic joint="thigh_r_02_joint" multiplier="-1" offset="0" />
@@ -168,5 +168,5 @@
 			<origin xyz="0 0 0" rpy="0 0.785398163 0" />
 			<axis xyz="0 1 0" />
-			<limit effort="1000.0" lower="-3.1" upper="3.1" velocity="10.0" />
+			<limit effort="1000.0" lower="-1.8588" upper="0.4974" velocity="10.0" />
 			<dynamics damping="0.0" friction="0.0" />
 			<mimic joint="thigh_r_03_joint" multiplier="1" offset="0" />
@@ -187,5 +187,5 @@
 			<origin xyz="-0.0335 0 0" rpy="0 0.785398163 0" />
 			<axis xyz="0 1 0" />
-			<limit effort="1000.0" lower="-3.1" upper="3.1" velocity="10.0" />
+			<limit effort="1000.0" lower="-1.8588" upper="0.4974" velocity="10.0" />
 			<dynamics damping="0.0" friction="0.0" />
 			<mimic joint="thigh_r_03_joint" multiplier="1" offset="0" />
@@ -210,5 +210,5 @@
 			<origin xyz="0 0 -0.1" rpy="0 -0.785398163 0" />
 			<axis xyz="0 1 0" />
-			<limit effort="1000.0" lower="-3.1" upper="3.1" velocity="10.0" />
+			<limit effort="1000.0" lower="-0.4974" upper="1.8588" velocity="10.0" />
 			<dynamics damping="0.0" friction="0.0" />
 			<mimic joint="thigh_r_03_joint" multiplier="-1" offset="0" />
@@ -230,5 +230,5 @@
 			<origin xyz="-0.015 0 -0.025" rpy="0 0 0" />
 			<axis xyz="1 0 0" />
-			<limit effort="1000.0" lower="-3.1" upper="3.1" velocity="10.0" />
+			<limit effort="1000.0" lower="-0.3704" upper="1.5708" velocity="10.0" />
 			<dynamics damping="0.0" friction="0.0" />
 		</joint>

Commit message: rename links

File: kuroko_description/xacro/kuroko/parts/arm_l.xacro (robot description, xacro)
@@ -3,77 +3,77 @@
   <xacro:macro name="arm_l_xacro">
     <!-- Link conencts from body. Shoulder first. -->
-    <joint name="shoulder_l_joint" type="revolute">
-      <parent link="chest" />
-      <child link="shoulder_l" />
-      <origin xyz="0 0.108 0.01275" rpy="0 0 0" />
-      <axis xyz="0 1 0" />
-      <limit effort="1000.0" lower="-3.1" upper="3.1" velocity="10.0" />
-      <dynamics damping="0.0" friction="0.0" />
+    <joint name="shoulder_l_pitch_joint" type="revolute">
+      <parent link="chest"/>
+      <child link="shoulder_l_pitch"/>
+      <origin xyz="0 0.108 0.01275" rpy="0 0 0"/>
+      <axis xyz="0 1 0"/>
+      <limit effort="1000.0" lower="-3.1" upper="3.1" velocity="10.0"/>
+      <dynamics damping="0.0" friction="0.0"/>
     </joint>
-    <link name="shoulder_l">
+    <link name="shoulder_l_pitch">
       <visual>
-        <origin xyz="0 0 0" rpy="0 0 0" />
+        <origin xyz="0 0 0" rpy="0 0 0"/>
         <geometry>
-          <mesh filename="package://kuroko_description/meshes/kuroko/obj/shoulder_l.obj" />
+          <mesh filename="package://kuroko_description/meshes/kuroko/obj/shoulder_l_pitch.obj"/>
         </geometry>
       </visual>
-      <xacro:box_collision xyz="0 0.0205 0" rpy="0 0 0" size="0.042 0.041 0.04" />
-      <xacro:box_inertial xyz="0 0.0205 0" rpy="0 0 0" size="0.042 0.041 0.04" mass="0.022" />
+      <xacro:box_collision xyz="0 0.0205 0" rpy="0 0 0" size="0.042 0.041 0.04"/>
+      <xacro:box_inertial xyz="0 0.0205 0" rpy="0 0 0" size="0.042 0.041 0.04" mass="0.022"/>
     </link>
     <joint name="arm_l_joint" type="revolute">
-      <parent link="shoulder_l" />
-      <child link="arm_l" />
-      <origin xyz="0 0.028 0" rpy="0 0 0" />
-      <axis xyz="-1 0 0" />
-      <limit effort="1000.0" lower="-2.0071" upper="1.0472" velocity="10.0" />
-      <dynamics damping="0.0" friction="0.0" />
+      <parent link="shoulder_l_pitch"/>
+      <child link="arm_l"/>
+      <origin xyz="0 0.028 0" rpy="0 0 0"/>
+      <axis xyz="-1 0 0"/>
+      <limit effort="1000.0" lower="-2.0071" upper="1.0472" velocity="10.0"/>
+      <dynamics damping="0.0" friction="0.0"/>
     </joint>
     <link name="arm_l">
       <visual>
-        <origin xyz="0 0 0" rpy="0 0 0" />
+        <origin xyz="0 0 0" rpy="0 0 0"/>
         <geometry>
-          <mesh filename="package://kuroko_description/meshes/kuroko/obj/arm_l.obj" />
+          <mesh filename="package://kuroko_description/meshes/kuroko/obj/arm_l.obj"/>
         </geometry>
       </visual>
-      <xacro:box_collision xyz="0 0.0385 -0.02575" rpy="0 0 0" size="0.0285 0.1045 0.08" />
-      <xacro:box_inertial xyz="0 0.0385 -0.02575" rpy="0 0 0" size="0.0285 0.1045 0.08" mass="0.342" />
+      <xacro:box_collision xyz="0 0.0385 -0.02575" rpy="0 0 0" size="0.0285 0.1045 0.08"/>
+      <xacro:box_inertial xyz="0 0.0385 -0.02575" rpy="0 0 0" size="0.0285 0.1045 0.08" mass="0.342"/>
     </link>
     <joint name="scissor_lf_joint" type="revolute">
-      <parent link="arm_l" />
-      <child link="scissor_lf" />
-      <origin xyz="0 0.0265 -0.0545" rpy="0 0 0" />
-      <axis xyz="0 -1 0" />
-      <limit effort="1000.0" lower="-2.6180" upper="2.6180" velocity="10.0" />
-      <dynamics damping="0.0" friction="0.0" />
+      <parent link="arm_l"/>
+      <child link="scissor_lf"/>
+      <origin xyz="0 0.0265 -0.0545" rpy="0 0 0"/>
+      <axis xyz="0 -1 0"/>
+      <limit effort="1000.0" lower="-2.6180" upper="2.6180" velocity="10.0"/>
+      <dynamics damping="0.0" friction="0.0"/>
     </joint>
     <link name="scissor_lf">
       <visual>
-        <origin xyz="0 0 0" rpy="0 0 0" />
+        <origin xyz="0 0 0" rpy="0 0 0"/>
         <geometry>
-          <mesh filename="package://kuroko_description/meshes/kuroko/obj/scissor_lf.obj" />
+          <mesh filename="package://kuroko_description/meshes/kuroko/obj/scissor_lf.obj"/>
         </geometry>
       </visual>
-      <xacro:box_collision xyz="0.0043 0 -0.104" rpy="0 0 0" size="0.01085 0.058 0.208" />
-      <xacro:box_collision xyz="-0.0206 0 -0.201" rpy="0 0 0" size="0.039 0.058 0.014" />
-      <xacro:box_inertial xyz="0.0043 0 -0.104" rpy="0 0 0" size="0.044 0.058 0.208" mass="0.032" />
+      <xacro:box_collision xyz="0.0043 0 -0.104" rpy="0 0 0" size="0.01085 0.058 0.208"/>
+      <xacro:box_collision xyz="-0.0206 0 -0.201" rpy="0 0 0" size="0.039 0.058 0.014"/>
+      <xacro:box_inertial xyz="0.0043 0 -0.104" rpy="0 0 0" size="0.044 0.058 0.208" mass="0.032"/>
     </link>
     <joint name="scissor_lr_joint" type="revolute">
-      <parent link="arm_l" />
-      <child link="scissor_lr" />
-      <origin xyz="0 0.0265 -0.0545" rpy="0 0 0" />
-      <axis xyz="0 1 0" />
-      <limit effort="1000.0" lower="-2.6180" upper="2.6180" velocity="10.0" />
-      <dynamics damping="0.0" friction="0.0" />
+      <parent link="arm_l"/>
+      <child link="scissor_lr"/>
+      <origin xyz="0 0.0265 -0.0545" rpy="0 0 0"/>
+      <axis xyz="0 1 0"/>
+      <limit effort="1000.0" lower="-2.6180" upper="2.6180" velocity="10.0"/>
+      <dynamics damping="0.0" friction="0.0"/>
     </joint>
     <link name="scissor_lr">
       <visual>
-        <origin xyz="0 0 0" rpy="0 0 0" />
+        <origin xyz="0 0 0" rpy="0 0 0"/>
         <geometry>
-          <mesh filename="package://kuroko_description/meshes/kuroko/obj/scissor_lr.obj" />
+          <mesh filename="package://kuroko_description/meshes/kuroko/obj/scissor_lr.obj"/>
         </geometry>
       </visual>
-      <xacro:box_collision xyz="-0.0043 0 -0.1" rpy="0 0 0" size="0.01085 0.044 0.2" />
-      <xacro:box_collision xyz="0.0206 0 -0.193" rpy="0 0 0" size="0.039 0.044 0.014" />
-      <xacro:box_inertial xyz="-0.0043 0 -0.1" rpy="0 0 0" size="0.044 0.044 0.2" mass="0.031" />
+      <xacro:box_collision xyz="-0.0043 0 -0.1" rpy="0 0 0" size="0.01085 0.044 0.2"/>
+      <xacro:box_collision xyz="0.0206 0 -0.193" rpy="0 0 0" size="0.039 0.044 0.014"/>
+      <xacro:box_inertial xyz="-0.0043 0 -0.1" rpy="0 0 0" size="0.044 0.044 0.2" mass="0.031"/>
     </link>
   </xacro:macro>

File: kuroko_description/xacro/kuroko/parts/arm_r.xacro (robot description, xacro)
@@ -3,78 +3,78 @@
   <xacro:macro name="arm_r_xacro">
     <!-- Link conencts from body. Shoulder first. -->
-    <joint name="shoulder_r_joint" type="revolute">
-      <parent link="chest" />
-      <child link="shoulder_r" />
-      <origin xyz="0 -0.108 0.01275" rpy="0 0 0" />
-      <axis xyz="0 -1 0" />
-      <limit effort="1000.0" lower="-3.1" upper="3.1" velocity="10.0" />
-      <dynamics damping="0.0" friction="0.0" />
+    <joint name="shoulder_r_pitch_joint" type="revolute">
+      <parent link="chest"/>
+      <child link="shoulder_r_pitch"/>
+      <origin xyz="0 -0.108 0.01275" rpy="0 0 0"/>
+      <axis xyz="0 -1 0"/>
+      <limit effort="1000.0" lower="-3.1" upper="3.1" velocity="10.0"/>
+      <dynamics damping="0.0" friction="0.0"/>
     </joint>
-    <link name="shoulder_r">
+    <link name="shoulder_r_pitch">
       <visual>
-        <origin xyz="0 0 0" rpy="0 0 0" />
+        <origin xyz="0 0 0" rpy="0 0 0"/>
         <geometry>
-          <mesh filename="package://kuroko_description/meshes/kuroko/obj/shoulder_r.obj" />
+          <mesh filename="package://kuroko_description/meshes/kuroko/obj/shoulder_r_pitch.obj"/>
         </geometry>
       </visual>
-      <xacro:box_collision xyz="0 -0.0205 0" rpy="0 0 0" size="0.042 0.041 0.04" />
-      <xacro:box_inertial xyz="0 -0.0205 0" rpy="0 0 0" size="0.042 0.041 0.04" mass="0.022" />
+      <xacro:box_collision xyz="0 -0.0205 0" rpy="0 0 0" size="0.042 0.041 0.04"/>
+      <xacro:box_inertial xyz="0 -0.0205 0" rpy="0 0 0" size="0.042 0.041 0.04" mass="0.022"/>
     </link>
     <joint name="arm_r_joint" type="revolute">
-      <parent link="shoulder_r" />
-      <child link="arm_r" />
-      <origin xyz="0 -0.028 0" rpy="0 0 0" />
-      <axis xyz="-1 0 0" />
-      <limit effort="1000.0" lower="-1.0472" upper="2.0071" velocity="10.0" />
-      <dynamics damping="0.0" friction="0.0" />
+      <parent link="shoulder_r_pitch"/>
+      <child link="arm_r"/>
+      <origin xyz="0 -0.028 0" rpy="0 0 0"/>
+      <axis xyz="-1 0 0"/>
+      <limit effort="1000.0" lower="-1.0472" upper="2.0071" velocity="10.0"/>
+      <dynamics damping="0.0" friction="0.0"/>
     </joint>
     <link name="arm_r">
       <visual>
-        <origin xyz="0 0 0" rpy="0 0 0" />
+        <origin xyz="0 0 0" rpy="0 0 0"/>
         <geometry>
-          <mesh filename="package://kuroko_description/meshes/kuroko/obj/arm_r.obj" />
+          <mesh filename="package://kuroko_description/meshes/kuroko/obj/arm_r.obj"/>
         </geometry>
       </visual>
-      <xacro:box_collision xyz="0 -0.0385 -0.02575" rpy="0 0 0" size="0.0285 0.1045 0.08" />
+      <xacro:box_collision xyz="0 -0.0385 -0.02575" rpy="0 0 0" size="0.0285 0.1045 0.08"/>
       <xacro:box_inertial xyz="0 -0.0385 -0.02575" rpy="0 0 0" size="0.0285 0.1045 0.08"
-        mass="0.342" />
+        mass="0.342"/>
     </link>
     <joint name="scissor_rf_joint" type="revolute">
-      <parent link="arm_r" />
-      <child link="scissor_rf" />
-      <origin xyz="0 -0.0265 -0.0545" rpy="0 0 0" />
-      <axis xyz="0 1 0" />
-      <limit effort="1000.0" lower="-2.6180" upper="2.6180" velocity="10.0" />
-      <dynamics damping="0.0" friction="0.0" />
+      <parent link="arm_r"/>
+      <child link="scissor_rf"/>
+      <origin xyz="0 -0.0265 -0.0545" rpy="0 0 0"/>
+      <axis xyz="0 1 0"/>
+      <limit effort="1000.0" lower="-2.6180" upper="2.6180" velocity="10.0"/>
+      <dynamics damping="0.0" friction="0.0"/>
     </joint>
     <link name="scissor_rf">
       <visual>
-        <origin xyz="0 0 0" rpy="0 0 0" />
+        <origin xyz="0 0 0" rpy="0 0 0"/>
         <geometry>
-          <mesh filename="package://kuroko_description/meshes/kuroko/obj/scissor_rf.obj" />
+          <mesh filename="package://kuroko_description/meshes/kuroko/obj/scissor_rf.obj"/>
         </geometry>
       </visual>
-      <xacro:box_collision xyz="0.0043 0 -0.104" rpy="0 0 0" size="0.01085 0.058 0.208" />
-      <xacro:box_collision xyz="-0.0206 0 -0.201" rpy="0 0 0" size="0.039 0.058 0.014" />
-      <xacro:box_inertial xyz="0.0043 0 -0.104" rpy="0 0 0" size="0.044 0.058 0.208" mass="0.032" />
+      <xacro:box_collision xyz="0.0043 0 -0.104" rpy="0 0 0" size="0.01085 0.058 0.208"/>
+      <xacro:box_collision xyz="-0.0206 0 -0.201" rpy="0 0 0" size="0.039 0.058 0.014"/>
+      <xacro:box_inertial xyz="0.0043 0 -0.104" rpy="0 0 0" size="0.044 0.058 0.208" mass="0.032"/>
     </link>
     <joint name="scissor_rr_joint" type="revolute">
-      <parent link="arm_r" />
-      <child link="scissor_rr" />
-      <origin xyz="0 -0.0265 -0.0545" rpy="0 0 0" />
-      <axis xyz="0 -1 0" />
-      <limit effort="1000.0" lower="-2.6180" upper="2.6180" velocity="10.0" />
-      <dynamics damping="0.0" friction="0.0" />
+      <parent link="arm_r"/>
+      <child link="scissor_rr"/>
+      <origin xyz="0 -0.0265 -0.0545" rpy="0 0 0"/>
+      <axis xyz="0 -1 0"/>
+      <limit effort="1000.0" lower="-2.6180" upper="2.6180" velocity="10.0"/>
+      <dynamics damping="0.0" friction="0.0"/>
     </joint>
     <link name="scissor_rr">
       <visual>
-        <origin xyz="0 0 0" rpy="0 0 0" />
+        <origin xyz="0 0 0" rpy="0 0 0"/>
         <geometry>
-          <mesh filename="package://kuroko_description/meshes/kuroko/obj/scissor_rr.obj" />
+          <mesh filename="package://kuroko_description/meshes/kuroko/obj/scissor_rr.obj"/>
         </geometry>
       </visual>
-      <xacro:box_collision xyz="-0.0043 0 -0.1" rpy="0 0 0" size="0.01085 0.044 0.2" />
-      <xacro:box_collision xyz="0.0206 0 -0.193" rpy="0 0 0" size="0.039 0.044 0.014" />
-      <xacro:box_inertial xyz="-0.0043 0 -0.1" rpy="0 0 0" size="0.044 0.044 0.2" mass="0.031" />
+      <xacro:box_collision xyz="-0.0043 0 -0.1" rpy="0 0 0" size="0.01085 0.044 0.2"/>
+      <xacro:box_collision xyz="0.0206 0 -0.193" rpy="0 0 0" size="0.039 0.044 0.014"/>
+      <xacro:box_inertial xyz="-0.0043 0 -0.1" rpy="0 0 0" size="0.044 0.044 0.2" mass="0.031"/>
     </link>
   </xacro:macro>

Commit message: rename links

File: kuroko_description/xacro/kuroko/parts/arm_l.xacro (robot description, xacro)
@@ -21,7 +21,7 @@
       <xacro:box_inertial xyz="0 0.0205 0" rpy="0 0 0" size="0.042 0.041 0.04" mass="0.022"/>
     </link>
-    <joint name="arm_l_joint" type="revolute">
+    <joint name="shoulder_l_roll_joint" type="revolute">
       <parent link="shoulder_l_pitch"/>
-      <child link="arm_l"/>
+      <child link="shoulder_l_roll"/>
       <origin xyz="0 0.028 0" rpy="0 0 0"/>
       <axis xyz="-1 0 0"/>
@@ -29,9 +29,9 @@
       <dynamics damping="0.0" friction="0.0"/>
     </joint>
-    <link name="arm_l">
+    <link name="shoulder_l_roll">
       <visual>
         <origin xyz="0 0 0" rpy="0 0 0"/>
         <geometry>
-          <mesh filename="package://kuroko_description/meshes/kuroko/obj/arm_l.obj"/>
+          <mesh filename="package://kuroko_description/meshes/kuroko/obj/shoulder_l_roll.obj"/>
         </geometry>
       </visual>
@@ -40,5 +40,5 @@
     </link>
     <joint name="scissor_lf_joint" type="revolute">
-      <parent link="arm_l"/>
+      <parent link="shoulder_l_roll"/>
       <child link="scissor_lf"/>
       <origin xyz="0 0.0265 -0.0545" rpy="0 0 0"/>
@@ -59,5 +59,5 @@
     </link>
     <joint name="scissor_lr_joint" type="revolute">
-      <parent link="arm_l"/>
+      <parent link="shoulder_l_roll"/>
       <child link="scissor_lr"/>
       <origin xyz="0 0.0265 -0.0545" rpy="0 0 0"/>

File: kuroko_description/xacro/kuroko/parts/arm_r.xacro (robot description, xacro)
@@ -21,7 +21,7 @@
       <xacro:box_inertial xyz="0 -0.0205 0" rpy="0 0 0" size="0.042 0.041 0.04" mass="0.022"/>
     </link>
-    <joint name="arm_r_joint" type="revolute">
+    <joint name="shoulder_r_roll_joint" type="revolute">
       <parent link="shoulder_r_pitch"/>
-      <child link="arm_r"/>
+      <child link="shoulder_r_roll"/>
       <origin xyz="0 -0.028 0" rpy="0 0 0"/>
       <axis xyz="-1 0 0"/>
@@ -29,9 +29,9 @@
       <dynamics damping="0.0" friction="0.0"/>
     </joint>
-    <link name="arm_r">
+    <link name="shoulder_r_roll">
       <visual>
         <origin xyz="0 0 0" rpy="0 0 0"/>
         <geometry>
-          <mesh filename="package://kuroko_description/meshes/kuroko/obj/arm_r.obj"/>
+          <mesh filename="package://kuroko_description/meshes/kuroko/obj/shoulder_r_roll.obj"/>
         </geometry>
       </visual>
@@ -41,5 +41,5 @@
     </link>
     <joint name="scissor_rf_joint" type="revolute">
-      <parent link="arm_r"/>
+      <parent link="shoulder_r_roll"/>
       <child link="scissor_rf"/>
       <origin xyz="0 -0.0265 -0.0545" rpy="0 0 0"/>
@@ -60,5 +60,5 @@
     </link>
     <joint name="scissor_rr_joint" type="revolute">
-      <parent link="arm_r"/>
+      <parent link="shoulder_r_roll"/>
       <child link="scissor_rr"/>
       <origin xyz="0 -0.0265 -0.0545" rpy="0 0 0"/>
