Commit message: rename links

File: kuroko_description/xacro/kuroko/parts/arm_l.xacro (robot description, xacro)
@@ -39,7 +39,7 @@
       <xacro:box_inertial xyz="0 0.0385 -0.02575" rpy="0 0 0" size="0.0285 0.1045 0.08" mass="0.342"/>
     </link>
-    <joint name="scissor_lf_joint" type="revolute">
+    <joint name="elbow_l_front_joint" type="revolute">
       <parent link="shoulder_l_roll"/>
-      <child link="scissor_lf"/>
+      <child link="elbow_l_front"/>
       <origin xyz="0 0.0265 -0.0545" rpy="0 0 0"/>
       <axis xyz="0 -1 0"/>
@@ -47,9 +47,9 @@
       <dynamics damping="0.0" friction="0.0"/>
     </joint>
-    <link name="scissor_lf">
+    <link name="elbow_l_front">
       <visual>
         <origin xyz="0 0 0" rpy="0 0 0"/>
         <geometry>
-          <mesh filename="package://kuroko_description/meshes/kuroko/obj/scissor_lf.obj"/>
+          <mesh filename="package://kuroko_description/meshes/kuroko/obj/elbow_l_front.obj"/>
         </geometry>
       </visual>
@@ -58,7 +58,7 @@
       <xacro:box_inertial xyz="0.0043 0 -0.104" rpy="0 0 0" size="0.044 0.058 0.208" mass="0.032"/>
     </link>
-    <joint name="scissor_lr_joint" type="revolute">
+    <joint name="elbow_l_rear_joint" type="revolute">
       <parent link="shoulder_l_roll"/>
-      <child link="scissor_lr"/>
+      <child link="elbow_l_rear"/>
       <origin xyz="0 0.0265 -0.0545" rpy="0 0 0"/>
       <axis xyz="0 1 0"/>
@@ -66,9 +66,9 @@
       <dynamics damping="0.0" friction="0.0"/>
     </joint>
-    <link name="scissor_lr">
+    <link name="elbow_l_rear">
       <visual>
         <origin xyz="0 0 0" rpy="0 0 0"/>
         <geometry>
-          <mesh filename="package://kuroko_description/meshes/kuroko/obj/scissor_lr.obj"/>
+          <mesh filename="package://kuroko_description/meshes/kuroko/obj/elbow_l_rear.obj"/>
         </geometry>
       </visual>

File: kuroko_description/xacro/kuroko/parts/arm_r.xacro (robot description, xacro)
@@ -40,7 +40,7 @@
         mass="0.342"/>
     </link>
-    <joint name="scissor_rf_joint" type="revolute">
+    <joint name="elbow_r_front_joint" type="revolute">
       <parent link="shoulder_r_roll"/>
-      <child link="scissor_rf"/>
+      <child link="elbow_r_front"/>
       <origin xyz="0 -0.0265 -0.0545" rpy="0 0 0"/>
       <axis xyz="0 1 0"/>
@@ -48,9 +48,9 @@
       <dynamics damping="0.0" friction="0.0"/>
     </joint>
-    <link name="scissor_rf">
+    <link name="elbow_r_front">
       <visual>
         <origin xyz="0 0 0" rpy="0 0 0"/>
         <geometry>
-          <mesh filename="package://kuroko_description/meshes/kuroko/obj/scissor_rf.obj"/>
+          <mesh filename="package://kuroko_description/meshes/kuroko/obj/elbow_r_front.obj"/>
         </geometry>
       </visual>
@@ -59,7 +59,7 @@
       <xacro:box_inertial xyz="0.0043 0 -0.104" rpy="0 0 0" size="0.044 0.058 0.208" mass="0.032"/>
     </link>
-    <joint name="scissor_rr_joint" type="revolute">
+    <joint name="elbow_r_rear_joint" type="revolute">
       <parent link="shoulder_r_roll"/>
-      <child link="scissor_rr"/>
+      <child link="elbow_r_rear"/>
       <origin xyz="0 -0.0265 -0.0545" rpy="0 0 0"/>
       <axis xyz="0 -1 0"/>
@@ -67,9 +67,9 @@
       <dynamics damping="0.0" friction="0.0"/>
     </joint>
-    <link name="scissor_rr">
+    <link name="elbow_r_rear">
       <visual>
         <origin xyz="0 0 0" rpy="0 0 0"/>
         <geometry>
-          <mesh filename="package://kuroko_description/meshes/kuroko/obj/scissor_rr.obj"/>
+          <mesh filename="package://kuroko_description/meshes/kuroko/obj/elbow_r_rear.obj"/>
         </geometry>
       </visual>

Commit message: Fix xacro

File: kuroko_description/xacro/kuroko/parts/arm_l.xacro (robot description, xacro)
@@ -24,7 +24,7 @@
       <parent link="shoulder_l_pitch_link"/>
       <child link="shoulder_l_roll_link"/>
-      <origin xyz="0 0.05425 0" rpy="0 0 0"/>
+      <origin xyz="0 0.05425 0" rpy="1.5708 0 0"/>
       <axis xyz="-1 0 0"/>
-      <limit effort="1000.0" lower="-2.0071" upper="1.0472" velocity="10.0"/>
+      <limit effort="1000.0" lower="-3.1" upper="3.1" velocity="10.0"/>
       <dynamics damping="0.0" friction="0.0"/>
     </joint>

File: kuroko_description/xacro/kuroko/parts/arm_r.xacro (robot description, xacro)
@@ -24,7 +24,7 @@
       <parent link="shoulder_r_pitch_link"/>
       <child link="shoulder_r_roll_link"/>
-      <origin xyz="0 -0.05425 0" rpy="0 0 0"/>
+      <origin xyz="0 -0.05425 0" rpy="-1.5708 0 0"/>
       <axis xyz="-1 0 0"/>
-      <limit effort="1000.0" lower="-1.0472" upper="2.0071" velocity="10.0"/>
+      <limit effort="1000.0" lower="-3.1" upper="3.1" velocity="10.0"/>
       <dynamics damping="0.0" friction="0.0"/>
     </joint>

Commit message: invert shoulder roll

File: kuroko_description/xacro/kuroko/parts/arm_l.xacro (robot description, xacro)
@@ -25,5 +25,5 @@
       <child link="shoulder_l_roll_link"/>
       <origin xyz="0 0.05425 0" rpy="1.5708 0 0"/>
-      <axis xyz="-1 0 0"/>
+      <axis xyz="1 0 0"/>
       <limit effort="1000.0" lower="-3.1" upper="3.1" velocity="10.0"/>
       <dynamics damping="0.0" friction="0.0"/>

File: kuroko_description/xacro/kuroko/parts/arm_r.xacro (robot description, xacro)
@@ -25,5 +25,5 @@
       <child link="shoulder_r_roll_link"/>
       <origin xyz="0 -0.05425 0" rpy="-1.5708 0 0"/>
-      <axis xyz="-1 0 0"/>
+      <axis xyz="1 0 0"/>
       <limit effort="1000.0" lower="-3.1" upper="3.1" velocity="10.0"/>
       <dynamics damping="0.0" friction="0.0"/>

Commit message: Use stl

File: kuroko_description/xacro/kuroko/parts/arm_l.xacro (robot description, xacro)
@@ -15,5 +15,5 @@
         <origin xyz="0 0 0" rpy="0 0 0"/>
         <geometry>
-          <mesh filename="${MESH_DIR}/kuroko/obj/shoulder_l_pitch.obj"/>
+          <mesh filename="${MESH_DIR}/kuroko/stl/shoulder_l_pitch.stl"/>
         </geometry>
       </visual>
@@ -33,5 +33,5 @@
         <origin xyz="0 0 0" rpy="0 0 0"/>
         <geometry>
-          <mesh filename="${MESH_DIR}/kuroko/obj/shoulder_l_roll.obj"/>
+          <mesh filename="${MESH_DIR}/kuroko/stl/shoulder_l_roll.stl"/>
         </geometry>
       </visual>
@@ -51,5 +51,5 @@
         <origin xyz="0 0 0" rpy="0 0 0"/>
         <geometry>
-          <mesh filename="${MESH_DIR}/kuroko/obj/elbow_l_front.obj"/>
+          <mesh filename="${MESH_DIR}/kuroko/stl/elbow_l_front.stl"/>
         </geometry>
       </visual>
@@ -70,5 +70,5 @@
         <origin xyz="0 0 0" rpy="0 0 0"/>
         <geometry>
-          <mesh filename="${MESH_DIR}/kuroko/obj/elbow_l_rear.obj"/>
+          <mesh filename="${MESH_DIR}/kuroko/stl/elbow_l_rear.stl"/>
         </geometry>
       </visual>

File: kuroko_description/xacro/kuroko/parts/arm_r.xacro (robot description, xacro)
@@ -15,5 +15,5 @@
         <origin xyz="0 0 0" rpy="0 0 0"/>
         <geometry>
-          <mesh filename="${MESH_DIR}/kuroko/obj/shoulder_r_pitch.obj"/>
+          <mesh filename="${MESH_DIR}/kuroko/stl/shoulder_r_pitch.stl"/>
         </geometry>
       </visual>
@@ -33,5 +33,5 @@
         <origin xyz="0 0 0" rpy="0 0 0"/>
         <geometry>
-          <mesh filename="${MESH_DIR}/kuroko/obj/shoulder_r_roll.obj"/>
+          <mesh filename="${MESH_DIR}/kuroko/stl/shoulder_r_roll.stl"/>
         </geometry>
       </visual>
@@ -51,5 +51,5 @@
         <origin xyz="0 0 0" rpy="0 0 0"/>
         <geometry>
-          <mesh filename="${MESH_DIR}/kuroko/obj/elbow_r_front.obj"/>
+          <mesh filename="${MESH_DIR}/kuroko/stl/elbow_r_front.stl"/>
         </geometry>
       </visual>
@@ -70,5 +70,5 @@
         <origin xyz="0 0 0" rpy="0 0 0"/>
         <geometry>
-          <mesh filename="${MESH_DIR}/kuroko/obj/elbow_r_rear.obj"/>
+          <mesh filename="${MESH_DIR}/kuroko/stl/elbow_r_rear.stl"/>
         </geometry>
       </visual>

File: kuroko_description/xacro/kuroko/parts/body.xacro (robot description, xacro)
@@ -7,5 +7,5 @@
         <origin xyz="0 0 0" rpy="0 0 0"/>
         <geometry>
-          <mesh filename="${MESH_DIR}/kuroko/obj/waist.obj"/>
+          <mesh filename="${MESH_DIR}/kuroko/stl/waist.stl"/>
         </geometry>
       </visual>
@@ -27,5 +27,5 @@
         <origin xyz="0 0 0" rpy="0 0 0"/>
         <geometry>
-          <mesh filename="${MESH_DIR}/kuroko/obj/chest.obj"/>
+          <mesh filename="${MESH_DIR}/kuroko/stl/chest.stl"/>
         </geometry>
       </visual>

File: kuroko_description/xacro/kuroko/parts/leg_l.xacro (robot description, xacro)
@@ -15,5 +15,5 @@
         <origin xyz="0 0 0" rpy="0 0 0"/>
         <geometry>
-          <mesh filename="${MESH_DIR}/kuroko/obj/hip_l_roll.obj"/>
+          <mesh filename="${MESH_DIR}/kuroko/stl/hip_l_roll.stl"/>
         </geometry>
       </visual>
@@ -34,5 +34,5 @@
         <origin xyz="0 0 0" rpy="0 0 0"/>
         <geometry>
-          <mesh filename="${MESH_DIR}/kuroko/obj/hip_l_pitch.obj"/>
+          <mesh filename="${MESH_DIR}/kuroko/stl/hip_l_pitch.stl"/>
         </geometry>
       </visual>
@@ -53,5 +53,5 @@
         <origin xyz="0 0 0" rpy="0 0 0"/>
         <geometry>
-          <mesh filename="${MESH_DIR}/kuroko/obj/thigh_l_active.obj"/>
+          <mesh filename="${MESH_DIR}/kuroko/stl/thigh_l_active.stl"/>
         </geometry>
       </visual>
@@ -71,5 +71,5 @@
         <origin xyz="0 0 0" rpy="0 0 0"/>
         <geometry>
-          <mesh filename="${MESH_DIR}/kuroko/obj/shin_l_active.obj"/>
+          <mesh filename="${MESH_DIR}/kuroko/stl/shin_l_active.stl"/>
         </geometry>
       </visual>
@@ -95,5 +95,5 @@
         <origin xyz="0 0 0" rpy="0 0 0"/>
         <geometry>
-          <mesh filename="${MESH_DIR}/kuroko/obj/thigh_r_middle_passive.obj"/>
+          <mesh filename="${MESH_DIR}/kuroko/stl/thigh_r_middle_passive.stl"/>
         </geometry>
       </visual>
@@ -138,5 +138,5 @@
         <origin xyz="0 0 0" rpy="0 0 0"/>
         <geometry>
-          <mesh filename="${MESH_DIR}/kuroko/obj/thigh_r_rear_passive.obj"/>
+          <mesh filename="${MESH_DIR}/kuroko/stl/thigh_r_rear_passive.stl"/>
         </geometry>
       </visual>
@@ -157,5 +157,5 @@
         <origin xyz="0 0 0" rpy="0 0 0"/>
         <geometry>
-          <mesh filename="${MESH_DIR}/kuroko/obj/knee_r_passive.obj"/>
+          <mesh filename="${MESH_DIR}/kuroko/stl/knee_r_passive.stl"/>
         </geometry>
       </visual>
@@ -176,5 +176,5 @@
         <origin xyz="0 0 0" rpy="0 0 0"/>
         <geometry>
-          <mesh filename="${MESH_DIR}/kuroko/obj/shin_r_front_passive.obj"/>
+          <mesh filename="${MESH_DIR}/kuroko/stl/shin_r_front_passive.stl"/>
         </geometry>
       </visual>
@@ -199,5 +199,5 @@
         <origin xyz="0 0 0" rpy="0 0 0"/>
         <geometry>
-          <mesh filename="${MESH_DIR}/kuroko/obj/shin_r_rear_passive.obj"/>
+          <mesh filename="${MESH_DIR}/kuroko/stl/shin_r_rear_passive.stl"/>
         </geometry>
       </visual>
@@ -218,5 +218,5 @@
         <origin xyz="0 0 0" rpy="0 0 0"/>
         <geometry>
-          <mesh filename="${MESH_DIR}/kuroko/obj/ankle_r_pitch_passive.obj"/>
+          <mesh filename="${MESH_DIR}/kuroko/stl/ankle_r_pitch_passive.stl"/>
         </geometry>
       </visual>
@@ -237,5 +237,5 @@
         <origin xyz="0 0 0" rpy="0 0 0"/>
         <geometry>
-          <mesh filename="${MESH_DIR}/kuroko/obj/ankle_l_roll.obj"/>
+          <mesh filename="${MESH_DIR}/kuroko/stl/ankle_l_roll.stl"/>
         </geometry>
       </visual>
@@ -256,5 +256,5 @@
         <origin xyz="0 0 0" rpy="0 0 0"/>
         <geometry>
-          <mesh filename="${MESH_DIR}/kuroko/obj/ankle_r_yaw.obj"/>
+          <mesh filename="${MESH_DIR}/kuroko/stl/ankle_r_yaw.stl"/>
         </geometry>
       </visual>

File: kuroko_description/xacro/kuroko/parts/leg_r.xacro (robot description, xacro)
@@ -15,5 +15,5 @@
         <origin xyz="0 0 0" rpy="0 0 0"/>
         <geometry>
-          <mesh filename="${MESH_DIR}/kuroko/obj/hip_r_roll.obj"/>
+          <mesh filename="${MESH_DIR}/kuroko/stl/hip_r_roll.stl"/>
         </geometry>
       </visual>
@@ -34,5 +34,5 @@
         <origin xyz="0 0 0" rpy="0 0 0"/>
         <geometry>
-          <mesh filename="${MESH_DIR}/kuroko/obj/hip_r_pitch.obj"/>
+          <mesh filename="${MESH_DIR}/kuroko/stl/hip_r_pitch.stl"/>
         </geometry>
       </visual>
@@ -53,5 +53,5 @@
         <origin xyz="0 0 0" rpy="0 0 0"/>
         <geometry>
-          <mesh filename="${MESH_DIR}/kuroko/obj/thigh_r_active.obj"/>
+          <mesh filename="${MESH_DIR}/kuroko/stl/thigh_r_active.stl"/>
         </geometry>
       </visual>
@@ -71,5 +71,5 @@
         <origin xyz="0 0 0" rpy="0 0 0"/>
         <geometry>
-          <mesh filename="${MESH_DIR}/kuroko/obj/shin_r_active.obj"/>
+          <mesh filename="${MESH_DIR}/kuroko/stl/shin_r_active.stl"/>
         </geometry>
       </visual>
@@ -95,5 +95,5 @@
         <origin xyz="0 0 0" rpy="0 0 0"/>
         <geometry>
-          <mesh filename="${MESH_DIR}/kuroko/obj/thigh_r_middle_passive.obj"/>
+          <mesh filename="${MESH_DIR}/kuroko/stl/thigh_r_middle_passive.stl"/>
         </geometry>
       </visual>
@@ -138,5 +138,5 @@
         <origin xyz="0 0 0" rpy="0 0 0"/>
         <geometry>
-          <mesh filename="${MESH_DIR}/kuroko/obj/thigh_r_rear_passive.obj"/>
+          <mesh filename="${MESH_DIR}/kuroko/stl/thigh_r_rear_passive.stl"/>
         </geometry>
       </visual>
@@ -157,5 +157,5 @@
         <origin xyz="0 0 0" rpy="0 0 0"/>
         <geometry>
-          <mesh filename="${MESH_DIR}/kuroko/obj/knee_r_passive.obj"/>
+          <mesh filename="${MESH_DIR}/kuroko/stl/knee_r_passive.stl"/>
         </geometry>
       </visual>
@@ -176,5 +176,5 @@
         <origin xyz="0 0 0" rpy="0 0 0"/>
         <geometry>
-          <mesh filename="${MESH_DIR}/kuroko/obj/shin_r_front_passive.obj"/>
+          <mesh filename="${MESH_DIR}/kuroko/stl/shin_r_front_passive.stl"/>
         </geometry>
       </visual>
@@ -199,5 +199,5 @@
         <origin xyz="0 0 0" rpy="0 0 0"/>
         <geometry>
-          <mesh filename="${MESH_DIR}/kuroko/obj/shin_r_rear_passive.obj"/>
+          <mesh filename="${MESH_DIR}/kuroko/stl/shin_r_rear_passive.stl"/>
         </geometry>
       </visual>
@@ -218,5 +218,5 @@
         <origin xyz="0 0 0" rpy="0 0 0"/>
         <geometry>
-          <mesh filename="${MESH_DIR}/kuroko/obj/ankle_r_pitch_passive.obj"/>
+          <mesh filename="${MESH_DIR}/kuroko/stl/ankle_r_pitch_passive.stl"/>
         </geometry>
       </visual>
@@ -237,5 +237,5 @@
         <origin xyz="0 0 0" rpy="0 0 0"/>
         <geometry>
-          <mesh filename="${MESH_DIR}/kuroko/obj/ankle_r_roll.obj"/>
+          <mesh filename="${MESH_DIR}/kuroko/stl/ankle_r_roll.stl"/>
         </geometry>
       </visual>
@@ -256,5 +256,5 @@
         <origin xyz="0 0 0" rpy="0 0 0"/>
         <geometry>
-          <mesh filename="${MESH_DIR}/kuroko/obj/ankle_r_yaw.obj"/>
+          <mesh filename="${MESH_DIR}/kuroko/stl/ankle_r_yaw.stl"/>
         </geometry>
       </visual>
