Commit message: All joint axis positive

File: kuroko_description/xacro/kuroko/parts/arm_l.xacro (robot description, xacro)
@@ -2,78 +2,77 @@
 <robot xmlns:xacro="http://www.ros.org/wiki/xacro">
   <xacro:macro name="arm_l_xacro">
-    <!-- Link conencts from body. Shoulder first. -->
     <joint name="shoulder_l_pitch" type="revolute">
-      <parent link="chest_link"/>
-      <child link="shoulder_l_pitch_link"/>
-      <origin xyz="0 0.128 0.01275" rpy="0 0 0"/>
-      <axis xyz="0 1 0"/>
-      <limit effort="3.1" lower="-3.1" upper="3.1" velocity="6.5"/>
-      <dynamics damping="0.4769" friction="0.0"/>
+      <parent link="chest_link" />
+      <child link="shoulder_l_pitch_link" />
+      <origin xyz="0 0.128 0.01275" rpy="0 0 0" />
+      <axis xyz="0 1 0" />
+      <limit effort="3.1" lower="-3.1" upper="3.1" velocity="6.5" />
+      <dynamics damping="0.476923" friction="0.0" />
     </joint>
     <link name="shoulder_l_pitch_link">
       <visual>
-        <origin xyz="0 0 0" rpy="0 0 0"/>
+        <origin xyz="0 0 0" rpy="0 0 0" />
         <geometry>
-          <mesh filename="${MESH_DIR}/kuroko/stl/shoulder_l_pitch.stl"/>
+          <mesh filename="${MESH_DIR}/kuroko/stl/shoulder_l_pitch.stl" />
         </geometry>
       </visual>
-      <xacro:box_collision xyz="-0.0096 0.0340 0.0000" rpy="0 0 0" size="0.0513 0.0680 0.0475"/>
-      <xacro:box_inertial xyz="-0.0096 0.0340 0.0000" rpy="0 0 0" size="0.0513 0.0680 0.0475" mass="0.165"/>
+      <xacro:box_collision xyz="-0.0096 0.0340 0.0000" rpy="0 0 0" size="0.0513 0.0680 0.0475" />
+      <xacro:box_inertial xyz="-0.0096 0.0340 0.0000" rpy="0 0 0" size="0.0513 0.0680 0.0475" mass="0.165" />
     </link>
     <joint name="shoulder_l_roll" type="revolute">
-      <parent link="shoulder_l_pitch_link"/>
-      <child link="shoulder_l_roll_link"/>
-      <origin xyz="0 0.05425 0" rpy="1.5708 0 0"/>
-      <axis xyz="1 0 0"/>
-      <limit effort="8.9" lower="-3.1" upper="3.1" velocity="6.9"/>
-      <dynamics damping="1.290" friction="0.0"/>
+      <parent link="shoulder_l_pitch_link" />
+      <child link="shoulder_l_roll_link" />
+      <origin xyz="0 0.05425 0" rpy="1.5708 0 0" />
+      <axis xyz="1 0 0" />
+      <limit effort="8.9" lower="-3.1" upper="3.1" velocity="6.9" />
+      <dynamics damping="1.289855" friction="0.0" />
     </joint>
     <link name="shoulder_l_roll_link">
       <visual>
-        <origin xyz="0 0 0" rpy="0 0 0"/>
+        <origin xyz="0 0 0" rpy="0 0 0" />
         <geometry>
-          <mesh filename="${MESH_DIR}/kuroko/stl/shoulder_l_roll.stl"/>
+          <mesh filename="${MESH_DIR}/kuroko/stl/shoulder_l_roll.stl" />
         </geometry>
       </visual>
-      <xacro:box_collision xyz="-0.0108 0.0000 -0.0186" rpy="0 0 0" size="0.0530 0.0860 0.0633"/>
-      <xacro:box_inertial xyz="-0.0108 0.0000 -0.0186" rpy="0 0 0" size="0.0530 0.0860 0.0633" mass="0.183"/>
+      <xacro:box_collision xyz="-0.0108 0.0000 -0.0186" rpy="0 0 0" size="0.0530 0.0860 0.0633" />
+      <xacro:box_inertial xyz="-0.0108 0.0000 -0.0186" rpy="0 0 0" size="0.0530 0.0860 0.0633" mass="0.183" />
     </link>
     <joint name="elbow_l_front" type="revolute">
-      <parent link="shoulder_l_roll_link"/>
-      <child link="elbow_l_front_link"/>
-      <origin xyz="0 -0.023 -0.036" rpy="0 0 0"/>
-      <axis xyz="0 -1 0"/>
-      <limit effort="3.1" lower="-2.6180" upper="2.6180" velocity="6.5"/>
-      <dynamics damping="0.4769" friction="0.0"/>
+      <parent link="shoulder_l_roll_link" />
+      <child link="elbow_l_front_link" />
+      <origin xyz="0 -0.023 -0.036" rpy="0 0 0" />
+      <axis xyz="0 1 0" />
+      <limit effort="3.1" lower="-2.618" upper="2.618" velocity="6.5" />
+      <dynamics damping="0.476923" friction="0.0" />
     </joint>
     <link name="elbow_l_front_link">
       <visual>
-        <origin xyz="0 0 0" rpy="0 0 0"/>
+        <origin xyz="0 0 0" rpy="0 0 0" />
         <geometry>
-          <mesh filename="${MESH_DIR}/kuroko/stl/elbow_l_front.stl"/>
+          <mesh filename="${MESH_DIR}/kuroko/stl/elbow_l_front.stl" />
         </geometry>
       </visual>
-      <xacro:box_collision xyz="0.0043 0 -0.104" rpy="0 0 0" size="0.01085 0.058 0.208"/>
-      <xacro:box_collision xyz="-0.0206 0 -0.201" rpy="0 0 0" size="0.039 0.058 0.014"/>
-      <xacro:box_inertial xyz="0.0043 0 -0.104" rpy="0 0 0" size="0.044 0.058 0.208" mass="0.032"/>
+      <xacro:box_collision xyz="0.0043 0 -0.104" rpy="0 0 0" size="0.01085 0.058 0.208" />
+      <xacro:box_collision xyz="-0.0206 0 -0.201" rpy="0 0 0" size="0.039 0.058 0.014" />
+      <xacro:box_inertial xyz="0.0043 0 -0.104" rpy="0 0 0" size="0.044 0.058 0.208" mass="0.032" />
     </link>
     <joint name="elbow_l_rear" type="revolute">
-      <parent link="shoulder_l_roll_link"/>
-      <child link="elbow_l_rear_link"/>
-      <origin xyz="0 -0.024 -0.036" rpy="0 0 0"/>
-      <axis xyz="0 1 0"/>
-      <limit effort="3.1" lower="-2.6180" upper="2.6180" velocity="6.5"/>
-      <dynamics damping="0.4769" friction="0.0"/>
+      <parent link="shoulder_l_roll_link" />
+      <child link="elbow_l_rear_link" />
+      <origin xyz="0 -0.024 -0.036" rpy="0 0 0" />
+      <axis xyz="0 1 0" />
+      <limit effort="3.1" lower="-2.6180" upper="2.6180" velocity="6.5" />
+      <dynamics damping="0.476923" friction="0.0" />
     </joint>
     <link name="elbow_l_rear_link">
       <visual>
-        <origin xyz="0 0 0" rpy="0 0 0"/>
+        <origin xyz="0 0 0" rpy="0 0 0" />
         <geometry>
-          <mesh filename="${MESH_DIR}/kuroko/stl/elbow_l_rear.stl"/>
+          <mesh filename="${MESH_DIR}/kuroko/stl/elbow_l_rear.stl" />
         </geometry>
       </visual>
-      <xacro:box_collision xyz="-0.0043 0 -0.1" rpy="0 0 0" size="0.01085 0.044 0.2"/>
-      <xacro:box_collision xyz="0.0206 0 -0.193" rpy="0 0 0" size="0.039 0.044 0.014"/>
-      <xacro:box_inertial xyz="-0.0043 0 -0.1" rpy="0 0 0" size="0.044 0.044 0.2" mass="0.031"/>
+      <xacro:box_collision xyz="-0.0043 0 -0.1" rpy="0 0 0" size="0.01085 0.044 0.2" />
+      <xacro:box_collision xyz="0.0206 0 -0.193" rpy="0 0 0" size="0.039 0.044 0.014" />
+      <xacro:box_inertial xyz="-0.0043 0 -0.1" rpy="0 0 0" size="0.044 0.044 0.2" mass="0.031" />
     </link>
   </xacro:macro>

File: kuroko_description/xacro/kuroko/parts/arm_r.xacro (robot description, xacro)
@@ -2,78 +2,77 @@
 <robot xmlns:xacro="http://www.ros.org/wiki/xacro">
   <xacro:macro name="arm_r_xacro">
-    <!-- Link conencts from body. Shoulder first. -->
     <joint name="shoulder_r_pitch" type="revolute">
-      <parent link="chest_link"/>
-      <child link="shoulder_r_pitch_link"/>
-      <origin xyz="0 -0.128 0.01275" rpy="0 0 0"/>
-      <axis xyz="0 -1 0"/>
-      <limit effort="3.1" lower="-3.1" upper="3.1" velocity="6.5"/>
-      <dynamics damping="0.4769" friction="0.0"/>
+      <parent link="chest_link" />
+      <child link="shoulder_r_pitch_link" />
+      <origin xyz="0 -0.128 0.01275" rpy="0 0 0" />
+      <axis xyz="0 1 0" />
+      <limit effort="3.1" lower="-3.1" upper="3.1" velocity="6.5" />
+      <dynamics damping="0.476923" friction="0.0" />
     </joint>
     <link name="shoulder_r_pitch_link">
       <visual>
-        <origin xyz="0 0 0" rpy="0 0 0"/>
+        <origin xyz="0 0 0" rpy="0 0 0" />
         <geometry>
-          <mesh filename="${MESH_DIR}/kuroko/stl/shoulder_r_pitch.stl"/>
+          <mesh filename="${MESH_DIR}/kuroko/stl/shoulder_r_pitch.stl" />
         </geometry>
       </visual>
-      <xacro:box_collision xyz="-0.0096 -0.0340 0.0000" rpy="0 0 0" size="0.0513 0.0680 0.0475"/>
-      <xacro:box_inertial xyz="-0.0096 -0.0340 0.0000" rpy="0 0 0" size="0.0513 0.0680 0.0475" mass="0.165"/>
+      <xacro:box_collision xyz="-0.0096 -0.0340 0.0000" rpy="0 0 0" size="0.0513 0.0680 0.0475" />
+      <xacro:box_inertial xyz="-0.0096 -0.0340 0.0000" rpy="0 0 0" size="0.0513 0.0680 0.0475" mass="0.165" />
     </link>
     <joint name="shoulder_r_roll" type="revolute">
-      <parent link="shoulder_r_pitch_link"/>
-      <child link="shoulder_r_roll_link"/>
-      <origin xyz="0 -0.05425 0" rpy="-1.5708 0 0"/>
-      <axis xyz="1 0 0"/>
-      <limit effort="8.9" lower="-3.1" upper="3.1" velocity="6.9"/>
-      <dynamics damping="1.290" friction="0.0"/>
+      <parent link="shoulder_r_pitch_link" />
+      <child link="shoulder_r_roll_link" />
+      <origin xyz="0 -0.05425 0" rpy="-1.5708 0 0" />
+      <axis xyz="1 0 0" />
+      <limit effort="8.9" lower="-3.1" upper="3.1" velocity="6.9" />
+      <dynamics damping="1.289855" friction="0.0" />
     </joint>
     <link name="shoulder_r_roll_link">
       <visual>
-        <origin xyz="0 0 0" rpy="0 0 0"/>
+        <origin xyz="0 0 0" rpy="0 0 0" />
         <geometry>
-          <mesh filename="${MESH_DIR}/kuroko/stl/shoulder_r_roll.stl"/>
+          <mesh filename="${MESH_DIR}/kuroko/stl/shoulder_r_roll.stl" />
         </geometry>
       </visual>
-      <xacro:box_collision xyz="-0.0108 0.0000 -0.0186" rpy="0 0 0" size="0.0530 0.0860 0.0633"/>
-      <xacro:box_inertial xyz="-0.0108 0.0000 -0.0186" rpy="0 0 0" size="0.0530 0.0860 0.0633" mass="0.183"/>
+      <xacro:box_collision xyz="-0.0108 0.0000 -0.0186" rpy="0 0 0" size="0.0530 0.0860 0.0633" />
+      <xacro:box_inertial xyz="-0.0108 0.0000 -0.0186" rpy="0 0 0" size="0.0530 0.0860 0.0633" mass="0.183" />
     </link>
     <joint name="elbow_r_front" type="revolute">
-      <parent link="shoulder_r_roll_link"/>
-      <child link="elbow_r_front_link"/>
-      <origin xyz="0 0.023 -0.036" rpy="0 0 0"/>
-      <axis xyz="0 1 0"/>
-      <limit effort="3.1" lower="-2.6180" upper="2.6180" velocity="6.6"/>
-      <dynamics damping="0.4769" friction="0.0"/>
+      <parent link="shoulder_r_roll_link" />
+      <child link="elbow_r_front_link" />
+      <origin xyz="0 0.023 -0.036" rpy="0 0 0" />
+      <axis xyz="0 1 0" />
+      <limit effort="3.1" lower="-2.6180" upper="2.6180" velocity="6.6" />
+      <dynamics damping="0.469697" friction="0.0" />
     </joint>
     <link name="elbow_r_front_link">
       <visual>
-        <origin xyz="0 0 0" rpy="0 0 0"/>
+        <origin xyz="0 0 0" rpy="0 0 0" />
         <geometry>
-          <mesh filename="${MESH_DIR}/kuroko/stl/elbow_r_front.stl"/>
+          <mesh filename="${MESH_DIR}/kuroko/stl/elbow_r_front.stl" />
         </geometry>
       </visual>
-      <xacro:box_collision xyz="0.0043 0 -0.104" rpy="0 0 0" size="0.01085 0.058 0.208"/>
-      <xacro:box_collision xyz="-0.0206 0 -0.201" rpy="0 0 0" size="0.039 0.058 0.014"/>
-      <xacro:box_inertial xyz="0.0043 0 -0.104" rpy="0 0 0" size="0.044 0.058 0.208" mass="0.032"/>
+      <xacro:box_collision xyz="0.0043 0 -0.104" rpy="0 0 0" size="0.01085 0.058 0.208" />
+      <xacro:box_collision xyz="-0.0206 0 -0.201" rpy="0 0 0" size="0.039 0.058 0.014" />
+      <xacro:box_inertial xyz="0.0043 0 -0.104" rpy="0 0 0" size="0.044 0.058 0.208" mass="0.032" />
     </link>
     <joint name="elbow_r_rear" type="revolute">
-      <parent link="shoulder_r_roll_link"/>
-      <child link="elbow_r_rear_link"/>
-      <origin xyz="0 0.024 -0.036" rpy="0 0 0"/>
-      <axis xyz="0 -1 0"/>
-      <limit effort="3.1" lower="-2.6180" upper="2.6180" velocity="6.5"/>
-      <dynamics damping="0.4769" friction="0.0"/>
+      <parent link="shoulder_r_roll_link" />
+      <child link="elbow_r_rear_link" />
+      <origin xyz="0 0.024 -0.036" rpy="0 0 0" />
+      <axis xyz="0 1 0" />
+      <limit effort="3.1" lower="-2.618" upper="2.618" velocity="6.5" />
+      <dynamics damping="0.476923" friction="0.0" />
     </joint>
     <link name="elbow_r_rear_link">
       <visual>
-        <origin xyz="0 0 0" rpy="0 0 0"/>
+        <origin xyz="0 0 0" rpy="0 0 0" />
         <geometry>
-          <mesh filename="${MESH_DIR}/kuroko/stl/elbow_r_rear.stl"/>
+          <mesh filename="${MESH_DIR}/kuroko/stl/elbow_r_rear.stl" />
         </geometry>
       </visual>
-      <xacro:box_collision xyz="-0.0043 0 -0.1" rpy="0 0 0" size="0.01085 0.044 0.2"/>
-      <xacro:box_collision xyz="0.0206 0 -0.193" rpy="0 0 0" size="0.039 0.044 0.014"/>
-      <xacro:box_inertial xyz="-0.0043 0 -0.1" rpy="0 0 0" size="0.044 0.044 0.2" mass="0.031"/>
+      <xacro:box_collision xyz="-0.0043 0 -0.1" rpy="0 0 0" size="0.01085 0.044 0.2" />
+      <xacro:box_collision xyz="0.0206 0 -0.193" rpy="0 0 0" size="0.039 0.044 0.014" />
+      <xacro:box_inertial xyz="-0.0043 0 -0.1" rpy="0 0 0" size="0.044 0.044 0.2" mass="0.031" />
     </link>
   </xacro:macro>

File: kuroko_description/xacro/kuroko/parts/body.xacro (robot description, xacro)
@@ -2,34 +2,31 @@
 <robot xmlns:xacro="http://www.ros.org/wiki/xacro">
   <xacro:macro name="body_xacro">
-    <!-- waist -->
     <link name="waist_link">
       <visual>
-        <origin xyz="0 0 0" rpy="0 0 0"/>
+        <origin xyz="0 0 0" rpy="0 0 0" />
         <geometry>
-          <mesh filename="${MESH_DIR}/kuroko/stl/waist.stl"/>
+          <mesh filename="${MESH_DIR}/kuroko/stl/waist.stl" />
         </geometry>
       </visual>
-      <xacro:box_collision xyz="0.0084 0.0000 -0.0483" rpy="0 0 0" size="0.1247 0.0560 0.0965"/>
-      <xacro:box_inertial xyz="0.0084 0.0000 -0.0483" rpy="0 0 0" size="0.1247 0.0560 0.0965" mass="0.388"/>
+      <xacro:box_collision xyz="0.0084 0.0000 -0.0483" rpy="0 0 0" size="0.1247 0.0560 0.0965" />
+      <xacro:box_inertial xyz="0.0084 0.0000 -0.0483" rpy="0 0 0" size="0.1247 0.0560 0.0965" mass="0.388" />
     </link>
-    <!-- Joint1 -->
     <joint name="chest" type="revolute">
-      <parent link="waist_link"/>
-      <child link="chest_link"/>
-      <origin xyz="0 0 0" rpy="0 0 0"/>
-      <axis xyz="0 0 1"/>
-      <limit effort="3.1" lower="-3.1" upper="3.1" velocity="6.5"/>
-      <dynamics damping="4769.0" friction="0.0"/>
+      <parent link="waist_link" />
+      <child link="chest_link" />
+      <origin xyz="0 0 0" rpy="0 0 0" />
+      <axis xyz="0 0 1" />
+      <limit effort="3.1" lower="-3.1" upper="3.1" velocity="6.5" />
+      <dynamics damping="0.476923" friction="0.0" />
     </joint>
-    <!-- chest -->
     <link name="chest_link">
       <visual>
-        <origin xyz="0 0 0" rpy="0 0 0"/>
+        <origin xyz="0 0 0" rpy="0 0 0" />
         <geometry>
-          <mesh filename="${MESH_DIR}/kuroko/stl/chest.stl"/>
+          <mesh filename="${MESH_DIR}/kuroko/stl/chest.stl" />
         </geometry>
       </visual>
-      <xacro:box_collision xyz="0.0120 0.0000 0.0635" rpy="0 0 0" size="0.1480 0.2560 0.1364"/>
-      <xacro:box_inertial xyz="0.0120 0.0000 0.0635" rpy="0 0 0" size="0.1480 0.2560 0.1364" mass="0.806"/>
+      <xacro:box_collision xyz="0.0120 0.0000 0.0635" rpy="0 0 0" size="0.1480 0.2560 0.1364" />
+      <xacro:box_inertial xyz="0.0120 0.0000 0.0635" rpy="0 0 0" size="0.1480 0.2560 0.1364" mass="0.806" />
     </link>
   </xacro:macro>
