Commit message: All joint axis positive

File: kuroko_description/xacro/kuroko/parts/leg_l.xacro (robot description, xacro)
@@ -2,12 +2,11 @@
 <robot xmlns:xacro="http://www.ros.org/wiki/xacro">
   <xacro:macro name="leg_l_xacro" params="gazebo:=false">
-    <!-- Link conencts from body. Hip first. -->
     <joint name="hip_l_roll" type="revolute">
       <parent link="waist_link"/>
       <child link="hip_l_roll_link"/>
       <origin xyz="0 0 -0.08425" rpy="0 0 0"/>
-      <axis xyz="-1 0 0"/>
-      <limit effort="3.1" lower="-0.5550" upper="1.8640" velocity="6.5"/>
-      <dynamics damping="0.4796" friction="0.0"/>
+      <axis xyz="1 0 0"/>
+      <limit effort="3.1" lower="-1.864" upper="0.555" velocity="6.5"/>
+      <dynamics damping="0.476923" friction="0.0"/>
     </joint>
     <link name="hip_l_roll_link">
@@ -19,6 +18,5 @@
       </visual>
       <xacro:box_collision xyz="0.00125 0.0065 -0.004125" rpy="0 0 0" size="0.092 0.041 0.03625"/>
-      <xacro:box_inertial xyz="0.00125 0.0065 -0.004125" rpy="0 0 0" size="0.092 0.041 0.03625"
-        mass="0.026"/>
+      <xacro:box_inertial xyz="0.00125 0.0065 -0.004125" rpy="0 0 0" size="0.092 0.041 0.03625" mass="0.026"/>
     </link>
     <joint name="hip_l_pitch" type="revolute">
@@ -28,5 +26,5 @@
       <axis xyz="0 1 0"/>
       <limit effort="3.1" lower="-3.1" upper="3.1" velocity="6.9"/>
-      <dynamics damping="1.290" friction="0.0"/>
+      <dynamics damping="0.449275" friction="0.0"/>
     </joint>
     <link name="hip_l_pitch_link">
@@ -38,6 +36,5 @@
       </visual>
       <xacro:box_collision xyz="-0.00175 0.049 -0.015" rpy="0 0 0" size="0.067 0.098 0.0585"/>
-      <xacro:box_inertial xyz="-0.00175 0.049 -0.015" rpy="0 0 0" size="0.067 0.098 0.0585"
-        mass="0.478"/>
+      <xacro:box_inertial xyz="-0.00175 0.049 -0.015" rpy="0 0 0" size="0.067 0.098 0.0585" mass="0.478"/>
     </link>
     <joint name="thigh_l_active" type="revolute">
@@ -45,7 +42,7 @@
       <child link="thigh_l_active_link"/>
       <origin xyz="0.015 0.02925 -0.0305" rpy="0 -0.785398163 0"/>
-      <axis xyz="0 -1 0"/>
-      <limit effort="8.9" lower="-1.8588" upper="0.4974" velocity="6.9"/>
-      <dynamics damping="1.290" friction="0.0"/>
+      <axis xyz="0 1 0"/>
+      <limit effort="8.9" lower="-0.4974" upper="1.8588" velocity="6.9"/>
+      <dynamics damping="1.289855" friction="0.0"/>
     </joint>
     <link name="thigh_l_active_link">
@@ -63,7 +60,7 @@
       <child link="shin_l_active_link"/>
       <origin xyz="-0.0185 0.02925 -0.0305" rpy="0 1.047197551 0"/>
-      <axis xyz="0 -1 0"/>
-      <limit effort="8.9" lower="-0.4974" upper="1.8588" velocity="6.9"/>
-      <dynamics damping="1.290" friction="0.0"/>
+      <axis xyz="0 1 0"/>
+      <limit effort="8.9" lower="-1.8588" upper="0.4974" velocity="6.9"/>
+      <dynamics damping="1.289855" friction="0.0"/>
     </joint>
     <link name="shin_l_active_link">
@@ -75,6 +72,5 @@
       </visual>
       <xacro:box_collision xyz="-0.004745 0 -0.015" rpy="0 0 0" size="0.02349 0.0445 0.044"/>
-      <xacro:box_inertial xyz="-0.004745 0 -0.015" rpy="0 0 0" size="0.02349 0.0445 0.044"
-        mass="0.008"/>
+      <xacro:box_inertial xyz="-0.004745 0 -0.015" rpy="0 0 0" size="0.02349 0.0445 0.044" mass="0.008"/>
     </link>
     <joint name="thigh_l_middle_passive" type="revolute">
@@ -82,12 +78,11 @@
       <child link="thigh_l_middle_passive_link"/>
       <origin xyz="-0.0185 0.02925 -0.0305" rpy="0 -0.785398163 0"/>
-      <axis xyz="0 -1 0"/>
-      <limit effort="0.0" lower="-3.1" upper="3.1" velocity="10.0"/>
-      <dynamics damping="0.0" friction="0.0"/>
+      <axis xyz="0 1 0"/>
+      <limit effort="0.0" lower="-3.1" upper="3.1" velocity="100.0"/>
+      <dynamics damping="0" friction="0.0"/>
       <mimic joint="thigh_l_active" multiplier="1" offset="0"/>
     </joint>
     <xacro:if value="$(arg gazebo)">
-      <xacro:gazebo_poassive_joint name="thigh_l_middle_passive_loop" xyz="-0.0335 0 0"
-        parent="knee_l_passive_link" child="thigh_l_middle_passive_link" axis="0 -1 0"/>
+      <xacro:gazebo_poassive_joint name="thigh_l_middle_passive_loop" xyz="-0.0335 0 0" parent="knee_l_passive_link" child="thigh_l_middle_passive_link" axis="0 1 0"/>
     </xacro:if>
     <link name="thigh_l_middle_passive_link">
@@ -106,7 +101,7 @@
         <child link="thigh_l_rear_passive_mimic_link"/>
         <origin xyz="0 0 -0.03" rpy="0 -1.832597551 0"/>
-        <axis xyz="0 -1 0"/>
+        <axis xyz="0 1 0"/>
         <limit effort="0.0" lower="-3.1" upper="3.1" velocity="100.0"/>
-        <dynamics damping="0.0" friction="0.0"/>
+        <dynamics damping="0" friction="0.0"/>
         <mimic joint="shin_l_active" multiplier="-1" offset="0"/>
       </joint>
@@ -116,7 +111,7 @@
         <child link="thigh_l_rear_passive_link"/>
         <origin xyz="0 0 0" rpy="0 0 0"/>
-        <axis xyz="0 -1 0"/>
+        <axis xyz="0 1 0"/>
         <limit effort="0.0" lower="-3.1" upper="3.1" velocity="100.0"/>
-        <dynamics damping="0.0" friction="0.0"/>
+        <dynamics damping="0" friction="0.0"/>
         <mimic joint="thigh_l_active" multiplier="1" offset="0"/>
       </joint>
@@ -127,10 +122,9 @@
         <child link="thigh_l_rear_passive_link"/>
         <origin xyz="0 0 -0.03" rpy="0 -1.832597551 0"/>
-        <axis xyz="0 -1 0"/>
-        <limit effort="0.0" lower="-1.5708" upper="0.9948" velocity="100.0"/>
-        <dynamics damping="0.0" friction="0.0"/>
+        <axis xyz="0 1 0"/>
+        <limit effort="0.0" lower="-0.9948" upper="1.5708" velocity="100.0"/>
+        <dynamics damping="0" friction="0.0"/>
       </joint>
-      <xacro:gazebo_poassive_joint name="thigh_l_rear_passive_loop" xyz="-0.00765471 0 -0.02897777"
-        parent="shin_l_rear_passive_link" child="thigh_l_rear_passive_link" axis="0 -1 0"/>
+      <xacro:gazebo_poassive_joint name="thigh_l_rear_passive_loop" xyz="-0.00765471 0 -0.02897777" parent="shin_l_rear_passive_link" child="thigh_l_rear_passive_link" axis="0 1 0"/>
     </xacro:if>
     <link name="thigh_l_rear_passive_link">
@@ -148,7 +142,7 @@
       <child link="knee_l_passive_link"/>
       <origin xyz="0 0 -0.1" rpy="0 0.785398163 0"/>
-      <axis xyz="0 -1 0"/>
-      <limit effort="0.0" lower="-0.4974" upper="1.8588" velocity="100.0"/>
-      <dynamics damping="0.0" friction="0.0"/>
+      <axis xyz="0 1 0"/>
+      <limit effort="0.0" lower="-1.8588" upper="0.4974" velocity="100.0"/>
+      <dynamics damping="0" friction="0.0"/>
       <mimic joint="thigh_l_active" multiplier="-1" offset="0"/>
     </joint>
@@ -167,7 +161,7 @@
       <child link="shin_l_front_passive_link"/>
       <origin xyz="0 0 0" rpy="0 0.785398163 0"/>
-      <axis xyz="0 -1 0"/>
-      <limit effort="0.0" lower="-0.4974" upper="1.8588" velocity="100.0"/>
-      <dynamics damping="0.0" friction="0.0"/>
+      <axis xyz="0 1 0"/>
+      <limit effort="0.0" lower="-1.8588" upper="0.4974" velocity="100.0"/>
+      <dynamics damping="0" friction="0.0"/>
       <mimic joint="shin_l_active" multiplier="1" offset="0"/>
     </joint>
@@ -186,12 +180,11 @@
       <child link="shin_l_rear_passive_link"/>
       <origin xyz="-0.0335 0 0" rpy="0 0.785398163 0"/>
-      <axis xyz="0 -1 0"/>
-      <limit effort="0.0" lower="-0.4974" upper="1.8588" velocity="100.0"/>
-      <dynamics damping="0.0" friction="0.0"/>
+      <axis xyz="0 1 0"/>
+      <limit effort="0.0" lower="-1.8588" upper="0.4974" velocity="100.0"/>
+      <dynamics damping="0" friction="0.0"/>
       <mimic joint="shin_l_active" multiplier="1" offset="0"/>
     </joint>
     <xacro:if value="$(arg gazebo)">
-      <xacro:gazebo_poassive_joint name="shin_l_rear_passive_loop" xyz="-0.0335 0 0"
-        parent="ankle_l_pitch_passive_link" child="shin_l_rear_passive_link" axis="0 -1 0"/>
+      <xacro:gazebo_poassive_joint name="shin_l_rear_passive_loop" xyz="-0.0335 0 0" parent="ankle_l_pitch_passive_link" child="shin_l_rear_passive_link" axis="0 1 0"/>
     </xacro:if>
     <link name="shin_l_rear_passive_link">
@@ -209,7 +202,7 @@
       <child link="ankle_l_pitch_passive_link"/>
       <origin xyz="0 0 -0.1" rpy="0 -0.785398163 0"/>
-      <axis xyz="0 -1 0"/>
-      <limit effort="0.0" lower="-1.8588" upper="0.4974" velocity="100.0"/>
-      <dynamics damping="0.0" friction="0.0"/>
+      <axis xyz="0 1 0"/>
+      <limit effort="0.0" lower="-0.4974" upper="1.8588" velocity="100.0"/>
+      <dynamics damping="0" friction="0.0"/>
       <mimic joint="shin_l_active" multiplier="-1" offset="0"/>
     </joint>
@@ -222,6 +215,5 @@
       </visual>
       <xacro:box_collision xyz="-0.0285 0 -0.013" rpy="0 0 0" size="0.0855 0.0325 0.0465"/>
-      <xacro:box_inertial xyz="-0.0285 0 -0.013" rpy="0 0 0" size="0.0855 0.0325 0.0465"
-        mass="0.104"/>
+      <xacro:box_inertial xyz="-0.0285 0 -0.013" rpy="0 0 0" size="0.0855 0.0325 0.0465" mass="0.104"/>
     </link>
     <joint name="ankle_l_roll" type="revolute">
@@ -231,5 +223,5 @@
       <axis xyz="1 0 0"/>
       <limit effort="3.1" lower="-1.5708" upper="0.3704" velocity="6.5"/>
-      <dynamics damping="0.4769" friction="0.0"/>
+      <dynamics damping="0.476923" friction="0.0"/>
     </joint>
     <link name="ankle_l_roll_link">
@@ -241,6 +233,5 @@
       </visual>
       <xacro:box_collision xyz="0 0.009375 -0.01175" rpy="0 0 0" size="0.0365 0.05375 0.043"/>
-      <xacro:box_inertial xyz="0 0.009375 -0.01175" rpy="0 0 0" size="0.0365 0.05375 0.043"
-        mass="0.136"/>
+      <xacro:box_inertial xyz="0 0.009375 -0.01175" rpy="0 0 0" size="0.0365 0.05375 0.043" mass="0.136"/>
     </link>
     <joint name="ankle_l_yaw" type="revolute">
@@ -248,7 +239,7 @@
       <child link="ankle_l_yaw_link"/>
       <origin xyz="0 0 -0.03825" rpy="0 0 0"/>
-      <axis xyz="0 0 -1"/>
+      <axis xyz="0 0 1"/>
       <limit effort="3.1" lower="-3.1" upper="3.1" velocity="6.5"/>
-      <dynamics damping="0.4769" friction="0.0"/>
+      <dynamics damping="0.476923" friction="0.0"/>
     </joint>
     <link name="ankle_l_yaw_link">

File: kuroko_description/xacro/kuroko/parts/leg_r.xacro (robot description, xacro)
@@ -2,5 +2,4 @@
 <robot xmlns:xacro="http://www.ros.org/wiki/xacro">
   <xacro:macro name="leg_r_xacro" params="gazebo:=false">
-    <!-- Link conencts from body. Hip first. -->
     <joint name="hip_r_roll" type="revolute">
       <parent link="waist_link"/>
@@ -8,6 +7,6 @@
       <origin xyz="0 0 -0.08425" rpy="0 0 0"/>
       <axis xyz="1 0 0"/>
-      <limit effort="1000.0" lower="-0.5550" upper="1.8640" velocity="10.0"/>
-      <dynamics damping="0.0" friction="0.0"/>
+      <limit effort="3.1" lower="-0.5550" upper="1.8640" velocity="6.5"/>
+      <dynamics damping="0.476923" friction="0.0"/>
     </joint>
     <link name="hip_r_roll_link">
@@ -19,6 +18,5 @@
       </visual>
       <xacro:box_collision xyz="0.00125 -0.0065 -0.004125" rpy="0 0 0" size="0.092 0.041 0.03625"/>
-      <xacro:box_inertial xyz="0.00125 -0.0065 -0.004125" rpy="0 0 0" size="0.092 0.041 0.03625"
-        mass="0.026"/>
+      <xacro:box_inertial xyz="0.00125 -0.0065 -0.004125" rpy="0 0 0" size="0.092 0.041 0.03625" mass="0.026"/>
     </link>
     <joint name="hip_r_pitch" type="revolute">
@@ -26,7 +24,7 @@
       <child link="hip_r_pitch_link"/>
       <origin xyz="0 -0.027 0" rpy="0 0 0"/>
-      <axis xyz="0 -1 0"/>
-      <limit effort="1000.0" lower="-3.1" upper="3.1" velocity="10.0"/>
-      <dynamics damping="0.0" friction="0.0"/>
+      <axis xyz="0 1 0"/>
+      <limit effort="3.1" lower="-3.1" upper="3.1" velocity="6.5"/>
+      <dynamics damping="0.476923" friction="0.0"/>
     </joint>
     <link name="hip_r_pitch_link">
@@ -38,6 +36,5 @@
       </visual>
       <xacro:box_collision xyz="-0.00175 -0.049 -0.015" rpy="0 0 0" size="0.067 0.098 0.0585"/>
-      <xacro:box_inertial xyz="-0.00175 -0.049 -0.015" rpy="0 0 0" size="0.067 0.098 0.0585"
-        mass="0.478"/>
+      <xacro:box_inertial xyz="-0.00175 -0.049 -0.015" rpy="0 0 0" size="0.067 0.098 0.0585" mass="0.478"/>
     </link>
     <joint name="thigh_r_active" type="revolute">
@@ -46,6 +43,6 @@
       <origin xyz="0.015 -0.02925 -0.0305" rpy="0 -0.785398163 0"/>
       <axis xyz="0 1 0"/>
-      <limit effort="1000.0" lower="-0.4974" upper="1.8588" velocity="10.0"/>
-      <dynamics damping="0.0" friction="0.0"/>
+      <limit effort="8.9" lower="-0.4974" upper="1.8588" velocity="6.9"/>
+      <dynamics damping="1.289855" friction="0.0"/>
     </joint>
     <link name="thigh_r_active_link">
@@ -64,6 +61,6 @@
       <origin xyz="-0.0185 -0.02925 -0.0305" rpy="0 1.047197551 0"/>
       <axis xyz="0 1 0"/>
-      <limit effort="1000.0" lower="-1.8588" upper="0.4974" velocity="10.0"/>
-      <dynamics damping="0.0" friction="0.0"/>
+      <limit effort="8.9" lower="-1.8588" upper="0.4974" velocity="6.9"/>
+      <dynamics damping="1.289855" friction="0.0"/>
     </joint>
     <link name="shin_r_active_link">
@@ -75,6 +72,5 @@
       </visual>
       <xacro:box_collision xyz="-0.004745 0 -0.015" rpy="0 0 0" size="0.02349 0.0445 0.044"/>
-      <xacro:box_inertial xyz="-0.004745 0 -0.015" rpy="0 0 0" size="0.02349 0.0445 0.044"
-        mass="0.008"/>
+      <xacro:box_inertial xyz="-0.004745 0 -0.015" rpy="0 0 0" size="0.02349 0.0445 0.044" mass="0.008"/>
     </link>
     <joint name="thigh_r_middle_passive" type="revolute">
@@ -83,11 +79,10 @@
       <origin xyz="-0.0185 -0.02925 -0.0305" rpy="0 -0.785398163 0"/>
       <axis xyz="0 1 0"/>
-      <limit effort="1000.0" lower="-3.1" upper="3.1" velocity="10.0"/>
-      <dynamics damping="0.0" friction="0.0"/>
+      <limit effort="0.0" lower="-3.1" upper="3.1" velocity="100.0"/>
+      <dynamics damping="0" friction="0.0"/>
       <mimic joint="thigh_r_active" multiplier="1" offset="0"/>
     </joint>
     <xacro:if value="$(arg gazebo)">
-      <xacro:gazebo_poassive_joint name="thigh_r_middle_passive_loop" xyz="-0.0335 0 0"
-        parent="knee_r_passive_link" child="thigh_r_middle_passive_link"/>
+      <xacro:gazebo_poassive_joint name="thigh_r_middle_passive_loop" xyz="-0.0335 0 0" parent="knee_r_passive_link" child="thigh_r_middle_passive_link" axis="0 1 0"/>
     </xacro:if>
     <link name="thigh_r_middle_passive_link">
@@ -107,6 +102,6 @@
         <origin xyz="0 0 -0.03" rpy="0 -1.832597551 0"/>
         <axis xyz="0 1 0"/>
-        <limit effort="1000.0" lower="-3.1" upper="3.1" velocity="10.0"/>
-        <dynamics damping="0.0" friction="0.0"/>
+        <limit effort="0.0" lower="-3.1" upper="3.1" velocity="100.0"/>
+        <dynamics damping="0" friction="0.0"/>
         <mimic joint="shin_r_active" multiplier="-1" offset="0"/>
       </joint>
@@ -117,6 +112,6 @@
         <origin xyz="0 0 0" rpy="0 0 0"/>
         <axis xyz="0 1 0"/>
-        <limit effort="1000.0" lower="-3.1" upper="3.1" velocity="10.0"/>
-        <dynamics damping="0.0" friction="0.0"/>
+        <limit effort="0.0" lower="-3.1" upper="3.1" velocity="100.0"/>
+        <dynamics damping="0" friction="0.0"/>
         <mimic joint="thigh_r_active" multiplier="1" offset="0"/>
       </joint>
@@ -128,9 +123,8 @@
         <origin xyz="0 0 -0.03" rpy="0 -1.832597551 0"/>
         <axis xyz="0 1 0"/>
-        <limit effort="1000.0" lower="-0.9948" upper="1.5708" velocity="10.0"/>
-        <dynamics damping="0.0" friction="0.0"/>
+        <limit effort="0.0" lower="-0.9948" upper="1.5708" velocity="100.0"/>
+        <dynamics damping="0" friction="0.0"/>
       </joint>
-      <xacro:gazebo_poassive_joint name="thigh_r_rear_passive_loop" xyz="-0.00765471 0 -0.02897777"
-        parent="shin_r_rear_passive_link" child="thigh_r_rear_passive_link"/>
+      <xacro:gazebo_poassive_joint name="thigh_r_rear_passive_loop" xyz="-0.00765471 0 -0.02897777" parent="shin_r_rear_passive_link" child="thigh_r_rear_passive_link" axis="0 1 0"/>
     </xacro:if>
     <link name="thigh_r_rear_passive_link">
@@ -149,6 +143,6 @@
       <origin xyz="0 0 -0.1" rpy="0 0.785398163 0"/>
       <axis xyz="0 1 0"/>
-      <limit effort="1000.0" lower="-1.8588" upper="0.4974" velocity="10.0"/>
-      <dynamics damping="0.0" friction="0.0"/>
+      <limit effort="0.0" lower="-1.8588" upper="0.4974" velocity="100.0"/>
+      <dynamics damping="0" friction="0.0"/>
       <mimic joint="thigh_r_active" multiplier="-1" offset="0"/>
     </joint>
@@ -168,6 +162,6 @@
       <origin xyz="0 0 0" rpy="0 0.785398163 0"/>
       <axis xyz="0 1 0"/>
-      <limit effort="1000.0" lower="-1.8588" upper="0.4974" velocity="10.0"/>
-      <dynamics damping="0.0" friction="0.0"/>
+      <limit effort="0.0" lower="-1.8588" upper="0.4974" velocity="100.0"/>
+      <dynamics damping="0" friction="0.0"/>
       <mimic joint="shin_r_active" multiplier="1" offset="0"/>
     </joint>
@@ -187,11 +181,10 @@
       <origin xyz="-0.0335 0 0" rpy="0 0.785398163 0"/>
       <axis xyz="0 1 0"/>
-      <limit effort="1000.0" lower="-1.8588" upper="0.4974" velocity="10.0"/>
-      <dynamics damping="0.0" friction="0.0"/>
+      <limit effort="0.0" lower="-1.8588" upper="0.4974" velocity="100.0"/>
+      <dynamics damping="0" friction="0.0"/>
       <mimic joint="shin_r_active" multiplier="1" offset="0"/>
     </joint>
     <xacro:if value="$(arg gazebo)">
-      <xacro:gazebo_poassive_joint name="shin_r_rear_passive_loop" xyz="-0.0335 0 0"
-        parent="ankle_r_pitch_passive_link" child="shin_r_rear_passive_link"/>
+      <xacro:gazebo_poassive_joint name="shin_r_rear_passive_loop" xyz="-0.0335 0 0" parent="ankle_r_pitch_passive_link" child="shin_r_rear_passive_link" axis="0 1 0"/>
     </xacro:if>
     <link name="shin_r_rear_passive_link">
@@ -210,6 +203,6 @@
       <origin xyz="0 0 -0.1" rpy="0 -0.785398163 0"/>
       <axis xyz="0 1 0"/>
-      <limit effort="1000.0" lower="-0.4974" upper="1.8588" velocity="10.0"/>
-      <dynamics damping="0.0" friction="0.0"/>
+      <limit effort="0.0" lower="-0.4974" upper="1.8588" velocity="100.0"/>
+      <dynamics damping="0" friction="0.0"/>
       <mimic joint="shin_r_active" multiplier="-1" offset="0"/>
     </joint>
@@ -222,6 +215,5 @@
       </visual>
       <xacro:box_collision xyz="-0.0285 0 -0.013" rpy="0 0 0" size="0.0855 0.0325 0.0465"/>
-      <xacro:box_inertial xyz="-0.0285 0 -0.013" rpy="0 0 0" size="0.0855 0.0325 0.0465"
-        mass="0.104"/>
+      <xacro:box_inertial xyz="-0.0285 0 -0.013" rpy="0 0 0" size="0.0855 0.0325 0.0465" mass="0.104"/>
     </link>
     <joint name="ankle_r_roll" type="revolute">
@@ -230,6 +222,6 @@
       <origin xyz="-0.015 0 -0.027" rpy="0 0 0"/>
       <axis xyz="1 0 0"/>
-      <limit effort="1000.0" lower="-0.3704" upper="1.5708" velocity="10.0"/>
-      <dynamics damping="0.0" friction="0.0"/>
+      <limit effort="3.1" lower="-0.3704" upper="1.5708" velocity="6.5"/>
+      <dynamics damping="0.476923" friction="0.0"/>
     </joint>
     <link name="ankle_r_roll_link">
@@ -241,6 +233,5 @@
       </visual>
       <xacro:box_collision xyz="0 -0.009375 -0.01175" rpy="0 0 0" size="0.0365 0.05375 0.043"/>
-      <xacro:box_inertial xyz="0 -0.009375 -0.01175" rpy="0 0 0" size="0.0365 0.05375 0.043"
-        mass="0.136"/>
+      <xacro:box_inertial xyz="0 -0.009375 -0.01175" rpy="0 0 0" size="0.0365 0.05375 0.043" mass="0.136"/>
     </link>
     <joint name="ankle_r_yaw" type="revolute">
@@ -248,7 +239,7 @@
       <child link="ankle_r_yaw_link"/>
       <origin xyz="0 0 -0.03825" rpy="0 0 0"/>
-      <axis xyz="0 0 -1"/>
-      <limit effort="1000.0" lower="-3.1" upper="3.1" velocity="10.0"/>
-      <dynamics damping="0.0" friction="0.0"/>
+      <axis xyz="0 0 1"/>
+      <limit effort="3.1" lower="-3.1" upper="3.1" velocity="6.5"/>
+      <dynamics damping="0.476923" friction="0.0"/>
     </joint>
     <link name="ankle_r_yaw_link">
