Commit message: Update joint torque and speed

File: kuroko_description/xacro/kuroko/parts/arm_l.xacro (robot description, xacro)
@@ -8,6 +8,6 @@
       <origin xyz="0 0.128 0.01275" rpy="0 0 0"/>
       <axis xyz="0 1 0"/>
-      <limit effort="1000.0" lower="-3.1" upper="3.1" velocity="10.0"/>
-      <dynamics damping="0.0" friction="0.0"/>
+      <limit effort="3.1" lower="-3.14" upper="3.14" velocity="6.5"/>
+      <dynamics damping="0.477" friction="0.0"/>
     </joint>
     <link name="shoulder_l_pitch_link">
@@ -26,6 +26,6 @@
       <origin xyz="0 0.05425 0" rpy="1.5708 0 0"/>
       <axis xyz="1 0 0"/>
-      <limit effort="1000.0" lower="-3.1" upper="3.1" velocity="10.0"/>
-      <dynamics damping="0.0" friction="0.0"/>
+      <limit effort="8.9" lower="-3.14" upper="3.14" velocity="6.9"/>
+      <dynamics damping="1.29" friction="0.0"/>
     </joint>
     <link name="shoulder_l_roll_link">
@@ -44,6 +44,6 @@
       <origin xyz="0 -0.023 -0.036" rpy="0 0 0"/>
       <axis xyz="0 -1 0"/>
-      <limit effort="1000.0" lower="-2.6180" upper="2.6180" velocity="10.0"/>
-      <dynamics damping="0.0" friction="0.0"/>
+      <limit effort="3.1" lower="-2.6180" upper="2.6180" velocity="6.5"/>
+      <dynamics damping="0.477" friction="0.0"/>
     </joint>
     <link name="elbow_l_front_link">
@@ -63,6 +63,6 @@
       <origin xyz="0 -0.024 -0.036" rpy="0 0 0"/>
       <axis xyz="0 1 0"/>
-      <limit effort="1000.0" lower="-2.6180" upper="2.6180" velocity="10.0"/>
-      <dynamics damping="0.0" friction="0.0"/>
+      <limit effort="3.1" lower="-2.6180" upper="2.6180" velocity="6.5"/>
+      <dynamics damping="0.477" friction="0.0"/>
     </joint>
     <link name="elbow_l_rear_link">

File: kuroko_description/xacro/kuroko/parts/arm_r.xacro (robot description, xacro)
@@ -8,6 +8,6 @@
       <origin xyz="0 -0.128 0.01275" rpy="0 0 0"/>
       <axis xyz="0 -1 0"/>
-      <limit effort="1000.0" lower="-3.1" upper="3.1" velocity="10.0"/>
-      <dynamics damping="0.0" friction="0.0"/>
+      <limit effort="3.1" lower="-3.14" upper="3.14" velocity="6.5"/>
+      <dynamics damping="0.477" friction="0.0"/>
     </joint>
     <link name="shoulder_r_pitch_link">
@@ -26,6 +26,6 @@
       <origin xyz="0 -0.05425 0" rpy="-1.5708 0 0"/>
       <axis xyz="1 0 0"/>
-      <limit effort="1000.0" lower="-3.1" upper="3.1" velocity="10.0"/>
-      <dynamics damping="0.0" friction="0.0"/>
+      <limit effort="8.9" lower="-3.14" upper="3.14" velocity="6.9"/>
+      <dynamics damping="1.29" friction="0.0"/>
     </joint>
     <link name="shoulder_r_roll_link">
@@ -44,6 +44,6 @@
       <origin xyz="0 0.023 -0.036" rpy="0 0 0"/>
       <axis xyz="0 1 0"/>
-      <limit effort="1000.0" lower="-2.6180" upper="2.6180" velocity="10.0"/>
-      <dynamics damping="0.0" friction="0.0"/>
+      <limit effort="3.1" lower="-2.6180" upper="2.6180" velocity="6.5"/>
+      <dynamics damping="0.477" friction="0.0"/>
     </joint>
     <link name="elbow_r_front_link">
@@ -63,6 +63,6 @@
       <origin xyz="0 0.024 -0.036" rpy="0 0 0"/>
       <axis xyz="0 -1 0"/>
-      <limit effort="1000.0" lower="-2.6180" upper="2.6180" velocity="10.0"/>
-      <dynamics damping="0.0" friction="0.0"/>
+      <limit effort="3.1" lower="-2.6180" upper="2.6180" velocity="6.5"/>
+      <dynamics damping="0.477" friction="0.0"/>
     </joint>
     <link name="elbow_r_rear_link">

File: kuroko_description/xacro/kuroko/parts/body.xacro (robot description, xacro)
@@ -19,6 +19,6 @@
       <origin xyz="0 0 0" rpy="0 0 0"/>
       <axis xyz="0 0 1"/>
-      <limit effort="1000.0" lower="-3.1" upper="3.1" velocity="10.0"/>
-      <dynamics damping="0.0" friction="0.0"/>
+      <limit effort="3.1" lower="-3.14" upper="3.14" velocity="6.5"/>
+      <dynamics damping="0.477" friction="0.0"/>
     </joint>
     <!-- chest -->

Commit message: Use stl

File: kuroko_description/xacro/kuroko/parts/arm_l.xacro (robot description, xacro)
@@ -16,5 +16,5 @@
           <origin xyz="0 0 0" rpy="0 0 0"/>
           <geometry>
-            <mesh filename="${MESH_DIR}/kuroko/obj/shoulder_l_pitch.obj"/>
+            <mesh filename="${MESH_DIR}/kuroko/stl/shoulder_l_pitch.stl"/>
           </geometry>
         </visual>
@@ -39,5 +39,5 @@
           <origin xyz="0 0 0" rpy="0 0 0"/>
           <geometry>
-            <mesh filename="${MESH_DIR}/kuroko/obj/shoulder_l_roll.obj"/>
+            <mesh filename="${MESH_DIR}/kuroko/stl/shoulder_l_roll.stl"/>
           </geometry>
         </visual>
@@ -62,5 +62,5 @@
           <origin xyz="0 0 0" rpy="0 0 0"/>
           <geometry>
-            <mesh filename="${MESH_DIR}/kuroko/obj/elbow_l_front.obj"/>
+            <mesh filename="${MESH_DIR}/kuroko/stl/elbow_l_front.stl"/>
           </geometry>
         </visual>
@@ -87,5 +87,5 @@
           <origin xyz="0 0 0" rpy="0 0 0"/>
           <geometry>
-            <mesh filename="${MESH_DIR}/kuroko/obj/elbow_l_rear.obj"/>
+            <mesh filename="${MESH_DIR}/kuroko/stl/elbow_l_rear.stl"/>
           </geometry>
         </visual>

File: kuroko_description/xacro/kuroko/parts/arm_r.xacro (robot description, xacro)
@@ -16,5 +16,5 @@
           <origin xyz="0 0 0" rpy="0 0 0"/>
           <geometry>
-            <mesh filename="${MESH_DIR}/kuroko/obj/shoulder_r_pitch.obj"/>
+            <mesh filename="${MESH_DIR}/kuroko/stl/shoulder_r_pitch.stl"/>
           </geometry>
         </visual>
@@ -39,5 +39,5 @@
           <origin xyz="0 0 0" rpy="0 0 0"/>
           <geometry>
-            <mesh filename="${MESH_DIR}/kuroko/obj/shoulder_r_roll.obj"/>
+            <mesh filename="${MESH_DIR}/kuroko/stl/shoulder_r_roll.stl"/>
           </geometry>
         </visual>
@@ -62,5 +62,5 @@
           <origin xyz="0 0 0" rpy="0 0 0"/>
           <geometry>
-            <mesh filename="${MESH_DIR}/kuroko/obj/elbow_r_front.obj"/>
+            <mesh filename="${MESH_DIR}/kuroko/stl/elbow_r_front.stl"/>
           </geometry>
         </visual>
@@ -87,5 +87,5 @@
           <origin xyz="0 0 0" rpy="0 0 0"/>
           <geometry>
-            <mesh filename="${MESH_DIR}/kuroko/obj/elbow_r_rear.obj"/>
+            <mesh filename="${MESH_DIR}/kuroko/stl/elbow_r_rear.stl"/>
           </geometry>
         </visual>

File: kuroko_description/xacro/kuroko/parts/body.xacro (robot description, xacro)
@@ -8,5 +8,5 @@
           <origin xyz="0 0 0" rpy="0 0 0"/>
           <geometry>
-            <mesh filename="${MESH_DIR}/kuroko/obj/waist.obj"/>
+            <mesh filename="${MESH_DIR}/kuroko/stl/waist.stl"/>
           </geometry>
         </visual>
@@ -33,5 +33,5 @@
           <origin xyz="0 0 0" rpy="0 0 0"/>
           <geometry>
-            <mesh filename="${MESH_DIR}/kuroko/obj/chest.obj"/>
+            <mesh filename="${MESH_DIR}/kuroko/stl/chest.stl"/>
           </geometry>
         </visual>

File: kuroko_description/xacro/kuroko/parts/leg_l.xacro (robot description, xacro)
@@ -16,5 +16,5 @@
           <origin xyz="0 0 0" rpy="0 0 0"/>
           <geometry>
-            <mesh filename="${MESH_DIR}/kuroko/obj/hip_l_roll.obj"/>
+            <mesh filename="${MESH_DIR}/kuroko/stl/hip_l_roll.stl"/>
           </geometry>
         </visual>
@@ -40,5 +40,5 @@
           <origin xyz="0 0 0" rpy="0 0 0"/>
           <geometry>
-            <mesh filename="${MESH_DIR}/kuroko/obj/hip_l_pitch.obj"/>
+            <mesh filename="${MESH_DIR}/kuroko/stl/hip_l_pitch.stl"/>
           </geometry>
         </visual>
@@ -64,5 +64,5 @@
           <origin xyz="0 0 0" rpy="0 0 0"/>
           <geometry>
-            <mesh filename="${MESH_DIR}/kuroko/obj/shin_l_active.obj"/>
+            <mesh filename="${MESH_DIR}/kuroko/stl/shin_l_active.stl"/>
           </geometry>
         </visual>
@@ -88,5 +88,5 @@
           <origin xyz="0 0 0" rpy="0 0 0"/>
           <geometry>
-            <mesh filename="${MESH_DIR}/kuroko/obj/thigh_l_active.obj"/>
+            <mesh filename="${MESH_DIR}/kuroko/stl/thigh_l_active.stl"/>
           </geometry>
         </visual>
@@ -134,5 +134,5 @@
           <origin xyz="0 0 0" rpy="0 0 0"/>
           <geometry>
-            <mesh filename="package://kuroko_description/meshes/kuroko/obj/shin_r_front_passive.obj"/>
+            <mesh filename="package://kuroko_description/meshes/kuroko/stl/shin_r_front_passive.stl"/>
           </geometry>
         </visual>
@@ -158,5 +158,5 @@
           <origin xyz="0 0 0" rpy="0 0 0"/>
           <geometry>
-            <mesh filename="${MESH_DIR}/kuroko/obj/thigh_r_middle_passive.obj"/>
+            <mesh filename="${MESH_DIR}/kuroko/stl/thigh_r_middle_passive.stl"/>
           </geometry>
         </visual>
@@ -204,5 +204,5 @@
           <origin xyz="0 0 0" rpy="0 0 0"/>
           <geometry>
-            <mesh filename="${MESH_DIR}/kuroko/obj/shin_r_rear_passive.obj"/>
+            <mesh filename="${MESH_DIR}/kuroko/stl/shin_r_rear_passive.stl"/>
           </geometry>
         </visual>
@@ -228,5 +228,5 @@
           <origin xyz="0.0335 0 0" rpy="0 0 0"/>
           <geometry>
-            <mesh filename="${MESH_DIR}/kuroko/obj/knee_r_passive.obj"/>
+            <mesh filename="${MESH_DIR}/kuroko/stl/knee_r_passive.stl"/>
           </geometry>
         </visual>
@@ -278,5 +278,5 @@
           <origin xyz="0 0 0.1" rpy="0 0 0"/>
           <geometry>
-            <mesh filename="${MESH_DIR}/kuroko/obj/thigh_r_rear_passive.obj"/>
+            <mesh filename="${MESH_DIR}/kuroko/stl/thigh_r_rear_passive.stl"/>
           </geometry>
         </visual>
@@ -306,5 +306,5 @@
           <origin xyz="0.0335 0 0" rpy="0 0 0"/>
           <geometry>
-            <mesh filename="${MESH_DIR}/kuroko/obj/ankle_r_pitch_passive.obj"/>
+            <mesh filename="${MESH_DIR}/kuroko/stl/ankle_r_pitch_passive.stl"/>
           </geometry>
         </visual>
@@ -333,5 +333,5 @@
           <origin xyz="0 0 0" rpy="0 0 0"/>
           <geometry>
-            <mesh filename="${MESH_DIR}/kuroko/obj/ankle_l_roll.obj"/>
+            <mesh filename="${MESH_DIR}/kuroko/stl/ankle_l_roll.stl"/>
           </geometry>
         </visual>
@@ -357,5 +357,5 @@
           <origin xyz="0 0 0" rpy="0 0 0"/>
           <geometry>
-            <mesh filename="${MESH_DIR}/kuroko/obj/ankle_r_yaw.obj"/>
+            <mesh filename="${MESH_DIR}/kuroko/stl/ankle_r_yaw.stl"/>
           </geometry>
         </visual>

File: kuroko_description/xacro/kuroko/parts/leg_r.xacro (robot description, xacro)
@@ -16,5 +16,5 @@
           <origin xyz="0 0 0" rpy="0 0 0"/>
           <geometry>
-            <mesh filename="${MESH_DIR}/kuroko/obj/hip_r_roll.obj"/>
+            <mesh filename="${MESH_DIR}/kuroko/stl/hip_r_roll.stl"/>
           </geometry>
         </visual>
@@ -40,5 +40,5 @@
           <origin xyz="0 0 0" rpy="0 0 0"/>
           <geometry>
-            <mesh filename="${MESH_DIR}/kuroko/obj/hip_r_pitch.obj"/>
+            <mesh filename="${MESH_DIR}/kuroko/stl/hip_r_pitch.stl"/>
           </geometry>
         </visual>
@@ -64,5 +64,5 @@
           <origin xyz="0 0 0" rpy="0 0 0"/>
           <geometry>
-            <mesh filename="${MESH_DIR}/kuroko/obj/shin_r_active.obj"/>
+            <mesh filename="${MESH_DIR}/kuroko/stl/shin_r_active.stl"/>
           </geometry>
         </visual>
@@ -88,5 +88,5 @@
           <origin xyz="0 0 0" rpy="0 0 0"/>
           <geometry>
-            <mesh filename="${MESH_DIR}/kuroko/obj/thigh_r_active.obj"/>
+            <mesh filename="${MESH_DIR}/kuroko/stl/thigh_r_active.stl"/>
           </geometry>
         </visual>
@@ -134,5 +134,5 @@
           <origin xyz="0 0 0" rpy="0 0 0"/>
           <geometry>
-            <mesh filename="${MESH_DIR}/kuroko/obj/shin_r_front_passive.obj"/>
+            <mesh filename="${MESH_DIR}/kuroko/stl/shin_r_front_passive.stl"/>
           </geometry>
         </visual>
@@ -158,5 +158,5 @@
           <origin xyz="0 0 0" rpy="0 0 0"/>
           <geometry>
-            <mesh filename="${MESH_DIR}/kuroko/obj/thigh_r_middle_passive.obj"/>
+            <mesh filename="${MESH_DIR}/kuroko/stl/thigh_r_middle_passive.stl"/>
           </geometry>
         </visual>
@@ -204,5 +204,5 @@
           <origin xyz="0 0 0" rpy="0 0 0"/>
           <geometry>
-            <mesh filename="${MESH_DIR}/kuroko/obj/shin_r_rear_passive.obj"/>
+            <mesh filename="${MESH_DIR}/kuroko/stl/shin_r_rear_passive.stl"/>
           </geometry>
         </visual>
@@ -228,5 +228,5 @@
           <origin xyz="0.0335 0 0" rpy="0 0 0"/>
           <geometry>
-            <mesh filename="${MESH_DIR}/kuroko/obj/knee_r_passive.obj"/>
+            <mesh filename="${MESH_DIR}/kuroko/stl/knee_r_passive.stl"/>
           </geometry>
         </visual>
@@ -278,5 +278,5 @@
           <origin xyz="0 0 0.1" rpy="0 0 0"/>
           <geometry>
-            <mesh filename="${MESH_DIR}/kuroko/obj/thigh_r_rear_passive.obj"/>
+            <mesh filename="${MESH_DIR}/kuroko/stl/thigh_r_rear_passive.stl"/>
           </geometry>
         </visual>
@@ -306,5 +306,5 @@
           <origin xyz="0.0335 0 0" rpy="0 0 0"/>
           <geometry>
-            <mesh filename="${MESH_DIR}/kuroko/obj/ankle_r_pitch_passive.obj"/>
+            <mesh filename="${MESH_DIR}/kuroko/stl/ankle_r_pitch_passive.stl"/>
           </geometry>
         </visual>
@@ -334,5 +334,5 @@
           <origin xyz="0 0 0" rpy="0 0 0"/>
           <geometry>
-            <mesh filename="${MESH_DIR}/kuroko/obj/ankle_r_roll.obj"/>
+            <mesh filename="${MESH_DIR}/kuroko/stl/ankle_r_roll.stl"/>
           </geometry>
         </visual>
@@ -358,5 +358,5 @@
           <origin xyz="0 0 0" rpy="0 0 0"/>
           <geometry>
-            <mesh filename="${MESH_DIR}/kuroko/obj/ankle_r_yaw.obj"/>
+            <mesh filename="${MESH_DIR}/kuroko/stl/ankle_r_yaw.stl"/>
           </geometry>
         </visual>
