Commit message: rename links

File: kuroko_description/xacro/kuroko/parts/leg_l.xacro (robot description, xacro)
@@ -41,7 +41,7 @@
         mass="0.478"/>
     </link>
-    <joint name="thigh_l_02_joint" type="revolute">
+    <joint name="thigh_l_active_joint" type="revolute">
       <parent link="hip_l_pitch"/>
-      <child link="thigh_l_02"/>
+      <child link="thigh_l_active"/>
       <origin xyz="0.015 0.02925 -0.0305" rpy="0 -0.785398163 0"/>
       <axis xyz="0 -1 0"/>
@@ -49,9 +49,9 @@
       <dynamics damping="0.0" friction="0.0"/>
     </joint>
-    <link name="thigh_l_02">
-      <visual>
-        <origin xyz="0 0 0" rpy="0 0 0"/>
-        <geometry>
-          <mesh filename="package://kuroko_description/meshes/kuroko/obj/thigh_l_02.obj"/>
+    <link name="thigh_l_active">
+      <visual>
+        <origin xyz="0 0 0" rpy="0 0 0"/>
+        <geometry>
+          <mesh filename="package://kuroko_description/meshes/kuroko/obj/thigh_l_active.obj"/>
         </geometry>
       </visual>
@@ -59,7 +59,7 @@
       <xacro:box_inertial xyz="0 0 -0.05" rpy="0 0 0" size="0.014 0.0445 0.114" mass="0.012"/>
     </link>
-    <joint name="thigh_l_03_joint" type="revolute">
+    <joint name="shin_l_active_joint" type="revolute">
       <parent link="hip_l_pitch"/>
-      <child link="thigh_l_03"/>
+      <child link="shin_l_active"/>
       <origin xyz="-0.0185 0.02925 -0.0305" rpy="0 1.047197551 0"/>
       <axis xyz="0 -1 0"/>
@@ -67,9 +67,9 @@
       <dynamics damping="0.0" friction="0.0"/>
     </joint>
-    <link name="thigh_l_03">
-      <visual>
-        <origin xyz="0 0 0" rpy="0 0 0"/>
-        <geometry>
-          <mesh filename="package://kuroko_description/meshes/kuroko/obj/thigh_l_03.obj"/>
+    <link name="shin_l_active">
+      <visual>
+        <origin xyz="0 0 0" rpy="0 0 0"/>
+        <geometry>
+          <mesh filename="package://kuroko_description/meshes/kuroko/obj/shin_l_active.obj"/>
         </geometry>
       </visual>
@@ -78,22 +78,22 @@
         mass="0.008"/>
     </link>
-    <joint name="thigh_l_04_joint" type="revolute">
+    <joint name="thigh_l_passive_middle_joint" type="revolute">
       <parent link="hip_l_pitch"/>
-      <child link="thigh_l_04"/>
+      <child link="thigh_l_passive_middle"/>
       <origin xyz="-0.0185 0.02925 -0.0305" rpy="0 -0.785398163 0"/>
       <axis xyz="0 -1 0"/>
       <limit effort="1000.0" lower="-3.1" upper="3.1" velocity="10.0"/>
       <dynamics damping="0.0" friction="0.0"/>
-      <mimic joint="thigh_l_02_joint" multiplier="1" offset="0"/>
+      <mimic joint="thigh_l_active_joint" multiplier="1" offset="0"/>
     </joint>
     <xacro:if value="$(arg gazebo)">
-      <xacro:gazebo_poassive_joint name="thigh_l_04_loop" xyz="-0.0335 0 0"
-        parent="knee_l" child="thigh_l_04" axis="0 -1 0"/>
+      <xacro:gazebo_poassive_joint name="thigh_l_passive_middle_loop" xyz="-0.0335 0 0"
+        parent="knee_l" child="thigh_l_passive_middle" axis="0 -1 0"/>
     </xacro:if>
-    <link name="thigh_l_04">
-      <visual>
-        <origin xyz="0 0 0" rpy="0 0 0"/>
-        <geometry>
-          <mesh filename="package://kuroko_description/meshes/kuroko/obj/thigh_r_04.obj"/>
+    <link name="thigh_l_passive_middle">
+      <visual>
+        <origin xyz="0 0 0" rpy="0 0 0"/>
+        <geometry>
+          <mesh filename="package://kuroko_description/meshes/kuroko/obj/thigh_r_passive_middle.obj"/>
         </geometry>
       </visual>
@@ -102,28 +102,28 @@
     </link>
     <xacro:unless value="$(arg gazebo)">
-      <joint name="thigh_l_05_mimic1" type="revolute">
-        <parent link="thigh_l_03"/>
-        <child link="thigh_l_05_mimic"/>
+      <joint name="thigh_l_passive_rear_mimic1" type="revolute">
+        <parent link="shin_l_active"/>
+        <child link="thigh_l_passive_rear_mimic"/>
         <origin xyz="0 0 -0.03" rpy="0 -1.832597551 0"/>
         <axis xyz="0 -1 0"/>
         <limit effort="1000.0" lower="-3.1" upper="3.1" velocity="10.0"/>
         <dynamics damping="0.0" friction="0.0"/>
-        <mimic joint="thigh_l_03_joint" multiplier="-1" offset="0"/>
+        <mimic joint="shin_l_active_joint" multiplier="-1" offset="0"/>
       </joint>
-      <link name="thigh_l_05_mimic"/>
-      <joint name="thigh_l_05_mimic2" type="revolute">
-        <parent link="thigh_l_05_mimic"/>
-        <child link="thigh_l_05"/>
+      <link name="thigh_l_passive_rear_mimic"/>
+      <joint name="thigh_l_passive_rear_mimic2" type="revolute">
+        <parent link="thigh_l_passive_rear_mimic"/>
+        <child link="thigh_l_passive_rear"/>
         <origin xyz="0 0 0" rpy="0 0 0"/>
         <axis xyz="0 -1 0"/>
         <limit effort="1000.0" lower="-3.1" upper="3.1" velocity="10.0"/>
         <dynamics damping="0.0" friction="0.0"/>
-        <mimic joint="thigh_l_02_joint" multiplier="1" offset="0"/>
+        <mimic joint="thigh_l_active_joint" multiplier="1" offset="0"/>
       </joint>
     </xacro:unless>
     <xacro:if value="$(arg gazebo)">
-      <joint name="thigh_l_05_joint" type="revolute">
-        <parent link="thigh_l_03"/>
-        <child link="thigh_l_05"/>
+      <joint name="thigh_l_passive_rear_joint" type="revolute">
+        <parent link="shin_l_active"/>
+        <child link="thigh_l_passive_rear"/>
         <origin xyz="0 0 -0.03" rpy="0 -1.832597551 0"/>
         <axis xyz="0 -1 0"/>
@@ -131,12 +131,12 @@
         <dynamics damping="0.0" friction="0.0"/>
       </joint>
-      <xacro:gazebo_poassive_joint name="thigh_l_05_loop" xyz="-0.00765471 0 -0.02897777"
-        parent="leg_l_02" child="thigh_l_05" axis="0 -1 0"/>
+      <xacro:gazebo_poassive_joint name="thigh_l_passive_rear_loop" xyz="-0.00765471 0 -0.02897777"
+        parent="leg_l_02" child="thigh_l_passive_rear" axis="0 -1 0"/>
     </xacro:if>
-    <link name="thigh_l_05">
-      <visual>
-        <origin xyz="0 0 0" rpy="0 0 0"/>
-        <geometry>
-          <mesh filename="package://kuroko_description/meshes/kuroko/obj/thigh_r_05.obj"/>
+    <link name="thigh_l_passive_rear">
+      <visual>
+        <origin xyz="0 0 0" rpy="0 0 0"/>
+        <geometry>
+          <mesh filename="package://kuroko_description/meshes/kuroko/obj/thigh_r_passive_rear.obj"/>
         </geometry>
       </visual>
@@ -145,5 +145,5 @@
     </link>
     <joint name="knee_l_joint" type="revolute">
-      <parent link="thigh_l_02"/>
+      <parent link="thigh_l_active"/>
       <child link="knee_l"/>
       <origin xyz="0 0 -0.1" rpy="0 0.785398163 0"/>
@@ -151,5 +151,5 @@
       <limit effort="1000.0" lower="-0.4974" upper="1.8588" velocity="10.0"/>
       <dynamics damping="0.0" friction="0.0"/>
-      <mimic joint="thigh_l_02_joint" multiplier="-1" offset="0"/>
+      <mimic joint="thigh_l_active_joint" multiplier="-1" offset="0"/>
     </joint>
     <link name="knee_l">
@@ -170,5 +170,5 @@
       <limit effort="1000.0" lower="-0.4974" upper="1.8588" velocity="10.0"/>
       <dynamics damping="0.0" friction="0.0"/>
-      <mimic joint="thigh_l_03_joint" multiplier="1" offset="0"/>
+      <mimic joint="shin_l_active_joint" multiplier="1" offset="0"/>
     </joint>
     <link name="leg_l_01">
@@ -189,5 +189,5 @@
       <limit effort="1000.0" lower="-0.4974" upper="1.8588" velocity="10.0"/>
       <dynamics damping="0.0" friction="0.0"/>
-      <mimic joint="thigh_l_03_joint" multiplier="1" offset="0"/>
+      <mimic joint="shin_l_active_joint" multiplier="1" offset="0"/>
     </joint>
     <xacro:if value="$(arg gazebo)">
@@ -212,5 +212,5 @@
       <limit effort="1000.0" lower="-1.8588" upper="0.4974" velocity="10.0"/>
       <dynamics damping="0.0" friction="0.0"/>
-      <mimic joint="thigh_l_03_joint" multiplier="-1" offset="0"/>
+      <mimic joint="shin_l_active_joint" multiplier="-1" offset="0"/>
     </joint>
     <link name="ankle_l_01">

File: kuroko_description/xacro/kuroko/parts/leg_r.xacro (robot description, xacro)
@@ -41,7 +41,7 @@
         mass="0.478"/>
     </link>
-    <joint name="thigh_r_02_joint" type="revolute">
+    <joint name="thigh_r_active_joint" type="revolute">
       <parent link="hip_r_pitch"/>
-      <child link="thigh_r_02"/>
+      <child link="thigh_r_active"/>
       <origin xyz="0.015 -0.02925 -0.0305" rpy="0 -0.785398163 0"/>
       <axis xyz="0 1 0"/>
@@ -49,9 +49,9 @@
       <dynamics damping="0.0" friction="0.0"/>
     </joint>
-    <link name="thigh_r_02">
-      <visual>
-        <origin xyz="0 0 0" rpy="0 0 0"/>
-        <geometry>
-          <mesh filename="package://kuroko_description/meshes/kuroko/obj/thigh_r_02.obj"/>
+    <link name="thigh_r_active">
+      <visual>
+        <origin xyz="0 0 0" rpy="0 0 0"/>
+        <geometry>
+          <mesh filename="package://kuroko_description/meshes/kuroko/obj/thigh_r_active.obj"/>
         </geometry>
       </visual>
@@ -59,7 +59,7 @@
       <xacro:box_inertial xyz="0 0 -0.05" rpy="0 0 0" size="0.014 0.0445 0.114" mass="0.012"/>
     </link>
-    <joint name="thigh_r_03_joint" type="revolute">
+    <joint name="shin_r_active_joint" type="revolute">
       <parent link="hip_r_pitch"/>
-      <child link="thigh_r_03"/>
+      <child link="shin_r_active"/>
       <origin xyz="-0.0185 -0.02925 -0.0305" rpy="0 1.047197551 0"/>
       <axis xyz="0 1 0"/>
@@ -67,9 +67,9 @@
       <dynamics damping="0.0" friction="0.0"/>
     </joint>
-    <link name="thigh_r_03">
-      <visual>
-        <origin xyz="0 0 0" rpy="0 0 0"/>
-        <geometry>
-          <mesh filename="package://kuroko_description/meshes/kuroko/obj/thigh_r_03.obj"/>
+    <link name="shin_r_active">
+      <visual>
+        <origin xyz="0 0 0" rpy="0 0 0"/>
+        <geometry>
+          <mesh filename="package://kuroko_description/meshes/kuroko/obj/shin_r_active.obj"/>
         </geometry>
       </visual>
@@ -78,22 +78,22 @@
         mass="0.008"/>
     </link>
-    <joint name="thigh_r_04_joint" type="revolute">
+    <joint name="thigh_r_passive_middle_joint" type="revolute">
       <parent link="hip_r_pitch"/>
-      <child link="thigh_r_04"/>
+      <child link="thigh_r_passive_middle"/>
       <origin xyz="-0.0185 -0.02925 -0.0305" rpy="0 -0.785398163 0"/>
       <axis xyz="0 1 0"/>
       <limit effort="1000.0" lower="-3.1" upper="3.1" velocity="10.0"/>
       <dynamics damping="0.0" friction="0.0"/>
-      <mimic joint="thigh_r_02_joint" multiplier="1" offset="0"/>
+      <mimic joint="thigh_r_active_joint" multiplier="1" offset="0"/>
     </joint>
     <xacro:if value="$(arg gazebo)">
-      <xacro:gazebo_poassive_joint name="thigh_r_04_loop" xyz="-0.0335 0 0"
-        parent="knee_r" child="thigh_r_04"/>
+      <xacro:gazebo_poassive_joint name="thigh_r_passive_middle_loop" xyz="-0.0335 0 0"
+        parent="knee_r" child="thigh_r_passive_middle"/>
     </xacro:if>
-    <link name="thigh_r_04">
-      <visual>
-        <origin xyz="0 0 0" rpy="0 0 0"/>
-        <geometry>
-          <mesh filename="package://kuroko_description/meshes/kuroko/obj/thigh_r_04.obj"/>
+    <link name="thigh_r_passive_middle">
+      <visual>
+        <origin xyz="0 0 0" rpy="0 0 0"/>
+        <geometry>
+          <mesh filename="package://kuroko_description/meshes/kuroko/obj/thigh_r_passive_middle.obj"/>
         </geometry>
       </visual>
@@ -102,28 +102,28 @@
     </link>
     <xacro:unless value="$(arg gazebo)">
-      <joint name="thigh_r_05_mimic1" type="revolute">
-        <parent link="thigh_r_03"/>
-        <child link="thigh_r_05_mimic"/>
+      <joint name="thigh_r_passive_rear_mimic1" type="revolute">
+        <parent link="shin_r_active"/>
+        <child link="thigh_r_passive_rear_mimic"/>
         <origin xyz="0 0 -0.03" rpy="0 -1.832597551 0"/>
         <axis xyz="0 1 0"/>
         <limit effort="1000.0" lower="-3.1" upper="3.1" velocity="10.0"/>
         <dynamics damping="0.0" friction="0.0"/>
-        <mimic joint="thigh_r_03_joint" multiplier="-1" offset="0"/>
+        <mimic joint="shin_r_active_joint" multiplier="-1" offset="0"/>
       </joint>
-      <link name="thigh_r_05_mimic"/>
-      <joint name="thigh_r_05_mimic2" type="revolute">
-        <parent link="thigh_r_05_mimic"/>
-        <child link="thigh_r_05"/>
+      <link name="thigh_r_passive_rear_mimic"/>
+      <joint name="thigh_r_passive_rear_mimic2" type="revolute">
+        <parent link="thigh_r_passive_rear_mimic"/>
+        <child link="thigh_r_passive_rear"/>
         <origin xyz="0 0 0" rpy="0 0 0"/>
         <axis xyz="0 1 0"/>
         <limit effort="1000.0" lower="-3.1" upper="3.1" velocity="10.0"/>
         <dynamics damping="0.0" friction="0.0"/>
-        <mimic joint="thigh_r_02_joint" multiplier="1" offset="0"/>
+        <mimic joint="thigh_r_active_joint" multiplier="1" offset="0"/>
       </joint>
     </xacro:unless>
     <xacro:if value="$(arg gazebo)">
-      <joint name="thigh_r_05_joint" type="revolute">
-        <parent link="thigh_r_03"/>
-        <child link="thigh_r_05"/>
+      <joint name="thigh_r_passive_rear_joint" type="revolute">
+        <parent link="shin_r_active"/>
+        <child link="thigh_r_passive_rear"/>
         <origin xyz="0 0 -0.03" rpy="0 -1.832597551 0"/>
         <axis xyz="0 1 0"/>
@@ -131,12 +131,12 @@
         <dynamics damping="0.0" friction="0.0"/>
       </joint>
-      <xacro:gazebo_poassive_joint name="thigh_r_05_loop" xyz="-0.00765471 0 -0.02897777"
-        parent="leg_r_02" child="thigh_r_05"/>
+      <xacro:gazebo_poassive_joint name="thigh_r_passive_rear_loop" xyz="-0.00765471 0 -0.02897777"
+        parent="leg_r_02" child="thigh_r_passive_rear"/>
     </xacro:if>
-    <link name="thigh_r_05">
-      <visual>
-        <origin xyz="0 0 0" rpy="0 0 0"/>
-        <geometry>
-          <mesh filename="package://kuroko_description/meshes/kuroko/obj/thigh_r_05.obj"/>
+    <link name="thigh_r_passive_rear">
+      <visual>
+        <origin xyz="0 0 0" rpy="0 0 0"/>
+        <geometry>
+          <mesh filename="package://kuroko_description/meshes/kuroko/obj/thigh_r_passive_rear.obj"/>
         </geometry>
       </visual>
@@ -145,5 +145,5 @@
     </link>
     <joint name="knee_r_joint" type="revolute">
-      <parent link="thigh_r_02"/>
+      <parent link="thigh_r_active"/>
       <child link="knee_r"/>
       <origin xyz="0 0 -0.1" rpy="0 0.785398163 0"/>
@@ -151,5 +151,5 @@
       <limit effort="1000.0" lower="-1.8588" upper="0.4974" velocity="10.0"/>
       <dynamics damping="0.0" friction="0.0"/>
-      <mimic joint="thigh_r_02_joint" multiplier="-1" offset="0"/>
+      <mimic joint="thigh_r_active_joint" multiplier="-1" offset="0"/>
     </joint>
     <link name="knee_r">
@@ -170,5 +170,5 @@
       <limit effort="1000.0" lower="-1.8588" upper="0.4974" velocity="10.0"/>
       <dynamics damping="0.0" friction="0.0"/>
-      <mimic joint="thigh_r_03_joint" multiplier="1" offset="0"/>
+      <mimic joint="shin_r_active_joint" multiplier="1" offset="0"/>
     </joint>
     <link name="leg_r_01">
@@ -189,5 +189,5 @@
       <limit effort="1000.0" lower="-1.8588" upper="0.4974" velocity="10.0"/>
       <dynamics damping="0.0" friction="0.0"/>
-      <mimic joint="thigh_r_03_joint" multiplier="1" offset="0"/>
+      <mimic joint="shin_r_active_joint" multiplier="1" offset="0"/>
     </joint>
     <xacro:if value="$(arg gazebo)">
@@ -212,5 +212,5 @@
       <limit effort="1000.0" lower="-0.4974" upper="1.8588" velocity="10.0"/>
       <dynamics damping="0.0" friction="0.0"/>
-      <mimic joint="thigh_r_03_joint" multiplier="-1" offset="0"/>
+      <mimic joint="shin_r_active_joint" multiplier="-1" offset="0"/>
     </joint>
     <link name="ankle_r_01">
