Commit message: rename links

File: kuroko_description/xacro/kuroko/parts/leg_l.xacro (robot description, xacro)
@@ -163,7 +163,7 @@
       <xacro:box_inertial xyz="-0.01675 0 0" rpy="0 0 0" size="0.0475 0.0505 0.014" mass="0.007"/>
     </link>
-    <joint name="leg_l_01_joint" type="revolute">
+    <joint name="shin_l_passive_front_joint" type="revolute">
       <parent link="knee_l"/>
-      <child link="leg_l_01"/>
+      <child link="shin_l_passive_front"/>
       <origin xyz="0 0 0" rpy="0 0.785398163 0"/>
       <axis xyz="0 -1 0"/>
@@ -172,9 +172,9 @@
       <mimic joint="shin_l_active_joint" multiplier="1" offset="0"/>
     </joint>
-    <link name="leg_l_01">
-      <visual>
-        <origin xyz="0 0 0" rpy="0 0 0"/>
-        <geometry>
-          <mesh filename="package://kuroko_description/meshes/kuroko/obj/leg_r_01.obj"/>
+    <link name="shin_l_passive_front">
+      <visual>
+        <origin xyz="0 0 0" rpy="0 0 0"/>
+        <geometry>
+          <mesh filename="package://kuroko_description/meshes/kuroko/obj/shin_r_passive_front.obj"/>
         </geometry>
       </visual>
@@ -193,5 +193,5 @@
     <xacro:if value="$(arg gazebo)">
       <xacro:gazebo_poassive_joint name="leg_l_02_loop" xyz="-0.0335 0 0"
-        parent="ankle_l_01" child="leg_l_02" axis="0 -1 0"/>
+        parent="ankle_l_pitch_passive" child="leg_l_02" axis="0 -1 0"/>
     </xacro:if>
     <link name="leg_l_02">
@@ -199,5 +199,5 @@
         <origin xyz="0 0 0" rpy="0 0 0"/>
         <geometry>
-          <mesh filename="package://kuroko_description/meshes/kuroko/obj/leg_r_02.obj"/>
+          <mesh filename="package://kuroko_description/meshes/kuroko/obj/shin_r_passive_rear.obj"/>
         </geometry>
       </visual>
@@ -205,7 +205,7 @@
       <xacro:box_inertial xyz="0 0 -0.05" rpy="0 0 0" size="0.014 0.0445 0.114" mass="0.016"/>
     </link>
-    <joint name="ankle_l_01_joint" type="revolute">
-      <parent link="leg_l_01"/>
-      <child link="ankle_l_01"/>
+    <joint name="ankle_l_pitch_passive_joint" type="revolute">
+      <parent link="shin_l_passive_front"/>
+      <child link="ankle_l_pitch_passive"/>
       <origin xyz="0 0 -0.1" rpy="0 -0.785398163 0"/>
       <axis xyz="0 -1 0"/>
@@ -214,9 +214,9 @@
       <mimic joint="shin_l_active_joint" multiplier="-1" offset="0"/>
     </joint>
-    <link name="ankle_l_01">
-      <visual>
-        <origin xyz="0 0 0" rpy="0 0 0"/>
-        <geometry>
-          <mesh filename="package://kuroko_description/meshes/kuroko/obj/ankle_r_01.obj"/>
+    <link name="ankle_l_pitch_passive">
+      <visual>
+        <origin xyz="0 0 0" rpy="0 0 0"/>
+        <geometry>
+          <mesh filename="package://kuroko_description/meshes/kuroko/obj/ankle_r_pitch_passive.obj"/>
         </geometry>
       </visual>
@@ -225,7 +225,7 @@
         mass="0.104"/>
     </link>
-    <joint name="toe_l_01_joint" type="revolute">
-      <parent link="ankle_l_01"/>
-      <child link="toe_l_01"/>
+    <joint name="ankle_l_roll_joint" type="revolute">
+      <parent link="ankle_l_pitch_passive"/>
+      <child link="ankle_l_roll"/>
       <origin xyz="-0.015 0 -0.025" rpy="0 0 0"/>
       <axis xyz="1 0 0"/>
@@ -233,9 +233,9 @@
       <dynamics damping="0.0" friction="0.0"/>
     </joint>
-    <link name="toe_l_01">
-      <visual>
-        <origin xyz="0 0 0" rpy="0 0 0"/>
-        <geometry>
-          <mesh filename="package://kuroko_description/meshes/kuroko/obj/toe_l_01.obj"/>
+    <link name="ankle_l_roll">
+      <visual>
+        <origin xyz="0 0 0" rpy="0 0 0"/>
+        <geometry>
+          <mesh filename="package://kuroko_description/meshes/kuroko/obj/ankle_l_roll.obj"/>
         </geometry>
       </visual>
@@ -244,7 +244,7 @@
         mass="0.136"/>
     </link>
-    <joint name="toe_l_02_joint" type="revolute">
-      <parent link="toe_l_01"/>
-      <child link="toe_l_02"/>
+    <joint name="ankle_l_yaw_joint" type="revolute">
+      <parent link="ankle_l_roll"/>
+      <child link="ankle_l_yaw"/>
       <origin xyz="0 0 -0.03825" rpy="0 0 0"/>
       <axis xyz="0 0 -1"/>
@@ -252,9 +252,9 @@
       <dynamics damping="0.0" friction="0.0"/>
     </joint>
-    <link name="toe_l_02">
-      <visual>
-        <origin xyz="0 0 0" rpy="0 0 0"/>
-        <geometry>
-          <mesh filename="package://kuroko_description/meshes/kuroko/obj/toe_r_02.obj"/>
+    <link name="ankle_l_yaw">
+      <visual>
+        <origin xyz="0 0 0" rpy="0 0 0"/>
+        <geometry>
+          <mesh filename="package://kuroko_description/meshes/kuroko/obj/ankle_r_yaw.obj"/>
         </geometry>
       </visual>

File: kuroko_description/xacro/kuroko/parts/leg_r.xacro (robot description, xacro)
@@ -132,5 +132,5 @@
       </joint>
       <xacro:gazebo_poassive_joint name="thigh_r_passive_rear_loop" xyz="-0.00765471 0 -0.02897777"
-        parent="leg_r_02" child="thigh_r_passive_rear"/>
+        parent="shin_r_passive_rear" child="thigh_r_passive_rear"/>
     </xacro:if>
     <link name="thigh_r_passive_rear">
@@ -163,7 +163,7 @@
       <xacro:box_inertial xyz="-0.01675 0 0" rpy="0 0 0" size="0.0475 0.0505 0.014" mass="0.007"/>
     </link>
-    <joint name="leg_r_01_joint" type="revolute">
+    <joint name="shin_r_passive_front_joint" type="revolute">
       <parent link="knee_r"/>
-      <child link="leg_r_01"/>
+      <child link="shin_r_passive_front"/>
       <origin xyz="0 0 0" rpy="0 0.785398163 0"/>
       <axis xyz="0 1 0"/>
@@ -172,9 +172,9 @@
       <mimic joint="shin_r_active_joint" multiplier="1" offset="0"/>
     </joint>
-    <link name="leg_r_01">
-      <visual>
-        <origin xyz="0 0 0" rpy="0 0 0"/>
-        <geometry>
-          <mesh filename="package://kuroko_description/meshes/kuroko/obj/leg_r_01.obj"/>
+    <link name="shin_r_passive_front">
+      <visual>
+        <origin xyz="0 0 0" rpy="0 0 0"/>
+        <geometry>
+          <mesh filename="package://kuroko_description/meshes/kuroko/obj/shin_r_passive_front.obj"/>
         </geometry>
       </visual>
@@ -182,7 +182,7 @@
       <xacro:box_inertial xyz="0 0 -0.05" rpy="0 0 0" size="0.014 0.0385 0.114" mass="0.013"/>
     </link>
-    <joint name="leg_r_02_joint" type="revolute">
+    <joint name="shin_r_passive_rear_joint" type="revolute">
       <parent link="knee_r"/>
-      <child link="leg_r_02"/>
+      <child link="shin_r_passive_rear"/>
       <origin xyz="-0.0335 0 0" rpy="0 0.785398163 0"/>
       <axis xyz="0 1 0"/>
@@ -192,12 +192,12 @@
     </joint>
     <xacro:if value="$(arg gazebo)">
-      <xacro:gazebo_poassive_joint name="leg_r_02_loop" xyz="-0.0335 0 0"
-        parent="ankle_r_01" child="leg_r_02"/>
+      <xacro:gazebo_poassive_joint name="shin_r_passive_rear_loop" xyz="-0.0335 0 0"
+        parent="ankle_r_pitch_passive" child="shin_r_passive_rear"/>
     </xacro:if>
-    <link name="leg_r_02">
-      <visual>
-        <origin xyz="0 0 0" rpy="0 0 0"/>
-        <geometry>
-          <mesh filename="package://kuroko_description/meshes/kuroko/obj/leg_r_02.obj"/>
+    <link name="shin_r_passive_rear">
+      <visual>
+        <origin xyz="0 0 0" rpy="0 0 0"/>
+        <geometry>
+          <mesh filename="package://kuroko_description/meshes/kuroko/obj/shin_r_passive_rear.obj"/>
         </geometry>
       </visual>
@@ -205,7 +205,7 @@
       <xacro:box_inertial xyz="0 0 -0.05" rpy="0 0 0" size="0.014 0.0445 0.114" mass="0.016"/>
     </link>
-    <joint name="ankle_r_01_joint" type="revolute">
-      <parent link="leg_r_01"/>
-      <child link="ankle_r_01"/>
+    <joint name="ankle_r_pitch_passive_joint" type="revolute">
+      <parent link="shin_r_passive_front"/>
+      <child link="ankle_r_pitch_passive"/>
       <origin xyz="0 0 -0.1" rpy="0 -0.785398163 0"/>
       <axis xyz="0 1 0"/>
@@ -214,9 +214,9 @@
       <mimic joint="shin_r_active_joint" multiplier="-1" offset="0"/>
     </joint>
-    <link name="ankle_r_01">
-      <visual>
-        <origin xyz="0 0 0" rpy="0 0 0"/>
-        <geometry>
-          <mesh filename="package://kuroko_description/meshes/kuroko/obj/ankle_r_01.obj"/>
+    <link name="ankle_r_pitch_passive">
+      <visual>
+        <origin xyz="0 0 0" rpy="0 0 0"/>
+        <geometry>
+          <mesh filename="package://kuroko_description/meshes/kuroko/obj/ankle_r_pitch_passive.obj"/>
         </geometry>
       </visual>
@@ -225,7 +225,7 @@
         mass="0.104"/>
     </link>
-    <joint name="toe_r_01_joint" type="revolute">
-      <parent link="ankle_r_01"/>
-      <child link="toe_r_01"/>
+    <joint name="ankle_r_roll_joint" type="revolute">
+      <parent link="ankle_r_pitch_passive"/>
+      <child link="ankle_r_roll"/>
       <origin xyz="-0.015 0 -0.025" rpy="0 0 0"/>
       <axis xyz="1 0 0"/>
@@ -233,9 +233,9 @@
       <dynamics damping="0.0" friction="0.0"/>
     </joint>
-    <link name="toe_r_01">
-      <visual>
-        <origin xyz="0 0 0" rpy="0 0 0"/>
-        <geometry>
-          <mesh filename="package://kuroko_description/meshes/kuroko/obj/toe_r_01.obj"/>
+    <link name="ankle_r_roll">
+      <visual>
+        <origin xyz="0 0 0" rpy="0 0 0"/>
+        <geometry>
+          <mesh filename="package://kuroko_description/meshes/kuroko/obj/ankle_r_roll.obj"/>
         </geometry>
       </visual>
@@ -244,7 +244,7 @@
         mass="0.136"/>
     </link>
-    <joint name="toe_r_02_joint" type="revolute">
-      <parent link="toe_r_01"/>
-      <child link="toe_r_02"/>
+    <joint name="ankle_r_yaw_joint" type="revolute">
+      <parent link="ankle_r_roll"/>
+      <child link="ankle_r_yaw"/>
       <origin xyz="0 0 -0.03825" rpy="0 0 0"/>
       <axis xyz="0 0 -1"/>
@@ -252,9 +252,9 @@
       <dynamics damping="0.0" friction="0.0"/>
     </joint>
-    <link name="toe_r_02">
-      <visual>
-        <origin xyz="0 0 0" rpy="0 0 0"/>
-        <geometry>
-          <mesh filename="package://kuroko_description/meshes/kuroko/obj/toe_r_02.obj"/>
+    <link name="ankle_r_yaw">
+      <visual>
+        <origin xyz="0 0 0" rpy="0 0 0"/>
+        <geometry>
+          <mesh filename="package://kuroko_description/meshes/kuroko/obj/ankle_r_yaw.obj"/>
         </geometry>
       </visual>

Commit message: Fix bug

File: kuroko_description/xacro/kuroko/parts/leg_l.xacro (robot description, xacro)
@@ -132,5 +132,5 @@
       </joint>
       <xacro:gazebo_poassive_joint name="thigh_l_passive_rear_loop" xyz="-0.00765471 0 -0.02897777"
-        parent="leg_l_02" child="thigh_l_passive_rear" axis="0 -1 0"/>
+        parent="shin_l_passive_rear" child="thigh_l_passive_rear" axis="0 -1 0"/>
     </xacro:if>
     <link name="thigh_l_passive_rear">
@@ -182,7 +182,7 @@
       <xacro:box_inertial xyz="0 0 -0.05" rpy="0 0 0" size="0.014 0.0385 0.114" mass="0.013"/>
     </link>
-    <joint name="leg_l_02_joint" type="revolute">
+    <joint name="shin_l_passive_rear_joint" type="revolute">
       <parent link="knee_l"/>
-      <child link="leg_l_02"/>
+      <child link="shin_l_passive_rear"/>
       <origin xyz="-0.0335 0 0" rpy="0 0.785398163 0"/>
       <axis xyz="0 -1 0"/>
@@ -192,8 +192,8 @@
     </joint>
     <xacro:if value="$(arg gazebo)">
-      <xacro:gazebo_poassive_joint name="leg_l_02_loop" xyz="-0.0335 0 0"
-        parent="ankle_l_pitch_passive" child="leg_l_02" axis="0 -1 0"/>
+      <xacro:gazebo_poassive_joint name="shin_l_passive_rear_loop" xyz="-0.0335 0 0"
+        parent="ankle_l_pitch_passive" child="shin_l_passive_rear" axis="0 -1 0"/>
     </xacro:if>
-    <link name="leg_l_02">
+    <link name="shin_l_passive_rear">
       <visual>
         <origin xyz="0 0 0" rpy="0 0 0"/>
