Commit message: [WIP] Create kinematics tree

File: kuroko_description/xacro/kuroko/parts/leg_l.xacro (robot description, xacro)
@@ -102,5 +102,5 @@
     </link>
     <xacro:unless value="$(arg gazebo)">
-      <joint name="thigh_l_rear_passive_mimic1" type="revolute">
+      <joint name="thigh_l_rear_passive_mimic" type="revolute">
         <parent link="shin_l_active_link"/>
         <child link="thigh_l_rear_passive_mimic_link"/>
@@ -112,5 +112,5 @@
       </joint>
       <link name="thigh_l_rear_passive_mimic_link"/>
-      <joint name="thigh_l_rear_passive_mimic2" type="revolute">
+      <joint name="thigh_l_rear_passive" type="revolute">
         <parent link="thigh_l_rear_passive_mimic_link"/>
         <child link="thigh_l_rear_passive_link"/>

File: kuroko_description/xacro/kuroko/parts/leg_r.xacro (robot description, xacro)
@@ -102,5 +102,5 @@
     </link>
     <xacro:unless value="$(arg gazebo)">
-      <joint name="thigh_r_rear_passive_mimic1" type="revolute">
+      <joint name="thigh_r_rear_passive_mimic" type="revolute">
         <parent link="shin_r_active_link"/>
         <child link="thigh_r_rear_passive_mimic_link"/>
@@ -112,5 +112,5 @@
       </joint>
       <link name="thigh_r_rear_passive_mimic_link"/>
-      <joint name="thigh_r_rear_passive_mimic2" type="revolute">
+      <joint name="thigh_r_rear_passive" type="revolute">
         <parent link="thigh_r_rear_passive_mimic_link"/>
         <child link="thigh_r_rear_passive_link"/>

Commit message: Rename thigh joints

File: kuroko_description/xacro/kuroko/parts/leg_l.xacro (robot description, xacro)
@@ -41,7 +41,7 @@
         mass="0.478"/>
     </link>
-    <joint name="thigh_l_front_active" type="revolute">
+    <joint name="thigh_l_active" type="revolute">
       <parent link="hip_l_pitch_link"/>
-      <child link="thigh_l_front_active_link"/>
+      <child link="thigh_l_active_link"/>
       <origin xyz="0.015 0.02925 -0.0305" rpy="0 -0.785398163 0"/>
       <axis xyz="0 -1 0"/>
@@ -49,9 +49,9 @@
       <dynamics damping="0.0" friction="0.0"/>
     </joint>
-    <link name="thigh_l_front_active_link">
-      <visual>
-        <origin xyz="0 0 0" rpy="0 0 0"/>
-        <geometry>
-          <mesh filename="package://kuroko_description/meshes/kuroko/obj/thigh_l_front_active.obj"/>
+    <link name="thigh_l_active_link">
+      <visual>
+        <origin xyz="0 0 0" rpy="0 0 0"/>
+        <geometry>
+          <mesh filename="package://kuroko_description/meshes/kuroko/obj/thigh_l_active.obj"/>
         </geometry>
       </visual>
@@ -85,5 +85,5 @@
       <limit effort="1000.0" lower="-3.1" upper="3.1" velocity="10.0"/>
       <dynamics damping="0.0" friction="0.0"/>
-      <mimic joint="thigh_l_front_active" multiplier="1" offset="0"/>
+      <mimic joint="thigh_l_active" multiplier="1" offset="0"/>
     </joint>
     <xacro:if value="$(arg gazebo)">
@@ -119,5 +119,5 @@
         <limit effort="1000.0" lower="-3.1" upper="3.1" velocity="10.0"/>
         <dynamics damping="0.0" friction="0.0"/>
-        <mimic joint="thigh_l_front_active" multiplier="1" offset="0"/>
+        <mimic joint="thigh_l_active" multiplier="1" offset="0"/>
       </joint>
     </xacro:unless>
@@ -145,5 +145,5 @@
     </link>
     <joint name="knee_l_passive" type="revolute">
-      <parent link="thigh_l_front_active_link"/>
+      <parent link="thigh_l_active_link"/>
       <child link="knee_l_passive_link"/>
       <origin xyz="0 0 -0.1" rpy="0 0.785398163 0"/>
@@ -151,5 +151,5 @@
       <limit effort="1000.0" lower="-0.4974" upper="1.8588" velocity="10.0"/>
       <dynamics damping="0.0" friction="0.0"/>
-      <mimic joint="thigh_l_front_active" multiplier="-1" offset="0"/>
+      <mimic joint="thigh_l_active" multiplier="-1" offset="0"/>
     </joint>
     <link name="knee_l_passive_link">

File: kuroko_description/xacro/kuroko/parts/leg_r.xacro (robot description, xacro)
@@ -41,7 +41,7 @@
         mass="0.478"/>
     </link>
-    <joint name="thigh_r_front_active" type="revolute">
+    <joint name="thigh_r_active" type="revolute">
       <parent link="hip_r_pitch_link"/>
-      <child link="thigh_r_front_active_link"/>
+      <child link="thigh_r_active_link"/>
       <origin xyz="0.015 -0.02925 -0.0305" rpy="0 -0.785398163 0"/>
       <axis xyz="0 1 0"/>
@@ -49,9 +49,9 @@
       <dynamics damping="0.0" friction="0.0"/>
     </joint>
-    <link name="thigh_r_front_active_link">
-      <visual>
-        <origin xyz="0 0 0" rpy="0 0 0"/>
-        <geometry>
-          <mesh filename="package://kuroko_description/meshes/kuroko/obj/thigh_r_front_active.obj"/>
+    <link name="thigh_r_active_link">
+      <visual>
+        <origin xyz="0 0 0" rpy="0 0 0"/>
+        <geometry>
+          <mesh filename="package://kuroko_description/meshes/kuroko/obj/thigh_r_active.obj"/>
         </geometry>
       </visual>
@@ -85,5 +85,5 @@
       <limit effort="1000.0" lower="-3.1" upper="3.1" velocity="10.0"/>
       <dynamics damping="0.0" friction="0.0"/>
-      <mimic joint="thigh_r_front_active" multiplier="1" offset="0"/>
+      <mimic joint="thigh_r_active" multiplier="1" offset="0"/>
     </joint>
     <xacro:if value="$(arg gazebo)">
@@ -119,5 +119,5 @@
         <limit effort="1000.0" lower="-3.1" upper="3.1" velocity="10.0"/>
         <dynamics damping="0.0" friction="0.0"/>
-        <mimic joint="thigh_r_front_active" multiplier="1" offset="0"/>
+        <mimic joint="thigh_r_active" multiplier="1" offset="0"/>
       </joint>
     </xacro:unless>
@@ -145,5 +145,5 @@
     </link>
     <joint name="knee_r_passive" type="revolute">
-      <parent link="thigh_r_front_active_link"/>
+      <parent link="thigh_r_active_link"/>
       <child link="knee_r_passive_link"/>
       <origin xyz="0 0 -0.1" rpy="0 0.785398163 0"/>
@@ -151,5 +151,5 @@
       <limit effort="1000.0" lower="-1.8588" upper="0.4974" velocity="10.0"/>
       <dynamics damping="0.0" friction="0.0"/>
-      <mimic joint="thigh_r_front_active" multiplier="-1" offset="0"/>
+      <mimic joint="thigh_r_active" multiplier="-1" offset="0"/>
     </joint>
     <link name="knee_r_passive_link">

Commit message: Simplify leg

File: kuroko_description/xacro/kuroko/parts/leg_l.xacro (robot description, xacro)
@@ -38,7 +38,7 @@
       <xacro:box_inertial xyz="-0.00175 0.049 -0.015" rpy="0 0 0" size="0.067 0.098 0.0585" mass="0.478"/>
     </link>
-    <joint name="thigh_l_active" type="revolute">
+    <joint name="thigh_l_front" type="revolute">
       <parent link="hip_l_pitch_link"/>
-      <child link="thigh_l_active_link"/>
+      <child link="thigh_l_front_link"/>
       <origin xyz="0.015 0.02925 -0.0305" rpy="0 -0.785398163 0"/>
       <axis xyz="0 1 0"/>
@@ -46,5 +46,5 @@
       <dynamics damping="1.289855" friction="0.0"/>
     </joint>
-    <link name="thigh_l_active_link">
+    <link name="thigh_l_front_link">
       <visual>
         <origin xyz="0 0 0" rpy="0 0 0"/>
@@ -56,35 +56,17 @@
       <xacro:box_inertial xyz="0 0 -0.05" rpy="0 0 0" size="0.014 0.0445 0.114" mass="0.012"/>
     </link>
-    <joint name="shin_l_active" type="revolute">
+    <joint name="thigh_l_rear" type="revolute">
       <parent link="hip_l_pitch_link"/>
-      <child link="shin_l_active_link"/>
-      <origin xyz="-0.0185 0.02925 -0.0305" rpy="0 1.047197551 0"/>
-      <axis xyz="0 1 0"/>
-      <limit effort="8.9" lower="-1.8588" upper="0.4974" velocity="6.9"/>
-      <dynamics damping="1.289855" friction="0.0"/>
-    </joint>
-    <link name="shin_l_active_link">
-      <visual>
-        <origin xyz="0 0 0" rpy="0 0 0"/>
-        <geometry>
-          <mesh filename="${MESH_DIR}/kuroko/stl/shin_l_active.stl"/>
-        </geometry>
-      </visual>
-      <xacro:box_collision xyz="-0.004745 0 -0.015" rpy="0 0 0" size="0.02349 0.0445 0.044"/>
-      <xacro:box_inertial xyz="-0.004745 0 -0.015" rpy="0 0 0" size="0.02349 0.0445 0.044" mass="0.008"/>
-    </link>
-    <joint name="thigh_l_middle_passive" type="revolute">
-      <parent link="hip_l_pitch_link"/>
-      <child link="thigh_l_middle_passive_link"/>
+      <child link="thigh_l_rear_link"/>
       <origin xyz="-0.0185 0.02925 -0.0305" rpy="0 -0.785398163 0"/>
       <axis xyz="0 1 0"/>
       <limit effort="0.0" lower="-3.1" upper="3.1" velocity="100.0"/>
       <dynamics damping="0" friction="0.0"/>
-      <mimic joint="thigh_l_active" multiplier="1" offset="0"/>
+      <mimic joint="thigh_l_front" multiplier="1" offset="0"/>
     </joint>
     <xacro:if value="$(arg gazebo)">
-      <xacro:gazebo_poassive_joint name="thigh_l_middle_passive_loop" xyz="-0.0335 0 0" parent="knee_l_passive_link" child="thigh_l_middle_passive_link" axis="0 1 0"/>
+      <xacro:gazebo_poassive_joint name="thigh_l_rear_loop" xyz="-0.0335 0 0" parent="knee_l_passive_link" child="thigh_l_rear_link" axis="0 1 0"/>
     </xacro:if>
-    <link name="thigh_l_middle_passive_link">
+    <link name="thigh_l_rear_link">
       <visual>
         <origin xyz="0 0 0" rpy="0 0 0"/>
@@ -96,48 +78,6 @@
       <xacro:box_inertial xyz="0 0 -0.05" rpy="0 0 0" size="0.014 0.0345 0.114" mass="0.012"/>
     </link>
-    <xacro:unless value="$(arg gazebo)">
-      <joint name="thigh_l_rear_passive_mimic" type="revolute">
-        <parent link="shin_l_active_link"/>
-        <child link="thigh_l_rear_passive_mimic_link"/>
-        <origin xyz="0 0 -0.03" rpy="0 -1.832597551 0"/>
-        <axis xyz="0 1 0"/>
-        <limit effort="0.0" lower="-3.1" upper="3.1" velocity="100.0"/>
-        <dynamics damping="0" friction="0.0"/>
-        <mimic joint="shin_l_active" multiplier="-1" offset="0"/>
-      </joint>
-      <link name="thigh_l_rear_passive_mimic_link"/>
-      <joint name="thigh_l_rear_passive" type="revolute">
-        <parent link="thigh_l_rear_passive_mimic_link"/>
-        <child link="thigh_l_rear_passive_link"/>
-        <origin xyz="0 0 0" rpy="0 0 0"/>
-        <axis xyz="0 1 0"/>
-        <limit effort="0.0" lower="-3.1" upper="3.1" velocity="100.0"/>
-        <dynamics damping="0" friction="0.0"/>
-        <mimic joint="thigh_l_active" multiplier="1" offset="0"/>
-      </joint>
-    </xacro:unless>
-    <xacro:if value="$(arg gazebo)">
-      <joint name="thigh_l_rear_passive" type="revolute">
-        <parent link="shin_l_active_link"/>
-        <child link="thigh_l_rear_passive_link"/>
-        <origin xyz="0 0 -0.03" rpy="0 -1.832597551 0"/>
-        <axis xyz="0 1 0"/>
-        <limit effort="0.0" lower="-0.9948" upper="1.5708" velocity="100.0"/>
-        <dynamics damping="0" friction="0.0"/>
-      </joint>
-      <xacro:gazebo_poassive_joint name="thigh_l_rear_passive_loop" xyz="-0.00765471 0 -0.02897777" parent="shin_l_rear_passive_link" child="thigh_l_rear_passive_link" axis="0 1 0"/>
-    </xacro:if>
-    <link name="thigh_l_rear_passive_link">
-      <visual>
-        <origin xyz="0 0 0" rpy="0 0 0"/>
-        <geometry>
-          <mesh filename="${MESH_DIR}/kuroko/stl/thigh_r_rear_passive.stl"/>
-        </geometry>
-      </visual>
-      <xacro:box_collision xyz="0 0 -0.05" rpy="0 0 0" size="0.014 0.0285 0.114"/>
-      <xacro:box_inertial xyz="0 0 -0.05" rpy="0 0 0" size="0.014 0.0285 0.114" mass="0.011"/>
-    </link>
     <joint name="knee_l_passive" type="revolute">
-      <parent link="thigh_l_active_link"/>
+      <parent link="thigh_l_front_link"/>
       <child link="knee_l_passive_link"/>
       <origin xyz="0 0 -0.1" rpy="0 0.785398163 0"/>
@@ -145,5 +85,5 @@
       <limit effort="0.0" lower="-1.8588" upper="0.4974" velocity="100.0"/>
       <dynamics damping="0" friction="0.0"/>
-      <mimic joint="thigh_l_active" multiplier="-1" offset="0"/>
+      <mimic joint="thigh_l_front" multiplier="-1" offset="0"/>
     </joint>
     <link name="knee_l_passive_link">
@@ -157,7 +97,7 @@
       <xacro:box_inertial xyz="-0.01675 0 0" rpy="0 0 0" size="0.0475 0.0505 0.014" mass="0.007"/>
     </link>
-    <joint name="shin_l_front_passive" type="revolute">
+    <joint name="shin_l_front" type="revolute">
       <parent link="knee_l_passive_link"/>
-      <child link="shin_l_front_passive_link"/>
+      <child link="shin_l_front_link"/>
       <origin xyz="0 0 0" rpy="0 0.785398163 0"/>
       <axis xyz="0 1 0"/>
@@ -166,5 +106,5 @@
       <mimic joint="shin_l_active" multiplier="1" offset="0"/>
     </joint>
-    <link name="shin_l_front_passive_link">
+    <link name="shin_l_front_link">
       <visual>
         <origin xyz="0 0 0" rpy="0 0 0"/>
@@ -176,7 +116,7 @@
       <xacro:box_inertial xyz="0 0 -0.05" rpy="0 0 0" size="0.014 0.0385 0.114" mass="0.013"/>
     </link>
-    <joint name="shin_l_rear_passive" type="revolute">
+    <joint name="shin_l_rear" type="revolute">
       <parent link="knee_l_passive_link"/>
-      <child link="shin_l_rear_passive_link"/>
+      <child link="shin_l_rear_link"/>
       <origin xyz="-0.0335 0 0" rpy="0 0.785398163 0"/>
       <axis xyz="0 1 0"/>
@@ -186,7 +126,7 @@
     </joint>
     <xacro:if value="$(arg gazebo)">
-      <xacro:gazebo_poassive_joint name="shin_l_rear_passive_loop" xyz="-0.0335 0 0" parent="ankle_l_pitch_passive_link" child="shin_l_rear_passive_link" axis="0 1 0"/>
+      <xacro:gazebo_poassive_joint name="shin_l_rear_loop" xyz="-0.0335 0 0" parent="ankle_l_pitch_passive_link" child="shin_l_rear_link" axis="0 1 0"/>
     </xacro:if>
-    <link name="shin_l_rear_passive_link">
+    <link name="shin_l_rear_link">
       <visual>
         <origin xyz="0 0 0" rpy="0 0 0"/>
@@ -199,5 +139,5 @@
     </link>
     <joint name="ankle_l_pitch_passive" type="revolute">
-      <parent link="shin_l_front_passive_link"/>
+      <parent link="shin_l_front_link"/>
       <child link="ankle_l_pitch_passive_link"/>
       <origin xyz="0 0 -0.1" rpy="0 -0.785398163 0"/>

File: kuroko_description/xacro/kuroko/parts/leg_r.xacro (robot description, xacro)
@@ -38,7 +38,7 @@
       <xacro:box_inertial xyz="-0.00175 -0.049 -0.015" rpy="0 0 0" size="0.067 0.098 0.0585" mass="0.478"/>
     </link>
-    <joint name="thigh_r_active" type="revolute">
+    <joint name="thigh_r_front" type="revolute">
       <parent link="hip_r_pitch_link"/>
-      <child link="thigh_r_active_link"/>
+      <child link="thigh_r_front_link"/>
       <origin xyz="0.015 -0.02925 -0.0305" rpy="0 -0.785398163 0"/>
       <axis xyz="0 1 0"/>
@@ -46,5 +46,5 @@
       <dynamics damping="1.289855" friction="0.0"/>
     </joint>
-    <link name="thigh_r_active_link">
+    <link name="thigh_r_front_link">
       <visual>
         <origin xyz="0 0 0" rpy="0 0 0"/>
@@ -56,35 +56,17 @@
       <xacro:box_inertial xyz="0 0 -0.05" rpy="0 0 0" size="0.014 0.0445 0.114" mass="0.012"/>
     </link>
-    <joint name="shin_r_active" type="revolute">
+    <joint name="thigh_r_rear" type="revolute">
       <parent link="hip_r_pitch_link"/>
-      <child link="shin_r_active_link"/>
-      <origin xyz="-0.0185 -0.02925 -0.0305" rpy="0 1.047197551 0"/>
-      <axis xyz="0 1 0"/>
-      <limit effort="8.9" lower="-1.8588" upper="0.4974" velocity="6.9"/>
-      <dynamics damping="1.289855" friction="0.0"/>
-    </joint>
-    <link name="shin_r_active_link">
-      <visual>
-        <origin xyz="0 0 0" rpy="0 0 0"/>
-        <geometry>
-          <mesh filename="${MESH_DIR}/kuroko/stl/shin_r_active.stl"/>
-        </geometry>
-      </visual>
-      <xacro:box_collision xyz="-0.004745 0 -0.015" rpy="0 0 0" size="0.02349 0.0445 0.044"/>
-      <xacro:box_inertial xyz="-0.004745 0 -0.015" rpy="0 0 0" size="0.02349 0.0445 0.044" mass="0.008"/>
-    </link>
-    <joint name="thigh_r_middle_passive" type="revolute">
-      <parent link="hip_r_pitch_link"/>
-      <child link="thigh_r_middle_passive_link"/>
+      <child link="thigh_r_rear_link"/>
       <origin xyz="-0.0185 -0.02925 -0.0305" rpy="0 -0.785398163 0"/>
       <axis xyz="0 1 0"/>
       <limit effort="0.0" lower="-3.1" upper="3.1" velocity="100.0"/>
       <dynamics damping="0" friction="0.0"/>
-      <mimic joint="thigh_r_active" multiplier="1" offset="0"/>
+      <mimic joint="thigh_r_front" multiplier="1" offset="0"/>
     </joint>
     <xacro:if value="$(arg gazebo)">
-      <xacro:gazebo_poassive_joint name="thigh_r_middle_passive_loop" xyz="-0.0335 0 0" parent="knee_r_passive_link" child="thigh_r_middle_passive_link" axis="0 1 0"/>
+      <xacro:gazebo_poassive_joint name="thigh_r_rear_loop" xyz="-0.0335 0 0" parent="knee_r_passive_link" child="thigh_r_rear_link" axis="0 1 0"/>
     </xacro:if>
-    <link name="thigh_r_middle_passive_link">
+    <link name="thigh_r_rear_link">
       <visual>
         <origin xyz="0 0 0" rpy="0 0 0"/>
@@ -96,48 +78,6 @@
       <xacro:box_inertial xyz="0 0 -0.05" rpy="0 0 0" size="0.014 0.0345 0.114" mass="0.012"/>
     </link>
-    <xacro:unless value="$(arg gazebo)">
-      <joint name="thigh_r_rear_passive_mimic" type="revolute">
-        <parent link="shin_r_active_link"/>
-        <child link="thigh_r_rear_passive_mimic_link"/>
-        <origin xyz="0 0 -0.03" rpy="0 -1.832597551 0"/>
-        <axis xyz="0 1 0"/>
-        <limit effort="0.0" lower="-3.1" upper="3.1" velocity="100.0"/>
-        <dynamics damping="0" friction="0.0"/>
-        <mimic joint="shin_r_active" multiplier="-1" offset="0"/>
-      </joint>
-      <link name="thigh_r_rear_passive_mimic_link"/>
-      <joint name="thigh_r_rear_passive" type="revolute">
-        <parent link="thigh_r_rear_passive_mimic_link"/>
-        <child link="thigh_r_rear_passive_link"/>
-        <origin xyz="0 0 0" rpy="0 0 0"/>
-        <axis xyz="0 1 0"/>
-        <limit effort="0.0" lower="-3.1" upper="3.1" velocity="100.0"/>
-        <dynamics damping="0" friction="0.0"/>
-        <mimic joint="thigh_r_active" multiplier="1" offset="0"/>
-      </joint>
-    </xacro:unless>
-    <xacro:if value="$(arg gazebo)">
-      <joint name="thigh_r_rear_passive" type="revolute">
-        <parent link="shin_r_active_link"/>
-        <child link="thigh_r_rear_passive_link"/>
-        <origin xyz="0 0 -0.03" rpy="0 -1.832597551 0"/>
-        <axis xyz="0 1 0"/>
-        <limit effort="0.0" lower="-0.9948" upper="1.5708" velocity="100.0"/>
-        <dynamics damping="0" friction="0.0"/>
-      </joint>
-      <xacro:gazebo_poassive_joint name="thigh_r_rear_passive_loop" xyz="-0.00765471 0 -0.02897777" parent="shin_r_rear_passive_link" child="thigh_r_rear_passive_link" axis="0 1 0"/>
-    </xacro:if>
-    <link name="thigh_r_rear_passive_link">
-      <visual>
-        <origin xyz="0 0 0" rpy="0 0 0"/>
-        <geometry>
-          <mesh filename="${MESH_DIR}/kuroko/stl/thigh_r_rear_passive.stl"/>
-        </geometry>
-      </visual>
-      <xacro:box_collision xyz="0 0 -0.05" rpy="0 0 0" size="0.014 0.0285 0.114"/>
-      <xacro:box_inertial xyz="0 0 -0.05" rpy="0 0 0" size="0.014 0.0285 0.114" mass="0.011"/>
-    </link>
     <joint name="knee_r_passive" type="revolute">
-      <parent link="thigh_r_active_link"/>
+      <parent link="thigh_r_front_link"/>
       <child link="knee_r_passive_link"/>
       <origin xyz="0 0 -0.1" rpy="0 0.785398163 0"/>
@@ -145,5 +85,5 @@
       <limit effort="0.0" lower="-1.8588" upper="0.4974" velocity="100.0"/>
       <dynamics damping="0" friction="0.0"/>
-      <mimic joint="thigh_r_active" multiplier="-1" offset="0"/>
+      <mimic joint="thigh_r_front" multiplier="-1" offset="0"/>
     </joint>
     <link name="knee_r_passive_link">
@@ -157,7 +97,7 @@
       <xacro:box_inertial xyz="-0.01675 0 0" rpy="0 0 0" size="0.0475 0.0505 0.014" mass="0.007"/>
     </link>
-    <joint name="shin_r_front_passive" type="revolute">
+    <joint name="shin_r_front" type="revolute">
       <parent link="knee_r_passive_link"/>
-      <child link="shin_r_front_passive_link"/>
+      <child link="shin_r_front_link"/>
       <origin xyz="0 0 0" rpy="0 0.785398163 0"/>
       <axis xyz="0 1 0"/>
@@ -166,5 +106,5 @@
       <mimic joint="shin_r_active" multiplier="1" offset="0"/>
     </joint>
-    <link name="shin_r_front_passive_link">
+    <link name="shin_r_front_link">
       <visual>
         <origin xyz="0 0 0" rpy="0 0 0"/>
@@ -176,7 +116,7 @@
       <xacro:box_inertial xyz="0 0 -0.05" rpy="0 0 0" size="0.014 0.0385 0.114" mass="0.013"/>
     </link>
-    <joint name="shin_r_rear_passive" type="revolute">
+    <joint name="shin_r_rear" type="revolute">
       <parent link="knee_r_passive_link"/>
-      <child link="shin_r_rear_passive_link"/>
+      <child link="shin_r_rear_link"/>
       <origin xyz="-0.0335 0 0" rpy="0 0.785398163 0"/>
       <axis xyz="0 1 0"/>
@@ -186,7 +126,7 @@
     </joint>
     <xacro:if value="$(arg gazebo)">
-      <xacro:gazebo_poassive_joint name="shin_r_rear_passive_loop" xyz="-0.0335 0 0" parent="ankle_r_pitch_passive_link" child="shin_r_rear_passive_link" axis="0 1 0"/>
+      <xacro:gazebo_poassive_joint name="shin_r_rear_loop" xyz="-0.0335 0 0" parent="ankle_r_pitch_passive_link" child="shin_r_rear_link" axis="0 1 0"/>
     </xacro:if>
-    <link name="shin_r_rear_passive_link">
+    <link name="shin_r_rear_link">
       <visual>
         <origin xyz="0 0 0" rpy="0 0 0"/>
@@ -199,5 +139,5 @@
     </link>
     <joint name="ankle_r_pitch_passive" type="revolute">
-      <parent link="shin_r_front_passive_link"/>
+      <parent link="shin_r_front_link"/>
       <child link="ankle_r_pitch_passive_link"/>
       <origin xyz="0 0 -0.1" rpy="0 -0.785398163 0"/>

File: kuroko_description/xacro/physics/box_physics.xacro (robot description, xacro)
@@ -1,5 +1,5 @@
 <?xml version="1.0"?>
 <robot xmlns:xacro="http://www.ros.org/wiki/xacro">
-  <xacro:macro name="box_inertial" params="xyz:='0 0 0' rpy:='0 0 0' size mass inertia_min:=0.00001">
+  <xacro:macro name="box_inertial" params="xyz:='0 0 0' rpy:='0 0 0' size mass inertia_min:=0.0001">
     <xacro:property name="d" value="${float(size.split()[0])}"/>
     <xacro:property name="w" value="${float(size.split()[1])}"/>
