Commit message: Update left leg joint tree

File: kuroko_description/xacro/kuroko/parts/leg_l.xacro (robot description, xacro)
@@ -8,6 +8,6 @@
       <origin xyz="0 0 -0.08425" rpy="0 0 0"/>
       <axis xyz="-1 0 0"/>
-      <limit effort="1000.0" lower="-0.5550" upper="1.8640" velocity="10.0"/>
-      <dynamics damping="0.0" friction="0.0"/>
+      <limit effort="3.1" lower="-0.5550" upper="1.8640" velocity="6.5"/>
+      <dynamics damping="0.477" friction="0.0"/>
     </joint>
     <link name="hip_l_roll_link">
@@ -27,6 +27,6 @@
       <origin xyz="0 0.027 0" rpy="0 0 0"/>
       <axis xyz="0 1 0"/>
-      <limit effort="1000.0" lower="-3.1" upper="3.1" velocity="10.0"/>
-      <dynamics damping="0.0" friction="0.0"/>
+      <limit effort="3.1" lower="-3.14" upper="3.14" velocity="6.5"/>
+      <dynamics damping="0.477" friction="0.0"/>
     </joint>
     <link name="hip_l_pitch_link">
@@ -40,4 +40,23 @@
       <xacro:box_inertial xyz="-0.00175 0.049 -0.015" rpy="0 0 0" size="0.067 0.098 0.0585"
         mass="0.478"/>
+    </link>
+    <joint name="shin_l_active" type="revolute">
+      <parent link="hip_l_pitch_link"/>
+      <child link="shin_l_active_link"/>
+      <origin xyz="-0.0185 0.02925 -0.0305" rpy="0 1.047197551 0"/>
+      <axis xyz="0 -1 0"/>
+      <limit effort="8.9" lower="-0.4974" upper="1.8588" velocity="6.9"/>
+      <dynamics damping="1.29" friction="0.0"/>
+    </joint>
+    <link name="shin_l_active_link">
+      <visual>
+        <origin xyz="0 0 0" rpy="0 0 0"/>
+        <geometry>
+          <mesh filename="package://kuroko_description/meshes/kuroko/obj/shin_l_active.obj"/>
+        </geometry>
+      </visual>
+      <xacro:box_collision xyz="-0.004745 0 -0.015" rpy="0 0 0" size="0.02349 0.0445 0.044"/>
+      <xacro:box_inertial xyz="-0.004745 0 -0.015" rpy="0 0 0" size="0.02349 0.0445 0.044"
+        mass="0.008"/>
     </link>
     <joint name="thigh_l_active" type="revolute">
@@ -46,6 +65,6 @@
       <origin xyz="0.015 0.02925 -0.0305" rpy="0 -0.785398163 0"/>
       <axis xyz="0 -1 0"/>
-      <limit effort="1000.0" lower="-1.8588" upper="0.4974" velocity="10.0"/>
-      <dynamics damping="0.0" friction="0.0"/>
+      <limit effort="8.9" lower="-1.8588" upper="0.4974" velocity="6.9"/>
+      <dynamics damping="1.29" friction="0.0"/>
     </joint>
     <link name="thigh_l_active_link">
@@ -59,22 +78,44 @@
       <xacro:box_inertial xyz="0 0 -0.05" rpy="0 0 0" size="0.014 0.0445 0.114" mass="0.012"/>
     </link>
-    <joint name="shin_l_active" type="revolute">
-      <parent link="hip_l_pitch_link"/>
-      <child link="shin_l_active_link"/>
-      <origin xyz="-0.0185 0.02925 -0.0305" rpy="0 1.047197551 0"/>
-      <axis xyz="0 -1 0"/>
-      <limit effort="1000.0" lower="-0.4974" upper="1.8588" velocity="10.0"/>
-      <dynamics damping="0.0" friction="0.0"/>
-    </joint>
-    <link name="shin_l_active_link">
-      <visual>
-        <origin xyz="0 0 0" rpy="0 0 0"/>
-        <geometry>
-          <mesh filename="package://kuroko_description/meshes/kuroko/obj/shin_l_active.obj"/>
-        </geometry>
-      </visual>
-      <xacro:box_collision xyz="-0.004745 0 -0.015" rpy="0 0 0" size="0.02349 0.0445 0.044"/>
-      <xacro:box_inertial xyz="-0.004745 0 -0.015" rpy="0 0 0" size="0.02349 0.0445 0.044"
-        mass="0.008"/>
+    <xacro:unless value="$(arg gazebo)">
+      <joint name="shin_l_front_mimic" type="revolute">
+        <parent link="thigh_l_active_link"/>
+        <child link="shin_l_front_mimic_link"/>
+        <origin xyz="0 0 -0.1" rpy="0 0.785398163 0"/>
+        <axis xyz="0 1 0"/>
+        <limit effort="0" lower="-3.1416" upper="3.1416" velocity="1000"/>
+        <dynamics damping="0.0" friction="0.0"/>
+        <mimic joint="thigh_l_active" multiplier="1" offset="0"/>
+      </joint>
+      <link name="shin_l_front_mimic_link"/>
+      <joint name="shin_l_front_passive" type="revolute">
+        <parent link="shin_l_front_mimic_link"/>
+        <child link="shin_l_front_passive_link"/>
+        <origin xyz="0 0 0" rpy="0 0.785398163 0"/>
+        <axis xyz="0 1 0"/>
+        <limit effort="0" lower="-3.1416" upper="3.1416" velocity="1000"/>
+        <dynamics damping="0.0" friction="0.0"/>
+        <mimic joint="shin_l_active" multiplier="-1" offset="0"/>
+      </joint>
+    </xacro:unless>
+    <xacro:if value="$(arg gazebo)">
+      <joint name="shin_l_front_passive" type="revolute">
+        <parent link="thigh_l_active_link"/>
+        <child link="shin_l_front_passive_link"/>
+        <origin xyz="0 0 -0.1" rpy="0 1.570796327 0"/>
+        <axis xyz="0 1 0"/>
+        <limit effort="0" lower="-1.570796327" upper="0.9948" velocity="1000.0"/>
+        <dynamics damping="0.0" friction="0.0"/>
+      </joint>
+    </xacro:if>
+    <link name="shin_l_front_passive_link">
+      <visual>
+        <origin xyz="0 0 0" rpy="0 0 0"/>
+        <geometry>
+          <mesh filename="package://kuroko_description/meshes/kuroko/obj/shin_r_front_passive.obj"/>
+        </geometry>
+      </visual>
+      <xacro:box_collision xyz="0 0 -0.05" rpy="0 0 0" size="0.014 0.0385 0.114"/>
+      <xacro:box_inertial xyz="0 0 -0.05" rpy="0 0 0" size="0.014 0.0385 0.114" mass="0.013"/>
     </link>
     <joint name="thigh_l_middle_passive" type="revolute">
@@ -82,13 +123,9 @@
       <child link="thigh_l_middle_passive_link"/>
       <origin xyz="-0.0185 0.02925 -0.0305" rpy="0 -0.785398163 0"/>
-      <axis xyz="0 -1 0"/>
-      <limit effort="1000.0" lower="-3.1" upper="3.1" velocity="10.0"/>
-      <dynamics damping="0.0" friction="0.0"/>
-      <mimic joint="thigh_l_active" multiplier="1" offset="0"/>
-    </joint>
-    <xacro:if value="$(arg gazebo)">
-      <xacro:gazebo_poassive_joint name="thigh_l_middle_passive_loop" xyz="-0.0335 0 0"
-        parent="knee_l_passive_link" child="thigh_l_middle_passive_link" axis="0 -1 0"/>
-    </xacro:if>
+      <axis xyz="0 1 0"/>
+      <limit effort="0" lower="-0.4974" upper="1.8588" velocity="1000"/>
+      <dynamics damping="0" friction="0"/>
+      <mimic joint="thigh_l_active" multiplier="-1" offset="0"/>
+    </joint>
     <link name="thigh_l_middle_passive_link">
       <visual>
@@ -102,131 +139,140 @@
     </link>
     <xacro:unless value="$(arg gazebo)">
-      <joint name="thigh_l_rear_passive_mimic" type="revolute">
-        <parent link="shin_l_active_link"/>
-        <child link="thigh_l_rear_passive_mimic_link"/>
-        <origin xyz="0 0 -0.03" rpy="0 -1.832597551 0"/>
-        <axis xyz="0 -1 0"/>
-        <limit effort="1000.0" lower="-3.1" upper="3.1" velocity="10.0"/>
+      <joint name="shin_l_rear_mimic" type="revolute">
+        <parent link="thigh_l_middle_passive_link"/>
+        <child link="shin_l_rear_mimic_link"/>
+        <origin xyz="0 0 -0.1" rpy="0 0.785398163 0"/>
+        <axis xyz="0 1 0"/>
+        <limit effort="0" lower="-3.1416" upper="3.1416" velocity="1000"/>
+        <dynamics damping="0.0" friction="0.0"/>
+        <mimic joint="thigh_l_active" multiplier="1" offset="0"/>
+      </joint>
+      <link name="shin_l_rear_mimic_link"/>
+      <joint name="shin_l_rear_passive" type="revolute">
+        <parent link="shin_l_rear_mimic_link"/>
+        <child link="shin_l_rear_passive_link"/>
+        <origin xyz="0 0 0" rpy="0 0.785398163 0"/>
+        <axis xyz="0 1 0"/>
+        <limit effort="0" lower="-3.1416" upper="3.1416" velocity="1000"/>
         <dynamics damping="0.0" friction="0.0"/>
         <mimic joint="shin_l_active" multiplier="-1" offset="0"/>
       </joint>
-      <link name="thigh_l_rear_passive_mimic_link"/>
-      <joint name="thigh_l_rear_passive" type="revolute">
-        <parent link="thigh_l_rear_passive_mimic_link"/>
-        <child link="thigh_l_rear_passive_link"/>
-        <origin xyz="0 0 0" rpy="0 0 0"/>
-        <axis xyz="0 -1 0"/>
-        <limit effort="1000.0" lower="-3.1" upper="3.1" velocity="10.0"/>
-        <dynamics damping="0.0" friction="0.0"/>
-        <mimic joint="thigh_l_active" multiplier="1" offset="0"/>
-      </joint>
     </xacro:unless>
     <xacro:if value="$(arg gazebo)">
-      <joint name="thigh_l_rear_passive" type="revolute">
-        <parent link="shin_l_active_link"/>
-        <child link="thigh_l_rear_passive_link"/>
-        <origin xyz="0 0 -0.03" rpy="0 -1.832597551 0"/>
-        <axis xyz="0 -1 0"/>
-        <limit effort="1000.0" lower="-1.5708" upper="0.9948" velocity="10.0"/>
-        <dynamics damping="0.0" friction="0.0"/>
-      </joint>
-      <xacro:gazebo_poassive_joint name="thigh_l_rear_passive_loop" xyz="-0.00765471 0 -0.02897777"
-        parent="shin_l_rear_passive_link" child="thigh_l_rear_passive_link" axis="0 -1 0"/>
-    </xacro:if>
-    <link name="thigh_l_rear_passive_link">
-      <visual>
-        <origin xyz="0 0 0" rpy="0 0 0"/>
-        <geometry>
-          <mesh filename="package://kuroko_description/meshes/kuroko/obj/thigh_r_rear_passive.obj"/>
-        </geometry>
-      </visual>
-      <xacro:box_collision xyz="0 0 -0.05" rpy="0 0 0" size="0.014 0.0285 0.114"/>
-      <xacro:box_inertial xyz="0 0 -0.05" rpy="0 0 0" size="0.014 0.0285 0.114" mass="0.011"/>
-    </link>
-    <joint name="knee_l_passive" type="revolute">
-      <parent link="thigh_l_active_link"/>
+      <joint name="shin_l_rear_passive" type="revolute">
+        <parent link="thigh_l_middle_passive_link"/>
+        <child link="shin_l_rear_passive_link"/>
+        <origin xyz="0 0 -0.1" rpy="0 1.570796327 0"/>
+        <axis xyz="0 1 0"/>
+        <limit effort="0" lower="-1.570796327" upper="0.9948" velocity="1000.0"/>
+        <dynamics damping="0.0" friction="0.0"/>
+      </joint>
+    </xacro:if>
+    <link name="shin_l_rear_passive_link">
+      <visual>
+        <origin xyz="0 0 0" rpy="0 0 0"/>
+        <geometry>
+          <mesh filename="package://kuroko_description/meshes/kuroko/obj/shin_r_rear_passive.obj"/>
+        </geometry>
+      </visual>
+      <xacro:box_collision xyz="0 0 -0.05" rpy="0 0 0" size="0.014 0.0445 0.114"/>
+      <xacro:box_inertial xyz="0 0 -0.05" rpy="0 0 0" size="0.014 0.0445 0.114" mass="0.016"/>
+    </link>
+    <joint name="knee_l_rear_passive" type="revolute">
+      <parent link="shin_l_rear_passive_link"/>
       <child link="knee_l_passive_link"/>
-      <origin xyz="0 0 -0.1" rpy="0 0.785398163 0"/>
-      <axis xyz="0 -1 0"/>
-      <limit effort="1000.0" lower="-0.4974" upper="1.8588" velocity="10.0"/>
-      <dynamics damping="0.0" friction="0.0"/>
-      <mimic joint="thigh_l_active" multiplier="-1" offset="0"/>
-    </joint>
-    <link name="knee_l_passive_link">
-      <visual>
-        <origin xyz="0 0 0" rpy="0 0 0"/>
-        <geometry>
-          <mesh filename="package://kuroko_description/meshes/kuroko/obj/knee_r_passive.obj"/>
-        </geometry>
-      </visual>
-      <xacro:box_collision xyz="-0.01675 0 0" rpy="0 0 0" size="0.0475 0.0505 0.014"/>
-      <xacro:box_inertial xyz="-0.01675 0 0" rpy="0 0 0" size="0.0475 0.0505 0.014" mass="0.007"/>
-    </link>
-    <joint name="shin_l_front_passive" type="revolute">
-      <parent link="knee_l_passive_link"/>
-      <child link="shin_l_front_passive_link"/>
-      <origin xyz="0 0 0" rpy="0 0.785398163 0"/>
-      <axis xyz="0 -1 0"/>
-      <limit effort="1000.0" lower="-0.4974" upper="1.8588" velocity="10.0"/>
+      <origin xyz="0 0 0" rpy="0 -0.785398164 0"/>
+      <axis xyz="0 1 0"/>
+      <limit effort="0" lower="-3.141592654" upper="3.141592654" velocity="1000.0"/>
       <dynamics damping="0.0" friction="0.0"/>
       <mimic joint="shin_l_active" multiplier="1" offset="0"/>
     </joint>
-    <link name="shin_l_front_passive_link">
-      <visual>
-        <origin xyz="0 0 0" rpy="0 0 0"/>
-        <geometry>
-          <mesh filename="package://kuroko_description/meshes/kuroko/obj/shin_r_front_passive.obj"/>
-        </geometry>
-      </visual>
-      <xacro:box_collision xyz="0 0 -0.05" rpy="0 0 0" size="0.014 0.0385 0.114"/>
-      <xacro:box_inertial xyz="0 0 -0.05" rpy="0 0 0" size="0.014 0.0385 0.114" mass="0.013"/>
-    </link>
-    <joint name="shin_l_rear_passive" type="revolute">
-      <parent link="knee_l_passive_link"/>
-      <child link="shin_l_rear_passive_link"/>
-      <origin xyz="-0.0335 0 0" rpy="0 0.785398163 0"/>
-      <axis xyz="0 -1 0"/>
-      <limit effort="1000.0" lower="-0.4974" upper="1.8588" velocity="10.0"/>
+    <link name="knee_l_passive_link">
+      <visual>
+        <origin xyz="0.0335 0 0" rpy="0 0 0"/>
+        <geometry>
+          <mesh filename="package://kuroko_description/meshes/kuroko/obj/knee_r_passive.obj"/>
+        </geometry>
+      </visual>
+      <xacro:box_collision xyz="0.01675 0 0" rpy="0 0 0" size="0.0475 0.0505 0.014"/>
+      <xacro:box_inertial xyz="0.01675 0 0" rpy="0 0 0" size="0.0475 0.0505 0.014" mass="0.007"/>
+    </link>
+    <xacro:if value="$(arg gazebo)">
+      <xacro:gazebo_poassive_joint name="knee_l_front_passive_loop" xyz="0.0335 0 0"
+        parent="knee_l_passive_link" child="thigh_l_active_link" axis="0 1 0" lower="-1.8588" upper="0.4974"/>
+    </xacro:if>
+    <xacro:unless value="$(arg gazebo)">
+      <joint name="thigh_l_rear_mimic" type="revolute">
+        <parent link="shin_l_rear_passive_link"/>
+        <child link="thigh_l_rear_mimic_link"/>
+        <origin xyz="-0.00776457 0 -0.0289778" rpy="0 -0.785398163 0"/>
+        <axis xyz="0 1 0"/>
+        <limit effort="0" lower="-3.1416" upper="3.1416" velocity="1000"/>
+        <dynamics damping="0.0" friction="0.0"/>
+        <mimic joint="thigh_l_active" multiplier="-1" offset="0"/>
+      </joint>
+      <link name="thigh_l_rear_mimic_link"/>
+      <joint name="thigh_l_rear_passive" type="revolute">
+        <parent link="thigh_l_rear_mimic_link"/>
+        <child link="thigh_l_rear_passive_link"/>
+        <origin xyz="0 0 0" rpy="0 -0.785398163 0"/>
+        <axis xyz="0 1 0"/>
+        <limit effort="0" lower="-3.1416" upper="3.1416" velocity="1000"/>
+        <dynamics damping="0.0" friction="0.0"/>
+        <mimic joint="shin_l_active" multiplier="1" offset="0"/>
+      </joint>
+    </xacro:unless>
+    <xacro:if value="$(arg gazebo)">
+      <joint name="thigh_l_rear_passive" type="revolute">
+        <parent link="shin_l_rear_passive_link"/>
+        <child link="thigh_l_rear_passive_link"/>
+        <origin xyz="-0.00776457 0 -0.0289778" rpy="0 -1.570796327 0"/>
+        <axis xyz="0 1 0"/>
+        <limit effort="0" lower="-0.9948" upper="1.570796327" velocity="1000.0"/>
+        <dynamics damping="0.0" friction="0.0"/>
+      </joint>
+    </xacro:if>
+    <link name="thigh_l_rear_passive_link">
+      <visual>
+        <origin xyz="0 0 0.1" rpy="0 0 0"/>
+        <geometry>
+          <mesh filename="package://kuroko_description/meshes/kuroko/obj/thigh_r_rear_passive.obj"/>
+        </geometry>
+      </visual>
+      <xacro:box_collision xyz="0 0 0.05" rpy="0 0 0" size="0.014 0.0285 0.114"/>
+      <xacro:box_inertial xyz="0 0 0.05" rpy="0 0 0" size="0.014 0.0285 0.114" mass="0.011"/>
+    </link>
+    <xacro:if value="$(arg gazebo)">
+      <xacro:gazebo_poassive_joint name="thigh_l_rear_passive_loop" xyz="0 0 0.1" rpy="0 1.832597551 0"
+        parent="thigh_l_rear_passive_link" child="shin_l_active_link" axis="0 1 0"/>
+    </xacro:if>
+    <joint name="ankle_l_rear_passive" type="revolute">
+      <parent link="shin_l_rear_passive_link"/>
+      <child link="ankle_l_rear_passive_link"/>
+      <origin xyz="0 0 -0.1" rpy="0 -0.785398163 0"/>
+      <axis xyz="0 1 0"/>
+      <limit effort="0" lower="-0.4974" upper="1.8588" velocity="1000.0"/>
       <dynamics damping="0.0" friction="0.0"/>
       <mimic joint="shin_l_active" multiplier="1" offset="0"/>
     </joint>
-    <xacro:if value="$(arg gazebo)">
-      <xacro:gazebo_poassive_joint name="shin_l_rear_passive_loop" xyz="-0.0335 0 0"
-        parent="ankle_l_pitch_passive_link" child="shin_l_rear_passive_link" axis="0 -1 0"/>
-    </xacro:if>
-    <link name="shin_l_rear_passive_link">
-      <visual>
-        <origin xyz="0 0 0" rpy="0 0 0"/>
-        <geometry>
-          <mesh filename="package://kuroko_description/meshes/kuroko/obj/shin_r_rear_passive.obj"/>
-        </geometry>
-      </visual>
-      <xacro:box_collision xyz="0 0 -0.05" rpy="0 0 0" size="0.014 0.0445 0.114"/>
-      <xacro:box_inertial xyz="0 0 -0.05" rpy="0 0 0" size="0.014 0.0445 0.114" mass="0.016"/>
-    </link>
-    <joint name="ankle_l_pitch_passive" type="revolute">
-      <parent link="shin_l_front_passive_link"/>
-      <child link="ankle_l_pitch_passive_link"/>
-      <origin xyz="0 0 -0.1" rpy="0 -0.785398163 0"/>
-      <axis xyz="0 -1 0"/>
-      <limit effort="1000.0" lower="-1.8588" upper="0.4974" velocity="10.0"/>
-      <dynamics damping="0.0" friction="0.0"/>
-      <mimic joint="shin_l_active" multiplier="-1" offset="0"/>
-    </joint>
-    <link name="ankle_l_pitch_passive_link">
-      <visual>
-        <origin xyz="0 0 0" rpy="0 0 0"/>
+    <link name="ankle_l_rear_passive_link">
+      <visual>
+        <origin xyz="0.0335 0 0" rpy="0 0 0"/>
         <geometry>
           <mesh filename="package://kuroko_description/meshes/kuroko/obj/ankle_r_pitch_passive.obj"/>
         </geometry>
       </visual>
-      <xacro:box_collision xyz="-0.0285 0 -0.013" rpy="0 0 0" size="0.0855 0.0325 0.0465"/>
-      <xacro:box_inertial xyz="-0.0285 0 -0.013" rpy="0 0 0" size="0.0855 0.0325 0.0465"
+      <xacro:box_collision xyz="0.005 0 -0.013" rpy="0 0 0" size="0.0855 0.0325 0.0465"/>
+      <xacro:box_inertial xyz="0.005 0 -0.013" rpy="0 0 0" size="0.0855 0.0325 0.0465"
         mass="0.104"/>
     </link>
+    <xacro:if value="$(arg gazebo)">
+      <xacro:gazebo_poassive_joint name="ankle_l_front_passive_loop" xyz="0.0335 0 0" rpy="0 -0.785398163 0"
+        parent="ankle_l_rear_passive_link" child="shin_l_front_passive_link" axis="0 1 0"/>
+    </xacro:if>
     <joint name="ankle_l_roll" type="revolute">
-      <parent link="ankle_l_pitch_passive_link"/>
+      <parent link="ankle_l_rear_passive_link"/>
       <child link="ankle_l_roll_link"/>
-      <origin xyz="-0.015 0 -0.027" rpy="0 0 0"/>
+      <origin xyz="0.0185 0 -0.027" rpy="0 0 0"/>
       <axis xyz="1 0 0"/>
       <limit effort="1000.0" lower="-1.5708" upper="0.3704" velocity="10.0"/>

Commit message: Use MESH_DIR

File: kuroko_description/xacro/kuroko/parts/leg_l.xacro (robot description, xacro)
@@ -134,5 +134,5 @@
           <origin xyz="0 0 0" rpy="0 0 0"/>
           <geometry>
-            <mesh filename="package://kuroko_description/meshes/kuroko/stl/shin_r_front_passive.stl"/>
+            <mesh filename="${MESH_DIR}/kuroko/stl/shin_r_front_passive.stl"/>
           </geometry>
         </visual>

Commit message: Fix bug

File: kuroko_description/xacro/kuroko/parts/leg_l.xacro (robot description, xacro)
@@ -325,6 +325,6 @@
       <origin xyz="0.0185 0 -0.027" rpy="0 0 0"/>
       <axis xyz="1 0 0"/>
-      <limit effort="1000.0" lower="-1.5708" upper="0.3704" velocity="10.0"/>
-      <dynamics damping="0.0" friction="0.0"/>
+      <limit effort="3.1" lower="-1.5708" upper="0.3704" velocity="6.5"/>
+      <dynamics damping="0.477" friction="0.0"/>
     </joint>
     <link name="ankle_l_roll_link">
@@ -349,6 +349,6 @@
       <origin xyz="0 0 -0.03825" rpy="0 0 0"/>
       <axis xyz="0 0 -1"/>
-      <limit effort="1000.0" lower="-3.1" upper="3.1" velocity="10.0"/>
-      <dynamics damping="0.0" friction="0.0"/>
+      <limit effort="3.1" lower="-3.1416" upper="3.1416" velocity="6.5"/>
+      <dynamics damping="0.477" friction="0.0"/>
     </joint>
     <link name="ankle_l_yaw_link">

File: kuroko_description/xacro/kuroko/parts/leg_r.xacro (robot description, xacro)
@@ -8,6 +8,6 @@
       <origin xyz="0 0 -0.08425" rpy="0 0 0"/>
       <axis xyz="1 0 0"/>
-      <limit effort="1000.0" lower="-0.5550" upper="1.8640" velocity="10.0"/>
-      <dynamics damping="0.0" friction="0.0"/>
+      <limit effort="3.1" lower="-0.5550" upper="1.8640" velocity="6.5"/>
+      <dynamics damping="0.477" friction="0.0"/>
     </joint>
     <link name="hip_r_roll_link">
@@ -32,6 +32,6 @@
       <origin xyz="0 -0.027 0" rpy="0 0 0"/>
       <axis xyz="0 -1 0"/>
-      <limit effort="1000.0" lower="-3.1" upper="3.1" velocity="10.0"/>
-      <dynamics damping="0.0" friction="0.0"/>
+      <limit effort="3.1" lower="-3.1" upper="3.1" velocity="6.5"/>
+      <dynamics damping="0.477" friction="0.0"/>
     </joint>
     <link name="hip_r_pitch_link">
@@ -326,6 +326,6 @@
       <origin xyz="0.0185 0 -0.027" rpy="0 0 0"/>
       <axis xyz="1 0 0"/>
-      <limit effort="1000.0" lower="-0.3704" upper="1.5708" velocity="10.0"/>
-      <dynamics damping="0.0" friction="0.0"/>
+      <limit effort="3.1" lower="-0.3704" upper="1.5708" velocity="6.5"/>
+      <dynamics damping="0.477" friction="0.0"/>
     </joint>
     <link name="ankle_r_roll_link">
@@ -350,6 +350,6 @@
       <origin xyz="0 0 -0.03825" rpy="0 0 0"/>
       <axis xyz="0 0 -1"/>
-      <limit effort="1000.0" lower="-3.1" upper="3.1" velocity="10.0"/>
-      <dynamics damping="0.0" friction="0.0"/>
+      <limit effort="3.1" lower="-3.1" upper="3.1" velocity="6.5"/>
+      <dynamics damping="0.477" friction="0.0"/>
     </joint>
     <link name="ankle_r_yaw_link">
