Commit message: finish arm

File: kuroko_description/xacro/kuroko/kuroko.xacro (robot description, xacro)
@@ -1,16 +1,17 @@
 <?xml version="1.0"?>
 <robot name="kuroko" xmlns:xacro="http://www.ros.org/wiki/xacro">
-  <xacro:arg name="model_mode" default="rviz"/>
-  <xacro:arg name="gazebo_motor_model" default="dc"/>
+  <xacro:arg name="model_mode" default="rviz" />
+  <xacro:arg name="gazebo_motor_model" default="dc" />
   <!-- <xacro:arg name="gazebo_motor_model" default="kuroko"/> -->
-  <xacro:arg name="gazebo_hw_interface" default="position"/>
-  <xacro:include filename="$(find kuroko_description)/xacro/kuroko/parts/body.xacro"/>
-  <xacro:include filename="$(find kuroko_description)/xacro/kuroko/transmission/body.gazebo"/>
-  <xacro:include filename="$(find kuroko_description)/xacro/kuroko/parts/arm_r.xacro"/>
-  <xacro:include filename="$(find kuroko_description)/xacro/kuroko/transmission/arm_r.gazebo"/>
-  <xacro:include filename="$(find kuroko_description)/xacro/kuroko/parts/arm_l.xacro"/>
-  <xacro:include filename="$(find kuroko_description)/xacro/kuroko/transmission/arm_l.gazebo"/>
-  <!-- <xacro:include filename="$(find kuroko_description)/xacro/kuroko/parts/leg_r.xacro"/>
-  <xacro:include filename="$(find kuroko_description)/xacro/kuroko/transmission/leg_r.gazebo"/>
+  <xacro:arg name="gazebo_hw_interface" default="position" />
+  <xacro:include filename="$(find kuroko_description)/xacro/kuroko/parts/body.xacro" />
+  <xacro:include filename="$(find kuroko_description)/xacro/kuroko/transmission/body.gazebo" />
+  <xacro:include filename="$(find kuroko_description)/xacro/kuroko/parts/arm_r.xacro" />
+  <xacro:include filename="$(find kuroko_description)/xacro/kuroko/transmission/arm_r.gazebo" />
+  <xacro:include filename="$(find kuroko_description)/xacro/kuroko/parts/arm_l.xacro" />
+  <xacro:include filename="$(find kuroko_description)/xacro/kuroko/transmission/arm_l.gazebo" />
+  <xacro:include filename="$(find kuroko_description)/xacro/kuroko/parts/leg_r.xacro" />
+  <xacro:include filename="$(find kuroko_description)/xacro/kuroko/transmission/leg_r.gazebo" />
+  <!--
   <xacro:include filename="$(find kuroko_description)/xacro/kuroko/parts/leg_l.xacro"/>
   <xacro:include filename="$(find kuroko_description)/xacro/kuroko/transmission/leg_l.gazebo"/>-->
@@ -38,26 +39,30 @@
   <!-- MACRO:Setting up a Robot Model -->
   <xacro:macro name="kuroko_xacro" params="model_mode gazebo_hw_interface">
-    <link name="root_link"/>
+    <link name="root_link" />
     <joint name="root_joint" type="fixed">
-        <parent link="root_link"/>
-        <child  link="chest"/>
-        <origin xyz="0 0 0" rpy="0 0 0"/>
+      <parent link="root_link" />
+      <child link="chest" />
+      <origin xyz="0 0 0" rpy="0 0 0" />
     </joint>
-    <xacro:body_xacro/>
-    <xacro:body_gazebo gazebo_hw_interface="${gazebo_hw_interface}"/>
-    <xacro:arm_r_xacro/>
-    <xacro:arm_r_gazebo gazebo_hw_interface="${gazebo_hw_interface}"/>
-    <xacro:arm_l_xacro/>
-    <xacro:arm_l_gazebo gazebo_hw_interface="${gazebo_hw_interface}"/>
-    <!-- <xacro:leg_r_xacro/>
-    <xacro:leg_r_gazebo gazebo_hw_interface="${gazebo_hw_interface}"/>
+    <xacro:body_xacro />
+    <xacro:body_gazebo gazebo_hw_interface="${gazebo_hw_interface}" />
+    <xacro:arm_r_xacro />
+    <xacro:arm_r_gazebo gazebo_hw_interface="${gazebo_hw_interface}" />
+    <xacro:arm_l_xacro />
+    <xacro:arm_l_gazebo gazebo_hw_interface="${gazebo_hw_interface}" />
+    <xacro:leg_r_xacro />
+    <xacro:leg_r_gazebo gazebo_hw_interface="${gazebo_hw_interface}" />
+    <!--
     <xacro:leg_l_xacro/>
     <xacro:leg_l_gazebo gazebo_hw_interface="${gazebo_hw_interface}"/>-->
   </xacro:macro>
   <!-- Load Macros -->
-  <xacro:kuroko_xacro model_mode="$(arg model_mode)" gazebo_hw_interface="$(arg gazebo_hw_interface)"/>
-  <xacro:gazebo_plugin_xacro gazebo_motor_model="$(arg gazebo_motor_model)"/>
+  <xacro:kuroko_xacro model_mode="$(arg model_mode)"
+    gazebo_hw_interface="$(arg gazebo_hw_interface)" />
+  <xacro:gazebo_plugin_xacro gazebo_motor_model="$(arg gazebo_motor_model)" />
   <!-- <xacro:imu_xacro model_mode="$(arg model_mode)"/> -->
-  <!-- <xacro:urg_xacro firame_id="arm_r_urg_link" topic_name="/sensor/urg/right/scan_raw" sensor_name="urg_right"/> -->
-  <!-- <xacro:urg_xacro firame_id="arm_l_urg_link" topic_name="/sensor/urg/left/scan_raw" sensor_name="urg_left"/> -->
+  <!-- <xacro:urg_xacro firame_id="arm_r_urg_link" topic_name="/sensor/urg/right/scan_raw"
+  sensor_name="urg_right"/> -->
+  <!-- <xacro:urg_xacro firame_id="arm_l_urg_link" topic_name="/sensor/urg/left/scan_raw"
+  sensor_name="urg_left"/> -->
 </robot>

File: kuroko_description/xacro/kuroko/parts/arm_l.xacro (robot description, xacro)
@@ -4,76 +4,76 @@
 		<!-- Link conencts from body. Shoulder first. -->
 		<joint name="shoulder_l_joint" type="revolute">
-			<parent link="chest"/>
-			<child link="shoulder_l"/>
-				<origin xyz="0 0.082 0.05075" rpy="0 0 0"/>
-				<axis xyz="0 1 0"/>
-			<limit effort="1000.0" lower="-3.1" upper="3.1" velocity="10.0"/>
-			<dynamics damping="0.0" friction="0.0"/>
+			<parent link="chest" />
+			<child link="shoulder_l" />
+			<origin xyz="0 0.082 0.05075" rpy="0 0 0" />
+			<axis xyz="0 1 0" />
+			<limit effort="1000.0" lower="-3.1" upper="3.1" velocity="10.0" />
+			<dynamics damping="0.0" friction="0.0" />
 		</joint>
 		<link name="shoulder_l">
 			<visual>
-				<origin xyz="0 0 0" rpy="0 0 0"/>
+				<origin xyz="0 0 0" rpy="0 0 0" />
 				<geometry>
-					<mesh filename="package://kuroko_description/meshes/kuroko/obj/shoulder_l.obj"/>
+					<mesh filename="package://kuroko_description/meshes/kuroko/obj/shoulder_l.obj" />
 				</geometry>
 			</visual>
-			<xacro:box_collision xyz="0 0.0205 0" rpy="0 0 0" size="0.053 0.041 0.04"/>
-			<xacro:box_inertial xyz="0 0.0205 0" rpy="0 0 0" size="0.053 0.041 0.04" mass="0.022"/>
+			<xacro:box_collision xyz="0 0.0205 0" rpy="0 0 0" size="0.053 0.041 0.04" />
+			<xacro:box_inertial xyz="0 0.0205 0" rpy="0 0 0" size="0.053 0.041 0.04" mass="0.022" />
 		</link>
 		<joint name="arm_l_joint" type="revolute">
-		  <parent link="shoulder_l"/>
-			<child link="arm_l"/>
-		    <origin xyz="0 0.028 0" rpy="0 0 0"/>
-		    <axis xyz="-1 0 0"/>
-			<limit effort="1000.0" lower="-3.1" upper="3.1" velocity="10.0"/>
-			<dynamics damping="0.0" friction="0.0"/>
+			<parent link="shoulder_l" />
+			<child link="arm_l" />
+			<origin xyz="0 0.028 0" rpy="0 0 0" />
+			<axis xyz="-1 0 0" />
+			<limit effort="1000.0" lower="-3.1" upper="3.1" velocity="10.0" />
+			<dynamics damping="0.0" friction="0.0" />
 		</joint>
 		<link name="arm_l">
 			<visual>
-				<origin xyz="0 0 0" rpy="0 0 0"/>
+				<origin xyz="0 0 0" rpy="0 0 0" />
 				<geometry>
-					<mesh filename="package://kuroko_description/meshes/kuroko/obj/arm_l.obj"/>
+					<mesh filename="package://kuroko_description/meshes/kuroko/obj/arm_l.obj" />
 				</geometry>
 			</visual>
-      <xacro:box_collision xyz="0 0.0385 -0.02575" rpy="0 0 0" size="0.044 0.1045 0.085"/>
-			<xacro:box_inertial xyz="0 0.0385 -0.02575" rpy="0 0 0" size="0.044 0.1045 0.085" mass="0.342"/>
+			<xacro:box_collision xyz="0 0.0385 -0.02575" rpy="0 0 0" size="0.044 0.1045 0.085" />
+			<xacro:box_inertial xyz="0 0.0385 -0.02575" rpy="0 0 0" size="0.044 0.1045 0.085" mass="0.342" />
 		</link>
 		<joint name="scissor_lf_joint" type="revolute">
-		  <parent link="arm_l"/>
-			<child link="scissor_lf"/>
-		    <origin xyz="0 0.02575 -0.057" rpy="0 0 0"/>
-		    <axis xyz="0 1 0"/>
-			<limit effort="1000.0" lower="-3.1" upper="3.1" velocity="10.0"/>
-			<dynamics damping="0.0" friction="0.0"/>
+			<parent link="arm_l" />
+			<child link="scissor_lf" />
+			<origin xyz="0 0.02575 -0.057" rpy="0 0 0" />
+			<axis xyz="0 1 0" />
+			<limit effort="1000.0" lower="-3.1" upper="3.1" velocity="10.0" />
+			<dynamics damping="0.0" friction="0.0" />
 		</joint>
 		<link name="scissor_lf">
 			<visual>
-				<origin xyz="0 0 0" rpy="0 0 0"/>
+				<origin xyz="0 0 0" rpy="0 0 0" />
 				<geometry>
-					<mesh filename="package://kuroko_description/meshes/kuroko/obj/scissor_lf.obj"/>
+					<mesh filename="package://kuroko_description/meshes/kuroko/obj/scissor_lf.obj" />
 				</geometry>
 			</visual>
-      <xacro:box_collision xyz="0.0043 0 -0.104" rpy="0 0 0" size="0.01085 0.058 0.208"/>
-      <xacro:box_collision xyz="-0.0206 0 -0.201" rpy="0 0 0" size="0.039 0.058 0.014"/>
-			<xacro:box_inertial xyz="0.0043 0 -0.104" rpy="0 0 0" size="0.044 0.058 0.208" mass="0.032"/>
+			<xacro:box_collision xyz="0.0043 0 -0.104" rpy="0 0 0" size="0.01085 0.058 0.208" />
+			<xacro:box_collision xyz="-0.0206 0 -0.201" rpy="0 0 0" size="0.039 0.058 0.014" />
+			<xacro:box_inertial xyz="0.0043 0 -0.104" rpy="0 0 0" size="0.044 0.058 0.208" mass="0.032" />
 		</link>
 		<joint name="scissor_lr_joint" type="revolute">
-		  <parent link="arm_l"/>
-			<child link="scissor_lr"/>
-		    <origin xyz="0 0.02575 -0.057" rpy="0 0 0"/>
-		    <axis xyz="0 -1 0"/>
-			<limit effort="1000.0" lower="-3.1" upper="3.1" velocity="10.0"/>
-			<dynamics damping="0.0" friction="0.0"/>
+			<parent link="arm_l" />
+			<child link="scissor_lr" />
+			<origin xyz="0 0.02575 -0.057" rpy="0 0 0" />
+			<axis xyz="0 -1 0" />
+			<limit effort="1000.0" lower="-3.1" upper="3.1" velocity="10.0" />
+			<dynamics damping="0.0" friction="0.0" />
 		</joint>
 		<link name="scissor_lr">
 			<visual>
-				<origin xyz="0 0 0" rpy="0 0 0"/>
+				<origin xyz="0 0 0" rpy="0 0 0" />
 				<geometry>
-					<mesh filename="package://kuroko_description/meshes/kuroko/obj/scissor_lr.obj"/>
+					<mesh filename="package://kuroko_description/meshes/kuroko/obj/scissor_lr.obj" />
 				</geometry>
 			</visual>
-      <xacro:box_collision xyz="-0.0043 0 -0.1" rpy="0 0 0" size="0.01085 0.044 0.2"/>
-      <xacro:box_collision xyz="0.0206 0 -0.193" rpy="0 0 0" size="0.039 0.044 0.014"/>
-			<xacro:box_inertial xyz="-0.0043 0 -0.1" rpy="0 0 0" size="0.044 0.044 0.2" mass="0.031"/>
+			<xacro:box_collision xyz="-0.0043 0 -0.1" rpy="0 0 0" size="0.01085 0.044 0.2" />
+			<xacro:box_collision xyz="0.0206 0 -0.193" rpy="0 0 0" size="0.039 0.044 0.014" />
+			<xacro:box_inertial xyz="-0.0043 0 -0.1" rpy="0 0 0" size="0.044 0.044 0.2" mass="0.031" />
 		</link>
 	</xacro:macro>

File: kuroko_description/xacro/kuroko/parts/arm_r.xacro (robot description, xacro)
@@ -4,76 +4,77 @@
 		<!-- Link conencts from body. Shoulder first. -->
 		<joint name="shoulder_r_joint" type="revolute">
-		  <parent link="chest"/>
-			<child link="shoulder_r"/>
-		    <origin xyz="0 -0.082 0.05075" rpy="0 0 0"/>
-		    <axis xyz="0 -1 0"/>
-			<limit effort="1000.0" lower="-3.1" upper="3.1" velocity="10.0"/>
-			<dynamics damping="0.0" friction="0.0"/>
+			<parent link="chest" />
+			<child link="shoulder_r" />
+			<origin xyz="0 -0.082 0.05075" rpy="0 0 0" />
+			<axis xyz="0 -1 0" />
+			<limit effort="1000.0" lower="-3.1" upper="3.1" velocity="10.0" />
+			<dynamics damping="0.0" friction="0.0" />
 		</joint>
 		<link name="shoulder_r">
 			<visual>
-				<origin xyz="0 0 0" rpy="0 0 0"/>
+				<origin xyz="0 0 0" rpy="0 0 0" />
 				<geometry>
-					<mesh filename="package://kuroko_description/meshes/kuroko/obj/shoulder_r.obj"/>
+					<mesh filename="package://kuroko_description/meshes/kuroko/obj/shoulder_r.obj" />
 				</geometry>
 			</visual>
-      <xacro:box_collision xyz="0 -0.0205 0" rpy="0 0 0" size="0.053 0.041 0.04"/>
-			<xacro:box_inertial xyz="0 -0.0205 0" rpy="0 0 0" size="0.053 0.041 0.04" mass="0.022"/>
+			<xacro:box_collision xyz="0 -0.0205 0" rpy="0 0 0" size="0.053 0.041 0.04" />
+			<xacro:box_inertial xyz="0 -0.0205 0" rpy="0 0 0" size="0.053 0.041 0.04" mass="0.022" />
 		</link>
 		<joint name="arm_r_joint" type="revolute">
-		  <parent link="shoulder_r"/>
-			<child link="arm_r"/>
-		    <origin xyz="0 -0.028 0" rpy="0 0 0"/>
-		    <axis xyz="-1 0 0"/>
-			<limit effort="1000.0" lower="-3.1" upper="3.1" velocity="10.0"/>
-			<dynamics damping="0.0" friction="0.0"/>
+			<parent link="shoulder_r" />
+			<child link="arm_r" />
+			<origin xyz="0 -0.028 0" rpy="0 0 0" />
+			<axis xyz="-1 0 0" />
+			<limit effort="1000.0" lower="-3.1" upper="3.1" velocity="10.0" />
+			<dynamics damping="0.0" friction="0.0" />
 		</joint>
 		<link name="arm_r">
 			<visual>
-				<origin xyz="0 0 0" rpy="0 0 0"/>
+				<origin xyz="0 0 0" rpy="0 0 0" />
 				<geometry>
-					<mesh filename="package://kuroko_description/meshes/kuroko/obj/arm_r.obj"/>
+					<mesh filename="package://kuroko_description/meshes/kuroko/obj/arm_r.obj" />
 				</geometry>
 			</visual>
-      <xacro:box_collision xyz="0 -0.0385 -0.02575" rpy="0 0 0" size="0.044 0.1045 0.085"/>
-			<xacro:box_inertial xyz="0 -0.0385 -0.02575" rpy="0 0 0" size="0.044 0.1045 0.085" mass="0.342"/>
+			<xacro:box_collision xyz="0 -0.0385 -0.02575" rpy="0 0 0" size="0.044 0.1045 0.085" />
+			<xacro:box_inertial xyz="0 -0.0385 -0.02575" rpy="0 0 0" size="0.044 0.1045 0.085"
+				mass="0.342" />
 		</link>
 		<joint name="scissor_rf_joint" type="revolute">
-		  <parent link="arm_r"/>
-			<child link="scissor_rf"/>
-		    <origin xyz="0 -0.02575 -0.057" rpy="0 0 0"/>
-		    <axis xyz="0 -1 0"/>
-			<limit effort="1000.0" lower="-3.1" upper="3.1" velocity="10.0"/>
-			<dynamics damping="0.0" friction="0.0"/>
+			<parent link="arm_r" />
+			<child link="scissor_rf" />
+			<origin xyz="0 -0.02575 -0.057" rpy="0 0 0" />
+			<axis xyz="0 -1 0" />
+			<limit effort="1000.0" lower="-3.1" upper="3.1" velocity="10.0" />
+			<dynamics damping="0.0" friction="0.0" />
 		</joint>
 		<link name="scissor_rf">
 			<visual>
-				<origin xyz="0 0 0" rpy="0 0 0"/>
+				<origin xyz="0 0 0" rpy="0 0 0" />
 				<geometry>
-					<mesh filename="package://kuroko_description/meshes/kuroko/obj/scissor_rf.obj"/>
+					<mesh filename="package://kuroko_description/meshes/kuroko/obj/scissor_rf.obj" />
 				</geometry>
 			</visual>
-      <xacro:box_collision xyz="0.0043 0 -0.104" rpy="0 0 0" size="0.01085 0.058 0.208"/>
-      <xacro:box_collision xyz="-0.0206 0 -0.201" rpy="0 0 0" size="0.039 0.058 0.014"/>
-			<xacro:box_inertial xyz="0.0043 0 -0.104" rpy="0 0 0" size="0.044 0.058 0.208" mass="0.032"/>
+			<xacro:box_collision xyz="0.0043 0 -0.104" rpy="0 0 0" size="0.01085 0.058 0.208" />
+			<xacro:box_collision xyz="-0.0206 0 -0.201" rpy="0 0 0" size="0.039 0.058 0.014" />
+			<xacro:box_inertial xyz="0.0043 0 -0.104" rpy="0 0 0" size="0.044 0.058 0.208" mass="0.032" />
 		</link>
 		<joint name="scissor_rr_joint" type="revolute">
-		  <parent link="arm_r"/>
-			<child link="scissor_rr"/>
-		    <origin xyz="0 -0.02575 -0.057" rpy="0 0 0"/>
-		    <axis xyz="0 1 0"/>
-			<limit effort="1000.0" lower="-3.1" upper="3.1" velocity="10.0"/>
-			<dynamics damping="0.0" friction="0.0"/>
+			<parent link="arm_r" />
+			<child link="scissor_rr" />
+			<origin xyz="0 -0.02575 -0.057" rpy="0 0 0" />
+			<axis xyz="0 1 0" />
+			<limit effort="1000.0" lower="-3.1" upper="3.1" velocity="10.0" />
+			<dynamics damping="0.0" friction="0.0" />
 		</joint>
 		<link name="scissor_rr">
 			<visual>
-				<origin xyz="0 0 0" rpy="0 0 0"/>
+				<origin xyz="0 0 0" rpy="0 0 0" />
 				<geometry>
-					<mesh filename="package://kuroko_description/meshes/kuroko/obj/scissor_rr.obj"/>
+					<mesh filename="package://kuroko_description/meshes/kuroko/obj/scissor_rr.obj" />
 				</geometry>
 			</visual>
-      <xacro:box_collision xyz="-0.0043 0 -0.1" rpy="0 0 0" size="0.01085 0.044 0.2"/>
-      <xacro:box_collision xyz="0.0206 0 -0.193" rpy="0 0 0" size="0.039 0.044 0.014"/>
-			<xacro:box_inertial xyz="-0.0043 0 -0.1" rpy="0 0 0" size="0.044 0.044 0.2" mass="0.031"/>
+			<xacro:box_collision xyz="-0.0043 0 -0.1" rpy="0 0 0" size="0.01085 0.044 0.2" />
+			<xacro:box_collision xyz="0.0206 0 -0.193" rpy="0 0 0" size="0.039 0.044 0.014" />
+			<xacro:box_inertial xyz="-0.0043 0 -0.1" rpy="0 0 0" size="0.044 0.044 0.2" mass="0.031" />
 		</link>
 	</xacro:macro>

File: kuroko_description/xacro/kuroko/parts/body.xacro (robot description, xacro)
@@ -32,5 +32,6 @@
 			</visual>
 			<xacro:box_collision xyz="0.00125 0 -0.04875" rpy="0 0 0" size="0.092 0.0325 0.0975" />
-			<xacro:box_inertial xyz="0.00125 0 -0.04875" rpy="0 0 0" size="0.092 0.0325 0.0975" mass="0.337" />
+			<xacro:box_inertial xyz="0.00125 0 -0.04875" rpy="0 0 0" size="0.092 0.0325 0.0975"
+				mass="0.337" />
 		</link>
 	</xacro:macro>
