Commit message: wip

File: kuroko_description/xacro/kuroko/kuroko.xacro (robot description, xacro)
@@ -1,5 +1,5 @@
 <?xml version="1.0"?>
 <robot name="kuroko" xmlns:xacro="http://www.ros.org/wiki/xacro">
-  <xacro:arg name="model_mode" default="rviz" />
+  <xacro:arg name="gazebo" default="false" />
   <xacro:arg name="gazebo_motor_model" default="dc" />
   <!-- <xacro:arg name="gazebo_motor_model" default="kuroko"/> -->
@@ -38,5 +38,5 @@
   </xacro:macro>
   <!-- MACRO:Setting up a Robot Model -->
-  <xacro:macro name="kuroko_xacro" params="model_mode gazebo_hw_interface">
+  <xacro:macro name="kuroko_xacro" params="gazebo gazebo_hw_interface">
     <link name="root_link" />
     <joint name="root_joint" type="fixed">
@@ -51,5 +51,5 @@
     <xacro:arm_l_xacro />
     <xacro:arm_l_gazebo gazebo_hw_interface="${gazebo_hw_interface}" />
-    <xacro:leg_r_xacro />
+    <xacro:leg_r_xacro gazebo="$(arg gazebo)" />
     <xacro:leg_r_gazebo gazebo_hw_interface="${gazebo_hw_interface}" />
     <!--
@@ -58,5 +58,5 @@
   </xacro:macro>
   <!-- Load Macros -->
-  <xacro:kuroko_xacro model_mode="$(arg model_mode)"
+  <xacro:kuroko_xacro gazebo="$(arg gazebo)"
     gazebo_hw_interface="$(arg gazebo_hw_interface)" />
   <xacro:gazebo_plugin_xacro gazebo_motor_model="$(arg gazebo_motor_model)" />

File: kuroko_description/xacro/kuroko/parts/arm_l.xacro (robot description, xacro)
@@ -6,5 +6,5 @@
 			<parent link="chest" />
 			<child link="shoulder_l" />
-			<origin xyz="0 0.082 0.05075" rpy="0 0 0" />
+			<origin xyz="0 0.108 0.01275" rpy="0 0 0" />
 			<axis xyz="0 1 0" />
 			<limit effort="1000.0" lower="-3.1" upper="3.1" velocity="10.0" />
@@ -18,6 +18,6 @@
 				</geometry>
 			</visual>
-			<xacro:box_collision xyz="0 0.0205 0" rpy="0 0 0" size="0.053 0.041 0.04" />
-			<xacro:box_inertial xyz="0 0.0205 0" rpy="0 0 0" size="0.053 0.041 0.04" mass="0.022" />
+			<xacro:box_collision xyz="0 0.0205 0" rpy="0 0 0" size="0.042 0.041 0.04" />
+			<xacro:box_inertial xyz="0 0.0205 0" rpy="0 0 0" size="0.042 0.041 0.04" mass="0.022" />
 		</link>
 		<joint name="arm_l_joint" type="revolute">
@@ -36,11 +36,11 @@
 				</geometry>
 			</visual>
-			<xacro:box_collision xyz="0 0.0385 -0.02575" rpy="0 0 0" size="0.044 0.1045 0.085" />
-			<xacro:box_inertial xyz="0 0.0385 -0.02575" rpy="0 0 0" size="0.044 0.1045 0.085" mass="0.342" />
+			<xacro:box_collision xyz="0 0.0385 -0.02575" rpy="0 0 0" size="0.0285 0.1045 0.08" />
+			<xacro:box_inertial xyz="0 0.0385 -0.02575" rpy="0 0 0" size="0.0285 0.1045 0.08" mass="0.342" />
 		</link>
 		<joint name="scissor_lf_joint" type="revolute">
 			<parent link="arm_l" />
 			<child link="scissor_lf" />
-			<origin xyz="0 0.02575 -0.057" rpy="0 0 0" />
+			<origin xyz="0 0.0265 -0.0545" rpy="0 0 0" />
 			<axis xyz="0 1 0" />
 			<limit effort="1000.0" lower="-3.1" upper="3.1" velocity="10.0" />
@@ -61,5 +61,5 @@
 			<parent link="arm_l" />
 			<child link="scissor_lr" />
-			<origin xyz="0 0.02575 -0.057" rpy="0 0 0" />
+			<origin xyz="0 0.0265 -0.0545" rpy="0 0 0" />
 			<axis xyz="0 -1 0" />
 			<limit effort="1000.0" lower="-3.1" upper="3.1" velocity="10.0" />

File: kuroko_description/xacro/kuroko/parts/arm_r.xacro (robot description, xacro)
@@ -6,5 +6,5 @@
 			<parent link="chest" />
 			<child link="shoulder_r" />
-			<origin xyz="0 -0.082 0.05075" rpy="0 0 0" />
+			<origin xyz="0 -0.108 0.01275" rpy="0 0 0" />
 			<axis xyz="0 -1 0" />
 			<limit effort="1000.0" lower="-3.1" upper="3.1" velocity="10.0" />
@@ -18,6 +18,6 @@
 				</geometry>
 			</visual>
-			<xacro:box_collision xyz="0 -0.0205 0" rpy="0 0 0" size="0.053 0.041 0.04" />
-			<xacro:box_inertial xyz="0 -0.0205 0" rpy="0 0 0" size="0.053 0.041 0.04" mass="0.022" />
+			<xacro:box_collision xyz="0 -0.0205 0" rpy="0 0 0" size="0.042 0.041 0.04" />
+			<xacro:box_inertial xyz="0 -0.0205 0" rpy="0 0 0" size="0.042 0.041 0.04" mass="0.022" />
 		</link>
 		<joint name="arm_r_joint" type="revolute">
@@ -36,6 +36,6 @@
 				</geometry>
 			</visual>
-			<xacro:box_collision xyz="0 -0.0385 -0.02575" rpy="0 0 0" size="0.044 0.1045 0.085" />
-			<xacro:box_inertial xyz="0 -0.0385 -0.02575" rpy="0 0 0" size="0.044 0.1045 0.085"
+			<xacro:box_collision xyz="0 -0.0385 -0.02575" rpy="0 0 0" size="0.0285 0.1045 0.08" />
+			<xacro:box_inertial xyz="0 -0.0385 -0.02575" rpy="0 0 0" size="0.0285 0.1045 0.08"
 				mass="0.342" />
 		</link>
@@ -43,5 +43,5 @@
 			<parent link="arm_r" />
 			<child link="scissor_rf" />
-			<origin xyz="0 -0.02575 -0.057" rpy="0 0 0" />
+			<origin xyz="0 -0.0265 -0.0545" rpy="0 0 0" />
 			<axis xyz="0 -1 0" />
 			<limit effort="1000.0" lower="-3.1" upper="3.1" velocity="10.0" />
@@ -62,5 +62,5 @@
 			<parent link="arm_r" />
 			<child link="scissor_rr" />
-			<origin xyz="0 -0.02575 -0.057" rpy="0 0 0" />
+			<origin xyz="0 -0.0265 -0.0545" rpy="0 0 0" />
 			<axis xyz="0 1 0" />
 			<limit effort="1000.0" lower="-3.1" upper="3.1" velocity="10.0" />

File: kuroko_description/xacro/kuroko/parts/body.xacro (robot description, xacro)
@@ -11,6 +11,6 @@
 				</geometry>
 			</visual>
-			<xacro:box_collision xyz="0 0 0.057" rpy="0 0 0" size="0.1 0.16 0.114" />
-			<xacro:box_inertial xyz="0 0 0.057" rpy="0 0 0" size="0.1 0.16 0.114" mass="0.991" />
+			<xacro:box_collision xyz="0 0 0.057" rpy="0 0 0" size="0.1 0.204 0.114" />
+			<xacro:box_inertial xyz="0 0 0.057" rpy="0 0 0" size="0.1 0.204 0.114" mass="0.991" />
 		</link>
 		<!-- Joint1 -->
@@ -31,6 +31,6 @@
 				</geometry>
 			</visual>
-			<xacro:box_collision xyz="0.00125 0 -0.04875" rpy="0 0 0" size="0.092 0.0325 0.0975" />
-			<xacro:box_inertial xyz="0.00125 0 -0.04875" rpy="0 0 0" size="0.092 0.0325 0.0975"
+			<xacro:box_collision xyz="0.00125 0 -0.04875" rpy="0 0 0" size="0.0705 0.0325 0.0975" />
+			<xacro:box_inertial xyz="0.00125 0 -0.04875" rpy="0 0 0" size="0.0705 0.0325 0.0975"
 				mass="0.337" />
 		</link>

File: kuroko_description/xacro/kuroko/parts/leg_r.xacro (robot description, xacro)
@@ -1,5 +1,5 @@
 <?xml version="1.0"?>
 <robot xmlns:xacro="http://www.ros.org/wiki/xacro">
-	<xacro:macro name="leg_r_xacro">
+	<xacro:macro name="leg_r_xacro" params="gazebo:=false">
 		<!-- Link conencts from body. Femoral first. -->
 		<joint name="crotch_r_joint" type="revolute">
@@ -37,12 +37,12 @@
 				</geometry>
 			</visual>
-			<xacro:box_collision xyz="-0.00175 -0.049 -0.015" rpy="0 0 0" size="0.067 0.098 0.0625" />
-			<xacro:box_inertial xyz="-0.00175 -0.049 -0.015" rpy="0 0 0" size="0.067 0.098 0.0625"
-				mass="0.484" />
+			<xacro:box_collision xyz="-0.00175 -0.049 -0.015" rpy="0 0 0" size="0.067 0.098 0.0585" />
+			<xacro:box_inertial xyz="-0.00175 -0.049 -0.015" rpy="0 0 0" size="0.067 0.098 0.0585"
+				mass="0.478" />
 		</link>
 		<joint name="thigh_r_02_joint" type="revolute">
 			<parent link="thigh_r_01" />
 			<child link="thigh_r_02" />
-			<origin xyz="0.015 -0.02925 -0.0305" rpy="0 0 0" />
+			<origin xyz="0.015 -0.02925 -0.0305" rpy="0 -0.785398163 0" />
 			<axis xyz="0 1 0" />
 			<limit effort="1000.0" lower="-3.1" upper="3.1" velocity="10.0" />
@@ -57,10 +57,10 @@
 			</visual>
 			<xacro:box_collision xyz="0 0 -0.05" rpy="0 0 0" size="0.014 0.0445 0.114" />
-			<xacro:box_inertial xyz="0 0 -0.05" rpy="0 0 0" size="0.014 0.0445 0.114" mass="0.011" />
+			<xacro:box_inertial xyz="0 0 -0.05" rpy="0 0 0" size="0.014 0.0445 0.114" mass="0.012" />
 		</link>
 		<joint name="thigh_r_03_joint" type="revolute">
 			<parent link="thigh_r_01" />
 			<child link="thigh_r_03" />
-			<origin xyz="-0.0185 -0.02925 -0.0305" rpy="0 0 0" />
+			<origin xyz="-0.0185 -0.02925 -0.0305" rpy="0 1.047197551 0" />
 			<axis xyz="0 1 0" />
 			<limit effort="1000.0" lower="-3.1" upper="3.1" velocity="10.0" />
@@ -76,10 +76,10 @@
 			<xacro:box_collision xyz="-0.004745 0 -0.015" rpy="0 0 0" size="0.02349 0.0445 0.044" />
 			<xacro:box_inertial xyz="-0.004745 0 -0.015" rpy="0 0 0" size="0.02349 0.0445 0.044"
-				mass="0.011" />
+				mass="0.008" />
 		</link>
 		<joint name="thigh_r_04_joint" type="revolute">
 			<parent link="thigh_r_01" />
 			<child link="thigh_r_04" />
-			<origin xyz="-0.0185 -0.02925 -0.0305" rpy="0 0 0" />
+			<origin xyz="-0.0185 -0.02925 -0.0305" rpy="0 -0.785398163 0" />
 			<axis xyz="0 1 0" />
 			<limit effort="1000.0" lower="-3.1" upper="3.1" velocity="10.0" />
@@ -95,25 +95,66 @@
 			</visual>
 			<xacro:box_collision xyz="0 0 -0.05" rpy="0 0 0" size="0.014 0.0345 0.114" />
-			<xacro:box_inertial xyz="0 0 -0.05" rpy="0 0 0" size="0.014 0.0345 0.114" mass="0.011" />
-		</link>
-		<joint name="thigh_r_05_mimic_joint" type="revolute">
-			<parent link="thigh_r_03" />
-			<child link="thigh_r_05_mimic" />
-			<origin xyz="0 0 -0.03" rpy="0 0 0" />
-			<axis xyz="0 1 0" />
-			<limit effort="1000.0" lower="-3.1" upper="3.1" velocity="10.0" />
-			<dynamics damping="0.0" friction="0.0" />
-			<mimic joint="thigh_r_03_joint" multiplier="-1" offset="0" />
-		</joint>
-		<link name="thigh_r_05_mimic" />
-		<joint name="thigh_r_05_joint" type="revolute">
-			<parent link="thigh_r_05_mimic" />
-			<child link="thigh_r_05" />
-			<origin xyz="0 0 0" rpy="0 0 0" />
-			<axis xyz="0 1 0" />
-			<limit effort="1000.0" lower="-3.1" upper="3.1" velocity="10.0" />
-			<dynamics damping="0.0" friction="0.0" />
-			<mimic joint="thigh_r_02_joint" multiplier="1" offset="0" />
-		</joint>
+			<xacro:box_inertial xyz="0 0 -0.05" rpy="0 0 0" size="0.014 0.0345 0.114" mass="0.012" />
+		</link>
+		<xacro:unless value="$(arg gazebo)">
+			<joint name="thigh_r_05_mimic1" type="revolute">
+				<parent link="thigh_r_03" />
+				<child link="thigh_r_05_mimic" />
+				<origin xyz="0 0 -0.03" rpy="0 -1.832597551 0" />
+				<axis xyz="0 1 0" />
+				<limit effort="1000.0" lower="-3.1" upper="3.1" velocity="10.0" />
+				<dynamics damping="0.0" friction="0.0" />
+				<mimic joint="thigh_r_03_joint" multiplier="-1" offset="0" />
+			</joint>
+			<link name="thigh_r_05_mimic" />
+			<joint name="thigh_r_05_mimic2" type="revolute">
+				<parent link="thigh_r_05_mimic" />
+				<child link="thigh_r_05" />
+				<origin xyz="0 0 0" rpy="0 0 0" />
+				<axis xyz="0 1 0" />
+				<limit effort="1000.0" lower="-3.1" upper="3.1" velocity="10.0" />
+				<dynamics damping="0.0" friction="0.0" />
+				<mimic joint="thigh_r_02_joint" multiplier="1" offset="0" />
+			</joint>
+		</xacro:unless>
+		<xacro:if value="$(arg gazebo)">
+			<joint name="thigh_r_05_joint" type="revolute">
+				<parent link="thigh_r_03" />
+				<child link="thigh_r_05" />
+				<origin xyz="0 0 -0.03" rpy="0 -1.832597551 0" />
+				<axis xyz="0 1 0" />
+				<limit effort="1000.0" lower="-3.1" upper="3.1" velocity="10.0" />
+				<dynamics damping="0.0" friction="0.0" />
+			</joint>
+			<gazebo>
+				<joint name="thigh_r_05_loop" type="revolute">
+					<parent>thigh_r_05</parent>
+					<child>leg_r_02</child>
+					<pose>-0.00765471 0 -0.02897777 0 0 0</pose>
+					<axis>
+						<xyz>0 1 0</xyz>
+						<limit>
+							<lower>-3.1</lower>
+							<upper>3.1</upper>
+						</limit>
+						<dynamics>
+							<spring_reference>0</spring_reference>
+							<spring_stiffness>0</spring_stiffness>
+						</dynamics>
+						<use_parent_model_frame>1</use_parent_model_frame>
+					</axis>
+					<physics>
+						<ode>
+							<implicit_spring_damper>1</implicit_spring_damper>
+							<cfm_damping>0</cfm_damping>
+							<limit>
+								<cfm>1e-7</cfm>
+								<erp>0.8</erp>
+							</limit>
+						</ode>
+					</physics>
+				</joint>
+			</gazebo>
+		</xacro:if>
 		<link name="thigh_r_05">
 			<visual>
@@ -129,5 +170,5 @@
 			<parent link="thigh_r_02" />
 			<child link="knee_r" />
-			<origin xyz="0 0 -0.1" rpy="0 0 0" />
+			<origin xyz="0 0 -0.1" rpy="0 0.785398163 0" />
 			<axis xyz="0 1 0" />
 			<limit effort="1000.0" lower="-3.1" upper="3.1" velocity="10.0" />
@@ -143,5 +184,100 @@
 			</visual>
 			<xacro:box_collision xyz="-0.01675 0 0" rpy="0 0 0" size="0.0475 0.0505 0.014" />
-			<xacro:box_inertial xyz="-0.01675 0 0" rpy="0 0 0" size="0.0475 0.0505 0.014" mass="0.0054" />
+			<xacro:box_inertial xyz="-0.01675 0 0" rpy="0 0 0" size="0.0475 0.0505 0.014" mass="0.007" />
+		</link>
+		<joint name="leg_r_01_joint" type="revolute">
+			<parent link="knee_r" />
+			<child link="leg_r_01" />
+			<origin xyz="0 0 0" rpy="0 0.785398163 0" />
+			<axis xyz="0 1 0" />
+			<limit effort="1000.0" lower="-3.1" upper="3.1" velocity="10.0" />
+			<dynamics damping="0.0" friction="0.0" />
+			<mimic joint="thigh_r_03_joint" multiplier="1" offset="0" />
+		</joint>
+		<link name="leg_r_01">
+			<visual>
+				<origin xyz="0 0 0" rpy="0 0 0" />
+				<geometry>
+					<mesh filename="package://kuroko_description/meshes/kuroko/obj/leg_r_01.obj" />
+				</geometry>
+			</visual>
+			<xacro:box_collision xyz="0 0 -0.05" rpy="0 0 0" size="0.014 0.0385 0.114" />
+			<xacro:box_inertial xyz="0 0 -0.05" rpy="0 0 0" size="0.014 0.0385 0.114" mass="0.013" />
+		</link>
+		<joint name="leg_r_02_joint" type="revolute">
+			<parent link="knee_r" />
+			<child link="leg_r_02" />
+			<origin xyz="-0.0335 0 0" rpy="0 0.785398163 0" />
+			<axis xyz="0 1 0" />
+			<limit effort="1000.0" lower="-3.1" upper="3.1" velocity="10.0" />
+			<dynamics damping="0.0" friction="0.0" />
+			<mimic joint="thigh_r_03_joint" multiplier="1" offset="0" />
+		</joint>
+		<link name="leg_r_02">
+			<visual>
+				<origin xyz="0 0 0" rpy="0 0 0" />
+				<geometry>
+					<mesh filename="package://kuroko_description/meshes/kuroko/obj/leg_r_02.obj" />
+				</geometry>
+			</visual>
+			<xacro:box_collision xyz="0 0 -0.05" rpy="0 0 0" size="0.014 0.0445 0.114" />
+			<xacro:box_inertial xyz="0 0 -0.05" rpy="0 0 0" size="0.014 0.0445 0.114" mass="0.016" />
+		</link>
+		<joint name="ankle_r_01_joint" type="revolute">
+			<parent link="leg_r_01" />
+			<child link="ankle_r_01" />
+			<origin xyz="0 0 -0.1" rpy="0 -0.785398163 0" />
+			<axis xyz="0 1 0" />
+			<limit effort="1000.0" lower="-3.1" upper="3.1" velocity="10.0" />
+			<dynamics damping="0.0" friction="0.0" />
+			<mimic joint="thigh_r_03_joint" multiplier="-1" offset="0" />
+		</joint>
+		<link name="ankle_r_01">
+			<visual>
+				<origin xyz="0 0 0" rpy="0 0 0" />
+				<geometry>
+					<mesh filename="package://kuroko_description/meshes/kuroko/obj/ankle_r_01.obj" />
+				</geometry>
+			</visual>
+			<xacro:box_collision xyz="-0.0285 0 -0.013" rpy="0 0 0" size="0.0855 0.0325 0.0465" />
+			<xacro:box_inertial xyz="-0.0285 0 -0.013" rpy="0 0 0" size="0.0855 0.0325 0.0465"
+				mass="0.104" />
+		</link>
+		<joint name="toe_r_01_joint" type="revolute">
+			<parent link="ankle_r_01" />
+			<child link="toe_r_01" />
+			<origin xyz="-0.015 0 -0.025" rpy="0 0 0" />
+			<axis xyz="1 0 0" />
+			<limit effort="1000.0" lower="-3.1" upper="3.1" velocity="10.0" />
+			<dynamics damping="0.0" friction="0.0" />
+		</joint>
+		<link name="toe_r_01">
+			<visual>
+				<origin xyz="0 0 0" rpy="0 0 0" />
+				<geometry>
+					<mesh filename="package://kuroko_description/meshes/kuroko/obj/toe_r_01.obj" />
+				</geometry>
+			</visual>
+			<xacro:box_collision xyz="0 -0.009375 -0.01175" rpy="0 0 0" size="0.0365 0.05375 0.043" />
+			<xacro:box_inertial xyz="0 -0.009375 -0.01175" rpy="0 0 0" size="0.0365 0.05375 0.043"
+				mass="0.136" />
+		</link>
+		<joint name="toe_r_02_joint" type="revolute">
+			<parent link="toe_r_01" />
+			<child link="toe_r_02" />
+			<origin xyz="0 0 -0.03825" rpy="0 0 0" />
+			<axis xyz="0 0 -1" />
+			<limit effort="1000.0" lower="-3.1" upper="3.1" velocity="10.0" />
+			<dynamics damping="0.0" friction="0.0" />
+		</joint>
+		<link name="toe_r_02">
+			<visual>
+				<origin xyz="0 0 0" rpy="0 0 0" />
+				<geometry>
+					<mesh filename="package://kuroko_description/meshes/kuroko/obj/toe_r_02.obj" />
+				</geometry>
+			</visual>
+			<xacro:box_collision xyz="0 0 -0.0025" rpy="0 0 0" size="0.12 0.075 0.005" />
+			<xacro:box_inertial xyz="0 0 -0.0025" rpy="0 0 0" size="0.12 0.075 0.005" mass="0.043" />
 		</link>
 	</xacro:macro>

File: kuroko_description/xacro/roboone_ring/large_ring.xacro (robot description, xacro)
@@ -1,26 +1,26 @@
 <?xml version="1.0"?>
-<robot name="large_ring"  xmlns:xacro="http://www.ros.org/wiki/xacro">
-	<xacro:include filename="./large_ring.gazebo"/>
+<robot name="large_ring" xmlns:xacro="http://www.ros.org/wiki/xacro">
+	<xacro:include filename="./large_ring.gazebo" />
 	<xacro:macro name="large_ring">
 		<link name="large_ring_link0">
 			<collision>
-				<origin xyz="0 0 -0.97" rpy="0 0 0"/>
+				<origin xyz="0 0 -0.97" rpy="0 0 0" />
 				<geometry>
-        			<mesh filename="package://ginko_description/meshes/roboone_ring/stl/large_ring.stl"/>
+					<mesh filename="package://kuroko_description/meshes/roboone_ring/stl/large_ring.stl" />
 				</geometry>
 			</collision>
 			<visual>
-				<origin xyz="0 0 0" rpy="0 0 0"/>
+				<origin xyz="0 0 0" rpy="0 0 0" />
 				<geometry>
-					<mesh filename="package://ginko_description/meshes/roboone_ring/obj/large_ring.obj"/>
+					<mesh filename="package://kuroko_description/meshes/roboone_ring/obj/large_ring.obj" />
 				</geometry>
 			</visual>
 			<inertial>
-				<mass value="484.78500000"/>
-				<origin xyz="0 0 0.01500000" rpy="0 0 0"/>
+				<mass value="484.78500000" />
+				<origin xyz="0 0 0.01500000" rpy="0 0 0" />
 				<inertia
 					ixx="439.45933388"
 					ixy="0.00000000" iyy="439.45933388"
-					ixz="0.00000000" iyz="0.00000000" izz="878.84595000"/>
+					ixz="0.00000000" iyz="0.00000000" izz="878.84595000" />
 			</inertial>
 		</link>

File: kuroko_description/xacro/roboone_ring/small_ring.xacro (robot description, xacro)
@@ -1,26 +1,26 @@
 <?xml version="1.0"?>
-<robot name="small_ring"  xmlns:xacro="http://www.ros.org/wiki/xacro">
-	<xacro:include filename="./small_ring.gazebo"/>
+<robot name="small_ring" xmlns:xacro="http://www.ros.org/wiki/xacro">
+	<xacro:include filename="./small_ring.gazebo" />
 	<xacro:macro name="small_ring">
 		<link name="small_ring_link0">
 			<collision>
-				<origin xyz="0 0 -0.97" rpy="0 0 0"/>
+				<origin xyz="0 0 -0.97" rpy="0 0 0" />
 				<geometry>
-        			<mesh filename="package://ginko_description/meshes/roboone_ring/stl/small_ring.stl"/>
+					<mesh filename="package://kuroko_description/meshes/roboone_ring/stl/small_ring.stl" />
 				</geometry>
 			</collision>
 			<visual>
-				<origin xyz="0 0 0" rpy="0 0 0"/>
+				<origin xyz="0 0 0" rpy="0 0 0" />
 				<geometry>
-					<mesh filename="package://ginko_description/meshes/roboone_ring/obj/small_ring.obj"/>
+					<mesh filename="package://kuroko_description/meshes/roboone_ring/obj/small_ring.obj" />
 				</geometry>
 			</visual>
 			<inertial>
-				<mass value="242.39250000"/>
-				<origin xyz="0 0 0.01500000" rpy="0 0 0"/>
+				<mass value="242.39250000" />
+				<origin xyz="0 0 0.01500000" rpy="0 0 0" />
 				<inertia
 					ixx="109.87392319"
 					ixy="0.00000000" iyy="109.87392319"
-					ixz="0.00000000" iyz="0.00000000" izz="219.71148750"/>
+					ixz="0.00000000" iyz="0.00000000" izz="219.71148750" />
 			</inertial>
 		</link>

File: kuroko_description/xacro/sensors/imu.xacro (robot description, xacro)
@@ -1,6 +1,6 @@
 <?xml version="1.0"?>
 <robot xmlns:xacro="http://www.ros.org/wiki/xacro">
-	<xacro:macro name="imu_xacro" params="model_mode">
-		<xacro:if value="${model_mode!='rviz'}">
+	<xacro:macro name="imu_xacro" params="gazebo">
+		<xacro:if value="$gazebo">
 			<link name="body_imu_attached_link">
 				<inertial>
@@ -40,5 +40,5 @@
 			</joint>
 		</xacro:if>
-		<xacro:if value="${model_mode=='rviz'}">
+		<xacro:unless value="gazebo">
 			<link name="body_imu_attached_link"/>
 			<joint name="body_imu_attached_joint" type="fixed">
@@ -53,5 +53,5 @@
 				<origin xyz="-0.09 0 -0.0379" rpy="0 0 0"/>
 			</joint>
-		</xacro:if>
+		</xacro:unless>
 		<gazebo>
 			<plugin name="imu_plugin" filename="libgazebo_ros_imu.so">
