Commit message: wip

File: kuroko_description/xacro/kuroko/kuroko.xacro (robot description, xacro)
@@ -5,4 +5,6 @@
   <!-- <xacro:arg name="gazebo_motor_model" default="kuroko"/> -->
   <xacro:arg name="gazebo_hw_interface" default="position" />
+	<xacro:include filename="$(find kuroko_description)/xacro/physics/box_physics.xacro" />
+	<xacro:include filename="$(find kuroko_description)/xacro/physics/gazebo_passive_joint.xacro" />
   <xacro:include filename="$(find kuroko_description)/xacro/kuroko/parts/body.xacro" />
   <xacro:include filename="$(find kuroko_description)/xacro/kuroko/transmission/body.gazebo" />

File: kuroko_description/xacro/kuroko/parts/body.xacro (robot description, xacro)
@@ -1,5 +1,4 @@
 <?xml version="1.0"?>
 <robot xmlns:xacro="http://www.ros.org/wiki/xacro">
-	<xacro:include filename="$(find kuroko_description)/xacro/physics/box_physics.xacro" />
 	<xacro:macro name="body_xacro">
 		<!-- chest -->

File: kuroko_description/xacro/kuroko/parts/leg_r.xacro (robot description, xacro)
@@ -87,4 +87,8 @@
 			<mimic joint="thigh_r_02_joint" multiplier="1" offset="0" />
 		</joint>
+		<xacro:if value="$(arg gazebo)">
+			<xacro:gazebo_poassive_joint name="thigh_r_04_loop" xyz="-0.0335 0 0"
+				parent="knee_r" child="thigh_r_04" />
+		</xacro:if>
 		<link name="thigh_r_04">
 			<visual>
@@ -127,33 +131,6 @@
 				<dynamics damping="0.0" friction="0.0" />
 			</joint>
-			<gazebo>
-				<joint name="thigh_r_05_loop" type="revolute">
-					<parent>thigh_r_05</parent>
-					<child>leg_r_02</child>
-					<pose>-0.00765471 0 -0.02897777 0 0 0</pose>
-					<axis>
-						<xyz>0 1 0</xyz>
-						<limit>
-							<lower>-3.1</lower>
-							<upper>3.1</upper>
-						</limit>
-						<dynamics>
-							<spring_reference>0</spring_reference>
-							<spring_stiffness>0</spring_stiffness>
-						</dynamics>
-						<use_parent_model_frame>1</use_parent_model_frame>
-					</axis>
-					<physics>
-						<ode>
-							<implicit_spring_damper>1</implicit_spring_damper>
-							<cfm_damping>0</cfm_damping>
-							<limit>
-								<cfm>1e-7</cfm>
-								<erp>0.8</erp>
-							</limit>
-						</ode>
-					</physics>
-				</joint>
-			</gazebo>
+			<xacro:gazebo_poassive_joint name="thigh_r_05_loop" xyz="-0.00765471 0 -0.02897777"
+				parent="leg_r_02" child="thigh_r_05" />
 		</xacro:if>
 		<link name="thigh_r_05">
@@ -214,4 +191,8 @@
 			<mimic joint="thigh_r_03_joint" multiplier="1" offset="0" />
 		</joint>
+		<xacro:if value="$(arg gazebo)">
+			<xacro:gazebo_poassive_joint name="leg_r_02_loop" xyz="-0.0335 0 0"
+				parent="ankle_r_01" child="leg_r_02" />
+		</xacro:if>
 		<link name="leg_r_02">
 			<visual>

File: kuroko_description/xacro/physics/gazebo_passive_joint.xacro (robot description, xacro)
@@ -1,15 +1,16 @@
 <?xml version="1.0"?>
 <robot xmlns:xacro="http://www.ros.org/wiki/xacro">
-	<xacro:macro name="gazebo_poassive_joint" params="parent child xyz:='0 0 0' rpy:='0 0 0' lower:=-3.1416 upper:=3.1416">
+	<xacro:macro name="gazebo_poassive_joint"
+		params="name:='joint' parent:='parent' child:='child' xyz:='0 0 0' rpy:='0 0 0' axis:='0 1 0' lower:=-3.1416 upper:=3.1416">
 		<gazebo>
-			<joint name="thigh_r_05_loop" type="revolute">
-				<parent>$(arg child)</parent>
-				<child>$(arg gazebo)</child>
-				<pose>$(arg xyz) $(arg rpy)</pose>
+			<joint name="${name}" type="revolute">
+				<parent>${child}</parent>
+				<child>${parent}</child>
+				<pose>${xyz} ${rpy}</pose>
 				<axis>
-					<xyz>0 1 0</xyz>
+					<xyz>${axis}</xyz>
 					<limit>
-						<lower>$(arg lower)</lower>
-						<upper>$(arg upper)</upper>
+						<lower>${lower}</lower>
+						<upper>${upper}</upper>
 					</limit>
 					<dynamics>

Commit message: Update leg_l

File: kuroko_description/xacro/kuroko/kuroko.xacro (robot description, xacro)
@@ -5,6 +5,6 @@
   <!-- <xacro:arg name="gazebo_motor_model" default="kuroko"/> -->
   <xacro:arg name="gazebo_hw_interface" default="position" />
-	<xacro:include filename="$(find kuroko_description)/xacro/physics/box_physics.xacro" />
-	<xacro:include filename="$(find kuroko_description)/xacro/physics/gazebo_passive_joint.xacro" />
+  <xacro:include filename="$(find kuroko_description)/xacro/physics/box_physics.xacro" />
+  <xacro:include filename="$(find kuroko_description)/xacro/physics/gazebo_passive_joint.xacro" />
   <xacro:include filename="$(find kuroko_description)/xacro/kuroko/parts/body.xacro" />
   <xacro:include filename="$(find kuroko_description)/xacro/kuroko/transmission/body.gazebo" />
@@ -15,7 +15,6 @@
   <xacro:include filename="$(find kuroko_description)/xacro/kuroko/parts/leg_r.xacro" />
   <xacro:include filename="$(find kuroko_description)/xacro/kuroko/transmission/leg_r.gazebo" />
-  <!--
-  <xacro:include filename="$(find kuroko_description)/xacro/kuroko/parts/leg_l.xacro"/>
-  <xacro:include filename="$(find kuroko_description)/xacro/kuroko/transmission/leg_l.gazebo"/>-->
+  <xacro:include filename="$(find kuroko_description)/xacro/kuroko/parts/leg_l.xacro" />
+  <xacro:include filename="$(find kuroko_description)/xacro/kuroko/transmission/leg_l.gazebo" />
   <!-- MACRO:Loading Gazebo Controllers for joints -->
   <xacro:macro name="gazebo_plugin_xacro" params="gazebo_motor_model">
@@ -55,7 +54,6 @@
     <xacro:leg_r_xacro gazebo="$(arg gazebo)" />
     <xacro:leg_r_gazebo gazebo_hw_interface="${gazebo_hw_interface}" />
-    <!--
-    <xacro:leg_l_xacro/>
-    <xacro:leg_l_gazebo gazebo_hw_interface="${gazebo_hw_interface}"/>-->
+    <xacro:leg_l_xacro gazebo="$(arg gazebo)" />
+    <xacro:leg_l_gazebo gazebo_hw_interface="${gazebo_hw_interface}" />
   </xacro:macro>
   <!-- Load Macros -->

File: kuroko_description/xacro/kuroko/parts/leg_l.xacro (robot description, xacro)
@@ -1,57 +1,57 @@
 <?xml version="1.0"?>
 <robot xmlns:xacro="http://www.ros.org/wiki/xacro">
-	<xacro:macro name="leg_r_xacro" params="gazebo:=false">
+	<xacro:macro name="leg_l_xacro" params="gazebo:=false">
 		<!-- Link conencts from body. Femoral first. -->
-		<joint name="crotch_r_joint" type="revolute">
+		<joint name="crotch_l_joint" type="revolute">
 			<parent link="waist" />
-			<child link="crotch_r" />
+			<child link="crotch_l" />
 			<origin xyz="0.00125 0 -0.08425" rpy="0 0 0" />
-			<axis xyz="1 0 0" />
+			<axis xyz="-1 0 0" />
 			<limit effort="1000.0" lower="-0.5550" upper="1.8640" velocity="10.0" />
 			<dynamics damping="0.0" friction="0.0" />
 		</joint>
-		<link name="crotch_r">
-			<visual>
-				<origin xyz="0 0 0" rpy="0 0 0" />
-				<geometry>
-					<mesh filename="package://kuroko_description/meshes/kuroko/obj/crotch_r.obj" />
-				</geometry>
-			</visual>
-			<xacro:box_collision xyz="0 -0.0065 -0.004125" rpy="0 0 0" size="0.092 0.041 0.03625" />
-			<xacro:box_inertial xyz="0 -0.0065 -0.004125" rpy="0 0 0" size="0.092 0.041 0.03625"
+		<link name="crotch_l">
+			<visual>
+				<origin xyz="0 0 0" rpy="0 0 0" />
+				<geometry>
+					<mesh filename="package://kuroko_description/meshes/kuroko/obj/crotch_l.obj" />
+				</geometry>
+			</visual>
+			<xacro:box_collision xyz="0 0.0065 -0.004125" rpy="0 0 0" size="0.092 0.041 0.03625" />
+			<xacro:box_inertial xyz="0 0.0065 -0.004125" rpy="0 0 0" size="0.092 0.041 0.03625"
 				mass="0.026" />
 		</link>
-		<joint name="thigh_r_01_joint" type="revolute">
-			<parent link="crotch_r" />
-			<child link="thigh_r_01" />
-			<origin xyz="0 -0.027 0" rpy="0 0 0" />
-			<axis xyz="0 -1 0" />
+		<joint name="thigh_l_01_joint" type="revolute">
+			<parent link="crotch_l" />
+			<child link="thigh_l_01" />
+			<origin xyz="0 0.027 0" rpy="0 0 0" />
+			<axis xyz="0 1 0" />
 			<limit effort="1000.0" lower="-3.1" upper="3.1" velocity="10.0" />
 			<dynamics damping="0.0" friction="0.0" />
 		</joint>
-		<link name="thigh_r_01">
-			<visual>
-				<origin xyz="0 0 0" rpy="0 0 0" />
-				<geometry>
-					<mesh filename="package://kuroko_description/meshes/kuroko/obj/thigh_r_01.obj" />
-				</geometry>
-			</visual>
-			<xacro:box_collision xyz="-0.00175 -0.049 -0.015" rpy="0 0 0" size="0.067 0.098 0.0585" />
-			<xacro:box_inertial xyz="-0.00175 -0.049 -0.015" rpy="0 0 0" size="0.067 0.098 0.0585"
+		<link name="thigh_l_01">
+			<visual>
+				<origin xyz="0 0 0" rpy="0 0 0" />
+				<geometry>
+					<mesh filename="package://kuroko_description/meshes/kuroko/obj/thigh_l_01.obj" />
+				</geometry>
+			</visual>
+			<xacro:box_collision xyz="-0.00175 0.049 -0.015" rpy="0 0 0" size="0.067 0.098 0.0585" />
+			<xacro:box_inertial xyz="-0.00175 0.049 -0.015" rpy="0 0 0" size="0.067 0.098 0.0585"
 				mass="0.478" />
 		</link>
-		<joint name="thigh_r_02_joint" type="revolute">
-			<parent link="thigh_r_01" />
-			<child link="thigh_r_02" />
-			<origin xyz="0.015 -0.02925 -0.0305" rpy="0 -0.785398163 0" />
-			<axis xyz="0 1 0" />
-			<limit effort="1000.0" lower="-0.4974" upper="1.8588" velocity="10.0" />
-			<dynamics damping="0.0" friction="0.0" />
-		</joint>
-		<link name="thigh_r_02">
-			<visual>
-				<origin xyz="0 0 0" rpy="0 0 0" />
-				<geometry>
-					<mesh filename="package://kuroko_description/meshes/kuroko/obj/thigh_r_02.obj" />
+		<joint name="thigh_l_02_joint" type="revolute">
+			<parent link="thigh_l_01" />
+			<child link="thigh_l_02" />
+			<origin xyz="0.015 0.02925 -0.0305" rpy="0 -0.785398163 0" />
+			<axis xyz="0 -1 0" />
+			<limit effort="1000.0" lower="-1.8588" upper="0.4974" velocity="10.0" />
+			<dynamics damping="0.0" friction="0.0" />
+		</joint>
+		<link name="thigh_l_02">
+			<visual>
+				<origin xyz="0 0 0" rpy="0 0 0" />
+				<geometry>
+					<mesh filename="package://kuroko_description/meshes/kuroko/obj/thigh_l_02.obj" />
 				</geometry>
 			</visual>
@@ -59,17 +59,17 @@
 			<xacro:box_inertial xyz="0 0 -0.05" rpy="0 0 0" size="0.014 0.0445 0.114" mass="0.012" />
 		</link>
-		<joint name="thigh_r_03_joint" type="revolute">
-			<parent link="thigh_r_01" />
-			<child link="thigh_r_03" />
-			<origin xyz="-0.0185 -0.02925 -0.0305" rpy="0 1.047197551 0" />
-			<axis xyz="0 1 0" />
-			<limit effort="1000.0" lower="-1.8588" upper="0.4974" velocity="10.0" />
-			<dynamics damping="0.0" friction="0.0" />
-		</joint>
-		<link name="thigh_r_03">
-			<visual>
-				<origin xyz="0 0 0" rpy="0 0 0" />
-				<geometry>
-					<mesh filename="package://kuroko_description/meshes/kuroko/obj/thigh_r_03.obj" />
+		<joint name="thigh_l_03_joint" type="revolute">
+			<parent link="thigh_l_01" />
+			<child link="thigh_l_03" />
+			<origin xyz="-0.0185 0.02925 -0.0305" rpy="0 1.047197551 0" />
+			<axis xyz="0 -1 0" />
+			<limit effort="1000.0" lower="-0.4974" upper="1.8588" velocity="10.0" />
+			<dynamics damping="0.0" friction="0.0" />
+		</joint>
+		<link name="thigh_l_03">
+			<visual>
+				<origin xyz="0 0 0" rpy="0 0 0" />
+				<geometry>
+					<mesh filename="package://kuroko_description/meshes/kuroko/obj/thigh_l_03.obj" />
 				</geometry>
 			</visual>
@@ -78,18 +78,18 @@
 				mass="0.008" />
 		</link>
-		<joint name="thigh_r_04_joint" type="revolute">
-			<parent link="thigh_r_01" />
-			<child link="thigh_r_04" />
-			<origin xyz="-0.0185 -0.02925 -0.0305" rpy="0 -0.785398163 0" />
-			<axis xyz="0 1 0" />
+		<joint name="thigh_l_04_joint" type="revolute">
+			<parent link="thigh_l_01" />
+			<child link="thigh_l_04" />
+			<origin xyz="-0.0185 0.02925 -0.0305" rpy="0 -0.785398163 0" />
+			<axis xyz="0 -1 0" />
 			<limit effort="1000.0" lower="-3.1" upper="3.1" velocity="10.0" />
 			<dynamics damping="0.0" friction="0.0" />
-			<mimic joint="thigh_r_02_joint" multiplier="1" offset="0" />
+			<mimic joint="thigh_l_02_joint" multiplier="1" offset="0" />
 		</joint>
 		<xacro:if value="$(arg gazebo)">
-			<xacro:gazebo_poassive_joint name="thigh_r_04_loop" xyz="-0.0335 0 0"
-				parent="knee_r" child="thigh_r_04" lower="-1.8588" upper="0.4974" />
+			<xacro:gazebo_poassive_joint name="thigh_l_04_loop" xyz="-0.0335 0 0"
+				parent="knee_l" child="thigh_l_04" axis="0 -1 0" />
 		</xacro:if>
-		<link name="thigh_r_04">
+		<link name="thigh_l_04">
 			<visual>
 				<origin xyz="0 0 0" rpy="0 0 0" />
@@ -102,37 +102,37 @@
 		</link>
 		<xacro:unless value="$(arg gazebo)">
-			<joint name="thigh_r_05_mimic1" type="revolute">
-				<parent link="thigh_r_03" />
-				<child link="thigh_r_05_mimic" />
+			<joint name="thigh_l_05_mimic1" type="revolute">
+				<parent link="thigh_l_03" />
+				<child link="thigh_l_05_mimic" />
 				<origin xyz="0 0 -0.03" rpy="0 -1.832597551 0" />
-				<axis xyz="0 1 0" />
+				<axis xyz="0 -1 0" />
 				<limit effort="1000.0" lower="-3.1" upper="3.1" velocity="10.0" />
 				<dynamics damping="0.0" friction="0.0" />
-				<mimic joint="thigh_r_03_joint" multiplier="-1" offset="0" />
+				<mimic joint="thigh_l_03_joint" multiplier="-1" offset="0" />
 			</joint>
-			<link name="thigh_r_05_mimic" />
-			<joint name="thigh_r_05_mimic2" type="revolute">
-				<parent link="thigh_r_05_mimic" />
-				<child link="thigh_r_05" />
-				<origin xyz="0 0 0" rpy="0 0 0" />
-				<axis xyz="0 1 0" />
+			<link name="thigh_l_05_mimic" />
+			<joint name="thigh_l_05_mimic2" type="revolute">
+				<parent link="thigh_l_05_mimic" />
+				<child link="thigh_l_05" />
+				<origin xyz="0 0 0" rpy="0 0 0" />
+				<axis xyz="0 -1 0" />
 				<limit effort="1000.0" lower="-3.1" upper="3.1" velocity="10.0" />
 				<dynamics damping="0.0" friction="0.0" />
-				<mimic joint="thigh_r_02_joint" multiplier="1" offset="0" />
+				<mimic joint="thigh_l_02_joint" multiplier="1" offset="0" />
 			</joint>
 		</xacro:unless>
 		<xacro:if value="$(arg gazebo)">
-			<joint name="thigh_r_05_joint" type="revolute">
-				<parent link="thigh_r_03" />
-				<child link="thigh_r_05" />
+			<joint name="thigh_l_05_joint" type="revolute">
+				<parent link="thigh_l_03" />
+				<child link="thigh_l_05" />
 				<origin xyz="0 0 -0.03" rpy="0 -1.832597551 0" />
-				<axis xyz="0 1 0" />
-				<limit effort="1000.0" lower="-0.7767" upper="1.5708" velocity="10.0" />
+				<axis xyz="0 -1 0" />
+				<limit effort="1000.0" lower="-1.5708" upper="0.7767" velocity="10.0" />
 				<dynamics damping="0.0" friction="0.0" />
 			</joint>
-			<xacro:gazebo_poassive_joint name="thigh_r_05_loop" xyz="-0.00765471 0 -0.02897777"
-				parent="leg_r_02" child="thigh_r_05"/>
+			<xacro:gazebo_poassive_joint name="thigh_l_05_loop" xyz="-0.00765471 0 -0.02897777"
+				parent="leg_l_02" child="thigh_l_05" axis="0 -1 0"/>
 		</xacro:if>
-		<link name="thigh_r_05">
+		<link name="thigh_l_05">
 			<visual>
 				<origin xyz="0 0 0" rpy="0 0 0" />
@@ -144,14 +144,14 @@
 			<xacro:box_inertial xyz="0 0 -0.05" rpy="0 0 0" size="0.014 0.0285 0.114" mass="0.011" />
 		</link>
-		<joint name="knee_r_joint" type="revolute">
-			<parent link="thigh_r_02" />
-			<child link="knee_r" />
+		<joint name="knee_l_joint" type="revolute">
+			<parent link="thigh_l_02" />
+			<child link="knee_l" />
 			<origin xyz="0 0 -0.1" rpy="0 0.785398163 0" />
-			<axis xyz="0 1 0" />
-			<limit effort="1000.0" lower="-1.8588" upper="0.4974" velocity="10.0" />
-			<dynamics damping="0.0" friction="0.0" />
-			<mimic joint="thigh_r_02_joint" multiplier="-1" offset="0" />
-		</joint>
-		<link name="knee_r">
+			<axis xyz="0 -1 0" />
+			<limit effort="1000.0" lower="-0.4974" upper="1.8588" velocity="10.0" />
+			<dynamics damping="0.0" friction="0.0" />
+			<mimic joint="thigh_l_02_joint" multiplier="-1" offset="0" />
+		</joint>
+		<link name="knee_l">
 			<visual>
 				<origin xyz="0 0 0" rpy="0 0 0" />
@@ -163,14 +163,14 @@
 			<xacro:box_inertial xyz="-0.01675 0 0" rpy="0 0 0" size="0.0475 0.0505 0.014" mass="0.007" />
 		</link>
-		<joint name="leg_r_01_joint" type="revolute">
-			<parent link="knee_r" />
-			<child link="leg_r_01" />
+		<joint name="leg_l_01_joint" type="revolute">
+			<parent link="knee_l" />
+			<child link="leg_l_01" />
 			<origin xyz="0 0 0" rpy="0 0.785398163 0" />
-			<axis xyz="0 1 0" />
-			<limit effort="1000.0" lower="-1.8588" upper="0.4974" velocity="10.0" />
-			<dynamics damping="0.0" friction="0.0" />
-			<mimic joint="thigh_r_03_joint" multiplier="1" offset="0" />
-		</joint>
-		<link name="leg_r_01">
+			<axis xyz="0 -1 0" />
+			<limit effort="1000.0" lower="-0.4974" upper="1.8588" velocity="10.0" />
+			<dynamics damping="0.0" friction="0.0" />
+			<mimic joint="thigh_l_03_joint" multiplier="1" offset="0" />
+		</joint>
+		<link name="leg_l_01">
 			<visual>
 				<origin xyz="0 0 0" rpy="0 0 0" />
@@ -182,18 +182,18 @@
 			<xacro:box_inertial xyz="0 0 -0.05" rpy="0 0 0" size="0.014 0.0385 0.114" mass="0.013" />
 		</link>
-		<joint name="leg_r_02_joint" type="revolute">
-			<parent link="knee_r" />
-			<child link="leg_r_02" />
+		<joint name="leg_l_02_joint" type="revolute">
+			<parent link="knee_l" />
+			<child link="leg_l_02" />
 			<origin xyz="-0.0335 0 0" rpy="0 0.785398163 0" />
-			<axis xyz="0 1 0" />
-			<limit effort="1000.0" lower="-1.8588" upper="0.4974" velocity="10.0" />
-			<dynamics damping="0.0" friction="0.0" />
-			<mimic joint="thigh_r_03_joint" multiplier="1" offset="0" />
+			<axis xyz="0 -1 0" />
+			<limit effort="1000.0" lower="-0.4974" upper="1.8588" velocity="10.0" />
+			<dynamics damping="0.0" friction="0.0" />
+			<mimic joint="thigh_l_03_joint" multiplier="1" offset="0" />
 		</joint>
 		<xacro:if value="$(arg gazebo)">
-			<xacro:gazebo_poassive_joint name="leg_r_02_loop" xyz="-0.0335 0 0"
-				parent="ankle_r_01" child="leg_r_02" />
+			<xacro:gazebo_poassive_joint name="leg_l_02_loop" xyz="-0.0335 0 0"
+				parent="ankle_l_01" child="leg_l_02" axis="0 -1 0"/>
 		</xacro:if>
-		<link name="leg_r_02">
+		<link name="leg_l_02">
 			<visual>
 				<origin xyz="0 0 0" rpy="0 0 0" />
@@ -205,14 +205,14 @@
 			<xacro:box_inertial xyz="0 0 -0.05" rpy="0 0 0" size="0.014 0.0445 0.114" mass="0.016" />
 		</link>
-		<joint name="ankle_r_01_joint" type="revolute">
-			<parent link="leg_r_01" />
-			<child link="ankle_r_01" />
+		<joint name="ankle_l_01_joint" type="revolute">
+			<parent link="leg_l_01" />
+			<child link="ankle_l_01" />
 			<origin xyz="0 0 -0.1" rpy="0 -0.785398163 0" />
-			<axis xyz="0 1 0" />
-			<limit effort="1000.0" lower="-0.4974" upper="1.8588" velocity="10.0" />
-			<dynamics damping="0.0" friction="0.0" />
-			<mimic joint="thigh_r_03_joint" multiplier="-1" offset="0" />
-		</joint>
-		<link name="ankle_r_01">
+			<axis xyz="0 -1 0" />
+			<limit effort="1000.0" lower="-1.8588" upper="0.4974" velocity="10.0" />
+			<dynamics damping="0.0" friction="0.0" />
+			<mimic joint="thigh_l_03_joint" multiplier="-1" offset="0" />
+		</joint>
+		<link name="ankle_l_01">
 			<visual>
 				<origin xyz="0 0 0" rpy="0 0 0" />
@@ -225,26 +225,26 @@
 				mass="0.104" />
 		</link>
-		<joint name="toe_r_01_joint" type="revolute">
-			<parent link="ankle_r_01" />
-			<child link="toe_r_01" />
+		<joint name="toe_l_01_joint" type="revolute">
+			<parent link="ankle_l_01" />
+			<child link="toe_l_01" />
 			<origin xyz="-0.015 0 -0.025" rpy="0 0 0" />
 			<axis xyz="1 0 0" />
-			<limit effort="1000.0" lower="-0.3704" upper="1.5708" velocity="10.0" />
-			<dynamics damping="0.0" friction="0.0" />
-		</joint>
-		<link name="toe_r_01">
-			<visual>
-				<origin xyz="0 0 0" rpy="0 0 0" />
-				<geometry>
-					<mesh filename="package://kuroko_description/meshes/kuroko/obj/toe_r_01.obj" />
-				</geometry>
-			</visual>
-			<xacro:box_collision xyz="0 -0.009375 -0.01175" rpy="0 0 0" size="0.0365 0.05375 0.043" />
-			<xacro:box_inertial xyz="0 -0.009375 -0.01175" rpy="0 0 0" size="0.0365 0.05375 0.043"
+			<limit effort="1000.0" lower="-1.5708" upper="0.3704" velocity="10.0" />
+			<dynamics damping="0.0" friction="0.0" />
+		</joint>
+		<link name="toe_l_01">
+			<visual>
+				<origin xyz="0 0 0" rpy="0 0 0" />
+				<geometry>
+					<mesh filename="package://kuroko_description/meshes/kuroko/obj/toe_l_01.obj" />
+				</geometry>
+			</visual>
+			<xacro:box_collision xyz="0 0.009375 -0.01175" rpy="0 0 0" size="0.0365 0.05375 0.043" />
+			<xacro:box_inertial xyz="0 0.009375 -0.01175" rpy="0 0 0" size="0.0365 0.05375 0.043"
 				mass="0.136" />
 		</link>
-		<joint name="toe_r_02_joint" type="revolute">
-			<parent link="toe_r_01" />
-			<child link="toe_r_02" />
+		<joint name="toe_l_02_joint" type="revolute">
+			<parent link="toe_l_01" />
+			<child link="toe_l_02" />
 			<origin xyz="0 0 -0.03825" rpy="0 0 0" />
 			<axis xyz="0 0 -1" />
@@ -252,5 +252,5 @@
 			<dynamics damping="0.0" friction="0.0" />
 		</joint>
-		<link name="toe_r_02">
+		<link name="toe_l_02">
 			<visual>
 				<origin xyz="0 0 0" rpy="0 0 0" />

File: kuroko_description/xacro/kuroko/parts/leg_r.xacro (robot description, xacro)
@@ -89,5 +89,5 @@
 		<xacro:if value="$(arg gazebo)">
 			<xacro:gazebo_poassive_joint name="thigh_r_04_loop" xyz="-0.0335 0 0"
-				parent="knee_r" child="thigh_r_04" lower="-1.8588" upper="0.4974" />
+				parent="knee_r" child="thigh_r_04" />
 		</xacro:if>
 		<link name="thigh_r_04">

Commit message: Attach sensors

File: kuroko_description/xacro/kuroko/kuroko.xacro (robot description, xacro)
@@ -17,4 +17,6 @@
   <xacro:include filename="$(find kuroko_description)/xacro/kuroko/parts/leg_l.xacro" />
   <xacro:include filename="$(find kuroko_description)/xacro/kuroko/transmission/leg_l.gazebo" />
+  <xacro:include filename="$(find kuroko_description)/xacro/sensors/imu/n100mini.xacro" />
+  <xacro:include filename="$(find kuroko_description)/xacro/sensors/depth/maixsense_a075v.xacro" />
   <!-- MACRO:Loading Gazebo Controllers for joints -->
   <xacro:macro name="gazebo_plugin_xacro" params="gazebo_motor_model">
@@ -56,4 +58,10 @@
     <xacro:leg_l_xacro gazebo="$(arg gazebo)" />
     <xacro:leg_l_gazebo gazebo_hw_interface="${gazebo_hw_interface}" />
+    <xacro:n100mini_imu parent="chest" name="imu">
+      <origin xyz="-0.05 0 0.04425" rpy="0 0 0"/>
+    </xacro:n100mini_imu>
+    <xacro:maixsense_rgbd parent="chest" name="rgbd">
+      <origin xyz="0.04425 0 0.017" rpy="0 0 0"/>
+    </xacro:maixsense_rgbd>
   </xacro:macro>
   <!-- Load Macros -->
@@ -61,8 +69,3 @@
     gazebo_hw_interface="$(arg gazebo_hw_interface)" />
   <xacro:gazebo_plugin_xacro gazebo_motor_model="$(arg gazebo_motor_model)" />
-  <!-- <xacro:imu_xacro model_mode="$(arg model_mode)"/> -->
-  <!-- <xacro:urg_xacro firame_id="arm_r_urg_link" topic_name="/sensor/urg/right/scan_raw"
-  sensor_name="urg_right"/> -->
-  <!-- <xacro:urg_xacro firame_id="arm_l_urg_link" topic_name="/sensor/urg/left/scan_raw"
-  sensor_name="urg_left"/> -->
 </robot>
