Commit message: Fix xacro

File: kuroko_description/xacro/kuroko/kuroko.xacro (robot description, xacro)
@@ -59,9 +59,6 @@
     <xacro:leg_l_gazebo gazebo_hw_interface="${gazebo_hw_interface}" />
     <xacro:n100mini_imu parent="chest" name="imu">
-      <origin xyz="-0.05 0 0.04425" rpy="0 0 0"/>
+      <origin xyz="0 0 0.008" rpy="0 0 0"/>
     </xacro:n100mini_imu>
-    <xacro:maixsense_rgbd parent="chest" name="rgbd">
-      <origin xyz="0.04425 0 0.017" rpy="0 0 0"/>
-    </xacro:maixsense_rgbd>
   </xacro:macro>
   <!-- Load Macros -->

File: kuroko_description/xacro/kuroko/parts/arm_l.xacro (robot description, xacro)
@@ -6,5 +6,5 @@
       <parent link="chest"/>
       <child link="shoulder_l_pitch"/>
-      <origin xyz="0 0.108 0.01275" rpy="0 0 0"/>
+      <origin xyz="0 0.1275 0.01275" rpy="0 0 0"/>
       <axis xyz="0 1 0"/>
       <limit effort="1000.0" lower="-3.1" upper="3.1" velocity="10.0"/>
@@ -18,11 +18,11 @@
         </geometry>
       </visual>
-      <xacro:box_collision xyz="0 0.0205 0" rpy="0 0 0" size="0.042 0.041 0.04"/>
-      <xacro:box_inertial xyz="0 0.0205 0" rpy="0 0 0" size="0.042 0.041 0.04" mass="0.022"/>
+      <xacro:box_collision xyz="0 0.024 0" rpy="0 0 0" size="0.042 0.048 0.04"/>
+      <xacro:box_inertial xyz="0 0.024 0" rpy="0 0 0" size="0.042 0.048 0.04" mass="0.022"/>
     </link>
     <joint name="shoulder_l_roll_joint" type="revolute">
       <parent link="shoulder_l_pitch"/>
       <child link="shoulder_l_roll"/>
-      <origin xyz="0 0.028 0" rpy="0 0 0"/>
+      <origin xyz="0 0.038 0" rpy="0 0 0"/>
       <axis xyz="-1 0 0"/>
       <limit effort="1000.0" lower="-2.0071" upper="1.0472" velocity="10.0"/>
@@ -36,11 +36,11 @@
         </geometry>
       </visual>
-      <xacro:box_collision xyz="0 0.0385 -0.02575" rpy="0 0 0" size="0.0285 0.1045 0.08"/>
-      <xacro:box_inertial xyz="0 0.0385 -0.02575" rpy="0 0 0" size="0.0285 0.1045 0.08" mass="0.342"/>
+      <xacro:box_collision xyz="0 0.016 -0.02575" rpy="0 0 0" size="0.0285 0.082 0.08"/>
+      <xacro:box_inertial xyz="0 0.016 -0.02575" rpy="0 0 0" size="0.0285 0.082 0.08" mass="0.342"/>
     </link>
     <joint name="elbow_l_front_joint" type="revolute">
       <parent link="shoulder_l_roll"/>
       <child link="elbow_l_front"/>
-      <origin xyz="0 0.0265 -0.0545" rpy="0 0 0"/>
+      <origin xyz="0 -0.008 -0.052" rpy="0 0 0"/>
       <axis xyz="0 -1 0"/>
       <limit effort="1000.0" lower="-2.6180" upper="2.6180" velocity="10.0"/>
@@ -61,5 +61,5 @@
       <parent link="shoulder_l_roll"/>
       <child link="elbow_l_rear"/>
-      <origin xyz="0 0.0265 -0.0545" rpy="0 0 0"/>
+      <origin xyz="0 -0.008 -0.052" rpy="0 0 0"/>
       <axis xyz="0 1 0"/>
       <limit effort="1000.0" lower="-2.6180" upper="2.6180" velocity="10.0"/>

File: kuroko_description/xacro/kuroko/parts/arm_r.xacro (robot description, xacro)
@@ -6,5 +6,5 @@
       <parent link="chest"/>
       <child link="shoulder_r_pitch"/>
-      <origin xyz="0 -0.108 0.01275" rpy="0 0 0"/>
+      <origin xyz="0 -0.1275 0.01275" rpy="0 0 0"/>
       <axis xyz="0 -1 0"/>
       <limit effort="1000.0" lower="-3.1" upper="3.1" velocity="10.0"/>
@@ -18,11 +18,11 @@
         </geometry>
       </visual>
-      <xacro:box_collision xyz="0 -0.0205 0" rpy="0 0 0" size="0.042 0.041 0.04"/>
-      <xacro:box_inertial xyz="0 -0.0205 0" rpy="0 0 0" size="0.042 0.041 0.04" mass="0.022"/>
+      <xacro:box_collision xyz="0 -0.024 0" rpy="0 0 0" size="0.042 0.048 0.04"/>
+      <xacro:box_inertial xyz="0 -0.024 0" rpy="0 0 0" size="0.042 0.048 0.04" mass="0.022"/>
     </link>
     <joint name="shoulder_r_roll_joint" type="revolute">
       <parent link="shoulder_r_pitch"/>
       <child link="shoulder_r_roll"/>
-      <origin xyz="0 -0.028 0" rpy="0 0 0"/>
+      <origin xyz="0 -0.038 0" rpy="0 0 0"/>
       <axis xyz="-1 0 0"/>
       <limit effort="1000.0" lower="-1.0472" upper="2.0071" velocity="10.0"/>
@@ -36,6 +36,6 @@
         </geometry>
       </visual>
-      <xacro:box_collision xyz="0 -0.0385 -0.02575" rpy="0 0 0" size="0.0285 0.1045 0.08"/>
-      <xacro:box_inertial xyz="0 -0.0385 -0.02575" rpy="0 0 0" size="0.0285 0.1045 0.08"
+      <xacro:box_collision xyz="0 -0.016 -0.02575" rpy="0 0 0" size="0.0285 0.082 0.08"/>
+      <xacro:box_inertial xyz="0 -0.016 -0.02575" rpy="0 0 0" size="0.0285 0.082 0.08"
         mass="0.342"/>
     </link>
@@ -43,5 +43,5 @@
       <parent link="shoulder_r_roll"/>
       <child link="elbow_r_front"/>
-      <origin xyz="0 -0.0265 -0.0545" rpy="0 0 0"/>
+      <origin xyz="0 0.008 -0.052" rpy="0 0 0"/>
       <axis xyz="0 1 0"/>
       <limit effort="1000.0" lower="-2.6180" upper="2.6180" velocity="10.0"/>
@@ -62,5 +62,5 @@
       <parent link="shoulder_r_roll"/>
       <child link="elbow_r_rear"/>
-      <origin xyz="0 -0.0265 -0.0545" rpy="0 0 0"/>
+      <origin xyz="0 0.008 -0.052" rpy="0 0 0"/>
       <axis xyz="0 -1 0"/>
       <limit effort="1000.0" lower="-2.6180" upper="2.6180" velocity="10.0"/>

File: kuroko_description/xacro/kuroko/parts/body.xacro (robot description, xacro)
@@ -10,6 +10,6 @@
         </geometry>
       </visual>
-      <xacro:box_collision xyz="0 0 0.057" rpy="0 0 0" size="0.1 0.204 0.114" />
-      <xacro:box_inertial xyz="0 0 0.057" rpy="0 0 0" size="0.1 0.204 0.114" mass="0.991" />
+      <xacro:box_collision xyz="0 0 0.057" rpy="0 0 0" size="0.1 0.242 0.114" />
+      <xacro:box_inertial xyz="0 0 0.057" rpy="0 0 0" size="0.1 0.242 0.114" mass="0.991" />
     </link>
     <!-- Joint1 -->

File: kuroko_description/xacro/kuroko/parts/leg_l.xacro (robot description, xacro)
@@ -6,5 +6,5 @@
       <parent link="waist"/>
       <child link="hip_l_roll"/>
-      <origin xyz="0.00125 0 -0.08425" rpy="0 0 0"/>
+      <origin xyz="0 0 -0.08425" rpy="0 0 0"/>
       <axis xyz="-1 0 0"/>
       <limit effort="1000.0" lower="-0.5550" upper="1.8640" velocity="10.0"/>
@@ -18,6 +18,6 @@
         </geometry>
       </visual>
-      <xacro:box_collision xyz="0 0.0065 -0.004125" rpy="0 0 0" size="0.092 0.041 0.03625"/>
-      <xacro:box_inertial xyz="0 0.0065 -0.004125" rpy="0 0 0" size="0.092 0.041 0.03625"
+      <xacro:box_collision xyz="0.00125 0.0065 -0.004125" rpy="0 0 0" size="0.092 0.041 0.03625"/>
+      <xacro:box_inertial xyz="0.00125 0.0065 -0.004125" rpy="0 0 0" size="0.092 0.041 0.03625"
         mass="0.026"/>
     </link>
@@ -228,5 +228,5 @@
       <parent link="ankle_l_pitch_passive"/>
       <child link="ankle_l_roll"/>
-      <origin xyz="-0.015 0 -0.025" rpy="0 0 0"/>
+      <origin xyz="-0.015 0 -0.027" rpy="0 0 0"/>
       <axis xyz="1 0 0"/>
       <limit effort="1000.0" lower="-1.5708" upper="0.3704" velocity="10.0"/>
@@ -259,6 +259,6 @@
         </geometry>
       </visual>
-      <xacro:box_collision xyz="0 0 -0.0025" rpy="0 0 0" size="0.12 0.075 0.005"/>
-      <xacro:box_inertial xyz="0 0 -0.0025" rpy="0 0 0" size="0.12 0.075 0.005" mass="0.043"/>
+      <xacro:box_collision xyz="0 0 -0.004" rpy="0 0 0" size="0.12 0.075 0.008"/>
+      <xacro:box_inertial xyz="0 0 -0.004" rpy="0 0 0" size="0.12 0.075 0.008" mass="0.043"/>
     </link>
   </xacro:macro>

File: kuroko_description/xacro/kuroko/parts/leg_r.xacro (robot description, xacro)
@@ -6,5 +6,5 @@
       <parent link="waist"/>
       <child link="hip_r_roll"/>
-      <origin xyz="0.00125 0 -0.08425" rpy="0 0 0"/>
+      <origin xyz="0 0 -0.08425" rpy="0 0 0"/>
       <axis xyz="1 0 0"/>
       <limit effort="1000.0" lower="-0.5550" upper="1.8640" velocity="10.0"/>
@@ -18,6 +18,6 @@
         </geometry>
       </visual>
-      <xacro:box_collision xyz="0 -0.0065 -0.004125" rpy="0 0 0" size="0.092 0.041 0.03625"/>
-      <xacro:box_inertial xyz="0 -0.0065 -0.004125" rpy="0 0 0" size="0.092 0.041 0.03625"
+      <xacro:box_collision xyz="0.00125 -0.0065 -0.004125" rpy="0 0 0" size="0.092 0.041 0.03625"/>
+      <xacro:box_inertial xyz="0.00125 -0.0065 -0.004125" rpy="0 0 0" size="0.092 0.041 0.03625"
         mass="0.026"/>
     </link>
@@ -228,5 +228,5 @@
       <parent link="ankle_r_pitch_passive"/>
       <child link="ankle_r_roll"/>
-      <origin xyz="-0.015 0 -0.025" rpy="0 0 0"/>
+      <origin xyz="-0.015 0 -0.027" rpy="0 0 0"/>
       <axis xyz="1 0 0"/>
       <limit effort="1000.0" lower="-0.3704" upper="1.5708" velocity="10.0"/>
@@ -259,6 +259,6 @@
         </geometry>
       </visual>
-      <xacro:box_collision xyz="0 0 -0.0025" rpy="0 0 0" size="0.12 0.075 0.005"/>
-      <xacro:box_inertial xyz="0 0 -0.0025" rpy="0 0 0" size="0.12 0.075 0.005" mass="0.043"/>
+      <xacro:box_collision xyz="0 0 -0.004" rpy="0 0 0" size="0.12 0.075 0.008"/>
+      <xacro:box_inertial xyz="0 0 -0.004" rpy="0 0 0" size="0.12 0.075 0.008" mass="0.043"/>
     </link>
   </xacro:macro>

Commit message: Edit joint names

File: kuroko_description/xacro/kuroko/kuroko.xacro (robot description, xacro)
@@ -1,22 +1,22 @@
 <?xml version="1.0"?>
 <robot name="kuroko" xmlns:xacro="http://www.ros.org/wiki/xacro">
-  <xacro:arg name="gazebo" default="false" />
-  <xacro:arg name="gazebo_motor_model" default="dc" />
+  <xacro:arg name="gazebo" default="false"/>
+  <xacro:arg name="gazebo_motor_model" default="dc"/>
   <!-- <xacro:arg name="gazebo_motor_model" default="kuroko"/> -->
-  <xacro:arg name="gazebo_hw_interface" default="position" />
-  <xacro:include filename="$(find kuroko_description)/xacro/physics/box_physics.xacro" />
-  <xacro:include filename="$(find kuroko_description)/xacro/physics/gazebo_passive_joint.xacro" />
-  <xacro:include filename="$(find kuroko_description)/xacro/kuroko/parts/body.xacro" />
-  <xacro:include filename="$(find kuroko_description)/xacro/kuroko/transmission/body.gazebo" />
-  <xacro:include filename="$(find kuroko_description)/xacro/kuroko/parts/arm_r.xacro" />
-  <xacro:include filename="$(find kuroko_description)/xacro/kuroko/transmission/arm_r.gazebo" />
-  <xacro:include filename="$(find kuroko_description)/xacro/kuroko/parts/arm_l.xacro" />
-  <xacro:include filename="$(find kuroko_description)/xacro/kuroko/transmission/arm_l.gazebo" />
-  <xacro:include filename="$(find kuroko_description)/xacro/kuroko/parts/leg_r.xacro" />
-  <xacro:include filename="$(find kuroko_description)/xacro/kuroko/transmission/leg_r.gazebo" />
-  <xacro:include filename="$(find kuroko_description)/xacro/kuroko/parts/leg_l.xacro" />
-  <xacro:include filename="$(find kuroko_description)/xacro/kuroko/transmission/leg_l.gazebo" />
-  <xacro:include filename="$(find kuroko_description)/xacro/sensors/imu/n100mini.xacro" />
-  <xacro:include filename="$(find kuroko_description)/xacro/sensors/depth/maixsense_a075v.xacro" />
+  <xacro:arg name="gazebo_hw_interface" default="position"/>
+  <xacro:include filename="$(find kuroko_description)/xacro/physics/box_physics.xacro"/>
+  <xacro:include filename="$(find kuroko_description)/xacro/physics/gazebo_passive_joint.xacro"/>
+  <xacro:include filename="$(find kuroko_description)/xacro/kuroko/parts/body.xacro"/>
+  <xacro:include filename="$(find kuroko_description)/xacro/kuroko/transmission/body.gazebo"/>
+  <xacro:include filename="$(find kuroko_description)/xacro/kuroko/parts/arm_r.xacro"/>
+  <xacro:include filename="$(find kuroko_description)/xacro/kuroko/transmission/arm_r.gazebo"/>
+  <xacro:include filename="$(find kuroko_description)/xacro/kuroko/parts/arm_l.xacro"/>
+  <xacro:include filename="$(find kuroko_description)/xacro/kuroko/transmission/arm_l.gazebo"/>
+  <xacro:include filename="$(find kuroko_description)/xacro/kuroko/parts/leg_r.xacro"/>
+  <xacro:include filename="$(find kuroko_description)/xacro/kuroko/transmission/leg_r.gazebo"/>
+  <xacro:include filename="$(find kuroko_description)/xacro/kuroko/parts/leg_l.xacro"/>
+  <xacro:include filename="$(find kuroko_description)/xacro/kuroko/transmission/leg_l.gazebo"/>
+  <xacro:include filename="$(find kuroko_description)/xacro/sensors/imu/n100mini.xacro"/>
+  <xacro:include filename="$(find kuroko_description)/xacro/sensors/depth/maixsense_a075v.xacro"/>
   <!-- MACRO:Loading Gazebo Controllers for joints -->
   <xacro:macro name="gazebo_plugin_xacro" params="gazebo_motor_model">
@@ -42,21 +42,21 @@
   <!-- MACRO:Setting up a Robot Model -->
   <xacro:macro name="kuroko_xacro" params="gazebo gazebo_hw_interface">
-    <link name="root_link" />
+    <link name="root_link"/>
     <joint name="root_joint" type="fixed">
-      <parent link="root_link" />
-      <child link="chest" />
-      <origin xyz="0 0 0" rpy="0 0 0" />
+      <parent link="root_link"/>
+      <child link="chest_link"/>
+      <origin xyz="0 0 0" rpy="0 0 0"/>
     </joint>
-    <xacro:body_xacro />
-    <xacro:body_gazebo gazebo_hw_interface="${gazebo_hw_interface}" />
-    <xacro:arm_r_xacro />
-    <xacro:arm_r_gazebo gazebo_hw_interface="${gazebo_hw_interface}" />
-    <xacro:arm_l_xacro />
-    <xacro:arm_l_gazebo gazebo_hw_interface="${gazebo_hw_interface}" />
-    <xacro:leg_r_xacro gazebo="$(arg gazebo)" />
-    <xacro:leg_r_gazebo gazebo_hw_interface="${gazebo_hw_interface}" />
-    <xacro:leg_l_xacro gazebo="$(arg gazebo)" />
-    <xacro:leg_l_gazebo gazebo_hw_interface="${gazebo_hw_interface}" />
-    <xacro:n100mini_imu parent="chest" name="imu">
+    <xacro:body_xacro/>
+    <xacro:body_gazebo gazebo_hw_interface="${gazebo_hw_interface}"/>
+    <xacro:arm_r_xacro/>
+    <xacro:arm_r_gazebo gazebo_hw_interface="${gazebo_hw_interface}"/>
+    <xacro:arm_l_xacro/>
+    <xacro:arm_l_gazebo gazebo_hw_interface="${gazebo_hw_interface}"/>
+    <xacro:leg_r_xacro gazebo="$(arg gazebo)"/>
+    <xacro:leg_r_gazebo gazebo_hw_interface="${gazebo_hw_interface}"/>
+    <xacro:leg_l_xacro gazebo="$(arg gazebo)"/>
+    <xacro:leg_l_gazebo gazebo_hw_interface="${gazebo_hw_interface}"/>
+    <xacro:n100mini_imu parent="chest_link" name="imu">
       <origin xyz="0 0 0.008" rpy="0 0 0"/>
     </xacro:n100mini_imu>
@@ -64,5 +64,5 @@
   <!-- Load Macros -->
   <xacro:kuroko_xacro gazebo="$(arg gazebo)"
-    gazebo_hw_interface="$(arg gazebo_hw_interface)" />
-  <xacro:gazebo_plugin_xacro gazebo_motor_model="$(arg gazebo_motor_model)" />
+    gazebo_hw_interface="$(arg gazebo_hw_interface)"/>
+  <xacro:gazebo_plugin_xacro gazebo_motor_model="$(arg gazebo_motor_model)"/>
 </robot>

File: kuroko_description/xacro/kuroko/parts/arm_l.xacro (robot description, xacro)
@@ -3,7 +3,7 @@
   <xacro:macro name="arm_l_xacro">
     <!-- Link conencts from body. Shoulder first. -->
-    <joint name="shoulder_l_pitch_joint" type="revolute">
-      <parent link="chest"/>
-      <child link="shoulder_l_pitch"/>
+    <joint name="shoulder_l_pitch" type="revolute">
+      <parent link="chest_link"/>
+      <child link="shoulder_l_pitch_link"/>
       <origin xyz="0 0.1275 0.01275" rpy="0 0 0"/>
       <axis xyz="0 1 0"/>
@@ -11,5 +11,5 @@
       <dynamics damping="0.0" friction="0.0"/>
     </joint>
-    <link name="shoulder_l_pitch">
+    <link name="shoulder_l_pitch_link">
       <visual>
         <origin xyz="0 0 0" rpy="0 0 0"/>
@@ -21,7 +21,7 @@
       <xacro:box_inertial xyz="0 0.024 0" rpy="0 0 0" size="0.042 0.048 0.04" mass="0.022"/>
     </link>
-    <joint name="shoulder_l_roll_joint" type="revolute">
-      <parent link="shoulder_l_pitch"/>
-      <child link="shoulder_l_roll"/>
+    <joint name="shoulder_l_roll" type="revolute">
+      <parent link="shoulder_l_pitch_link"/>
+      <child link="shoulder_l_roll_link"/>
       <origin xyz="0 0.038 0" rpy="0 0 0"/>
       <axis xyz="-1 0 0"/>
@@ -29,5 +29,5 @@
       <dynamics damping="0.0" friction="0.0"/>
     </joint>
-    <link name="shoulder_l_roll">
+    <link name="shoulder_l_roll_link">
       <visual>
         <origin xyz="0 0 0" rpy="0 0 0"/>
@@ -39,7 +39,7 @@
       <xacro:box_inertial xyz="0 0.016 -0.02575" rpy="0 0 0" size="0.0285 0.082 0.08" mass="0.342"/>
     </link>
-    <joint name="elbow_l_front_joint" type="revolute">
-      <parent link="shoulder_l_roll"/>
-      <child link="elbow_l_front"/>
+    <joint name="elbow_l_front" type="revolute">
+      <parent link="shoulder_l_roll_link"/>
+      <child link="elbow_l_front_link"/>
       <origin xyz="0 -0.008 -0.052" rpy="0 0 0"/>
       <axis xyz="0 -1 0"/>
@@ -47,5 +47,5 @@
       <dynamics damping="0.0" friction="0.0"/>
     </joint>
-    <link name="elbow_l_front">
+    <link name="elbow_l_front_link">
       <visual>
         <origin xyz="0 0 0" rpy="0 0 0"/>
@@ -58,7 +58,7 @@
       <xacro:box_inertial xyz="0.0043 0 -0.104" rpy="0 0 0" size="0.044 0.058 0.208" mass="0.032"/>
     </link>
-    <joint name="elbow_l_rear_joint" type="revolute">
-      <parent link="shoulder_l_roll"/>
-      <child link="elbow_l_rear"/>
+    <joint name="elbow_l_rear" type="revolute">
+      <parent link="shoulder_l_roll_link"/>
+      <child link="elbow_l_rear_link"/>
       <origin xyz="0 -0.008 -0.052" rpy="0 0 0"/>
       <axis xyz="0 1 0"/>
@@ -66,5 +66,5 @@
       <dynamics damping="0.0" friction="0.0"/>
     </joint>
-    <link name="elbow_l_rear">
+    <link name="elbow_l_rear_link">
       <visual>
         <origin xyz="0 0 0" rpy="0 0 0"/>

File: kuroko_description/xacro/kuroko/parts/arm_r.xacro (robot description, xacro)
@@ -3,7 +3,7 @@
   <xacro:macro name="arm_r_xacro">
     <!-- Link conencts from body. Shoulder first. -->
-    <joint name="shoulder_r_pitch_joint" type="revolute">
-      <parent link="chest"/>
-      <child link="shoulder_r_pitch"/>
+    <joint name="shoulder_r_pitch" type="revolute">
+      <parent link="chest_link"/>
+      <child link="shoulder_r_pitch_link"/>
       <origin xyz="0 -0.1275 0.01275" rpy="0 0 0"/>
       <axis xyz="0 -1 0"/>
@@ -11,5 +11,5 @@
       <dynamics damping="0.0" friction="0.0"/>
     </joint>
-    <link name="shoulder_r_pitch">
+    <link name="shoulder_r_pitch_link">
       <visual>
         <origin xyz="0 0 0" rpy="0 0 0"/>
@@ -21,7 +21,7 @@
       <xacro:box_inertial xyz="0 -0.024 0" rpy="0 0 0" size="0.042 0.048 0.04" mass="0.022"/>
     </link>
-    <joint name="shoulder_r_roll_joint" type="revolute">
-      <parent link="shoulder_r_pitch"/>
-      <child link="shoulder_r_roll"/>
+    <joint name="shoulder_r_roll" type="revolute">
+      <parent link="shoulder_r_pitch_link"/>
+      <child link="shoulder_r_roll_link"/>
       <origin xyz="0 -0.038 0" rpy="0 0 0"/>
       <axis xyz="-1 0 0"/>
@@ -29,5 +29,5 @@
       <dynamics damping="0.0" friction="0.0"/>
     </joint>
-    <link name="shoulder_r_roll">
+    <link name="shoulder_r_roll_link">
       <visual>
         <origin xyz="0 0 0" rpy="0 0 0"/>
@@ -40,7 +40,7 @@
         mass="0.342"/>
     </link>
-    <joint name="elbow_r_front_joint" type="revolute">
-      <parent link="shoulder_r_roll"/>
-      <child link="elbow_r_front"/>
+    <joint name="elbow_r_front" type="revolute">
+      <parent link="shoulder_r_roll_link"/>
+      <child link="elbow_r_front_link"/>
       <origin xyz="0 0.008 -0.052" rpy="0 0 0"/>
       <axis xyz="0 1 0"/>
@@ -48,5 +48,5 @@
       <dynamics damping="0.0" friction="0.0"/>
     </joint>
-    <link name="elbow_r_front">
+    <link name="elbow_r_front_link">
       <visual>
         <origin xyz="0 0 0" rpy="0 0 0"/>
@@ -59,7 +59,7 @@
       <xacro:box_inertial xyz="0.0043 0 -0.104" rpy="0 0 0" size="0.044 0.058 0.208" mass="0.032"/>
     </link>
-    <joint name="elbow_r_rear_joint" type="revolute">
-      <parent link="shoulder_r_roll"/>
-      <child link="elbow_r_rear"/>
+    <joint name="elbow_r_rear" type="revolute">
+      <parent link="shoulder_r_roll_link"/>
+      <child link="elbow_r_rear_link"/>
       <origin xyz="0 0.008 -0.052" rpy="0 0 0"/>
       <axis xyz="0 -1 0"/>
@@ -67,5 +67,5 @@
       <dynamics damping="0.0" friction="0.0"/>
     </joint>
-    <link name="elbow_r_rear">
+    <link name="elbow_r_rear_link">
       <visual>
         <origin xyz="0 0 0" rpy="0 0 0"/>

File: kuroko_description/xacro/kuroko/parts/body.xacro (robot description, xacro)
@@ -3,34 +3,34 @@
   <xacro:macro name="body_xacro">
     <!-- chest -->
-    <link name="chest">
+    <link name="chest_link">
       <visual>
-        <origin xyz="0 0 0" rpy="0 0 0" />
+        <origin xyz="0 0 0" rpy="0 0 0"/>
         <geometry>
-          <mesh filename="package://kuroko_description/meshes/kuroko/obj/chest.obj" />
+          <mesh filename="package://kuroko_description/meshes/kuroko/obj/chest.obj"/>
         </geometry>
       </visual>
-      <xacro:box_collision xyz="0 0 0.057" rpy="0 0 0" size="0.1 0.242 0.114" />
-      <xacro:box_inertial xyz="0 0 0.057" rpy="0 0 0" size="0.1 0.242 0.114" mass="0.991" />
+      <xacro:box_collision xyz="0 0 0.057" rpy="0 0 0" size="0.1 0.242 0.114"/>
+      <xacro:box_inertial xyz="0 0 0.057" rpy="0 0 0" size="0.1 0.242 0.114" mass="0.991"/>
     </link>
     <!-- Joint1 -->
-    <joint name="waist_joint" type="revolute">
-      <parent link="chest" />
-      <child link="waist" />
-      <origin xyz="0 0 0" rpy="0 0 0" />
-      <axis xyz="0 0 -1" />
-      <limit effort="1000.0" lower="-3.1" upper="3.1" velocity="10.0" />
-      <dynamics damping="0.0" friction="0.0" />
+    <joint name="waist" type="revolute">
+      <parent link="chest_link"/>
+      <child link="waist_link"/>
+      <origin xyz="0 0 0" rpy="0 0 0"/>
+      <axis xyz="0 0 -1"/>
+      <limit effort="1000.0" lower="-3.1" upper="3.1" velocity="10.0"/>
+      <dynamics damping="0.0" friction="0.0"/>
     </joint>
     <!-- waist -->
-    <link name="waist">
+    <link name="waist_link">
       <visual>
-        <origin xyz="0 0 0" rpy="0 0 0" />
+        <origin xyz="0 0 0" rpy="0 0 0"/>
         <geometry>
-          <mesh filename="package://kuroko_description/meshes/kuroko/obj/waist.obj" />
+          <mesh filename="package://kuroko_description/meshes/kuroko/obj/waist.obj"/>
         </geometry>
       </visual>
-      <xacro:box_collision xyz="0.00125 0 -0.04875" rpy="0 0 0" size="0.0705 0.0325 0.0975" />
+      <xacro:box_collision xyz="0.00125 0 -0.04875" rpy="0 0 0" size="0.0705 0.0325 0.0975"/>
       <xacro:box_inertial xyz="0.00125 0 -0.04875" rpy="0 0 0" size="0.0705 0.0325 0.0975"
-        mass="0.337" />
+        mass="0.337"/>
     </link>
   </xacro:macro>

File: kuroko_description/xacro/kuroko/parts/leg_l.xacro (robot description, xacro)
@@ -4,5 +4,5 @@
     <!-- Link conencts from body. Femoral first. -->
     <joint name="hip_l_roll_joint" type="revolute">
-      <parent link="waist"/>
+      <parent link="waist_link"/>
       <child link="hip_l_roll"/>
       <origin xyz="0 0 -0.08425" rpy="0 0 0"/>

File: kuroko_description/xacro/kuroko/parts/leg_r.xacro (robot description, xacro)
@@ -4,5 +4,5 @@
     <!-- Link conencts from body. Femoral first. -->
     <joint name="hip_r_roll_joint" type="revolute">
-      <parent link="waist"/>
+      <parent link="waist_link"/>
       <child link="hip_r_roll"/>
       <origin xyz="0 0 -0.08425" rpy="0 0 0"/>
