Commit message: root_link -> body_link

File: kuroko_description/xacro/kuroko/kuroko.xacro (robot description, xacro)
@@ -42,7 +42,7 @@
   <!-- MACRO:Setting up a Robot Model -->
   <xacro:macro name="kuroko_xacro" params="gazebo gazebo_hw_interface">
-    <link name="root_link"/>
+    <link name="body_link"/>
     <joint name="root_joint" type="fixed">
-      <parent link="root_link"/>
+      <parent link="body_link"/>
       <child link="chest_link"/>
       <origin xyz="0 0 0" rpy="0 0 0"/>

Commit message: Waist to root

File: kuroko_description/xacro/kuroko/kuroko.xacro (robot description, xacro)
@@ -45,5 +45,5 @@
     <joint name="root_joint" type="fixed">
       <parent link="body_link"/>
-      <child link="chest_link"/>
+      <child link="waist_link"/>
       <origin xyz="0 0 0" rpy="0 0 0"/>
     </joint>

File: kuroko_description/xacro/kuroko/parts/body.xacro (robot description, xacro)
@@ -2,24 +2,4 @@
 <robot xmlns:xacro="http://www.ros.org/wiki/xacro">
   <xacro:macro name="body_xacro">
-    <!-- chest -->
-    <link name="chest_link">
-      <visual>
-        <origin xyz="0 0 0" rpy="0 0 0"/>
-        <geometry>
-          <mesh filename="package://kuroko_description/meshes/kuroko/obj/chest.obj"/>
-        </geometry>
-      </visual>
-      <xacro:box_collision xyz="0 0 0.057" rpy="0 0 0" size="0.1 0.242 0.114"/>
-      <xacro:box_inertial xyz="0 0 0.057" rpy="0 0 0" size="0.1 0.242 0.114" mass="0.991"/>
-    </link>
-    <!-- Joint1 -->
-    <joint name="waist" type="revolute">
-      <parent link="chest_link"/>
-      <child link="waist_link"/>
-      <origin xyz="0 0 0" rpy="0 0 0"/>
-      <axis xyz="0 0 -1"/>
-      <limit effort="1000.0" lower="-3.1" upper="3.1" velocity="10.0"/>
-      <dynamics damping="0.0" friction="0.0"/>
-    </joint>
     <!-- waist -->
     <link name="waist_link">
@@ -34,4 +14,24 @@
         mass="0.337"/>
     </link>
+    <!-- Joint1 -->
+    <joint name="waist" type="revolute">
+      <parent link="waist_link"/>
+      <child link="chest_link"/>
+      <origin xyz="0 0 0" rpy="0 0 0"/>
+      <axis xyz="0 0 1"/>
+      <limit effort="1000.0" lower="-3.1" upper="3.1" velocity="10.0"/>
+      <dynamics damping="0.0" friction="0.0"/>
+    </joint>
+    <!-- chest -->
+    <link name="chest_link">
+      <visual>
+        <origin xyz="0 0 0" rpy="0 0 0"/>
+        <geometry>
+          <mesh filename="package://kuroko_description/meshes/kuroko/obj/chest.obj"/>
+        </geometry>
+      </visual>
+      <xacro:box_collision xyz="0 0 0.057" rpy="0 0 0" size="0.1 0.242 0.114"/>
+      <xacro:box_inertial xyz="0 0 0.057" rpy="0 0 0" size="0.1 0.242 0.114" mass="0.991"/>
+    </link>
   </xacro:macro>
 </robot>

File: kuroko_description/xacro/sensors/imu/n100mini.xacro (robot description, xacro)
@@ -4,31 +4,31 @@
   xmlns:interface="http://playerstage.sourceforge.net/gazebo/xmlschema/#interface"
   xmlns:xacro="http://www.ros.org/wiki/xacro">
-  <xacro:include filename="n100mini_gazebo.xacro" />
+  <xacro:include filename="n100mini_gazebo.xacro"/>
   <xacro:macro name="n100mini_imu" params="name parent:='base_link' update_rate:=400 *origin">
-    <xacro:property name="depth" value="0.0245" />
-    <xacro:property name="width" value="0.0245" />
-    <xacro:property name="height" value="0.0145" />
+    <xacro:property name="depth" value="0.0245"/>
+    <xacro:property name="width" value="0.0245"/>
+    <xacro:property name="height" value="0.0145"/>
     <joint name="${name}_joint" type="fixed">
-      <parent link="${parent}" />
-      <child link="${name}_link" />
-      <xacro:insert_block name="origin" />
+      <parent link="${parent}"/>
+      <child link="${name}_link"/>
+      <xacro:insert_block name="origin"/>
     </joint>
     <link name="${name}_link">
       <visual>
-        <origin xyz="0 0 0" rpy="0 0 0" />
+        <origin xyz="0 0 0" rpy="0 0 0"/>
         <geometry>
-          <box size="${depth} ${width} ${height}" />
+          <box size="${depth} ${width} ${height}"/>
         </geometry>
         <material name="gray">
-          <color rgba="0.5 0.5 0.5 1" />
+          <color rgba="0.5 0.5 0.5 1"/>
         </material>
       </visual>
       <collision>
-        <origin xyz="0 0 0" rpy="0 0 0" />
+        <origin xyz="0 0 0" rpy="0 0 0"/>
         <geometry>
-          <box size="${depth} ${width} ${height}" />
+          <box size="${depth} ${width} ${height}"/>
         </geometry>
       </collision>
-      <xacro:box_inertial xyz="0 0 0" rpy="0 0 0" size="${depth} ${width} ${height}" mass="0.013" />
+      <xacro:box_inertial xyz="0 0 0" rpy="0 0 0" size="${depth} ${width} ${height}" mass="0.013"/>
     </link>
     <!-- gazebo extensions -->
@@ -37,5 +37,5 @@
       <preserveFixedJoint>true</preserveFixedJoint>
     </gazebo>
-    <xacro:n100mini_gazebo name="${name}" update_rate="${update_rate}" />
+    <xacro:n100mini_gazebo name="${name}" update_rate="${update_rate}"/>
   </xacro:macro>
 </robot>

Commit message: Attach USB camera

File: kuroko_description/xacro/kuroko/kuroko.xacro (robot description, xacro)
@@ -18,5 +18,5 @@
   <xacro:include filename="$(find kuroko_description)/xacro/kuroko/transmission/leg_l.gazebo"/>
   <xacro:include filename="$(find kuroko_description)/xacro/sensors/imu/n100mini.xacro"/>
-  <xacro:include filename="$(find kuroko_description)/xacro/sensors/depth/maixsense_a075v.xacro"/>
+  <xacro:include filename="$(find kuroko_description)/xacro/sensors/camera/usb_camera.xacro"/>
   <!-- MACRO:Loading Gazebo Controllers for joints -->
   <xacro:macro name="gazebo_plugin_xacro" params="gazebo_motor_model">
@@ -61,4 +61,7 @@
       <origin xyz="0 0 0.008" rpy="0 0 0"/>
     </xacro:n100mini_imu>
+    <xacro:usb_camera parent="waist_link" name="usb_camera">
+      <origin xyz="0.075230 0 -0.032085" rpy="0 0.1745329 0"/>
+    </xacro:usb_camera>
   </xacro:macro>
   <!-- Load Macros -->

Commit message: Edit device names

File: kuroko_description/xacro/kuroko/kuroko.xacro (robot description, xacro)
@@ -17,5 +17,5 @@
   <xacro:include filename="$(find kuroko_description)/xacro/kuroko/parts/leg_l.xacro"/>
   <xacro:include filename="$(find kuroko_description)/xacro/kuroko/transmission/leg_l.gazebo"/>
-  <xacro:include filename="$(find kuroko_description)/xacro/sensors/imu/n100mini.xacro"/>
+  <xacro:include filename="$(find kuroko_description)/xacro/sensors/imu/imu_n100mini.xacro"/>
   <xacro:include filename="$(find kuroko_description)/xacro/sensors/camera/usb_camera.xacro"/>
   <!-- MACRO:Loading Gazebo Controllers for joints -->
@@ -58,8 +58,8 @@
     <xacro:leg_l_xacro gazebo="$(arg gazebo)"/>
     <xacro:leg_l_gazebo gazebo_hw_interface="${gazebo_hw_interface}"/>
-    <xacro:n100mini_imu parent="chest_link" name="imu">
+    <xacro:imu_n100mini parent="chest_link" name="imu">
       <origin xyz="0 0 0.008" rpy="0 0 0"/>
-    </xacro:n100mini_imu>
-    <xacro:usb_camera parent="waist_link" name="usb_camera">
+    </xacro:imu_n100mini>
+    <xacro:usb_camera parent="waist_link" name="camera">
       <origin xyz="0.075230 0 -0.032085" rpy="0 0.1745329 0"/>
     </xacro:usb_camera>

File: kuroko_description/xacro/sensors/camera/usb_camera.xacro (robot description, xacro)
@@ -55,7 +55,7 @@
           <alwaysOn>true</alwaysOn>
           <updateRate>30</updateRate>
-          <cameraName>usb_camera</cameraName>
-          <imageTopicName>image_raw</imageTopicName>
-          <cameraInfoTopicName>camera_info</cameraInfoTopicName>
+          <cameraName>camera</cameraName>
+          <imageTopicName>resized/image</imageTopicName>
+          <cameraInfoTopicName>resized/camera_info</cameraInfoTopicName>
           <frameName>${name}_optical_link</frameName>
           <hackBaseline>0</hackBaseline>

File: kuroko_description/xacro/sensors/imu/imu_n100mini.xacro (robot description, xacro)
@@ -4,6 +4,6 @@
   xmlns:interface="http://playerstage.sourceforge.net/gazebo/xmlschema/#interface"
   xmlns:xacro="http://www.ros.org/wiki/xacro">
-  <xacro:include filename="n100mini_gazebo.xacro"/>
-  <xacro:macro name="n100mini_imu" params="name parent:='base_link' update_rate:=400 *origin">
+  <xacro:include filename="imu_n100mini_gazebo.xacro"/>
+  <xacro:macro name="imu_n100mini" params="name parent:='base_link' update_rate:=400 *origin">
     <xacro:property name="depth" value="0.0245"/>
     <xacro:property name="width" value="0.0245"/>

File: kuroko_description/xacro/sensors/imu/imu_n100mini_gazebo.xacro (robot description, xacro)
@@ -1,5 +1,5 @@
 <?xml version="1.0" encoding="UTF-8"?>
 <robot xmlns:xacro="http://www.ros.org/wiki/xacro">
-  <xacro:macro name="n100_gazebo" params="name update_rate">
+  <xacro:macro name="n100mini_gazebo" params="name update_rate">
     <gazebo reference="${name}_link">
       <material>Gazebo/Gray</material>
@@ -10,6 +10,6 @@
         <updateRate>${update_rate}</updateRate>
         <bodyName>${name}_link</bodyName>
-        <topicName>${name}/data</topicName>
-        <serviceName>${name}/service</serviceName>
+        <topicName>/kuroko/sensors/imu/data</topicName>
+        <serviceName>/kuroko/sensors/imu/service</serviceName>
         <frameId>${name}_link</frameId>
         <gaussianNoise>0</gaussianNoise>
@@ -22,5 +22,5 @@
         <updateRate>${update_rate}</updateRate>
         <bodyName>${name}_link</bodyName>
-        <topicName>${name}/mag</topicName>
+        <topicName>/kuroko/sensors/imu/mag</topicName>
         <frameId>${name}_link</frameId>
         <useMagneticFieldMsgs>true</useMagneticFieldMsgs>

Commit message: Change shoulder motor

File: kuroko_description/xacro/kuroko/kuroko.xacro (robot description, xacro)
@@ -57,9 +57,9 @@
     <xacro:leg_l_xacro gazebo="$(arg gazebo)"/>
     <xacro:leg_l_gazebo gazebo_hw_interface="${gazebo_hw_interface}"/>
-    <xacro:imu_n100mini parent="chest_link" name="imu">
-      <origin xyz="0 0 0.008" rpy="0 0 0"/>
+    <xacro:imu_n100mini parent="waist_link" name="imu">
+      <origin xyz="-0.04 0 -0.01" rpy="0 0 0"/>
     </xacro:imu_n100mini>
     <xacro:usb_camera parent="waist_link" name="camera">
-      <origin xyz="0.075230 0 -0.032085" rpy="0 0.1745329 0"/>
+      <origin xyz="0.07 0 -0.026" rpy="0 0 0"/>
     </xacro:usb_camera>
   </xacro:macro>

File: kuroko_description/xacro/kuroko/parts/arm_l.xacro (robot description, xacro)
@@ -6,5 +6,5 @@
       <parent link="chest_link"/>
       <child link="shoulder_l_pitch_link"/>
-      <origin xyz="0 0.1275 0.01275" rpy="0 0 0"/>
+      <origin xyz="0 0.128 0.01275" rpy="0 0 0"/>
       <axis xyz="0 1 0"/>
       <limit effort="1000.0" lower="-3.1" upper="3.1" velocity="10.0"/>
@@ -18,11 +18,11 @@
         </geometry>
       </visual>
-      <xacro:box_collision xyz="0 0.024 0" rpy="0 0 0" size="0.042 0.048 0.04"/>
-      <xacro:box_inertial xyz="0 0.024 0" rpy="0 0 0" size="0.042 0.048 0.04" mass="0.022"/>
+      <xacro:box_collision xyz="-0.0096 0.0340 0.0000" rpy="0 0 0" size="0.0513 0.0680 0.0475"/>
+      <xacro:box_inertial xyz="-0.0096 0.0340 0.0000" rpy="0 0 0" size="0.0513 0.0680 0.0475" mass="0.165"/>
     </link>
     <joint name="shoulder_l_roll" type="revolute">
       <parent link="shoulder_l_pitch_link"/>
       <child link="shoulder_l_roll_link"/>
-      <origin xyz="0 0.038 0" rpy="0 0 0"/>
+      <origin xyz="0 0.05425 0" rpy="0 0 0"/>
       <axis xyz="-1 0 0"/>
       <limit effort="1000.0" lower="-2.0071" upper="1.0472" velocity="10.0"/>
@@ -36,11 +36,11 @@
         </geometry>
       </visual>
-      <xacro:box_collision xyz="0 0.016 -0.02575" rpy="0 0 0" size="0.0285 0.082 0.08"/>
-      <xacro:box_inertial xyz="0 0.016 -0.02575" rpy="0 0 0" size="0.0285 0.082 0.08" mass="0.342"/>
+      <xacro:box_collision xyz="-0.0108 0.0000 -0.0186" rpy="0 0 0" size="0.0530 0.0860 0.0633"/>
+      <xacro:box_inertial xyz="-0.0108 0.0000 -0.0186" rpy="0 0 0" size="0.0530 0.0860 0.0633" mass="0.183"/>
     </link>
     <joint name="elbow_l_front" type="revolute">
       <parent link="shoulder_l_roll_link"/>
       <child link="elbow_l_front_link"/>
-      <origin xyz="0 -0.008 -0.052" rpy="0 0 0"/>
+      <origin xyz="0 -0.023 -0.036" rpy="0 0 0"/>
       <axis xyz="0 -1 0"/>
       <limit effort="1000.0" lower="-2.6180" upper="2.6180" velocity="10.0"/>
@@ -61,5 +61,5 @@
       <parent link="shoulder_l_roll_link"/>
       <child link="elbow_l_rear_link"/>
-      <origin xyz="0 -0.008 -0.052" rpy="0 0 0"/>
+      <origin xyz="0 -0.024 -0.036" rpy="0 0 0"/>
       <axis xyz="0 1 0"/>
       <limit effort="1000.0" lower="-2.6180" upper="2.6180" velocity="10.0"/>

File: kuroko_description/xacro/kuroko/parts/arm_r.xacro (robot description, xacro)
@@ -6,5 +6,5 @@
       <parent link="chest_link"/>
       <child link="shoulder_r_pitch_link"/>
-      <origin xyz="0 -0.1275 0.01275" rpy="0 0 0"/>
+      <origin xyz="0 -0.128 0.01275" rpy="0 0 0"/>
       <axis xyz="0 -1 0"/>
       <limit effort="1000.0" lower="-3.1" upper="3.1" velocity="10.0"/>
@@ -18,11 +18,11 @@
         </geometry>
       </visual>
-      <xacro:box_collision xyz="0 -0.024 0" rpy="0 0 0" size="0.042 0.048 0.04"/>
-      <xacro:box_inertial xyz="0 -0.024 0" rpy="0 0 0" size="0.042 0.048 0.04" mass="0.022"/>
+      <xacro:box_collision xyz="-0.0096 -0.0340 0.0000" rpy="0 0 0" size="0.0513 0.0680 0.0475"/>
+      <xacro:box_inertial xyz="-0.0096 -0.0340 0.0000" rpy="0 0 0" size="0.0513 0.0680 0.0475" mass="0.165"/>
     </link>
     <joint name="shoulder_r_roll" type="revolute">
       <parent link="shoulder_r_pitch_link"/>
       <child link="shoulder_r_roll_link"/>
-      <origin xyz="0 -0.038 0" rpy="0 0 0"/>
+      <origin xyz="0 -0.05425 0" rpy="0 0 0"/>
       <axis xyz="-1 0 0"/>
       <limit effort="1000.0" lower="-1.0472" upper="2.0071" velocity="10.0"/>
@@ -36,12 +36,11 @@
         </geometry>
       </visual>
-      <xacro:box_collision xyz="0 -0.016 -0.02575" rpy="0 0 0" size="0.0285 0.082 0.08"/>
-      <xacro:box_inertial xyz="0 -0.016 -0.02575" rpy="0 0 0" size="0.0285 0.082 0.08"
-        mass="0.342"/>
+      <xacro:box_collision xyz="-0.0108 0.0000 -0.0186" rpy="0 0 0" size="0.0530 0.0860 0.0633"/>
+      <xacro:box_inertial xyz="-0.0108 0.0000 -0.0186" rpy="0 0 0" size="0.0530 0.0860 0.0633" mass="0.183"/>
     </link>
     <joint name="elbow_r_front" type="revolute">
       <parent link="shoulder_r_roll_link"/>
       <child link="elbow_r_front_link"/>
-      <origin xyz="0 0.008 -0.052" rpy="0 0 0"/>
+      <origin xyz="0 0.023 -0.036" rpy="0 0 0"/>
       <axis xyz="0 1 0"/>
       <limit effort="1000.0" lower="-2.6180" upper="2.6180" velocity="10.0"/>
@@ -62,5 +61,5 @@
       <parent link="shoulder_r_roll_link"/>
       <child link="elbow_r_rear_link"/>
-      <origin xyz="0 0.008 -0.052" rpy="0 0 0"/>
+      <origin xyz="0 0.024 -0.036" rpy="0 0 0"/>
       <axis xyz="0 -1 0"/>
       <limit effort="1000.0" lower="-2.6180" upper="2.6180" velocity="10.0"/>

File: kuroko_description/xacro/kuroko/parts/body.xacro (robot description, xacro)
@@ -10,7 +10,6 @@
         </geometry>
       </visual>
-      <xacro:box_collision xyz="0.00125 0 -0.04875" rpy="0 0 0" size="0.0705 0.0325 0.0975"/>
-      <xacro:box_inertial xyz="0.00125 0 -0.04875" rpy="0 0 0" size="0.0705 0.0325 0.0975"
-        mass="0.337"/>
+      <xacro:box_collision xyz="0.0084 0.0000 -0.0483" rpy="0 0 0" size="0.1247 0.0560 0.0965"/>
+      <xacro:box_inertial xyz="0.0084 0.0000 -0.0483" rpy="0 0 0" size="0.1247 0.0560 0.0965" mass="0.388"/>
     </link>
     <!-- Joint1 -->
@@ -31,6 +30,6 @@
         </geometry>
       </visual>
-      <xacro:box_collision xyz="0 0 0.057" rpy="0 0 0" size="0.1 0.242 0.114"/>
-      <xacro:box_inertial xyz="0 0 0.057" rpy="0 0 0" size="0.1 0.242 0.114" mass="0.991"/>
+      <xacro:box_collision xyz="0.0120 0.0000 0.0635" rpy="0 0 0" size="0.1480 0.2560 0.1364"/>
+      <xacro:box_inertial xyz="0.0120 0.0000 0.0635" rpy="0 0 0" size="0.1480 0.2560 0.1364" mass="0.806"/>
     </link>
   </xacro:macro>

Commit message: Add tf luna

File: kuroko_description/xacro/kuroko/kuroko.xacro (robot description, xacro)
@@ -16,4 +16,5 @@
   <xacro:include filename="$(find kuroko_description)/xacro/kuroko/parts/leg_l.xacro"/>
   <xacro:include filename="$(find kuroko_description)/xacro/kuroko/transmission/leg_l.gazebo"/>
+  <xacro:include filename="$(find kuroko_description)/xacro/sensors/range/tfluna.xacro"/>
   <xacro:include filename="$(find kuroko_description)/xacro/sensors/imu/imu_n100mini.xacro"/>
   <xacro:include filename="$(find kuroko_description)/xacro/sensors/camera/usb_camera.xacro"/>
@@ -63,4 +64,7 @@
       <origin xyz="0.07 0 -0.026" rpy="0 0 0"/>
     </xacro:usb_camera>
+    <xacro:tfluna parent="waist_link" name="tfluna" ros_topic="/kuroko/sensors/ragne">
+      <origin xyz="0.07 0 -0.044" rpy="0 0 0"/>
+    </xacro:tfluna>
   </xacro:macro>
   <!-- Load Macros -->

File: kuroko_description/xacro/physics/box_physics.xacro (robot description, xacro)
@@ -2,18 +2,18 @@
 <robot xmlns:xacro="http://www.ros.org/wiki/xacro">
   <xacro:macro name="box_inertial" params="xyz:='0 0 0' rpy:='0 0 0' size mass inertia_min:=0.00001">
-    <xacro:property name="d" value="${float(size.split()[0])}" />
-    <xacro:property name="w" value="${float(size.split()[1])}" />
-    <xacro:property name="h" value="${float(size.split()[2])}" />
-    <xacro:property name="ixx" value="${mass * (w ** 2 + h ** 2) / 12}" />
-    <xacro:property name="iyy" value="${mass * (d ** 2 + h ** 2) / 12}" />
-    <xacro:property name="izz" value="${mass * (w ** 2 + d ** 2) / 12}" />
+    <xacro:property name="d" value="${float(size.split()[0])}"/>
+    <xacro:property name="w" value="${float(size.split()[1])}"/>
+    <xacro:property name="h" value="${float(size.split()[2])}"/>
+    <xacro:property name="ixx" value="${mass * (w ** 2 + h ** 2) / 12}"/>
+    <xacro:property name="iyy" value="${mass * (d ** 2 + h ** 2) / 12}"/>
+    <xacro:property name="izz" value="${mass * (w ** 2 + d ** 2) / 12}"/>
     <xacro:if value="${int(inertia_min/ixx)}">
-      <xacro:property name="ixx" value="${inertia_min}" />
+      <xacro:property name="ixx" value="${inertia_min}"/>
     </xacro:if>
     <xacro:if value="${int(inertia_min/iyy)}">
-      <xacro:property name="iyy" value="${inertia_min}" />
+      <xacro:property name="iyy" value="${inertia_min}"/>
     </xacro:if>
     <xacro:if value="${int(inertia_min/izz)}">
-      <xacro:property name="izz" value="${inertia_min}" />
+      <xacro:property name="izz" value="${inertia_min}"/>
     </xacro:if>
     <inertial>
@@ -21,6 +21,6 @@
       <mass value="${mass}"/>
       <inertia ixx="${ixx}"
-               ixy="0.0" iyy="${iyy}"
-               ixz="0.0" iyz="0.0" izz="${izz}"/>
+        ixy="0.0" iyy="${iyy}"
+        ixz="0.0" iyz="0.0" izz="${izz}"/>
     </inertial>
   </xacro:macro>
@@ -33,3 +33,14 @@
     </collision>
   </xacro:macro>
+  <xacro:macro name="box_visual" params="xyz:='0 0 0' rpy:='0 0 0' size material_name:='gray' color:='0.5 0.5 0.5 1'">
+    <visual>
+      <origin xyz="${xyz}" rpy="${rpy}"/>
+      <geometry>
+        <box size="${size}"/>
+      </geometry>
+      <material name="${material_name}">
+        <color rgba="${color}"/>
+      </material>
+    </visual>
+  </xacro:macro>
 </robot>

File: kuroko_description/xacro/sensors/imu/imu_n100mini.xacro (robot description, xacro)
@@ -6,7 +6,7 @@
   <xacro:include filename="imu_n100mini_gazebo.xacro"/>
   <xacro:macro name="imu_n100mini" params="name parent:='base_link' update_rate:=400 *origin">
-    <xacro:property name="depth" value="0.0245"/>
-    <xacro:property name="width" value="0.0245"/>
-    <xacro:property name="height" value="0.0145"/>
+    <xacro:property name="depth" value="0.01"/>
+    <xacro:property name="width" value="0.01"/>
+    <xacro:property name="height" value="0.01"/>
     <joint name="${name}_joint" type="fixed">
       <parent link="${parent}"/>
