Commit message: Use relative path

File: kuroko_description/xacro/kuroko/kuroko.xacro (robot description, xacro)
@@ -4,19 +4,20 @@
   <xacro:arg name="gazebo_motor_model" default="dc"/>
   <xacro:arg name="gazebo_hw_interface" default="position"/>
-  <xacro:include filename="$(find kuroko_description)/xacro/physics/box_physics.xacro"/>
-  <xacro:include filename="$(find kuroko_description)/xacro/physics/gazebo_passive_joint.xacro"/>
-  <xacro:include filename="$(find kuroko_description)/xacro/kuroko/parts/body.xacro"/>
-  <xacro:include filename="$(find kuroko_description)/xacro/kuroko/transmission/body.gazebo"/>
-  <xacro:include filename="$(find kuroko_description)/xacro/kuroko/parts/arm_r.xacro"/>
-  <xacro:include filename="$(find kuroko_description)/xacro/kuroko/transmission/arm_r.gazebo"/>
-  <xacro:include filename="$(find kuroko_description)/xacro/kuroko/parts/arm_l.xacro"/>
-  <xacro:include filename="$(find kuroko_description)/xacro/kuroko/transmission/arm_l.gazebo"/>
-  <xacro:include filename="$(find kuroko_description)/xacro/kuroko/parts/leg_r.xacro"/>
-  <xacro:include filename="$(find kuroko_description)/xacro/kuroko/transmission/leg_r.gazebo"/>
-  <xacro:include filename="$(find kuroko_description)/xacro/kuroko/parts/leg_l.xacro"/>
-  <xacro:include filename="$(find kuroko_description)/xacro/kuroko/transmission/leg_l.gazebo"/>
-  <xacro:include filename="$(find kuroko_description)/xacro/sensors/range/tfluna.xacro"/>
-  <xacro:include filename="$(find kuroko_description)/xacro/sensors/imu/imu_n100mini.xacro"/>
-  <xacro:include filename="$(find kuroko_description)/xacro/sensors/camera/usb_camera.xacro"/>
+  <xacro:property name="XACRO_DIR" value="$(cwd)/${xacro.abs_filename('..')}" />
+  <xacro:include filename="${XACRO_DIR}/physics/box_physics.xacro"/>
+  <xacro:include filename="${XACRO_DIR}/physics/gazebo_passive_joint.xacro"/>
+  <xacro:include filename="${XACRO_DIR}/kuroko/parts/body.xacro"/>
+  <xacro:include filename="${XACRO_DIR}/kuroko/transmission/body.gazebo"/>
+  <xacro:include filename="${XACRO_DIR}/kuroko/parts/arm_r.xacro"/>
+  <xacro:include filename="${XACRO_DIR}/kuroko/transmission/arm_r.gazebo"/>
+  <xacro:include filename="${XACRO_DIR}/kuroko/parts/arm_l.xacro"/>
+  <xacro:include filename="${XACRO_DIR}/kuroko/transmission/arm_l.gazebo"/>
+  <xacro:include filename="${XACRO_DIR}/kuroko/parts/leg_r.xacro"/>
+  <xacro:include filename="${XACRO_DIR}/kuroko/transmission/leg_r.gazebo"/>
+  <xacro:include filename="${XACRO_DIR}/kuroko/parts/leg_l.xacro"/>
+  <xacro:include filename="${XACRO_DIR}/kuroko/transmission/leg_l.gazebo"/>
+  <xacro:include filename="${XACRO_DIR}/sensors/range/tfluna.xacro"/>
+  <xacro:include filename="${XACRO_DIR}/sensors/imu/imu_n100mini.xacro"/>
+  <xacro:include filename="${XACRO_DIR}/sensors/camera/usb_camera.xacro"/>
   <!-- MACRO:Loading Gazebo Controllers for joints -->
   <xacro:macro name="gazebo_plugin_xacro" params="gazebo_motor_model">

File: kuroko_description/xacro/kuroko/parts/arm_l.xacro (robot description, xacro)
@@ -1,4 +1,5 @@
 <?xml version="1.0"?>
 <robot xmlns:xacro="http://www.ros.org/wiki/xacro">
+  <xacro:property name="MESH_DIR" value="$(cwd)/${xacro.abs_filename('../../../meshes')}" />
   <xacro:macro name="arm_l_xacro">
     <!-- Link conencts from body. Shoulder first. -->
@@ -15,5 +16,5 @@
         <origin xyz="0 0 0" rpy="0 0 0"/>
         <geometry>
-          <mesh filename="package://kuroko_description/meshes/kuroko/obj/shoulder_l_pitch.obj"/>
+          <mesh filename="${MESH_DIR}/kuroko/obj/shoulder_l_pitch.obj"/>
         </geometry>
       </visual>
@@ -33,5 +34,5 @@
         <origin xyz="0 0 0" rpy="0 0 0"/>
         <geometry>
-          <mesh filename="package://kuroko_description/meshes/kuroko/obj/shoulder_l_roll.obj"/>
+          <mesh filename="${MESH_DIR}/kuroko/obj/shoulder_l_roll.obj"/>
         </geometry>
       </visual>
@@ -51,5 +52,5 @@
         <origin xyz="0 0 0" rpy="0 0 0"/>
         <geometry>
-          <mesh filename="package://kuroko_description/meshes/kuroko/obj/elbow_l_front.obj"/>
+          <mesh filename="${MESH_DIR}/kuroko/obj/elbow_l_front.obj"/>
         </geometry>
       </visual>
@@ -70,5 +71,5 @@
         <origin xyz="0 0 0" rpy="0 0 0"/>
         <geometry>
-          <mesh filename="package://kuroko_description/meshes/kuroko/obj/elbow_l_rear.obj"/>
+          <mesh filename="${MESH_DIR}/kuroko/obj/elbow_l_rear.obj"/>
         </geometry>
       </visual>

File: kuroko_description/xacro/kuroko/parts/arm_r.xacro (robot description, xacro)
@@ -1,4 +1,5 @@
 <?xml version="1.0"?>
 <robot xmlns:xacro="http://www.ros.org/wiki/xacro">
+  <xacro:property name="MESH_DIR" value="$(cwd)/${xacro.abs_filename('../../../meshes')}" />
   <xacro:macro name="arm_r_xacro">
     <!-- Link conencts from body. Shoulder first. -->
@@ -15,5 +16,5 @@
         <origin xyz="0 0 0" rpy="0 0 0"/>
         <geometry>
-          <mesh filename="package://kuroko_description/meshes/kuroko/obj/shoulder_r_pitch.obj"/>
+          <mesh filename="${MESH_DIR}/kuroko/obj/shoulder_r_pitch.obj"/>
         </geometry>
       </visual>
@@ -33,5 +34,5 @@
         <origin xyz="0 0 0" rpy="0 0 0"/>
         <geometry>
-          <mesh filename="package://kuroko_description/meshes/kuroko/obj/shoulder_r_roll.obj"/>
+          <mesh filename="${MESH_DIR}/kuroko/obj/shoulder_r_roll.obj"/>
         </geometry>
       </visual>
@@ -51,5 +52,5 @@
         <origin xyz="0 0 0" rpy="0 0 0"/>
         <geometry>
-          <mesh filename="package://kuroko_description/meshes/kuroko/obj/elbow_r_front.obj"/>
+          <mesh filename="${MESH_DIR}/kuroko/obj/elbow_r_front.obj"/>
         </geometry>
       </visual>
@@ -70,5 +71,5 @@
         <origin xyz="0 0 0" rpy="0 0 0"/>
         <geometry>
-          <mesh filename="package://kuroko_description/meshes/kuroko/obj/elbow_r_rear.obj"/>
+          <mesh filename="${MESH_DIR}/kuroko/obj/elbow_r_rear.obj"/>
         </geometry>
       </visual>

File: kuroko_description/xacro/kuroko/parts/body.xacro (robot description, xacro)
@@ -1,4 +1,5 @@
 <?xml version="1.0"?>
 <robot xmlns:xacro="http://www.ros.org/wiki/xacro">
+  <xacro:property name="MESH_DIR" value="$(cwd)/${xacro.abs_filename('../../../meshes')}" />
   <xacro:macro name="body_xacro">
     <!-- waist -->
@@ -7,5 +8,5 @@
         <origin xyz="0 0 0" rpy="0 0 0"/>
         <geometry>
-          <mesh filename="package://kuroko_description/meshes/kuroko/obj/waist.obj"/>
+          <mesh filename="${MESH_DIR}/kuroko/obj/waist.obj"/>
         </geometry>
       </visual>
@@ -27,5 +28,5 @@
         <origin xyz="0 0 0" rpy="0 0 0"/>
         <geometry>
-          <mesh filename="package://kuroko_description/meshes/kuroko/obj/chest.obj"/>
+          <mesh filename="${MESH_DIR}/kuroko/obj/chest.obj"/>
         </geometry>
       </visual>

File: kuroko_description/xacro/kuroko/parts/leg_l.xacro (robot description, xacro)
@@ -1,4 +1,5 @@
 <?xml version="1.0"?>
 <robot xmlns:xacro="http://www.ros.org/wiki/xacro">
+  <xacro:property name="MESH_DIR" value="$(cwd)/${xacro.abs_filename('../../../meshes')}" />
   <xacro:macro name="leg_l_xacro" params="gazebo:=false">
     <!-- Link conencts from body. Hip first. -->
@@ -15,5 +16,5 @@
         <origin xyz="0 0 0" rpy="0 0 0"/>
         <geometry>
-          <mesh filename="package://kuroko_description/meshes/kuroko/obj/hip_l_roll.obj"/>
+          <mesh filename="${MESH_DIR}/kuroko/obj/hip_l_roll.obj"/>
         </geometry>
       </visual>
@@ -34,5 +35,5 @@
         <origin xyz="0 0 0" rpy="0 0 0"/>
         <geometry>
-          <mesh filename="package://kuroko_description/meshes/kuroko/obj/hip_l_pitch.obj"/>
+          <mesh filename="${MESH_DIR}/kuroko/obj/hip_l_pitch.obj"/>
         </geometry>
       </visual>
@@ -53,5 +54,5 @@
         <origin xyz="0 0 0" rpy="0 0 0"/>
         <geometry>
-          <mesh filename="package://kuroko_description/meshes/kuroko/obj/thigh_l_active.obj"/>
+          <mesh filename="${MESH_DIR}/kuroko/obj/thigh_l_active.obj"/>
         </geometry>
       </visual>
@@ -71,5 +72,5 @@
         <origin xyz="0 0 0" rpy="0 0 0"/>
         <geometry>
-          <mesh filename="package://kuroko_description/meshes/kuroko/obj/shin_l_active.obj"/>
+          <mesh filename="${MESH_DIR}/kuroko/obj/shin_l_active.obj"/>
         </geometry>
       </visual>
@@ -95,5 +96,5 @@
         <origin xyz="0 0 0" rpy="0 0 0"/>
         <geometry>
-          <mesh filename="package://kuroko_description/meshes/kuroko/obj/thigh_r_middle_passive.obj"/>
+          <mesh filename="${MESH_DIR}/kuroko/obj/thigh_r_middle_passive.obj"/>
         </geometry>
       </visual>
@@ -138,5 +139,5 @@
         <origin xyz="0 0 0" rpy="0 0 0"/>
         <geometry>
-          <mesh filename="package://kuroko_description/meshes/kuroko/obj/thigh_r_rear_passive.obj"/>
+          <mesh filename="${MESH_DIR}/kuroko/obj/thigh_r_rear_passive.obj"/>
         </geometry>
       </visual>
@@ -157,5 +158,5 @@
         <origin xyz="0 0 0" rpy="0 0 0"/>
         <geometry>
-          <mesh filename="package://kuroko_description/meshes/kuroko/obj/knee_r_passive.obj"/>
+          <mesh filename="${MESH_DIR}/kuroko/obj/knee_r_passive.obj"/>
         </geometry>
       </visual>
@@ -176,5 +177,5 @@
         <origin xyz="0 0 0" rpy="0 0 0"/>
         <geometry>
-          <mesh filename="package://kuroko_description/meshes/kuroko/obj/shin_r_front_passive.obj"/>
+          <mesh filename="${MESH_DIR}/kuroko/obj/shin_r_front_passive.obj"/>
         </geometry>
       </visual>
@@ -199,5 +200,5 @@
         <origin xyz="0 0 0" rpy="0 0 0"/>
         <geometry>
-          <mesh filename="package://kuroko_description/meshes/kuroko/obj/shin_r_rear_passive.obj"/>
+          <mesh filename="${MESH_DIR}/kuroko/obj/shin_r_rear_passive.obj"/>
         </geometry>
       </visual>
@@ -218,5 +219,5 @@
         <origin xyz="0 0 0" rpy="0 0 0"/>
         <geometry>
-          <mesh filename="package://kuroko_description/meshes/kuroko/obj/ankle_r_pitch_passive.obj"/>
+          <mesh filename="${MESH_DIR}/kuroko/obj/ankle_r_pitch_passive.obj"/>
         </geometry>
       </visual>
@@ -237,5 +238,5 @@
         <origin xyz="0 0 0" rpy="0 0 0"/>
         <geometry>
-          <mesh filename="package://kuroko_description/meshes/kuroko/obj/ankle_l_roll.obj"/>
+          <mesh filename="${MESH_DIR}/kuroko/obj/ankle_l_roll.obj"/>
         </geometry>
       </visual>
@@ -256,5 +257,5 @@
         <origin xyz="0 0 0" rpy="0 0 0"/>
         <geometry>
-          <mesh filename="package://kuroko_description/meshes/kuroko/obj/ankle_r_yaw.obj"/>
+          <mesh filename="${MESH_DIR}/kuroko/obj/ankle_r_yaw.obj"/>
         </geometry>
       </visual>

File: kuroko_description/xacro/kuroko/parts/leg_r.xacro (robot description, xacro)
@@ -1,4 +1,5 @@
 <?xml version="1.0"?>
 <robot xmlns:xacro="http://www.ros.org/wiki/xacro">
+  <xacro:property name="MESH_DIR" value="$(cwd)/${xacro.abs_filename('../../../meshes')}" />
   <xacro:macro name="leg_r_xacro" params="gazebo:=false">
     <!-- Link conencts from body. Hip first. -->
@@ -15,5 +16,5 @@
         <origin xyz="0 0 0" rpy="0 0 0"/>
         <geometry>
-          <mesh filename="package://kuroko_description/meshes/kuroko/obj/hip_r_roll.obj"/>
+          <mesh filename="${MESH_DIR}/kuroko/obj/hip_r_roll.obj"/>
         </geometry>
       </visual>
@@ -34,5 +35,5 @@
         <origin xyz="0 0 0" rpy="0 0 0"/>
         <geometry>
-          <mesh filename="package://kuroko_description/meshes/kuroko/obj/hip_r_pitch.obj"/>
+          <mesh filename="${MESH_DIR}/kuroko/obj/hip_r_pitch.obj"/>
         </geometry>
       </visual>
@@ -53,5 +54,5 @@
         <origin xyz="0 0 0" rpy="0 0 0"/>
         <geometry>
-          <mesh filename="package://kuroko_description/meshes/kuroko/obj/thigh_r_active.obj"/>
+          <mesh filename="${MESH_DIR}/kuroko/obj/thigh_r_active.obj"/>
         </geometry>
       </visual>
@@ -71,5 +72,5 @@
         <origin xyz="0 0 0" rpy="0 0 0"/>
         <geometry>
-          <mesh filename="package://kuroko_description/meshes/kuroko/obj/shin_r_active.obj"/>
+          <mesh filename="${MESH_DIR}/kuroko/obj/shin_r_active.obj"/>
         </geometry>
       </visual>
@@ -95,5 +96,5 @@
         <origin xyz="0 0 0" rpy="0 0 0"/>
         <geometry>
-          <mesh filename="package://kuroko_description/meshes/kuroko/obj/thigh_r_middle_passive.obj"/>
+          <mesh filename="${MESH_DIR}/kuroko/obj/thigh_r_middle_passive.obj"/>
         </geometry>
       </visual>
@@ -138,5 +139,5 @@
         <origin xyz="0 0 0" rpy="0 0 0"/>
         <geometry>
-          <mesh filename="package://kuroko_description/meshes/kuroko/obj/thigh_r_rear_passive.obj"/>
+          <mesh filename="${MESH_DIR}/kuroko/obj/thigh_r_rear_passive.obj"/>
         </geometry>
       </visual>
@@ -157,5 +158,5 @@
         <origin xyz="0 0 0" rpy="0 0 0"/>
         <geometry>
-          <mesh filename="package://kuroko_description/meshes/kuroko/obj/knee_r_passive.obj"/>
+          <mesh filename="${MESH_DIR}/kuroko/obj/knee_r_passive.obj"/>
         </geometry>
       </visual>
@@ -176,5 +177,5 @@
         <origin xyz="0 0 0" rpy="0 0 0"/>
         <geometry>
-          <mesh filename="package://kuroko_description/meshes/kuroko/obj/shin_r_front_passive.obj"/>
+          <mesh filename="${MESH_DIR}/kuroko/obj/shin_r_front_passive.obj"/>
         </geometry>
       </visual>
@@ -199,5 +200,5 @@
         <origin xyz="0 0 0" rpy="0 0 0"/>
         <geometry>
-          <mesh filename="package://kuroko_description/meshes/kuroko/obj/shin_r_rear_passive.obj"/>
+          <mesh filename="${MESH_DIR}/kuroko/obj/shin_r_rear_passive.obj"/>
         </geometry>
       </visual>
@@ -218,5 +219,5 @@
         <origin xyz="0 0 0" rpy="0 0 0"/>
         <geometry>
-          <mesh filename="package://kuroko_description/meshes/kuroko/obj/ankle_r_pitch_passive.obj"/>
+          <mesh filename="${MESH_DIR}/kuroko/obj/ankle_r_pitch_passive.obj"/>
         </geometry>
       </visual>
@@ -237,5 +238,5 @@
         <origin xyz="0 0 0" rpy="0 0 0"/>
         <geometry>
-          <mesh filename="package://kuroko_description/meshes/kuroko/obj/ankle_r_roll.obj"/>
+          <mesh filename="${MESH_DIR}/kuroko/obj/ankle_r_roll.obj"/>
         </geometry>
       </visual>
@@ -256,5 +257,5 @@
         <origin xyz="0 0 0" rpy="0 0 0"/>
         <geometry>
-          <mesh filename="package://kuroko_description/meshes/kuroko/obj/ankle_r_yaw.obj"/>
+          <mesh filename="${MESH_DIR}/kuroko/obj/ankle_r_yaw.obj"/>
         </geometry>
       </visual>

Commit message: Fix path

File: kuroko_description/xacro/kuroko/kuroko.xacro (robot description, xacro)
@@ -5,5 +5,5 @@
   <xacro:arg name="gazebo_hw_interface" default="position"/>
   <xacro:property name="XACRO_DIR" value="$(find kuroko_description)/xacro" />
-  <xacro:property name="MESH_DIR" value="$(find kuroko_description)/xacro/meshes" />
+  <xacro:property name="MESH_DIR" value="package://kuroko_description/meshes" />
   <xacro:include filename="${XACRO_DIR}/physics/box_physics.xacro"/>
   <xacro:include filename="${XACRO_DIR}/physics/gazebo_passive_joint.xacro"/>

File: kuroko_description/xacro/kuroko/parts/leg_l.xacro (robot description, xacro)
@@ -45,4 +45,5 @@
       <limit effort="0" lower="-0.4974" upper="1.8588" velocity="100"/>
       <dynamics damping="0" friction="0.0"/>
+      <mimic joint="knee_l_rear" multiplier="-1" offset="0"/>
     </joint>
     <link name="thigh_l_rear_link">
@@ -63,5 +64,5 @@
       <limit effort="0" lower="-0.4974" upper="1.8588" velocity="100"/>
       <dynamics damping="0" friction="0"/>
-      <mimic joint="thigh_l_rear" multiplier="1" offset="0"/>
+      <mimic joint="knee_l_rear" multiplier="-1" offset="0"/>
     </joint>
     <link name="thigh_l_front_link">
@@ -116,11 +117,11 @@
     <link name="shin_l_front_link">
       <visual>
-        <origin xyz="0 0 0" rpy="0 0 0"/>
+        <origin xyz="0 0 0.1" rpy="0 0 0"/>
         <geometry>
           <mesh filename="${MESH_DIR}/kuroko/stl/shin_r_front_passive.stl"/>
         </geometry>
       </visual>
-      <xacro:box_collision xyz="0 0 -0.05" rpy="0 0 0" size="0.014 0.0385 0.114"/>
-      <xacro:box_inertial xyz="0 0 -0.05" rpy="0 0 0" size="0.014 0.0385 0.114" mass="0.013"/>
+      <xacro:box_collision xyz="0 0 0.05" rpy="0 0 0" size="0.014 0.0385 0.114"/>
+      <xacro:box_inertial xyz="0 0 0.05" rpy="0 0 0" size="0.014 0.0385 0.114" mass="0.013"/>
     </link>
     <xacro:if value="$(arg gazebo)">
@@ -149,5 +150,5 @@
       <parent link="ankle_l_pitch_link"/>
       <child link="shin_l_front_link"/>
-      <origin xyz="0 0 0.0335" rpy="0 0.785398163 0"/>
+      <origin xyz="0.0335 0 0" rpy="0 0.785398163 0"/>
       <axis xyz="0 1 0"/>
       <limit effort="0.0" lower="-1.8588" upper="0.4974" velocity="100.0"/>
@@ -158,5 +159,5 @@
       <parent link="ankle_l_pitch_link"/>
       <child link="ankle_l_roll_link"/>
-      <origin xyz="-0.015 0 -0.027" rpy="0 0 0"/>
+      <origin xyz="0.0185 0 -0.027" rpy="0 0 0"/>
       <axis xyz="1 0 0"/>
       <limit effort="3.1" lower="-1.5708" upper="0.3704" velocity="6.5"/>

File: kuroko_description/xacro/kuroko/parts/leg_r.xacro (robot description, xacro)
@@ -41,8 +41,9 @@
       <parent link="hip_r_pitch_link"/>
       <child link="thigh_r_rear_link"/>
-      <origin xyz="-0.0185 0.02925 -0.0305" rpy="0 -0.785398163 0"/>
+      <origin xyz="-0.0185 -0.02925 -0.0305" rpy="0 -0.785398163 0"/>
       <axis xyz="0 1 0"/>
       <limit effort="0" lower="-0.4974" upper="1.8588" velocity="100"/>
       <dynamics damping="0" friction="0.0"/>
+      <mimic joint="knee_r_rear" multiplier="-1" offset="0"/>
     </joint>
     <link name="thigh_r_rear_link">
@@ -59,9 +60,9 @@
       <parent link="hip_r_pitch_link"/>
       <child link="thigh_r_front_link"/>
-      <origin xyz="0.015 0.02925 -0.0305" rpy="0 -0.785398163 0"/>
+      <origin xyz="0.015 -0.02925 -0.0305" rpy="0 -0.785398163 0"/>
       <axis xyz="0 1 0"/>
       <limit effort="0" lower="-0.4974" upper="1.8588" velocity="100"/>
       <dynamics damping="0" friction="0"/>
-      <mimic joint="thigh_r_rear" multiplier="1" offset="0"/>
+      <mimic joint="knee_r_rear" multiplier="-1" offset="0"/>
     </joint>
     <link name="thigh_r_front_link">
@@ -116,11 +117,11 @@
     <link name="shin_r_front_link">
       <visual>
-        <origin xyz="0 0 0" rpy="0 0 0"/>
+        <origin xyz="0 0 0.1" rpy="0 0 0"/>
         <geometry>
           <mesh filename="${MESH_DIR}/kuroko/stl/shin_r_front_passive.stl"/>
         </geometry>
       </visual>
-      <xacro:box_collision xyz="0 0 -0.05" rpy="0 0 0" size="0.014 0.0385 0.114"/>
-      <xacro:box_inertial xyz="0 0 -0.05" rpy="0 0 0" size="0.014 0.0385 0.114" mass="0.013"/>
+      <xacro:box_collision xyz="0 0 0.05" rpy="0 0 0" size="0.014 0.0385 0.114"/>
+      <xacro:box_inertial xyz="0 0 0.05" rpy="0 0 0" size="0.014 0.0385 0.114" mass="0.013"/>
     </link>
     <xacro:if value="$(arg gazebo)">
@@ -149,5 +150,5 @@
       <parent link="ankle_r_pitch_link"/>
       <child link="shin_r_front_link"/>
-      <origin xyz="0 0 0.0335" rpy="0 0.785398163 0"/>
+      <origin xyz="0.0335 0 0" rpy="0 0.785398163 0"/>
       <axis xyz="0 1 0"/>
       <limit effort="0.0" lower="-1.8588" upper="0.4974" velocity="100.0"/>
@@ -158,5 +159,5 @@
       <parent link="ankle_r_pitch_link"/>
       <child link="ankle_r_roll_link"/>
-      <origin xyz="-0.015 0 -0.027" rpy="0 0 0"/>
+      <origin xyz="0.0185 0 -0.027" rpy="0 0 0"/>
       <axis xyz="1 0 0"/>
       <limit effort="3.1" lower="-1.5708" upper="0.3704" velocity="6.5"/>
