Commit message: Add box_visual option

File: kuroko_description/xacro/kuroko/kuroko.xacro (robot description, xacro)
@@ -2,4 +2,5 @@
 <robot name="kuroko" xmlns:xacro="http://www.ros.org/wiki/xacro">
   <xacro:arg name="gazebo" default="false"/>
+  <xacro:arg name="box_visual" default="false"/>
   <xacro:arg name="gazebo_motor_model" default="dc"/>
   <xacro:arg name="gazebo_hw_interface" default="position"/>
@@ -41,5 +42,5 @@
   </xacro:macro>
   <!-- MACRO:Setting up a Robot Model -->
-  <xacro:macro name="kuroko_xacro" params="gazebo gazebo_hw_interface">
+  <xacro:macro name="kuroko_xacro" params="gazebo box_visual gazebo_hw_interface">
     <link name="body_link"/>
     <joint name="root_joint" type="fixed">
@@ -48,13 +49,13 @@
       <origin xyz="0 0 0" rpy="0 0 0"/>
     </joint>
-    <xacro:body_xacro/>
+    <xacro:body_xacro box_visual="$(arg box_visual)"/>
     <xacro:body_gazebo gazebo_hw_interface="${gazebo_hw_interface}"/>
-    <xacro:arm_r_xacro/>
+    <xacro:arm_r_xacro box_visual="$(arg box_visual)"/>
     <xacro:arm_r_gazebo gazebo_hw_interface="${gazebo_hw_interface}"/>
-    <xacro:arm_l_xacro/>
+    <xacro:arm_l_xacro box_visual="$(arg box_visual)"/>
     <xacro:arm_l_gazebo gazebo_hw_interface="${gazebo_hw_interface}"/>
-    <xacro:leg_r_xacro gazebo="$(arg gazebo)"/>
+    <xacro:leg_r_xacro gazebo="$(arg gazebo)" box_visual="$(arg box_visual)"/>
     <xacro:leg_r_gazebo gazebo_hw_interface="${gazebo_hw_interface}"/>
-    <xacro:leg_l_xacro gazebo="$(arg gazebo)"/>
+    <xacro:leg_l_xacro gazebo="$(arg gazebo)" box_visual="$(arg box_visual)"/>
     <xacro:leg_l_gazebo gazebo_hw_interface="${gazebo_hw_interface}"/>
     <xacro:imu_n100mini parent="waist_link" name="imu">
@@ -69,5 +70,5 @@
   </xacro:macro>
   <!-- Load Macros -->
-  <xacro:kuroko_xacro gazebo="$(arg gazebo)"
+  <xacro:kuroko_xacro gazebo="$(arg gazebo)" box_visual="$(arg box_visual)"
     gazebo_hw_interface="$(arg gazebo_hw_interface)"/>
   <xacro:gazebo_plugin_xacro gazebo_motor_model="$(arg gazebo_motor_model)"/>

File: kuroko_description/xacro/kuroko/parts/arm_l.xacro (robot description, xacro)
@@ -1,5 +1,5 @@
 <?xml version="1.0"?>
 <robot xmlns:xacro="http://www.ros.org/wiki/xacro">
-  <xacro:macro name="arm_l_xacro">
+  <xacro:macro name="arm_l_xacro" params="box_visual:=false">
     <!-- Link conencts from body. Shoulder first. -->
     <joint name="shoulder_l_pitch" type="revolute">
@@ -12,10 +12,15 @@
     </joint>
     <link name="shoulder_l_pitch_link">
-      <visual>
-        <origin xyz="0 0 0" rpy="0 0 0"/>
-        <geometry>
-          <mesh filename="package://kuroko_description/meshes/kuroko/obj/shoulder_l_pitch.obj"/>
-        </geometry>
-      </visual>
+      <xacro:unless value="$(arg box_visual)">
+        <visual>
+          <origin xyz="0 0 0" rpy="0 0 0"/>
+          <geometry>
+            <mesh filename="package://kuroko_description/meshes/kuroko/obj/shoulder_l_pitch.obj"/>
+          </geometry>
+        </visual>
+      </xacro:unless>
+      <xacro:if value="$(arg box_visual)">
+        <xacro:box_visual xyz="-0.0096 0.0340 0.0000" rpy="0 0 0" size="0.0513 0.0680 0.0475"/>
+      </xacro:if>
       <xacro:box_collision xyz="-0.0096 0.0340 0.0000" rpy="0 0 0" size="0.0513 0.0680 0.0475"/>
       <xacro:box_inertial xyz="-0.0096 0.0340 0.0000" rpy="0 0 0" size="0.0513 0.0680 0.0475" mass="0.165"/>
@@ -30,10 +35,15 @@
     </joint>
     <link name="shoulder_l_roll_link">
-      <visual>
-        <origin xyz="0 0 0" rpy="0 0 0"/>
-        <geometry>
-          <mesh filename="package://kuroko_description/meshes/kuroko/obj/shoulder_l_roll.obj"/>
-        </geometry>
-      </visual>
+      <xacro:unless value="$(arg box_visual)">
+        <visual>
+          <origin xyz="0 0 0" rpy="0 0 0"/>
+          <geometry>
+            <mesh filename="package://kuroko_description/meshes/kuroko/obj/shoulder_l_roll.obj"/>
+          </geometry>
+        </visual>
+      </xacro:unless>
+      <xacro:if value="$(arg box_visual)">
+        <xacro:box_visual xyz="-0.0108 0.0000 -0.0186" rpy="0 0 0" size="0.0530 0.0860 0.0633"/>
+      </xacro:if>
       <xacro:box_collision xyz="-0.0108 0.0000 -0.0186" rpy="0 0 0" size="0.0530 0.0860 0.0633"/>
       <xacro:box_inertial xyz="-0.0108 0.0000 -0.0186" rpy="0 0 0" size="0.0530 0.0860 0.0633" mass="0.183"/>
@@ -48,10 +58,16 @@
     </joint>
     <link name="elbow_l_front_link">
-      <visual>
-        <origin xyz="0 0 0" rpy="0 0 0"/>
-        <geometry>
-          <mesh filename="package://kuroko_description/meshes/kuroko/obj/elbow_l_front.obj"/>
-        </geometry>
-      </visual>
+      <xacro:unless value="$(arg box_visual)">
+        <visual>
+          <origin xyz="0 0 0" rpy="0 0 0"/>
+          <geometry>
+            <mesh filename="package://kuroko_description/meshes/kuroko/obj/elbow_l_front.obj"/>
+          </geometry>
+        </visual>
+      </xacro:unless>
+      <xacro:if value="$(arg box_visual)">
+        <xacro:box_visual xyz="0.0043 0 -0.104" rpy="0 0 0" size="0.01085 0.058 0.208"/>
+        <xacro:box_visual xyz="-0.0206 0 -0.201" rpy="0 0 0" size="0.039 0.058 0.014"/>
+      </xacro:if>
       <xacro:box_collision xyz="0.0043 0 -0.104" rpy="0 0 0" size="0.01085 0.058 0.208"/>
       <xacro:box_collision xyz="-0.0206 0 -0.201" rpy="0 0 0" size="0.039 0.058 0.014"/>
@@ -67,10 +83,16 @@
     </joint>
     <link name="elbow_l_rear_link">
-      <visual>
-        <origin xyz="0 0 0" rpy="0 0 0"/>
-        <geometry>
-          <mesh filename="package://kuroko_description/meshes/kuroko/obj/elbow_l_rear.obj"/>
-        </geometry>
-      </visual>
+      <xacro:unless value="$(arg box_visual)">
+        <visual>
+          <origin xyz="0 0 0" rpy="0 0 0"/>
+          <geometry>
+            <mesh filename="package://kuroko_description/meshes/kuroko/obj/elbow_l_rear.obj"/>
+          </geometry>
+        </visual>
+      </xacro:unless>
+      <xacro:if value="$(arg box_visual)">
+        <xacro:box_visual xyz="-0.0043 0 -0.1" rpy="0 0 0" size="0.01085 0.044 0.2"/>
+        <xacro:box_visual xyz="0.0206 0 -0.193" rpy="0 0 0" size="0.039 0.044 0.014"/>
+      </xacro:if>
       <xacro:box_collision xyz="-0.0043 0 -0.1" rpy="0 0 0" size="0.01085 0.044 0.2"/>
       <xacro:box_collision xyz="0.0206 0 -0.193" rpy="0 0 0" size="0.039 0.044 0.014"/>

File: kuroko_description/xacro/kuroko/parts/arm_r.xacro (robot description, xacro)
@@ -1,5 +1,5 @@
 <?xml version="1.0"?>
 <robot xmlns:xacro="http://www.ros.org/wiki/xacro">
-  <xacro:macro name="arm_r_xacro">
+  <xacro:macro name="arm_r_xacro" params="box_visual:=false">
     <!-- Link conencts from body. Shoulder first. -->
     <joint name="shoulder_r_pitch" type="revolute">
@@ -12,10 +12,15 @@
     </joint>
     <link name="shoulder_r_pitch_link">
-      <visual>
-        <origin xyz="0 0 0" rpy="0 0 0"/>
-        <geometry>
-          <mesh filename="package://kuroko_description/meshes/kuroko/obj/shoulder_r_pitch.obj"/>
-        </geometry>
-      </visual>
+      <xacro:unless value="$(arg box_visual)">
+        <visual>
+          <origin xyz="0 0 0" rpy="0 0 0"/>
+          <geometry>
+            <mesh filename="package://kuroko_description/meshes/kuroko/obj/shoulder_r_pitch.obj"/>
+          </geometry>
+        </visual>
+      </xacro:unless>
+      <xacro:if value="$(arg box_visual)">
+        <xacro:box_visual xyz="-0.0096 -0.0340 0.0000" rpy="0 0 0" size="0.0513 0.0680 0.0475"/>
+      </xacro:if>
       <xacro:box_collision xyz="-0.0096 -0.0340 0.0000" rpy="0 0 0" size="0.0513 0.0680 0.0475"/>
       <xacro:box_inertial xyz="-0.0096 -0.0340 0.0000" rpy="0 0 0" size="0.0513 0.0680 0.0475" mass="0.165"/>
@@ -30,10 +35,15 @@
     </joint>
     <link name="shoulder_r_roll_link">
-      <visual>
-        <origin xyz="0 0 0" rpy="0 0 0"/>
-        <geometry>
-          <mesh filename="package://kuroko_description/meshes/kuroko/obj/shoulder_r_roll.obj"/>
-        </geometry>
-      </visual>
+      <xacro:unless value="$(arg box_visual)">
+        <visual>
+          <origin xyz="0 0 0" rpy="0 0 0"/>
+          <geometry>
+            <mesh filename="package://kuroko_description/meshes/kuroko/obj/shoulder_r_roll.obj"/>
+          </geometry>
+        </visual>
+      </xacro:unless>
+      <xacro:if value="$(arg box_visual)">
+        <xacro:box_visual xyz="-0.0108 0.0000 -0.0186" rpy="0 0 0" size="0.0530 0.0860 0.0633"/>
+      </xacro:if>
       <xacro:box_collision xyz="-0.0108 0.0000 -0.0186" rpy="0 0 0" size="0.0530 0.0860 0.0633"/>
       <xacro:box_inertial xyz="-0.0108 0.0000 -0.0186" rpy="0 0 0" size="0.0530 0.0860 0.0633" mass="0.183"/>
@@ -48,10 +58,16 @@
     </joint>
     <link name="elbow_r_front_link">
-      <visual>
-        <origin xyz="0 0 0" rpy="0 0 0"/>
-        <geometry>
-          <mesh filename="package://kuroko_description/meshes/kuroko/obj/elbow_r_front.obj"/>
-        </geometry>
-      </visual>
+      <xacro:unless value="$(arg box_visual)">
+        <visual>
+          <origin xyz="0 0 0" rpy="0 0 0"/>
+          <geometry>
+            <mesh filename="package://kuroko_description/meshes/kuroko/obj/elbow_r_front.obj"/>
+          </geometry>
+        </visual>
+      </xacro:unless>
+      <xacro:if value="$(arg box_visual)">
+        <xacro:box_visual xyz="0.0043 0 -0.104" rpy="0 0 0" size="0.01085 0.058 0.208"/>
+        <xacro:box_visual xyz="-0.0206 0 -0.201" rpy="0 0 0" size="0.039 0.058 0.014"/>
+      </xacro:if>
       <xacro:box_collision xyz="0.0043 0 -0.104" rpy="0 0 0" size="0.01085 0.058 0.208"/>
       <xacro:box_collision xyz="-0.0206 0 -0.201" rpy="0 0 0" size="0.039 0.058 0.014"/>
@@ -67,10 +83,16 @@
     </joint>
     <link name="elbow_r_rear_link">
-      <visual>
-        <origin xyz="0 0 0" rpy="0 0 0"/>
-        <geometry>
-          <mesh filename="package://kuroko_description/meshes/kuroko/obj/elbow_r_rear.obj"/>
-        </geometry>
-      </visual>
+      <xacro:unless value="$(arg box_visual)">
+        <visual>
+          <origin xyz="0 0 0" rpy="0 0 0"/>
+          <geometry>
+            <mesh filename="package://kuroko_description/meshes/kuroko/obj/elbow_r_rear.obj"/>
+          </geometry>
+        </visual>
+      </xacro:unless>
+      <xacro:if value="$(arg box_visual)">
+        <xacro:box_visual xyz="-0.0043 0 -0.1" rpy="0 0 0" size="0.01085 0.044 0.2"/>
+        <xacro:box_visual xyz="0.0206 0 -0.193" rpy="0 0 0" size="0.039 0.044 0.014"/>
+      </xacro:if>
       <xacro:box_collision xyz="-0.0043 0 -0.1" rpy="0 0 0" size="0.01085 0.044 0.2"/>
       <xacro:box_collision xyz="0.0206 0 -0.193" rpy="0 0 0" size="0.039 0.044 0.014"/>

File: kuroko_description/xacro/kuroko/parts/body.xacro (robot description, xacro)
@@ -1,13 +1,18 @@
 <?xml version="1.0"?>
 <robot xmlns:xacro="http://www.ros.org/wiki/xacro">
-  <xacro:macro name="body_xacro">
+  <xacro:macro name="body_xacro" params="box_visual:=false">
     <!-- waist -->
     <link name="waist_link">
-      <visual>
-        <origin xyz="0 0 0" rpy="0 0 0"/>
-        <geometry>
-          <mesh filename="package://kuroko_description/meshes/kuroko/obj/waist.obj"/>
-        </geometry>
-      </visual>
+      <xacro:unless value="$(arg box_visual)">
+        <visual>
+          <origin xyz="0 0 0" rpy="0 0 0"/>
+          <geometry>
+            <mesh filename="package://kuroko_description/meshes/kuroko/obj/waist.obj"/>
+          </geometry>
+        </visual>
+      </xacro:unless>
+      <xacro:if value="$(arg box_visual)">
+        <xacro:box_visual xyz="0.0084 0.0000 -0.0483" rpy="0 0 0" size="0.1247 0.0560 0.0965"/>
+      </xacro:if>
       <xacro:box_collision xyz="0.0084 0.0000 -0.0483" rpy="0 0 0" size="0.1247 0.0560 0.0965"/>
       <xacro:box_inertial xyz="0.0084 0.0000 -0.0483" rpy="0 0 0" size="0.1247 0.0560 0.0965" mass="0.388"/>
@@ -24,10 +29,15 @@
     <!-- chest -->
     <link name="chest_link">
-      <visual>
-        <origin xyz="0 0 0" rpy="0 0 0"/>
-        <geometry>
-          <mesh filename="package://kuroko_description/meshes/kuroko/obj/chest.obj"/>
-        </geometry>
-      </visual>
+      <xacro:unless value="$(arg box_visual)">
+        <visual>
+          <origin xyz="0 0 0" rpy="0 0 0"/>
+          <geometry>
+            <mesh filename="package://kuroko_description/meshes/kuroko/obj/chest.obj"/>
+          </geometry>
+        </visual>
+      </xacro:unless>
+      <xacro:if value="$(arg box_visual)">
+        <xacro:box_visual xyz="0.0120 0.0000 0.0635" rpy="0 0 0" size="0.1480 0.2560 0.1364"/>
+      </xacro:if>
       <xacro:box_collision xyz="0.0120 0.0000 0.0635" rpy="0 0 0" size="0.1480 0.2560 0.1364"/>
       <xacro:box_inertial xyz="0.0120 0.0000 0.0635" rpy="0 0 0" size="0.1480 0.2560 0.1364" mass="0.806"/>
