Commit message: Add XACRO_DIR and MESH_DIR

File: kuroko_description/xacro/kuroko/kuroko.xacro (robot description, xacro)
@@ -5,19 +5,21 @@
   <xacro:arg name="gazebo_motor_model" default="dc"/>
   <xacro:arg name="gazebo_hw_interface" default="position"/>
-  <xacro:include filename="$(find kuroko_description)/xacro/physics/box_physics.xacro"/>
-  <xacro:include filename="$(find kuroko_description)/xacro/physics/gazebo_passive_joint.xacro"/>
-  <xacro:include filename="$(find kuroko_description)/xacro/kuroko/parts/body.xacro"/>
-  <xacro:include filename="$(find kuroko_description)/xacro/kuroko/transmission/body.gazebo"/>
-  <xacro:include filename="$(find kuroko_description)/xacro/kuroko/parts/arm_r.xacro"/>
-  <xacro:include filename="$(find kuroko_description)/xacro/kuroko/transmission/arm_r.gazebo"/>
-  <xacro:include filename="$(find kuroko_description)/xacro/kuroko/parts/arm_l.xacro"/>
-  <xacro:include filename="$(find kuroko_description)/xacro/kuroko/transmission/arm_l.gazebo"/>
-  <xacro:include filename="$(find kuroko_description)/xacro/kuroko/parts/leg_r.xacro"/>
-  <xacro:include filename="$(find kuroko_description)/xacro/kuroko/transmission/leg_r.gazebo"/>
-  <xacro:include filename="$(find kuroko_description)/xacro/kuroko/parts/leg_l.xacro"/>
-  <xacro:include filename="$(find kuroko_description)/xacro/kuroko/transmission/leg_l.gazebo"/>
-  <xacro:include filename="$(find kuroko_description)/xacro/sensors/range/tfluna.xacro"/>
-  <xacro:include filename="$(find kuroko_description)/xacro/sensors/imu/imu_n100mini.xacro"/>
-  <xacro:include filename="$(find kuroko_description)/xacro/sensors/camera/usb_camera.xacro"/>
+  <xacro:property name="XACRO_DIR" value="$(find kuroko_description)/xacro" />
+  <xacro:property name="MESH_DIR" value="package://kuroko_description/meshes" />
+  <xacro:include filename="${XACRO_DIR}/physics/box_physics.xacro"/>
+  <xacro:include filename="${XACRO_DIR}/physics/gazebo_passive_joint.xacro"/>
+  <xacro:include filename="${XACRO_DIR}/kuroko/parts/body.xacro"/>
+  <xacro:include filename="${XACRO_DIR}/kuroko/transmission/body.gazebo"/>
+  <xacro:include filename="${XACRO_DIR}/kuroko/parts/arm_r.xacro"/>
+  <xacro:include filename="${XACRO_DIR}/kuroko/transmission/arm_r.gazebo"/>
+  <xacro:include filename="${XACRO_DIR}/kuroko/parts/arm_l.xacro"/>
+  <xacro:include filename="${XACRO_DIR}/kuroko/transmission/arm_l.gazebo"/>
+  <xacro:include filename="${XACRO_DIR}/kuroko/parts/leg_r.xacro"/>
+  <xacro:include filename="${XACRO_DIR}/kuroko/transmission/leg_r.gazebo"/>
+  <xacro:include filename="${XACRO_DIR}/kuroko/parts/leg_l.xacro"/>
+  <xacro:include filename="${XACRO_DIR}/kuroko/transmission/leg_l.gazebo"/>
+  <xacro:include filename="${XACRO_DIR}/sensors/range/tfluna.xacro"/>
+  <xacro:include filename="${XACRO_DIR}/sensors/imu/imu_n100mini.xacro"/>
+  <xacro:include filename="${XACRO_DIR}/sensors/camera/usb_camera.xacro"/>
   <!-- MACRO:Loading Gazebo Controllers for joints -->
   <xacro:macro name="gazebo_plugin_xacro" params="gazebo_motor_model">

File: kuroko_description/xacro/kuroko/parts/arm_l.xacro (robot description, xacro)
@@ -16,5 +16,5 @@
           <origin xyz="0 0 0" rpy="0 0 0"/>
           <geometry>
-            <mesh filename="package://kuroko_description/meshes/kuroko/obj/shoulder_l_pitch.obj"/>
+            <mesh filename="${MESH_DIR}/kuroko/obj/shoulder_l_pitch.obj"/>
           </geometry>
         </visual>
@@ -39,5 +39,5 @@
           <origin xyz="0 0 0" rpy="0 0 0"/>
           <geometry>
-            <mesh filename="package://kuroko_description/meshes/kuroko/obj/shoulder_l_roll.obj"/>
+            <mesh filename="${MESH_DIR}/kuroko/obj/shoulder_l_roll.obj"/>
           </geometry>
         </visual>
@@ -62,5 +62,5 @@
           <origin xyz="0 0 0" rpy="0 0 0"/>
           <geometry>
-            <mesh filename="package://kuroko_description/meshes/kuroko/obj/elbow_l_front.obj"/>
+            <mesh filename="${MESH_DIR}/kuroko/obj/elbow_l_front.obj"/>
           </geometry>
         </visual>
@@ -87,5 +87,5 @@
           <origin xyz="0 0 0" rpy="0 0 0"/>
           <geometry>
-            <mesh filename="package://kuroko_description/meshes/kuroko/obj/elbow_l_rear.obj"/>
+            <mesh filename="${MESH_DIR}/kuroko/obj/elbow_l_rear.obj"/>
           </geometry>
         </visual>

File: kuroko_description/xacro/kuroko/parts/arm_r.xacro (robot description, xacro)
@@ -16,5 +16,5 @@
           <origin xyz="0 0 0" rpy="0 0 0"/>
           <geometry>
-            <mesh filename="package://kuroko_description/meshes/kuroko/obj/shoulder_r_pitch.obj"/>
+            <mesh filename="${MESH_DIR}/kuroko/obj/shoulder_r_pitch.obj"/>
           </geometry>
         </visual>
@@ -39,5 +39,5 @@
           <origin xyz="0 0 0" rpy="0 0 0"/>
           <geometry>
-            <mesh filename="package://kuroko_description/meshes/kuroko/obj/shoulder_r_roll.obj"/>
+            <mesh filename="${MESH_DIR}/kuroko/obj/shoulder_r_roll.obj"/>
           </geometry>
         </visual>
@@ -62,5 +62,5 @@
           <origin xyz="0 0 0" rpy="0 0 0"/>
           <geometry>
-            <mesh filename="package://kuroko_description/meshes/kuroko/obj/elbow_r_front.obj"/>
+            <mesh filename="${MESH_DIR}/kuroko/obj/elbow_r_front.obj"/>
           </geometry>
         </visual>
@@ -87,5 +87,5 @@
           <origin xyz="0 0 0" rpy="0 0 0"/>
           <geometry>
-            <mesh filename="package://kuroko_description/meshes/kuroko/obj/elbow_r_rear.obj"/>
+            <mesh filename="${MESH_DIR}/kuroko/obj/elbow_r_rear.obj"/>
           </geometry>
         </visual>

File: kuroko_description/xacro/kuroko/parts/body.xacro (robot description, xacro)
@@ -8,5 +8,5 @@
           <origin xyz="0 0 0" rpy="0 0 0"/>
           <geometry>
-            <mesh filename="package://kuroko_description/meshes/kuroko/obj/waist.obj"/>
+            <mesh filename="${MESH_DIR}/kuroko/obj/waist.obj"/>
           </geometry>
         </visual>
@@ -33,5 +33,5 @@
           <origin xyz="0 0 0" rpy="0 0 0"/>
           <geometry>
-            <mesh filename="package://kuroko_description/meshes/kuroko/obj/chest.obj"/>
+            <mesh filename="${MESH_DIR}/kuroko/obj/chest.obj"/>
           </geometry>
         </visual>

File: kuroko_description/xacro/kuroko/parts/leg_l.xacro (robot description, xacro)
@@ -16,5 +16,5 @@
           <origin xyz="0 0 0" rpy="0 0 0"/>
           <geometry>
-            <mesh filename="package://kuroko_description/meshes/kuroko/obj/hip_l_roll.obj"/>
+            <mesh filename="${MESH_DIR}/kuroko/obj/hip_l_roll.obj"/>
           </geometry>
         </visual>
@@ -40,5 +40,5 @@
           <origin xyz="0 0 0" rpy="0 0 0"/>
           <geometry>
-            <mesh filename="package://kuroko_description/meshes/kuroko/obj/hip_l_pitch.obj"/>
+            <mesh filename="${MESH_DIR}/kuroko/obj/hip_l_pitch.obj"/>
           </geometry>
         </visual>
@@ -64,5 +64,5 @@
           <origin xyz="0 0 0" rpy="0 0 0"/>
           <geometry>
-            <mesh filename="package://kuroko_description/meshes/kuroko/obj/shin_l_active.obj"/>
+            <mesh filename="${MESH_DIR}/kuroko/obj/shin_l_active.obj"/>
           </geometry>
         </visual>
@@ -88,5 +88,5 @@
           <origin xyz="0 0 0" rpy="0 0 0"/>
           <geometry>
-            <mesh filename="package://kuroko_description/meshes/kuroko/obj/thigh_l_active.obj"/>
+            <mesh filename="${MESH_DIR}/kuroko/obj/thigh_l_active.obj"/>
           </geometry>
         </visual>
@@ -158,5 +158,5 @@
           <origin xyz="0 0 0" rpy="0 0 0"/>
           <geometry>
-            <mesh filename="package://kuroko_description/meshes/kuroko/obj/thigh_r_middle_passive.obj"/>
+            <mesh filename="${MESH_DIR}/kuroko/obj/thigh_r_middle_passive.obj"/>
           </geometry>
         </visual>
@@ -204,5 +204,5 @@
           <origin xyz="0 0 0" rpy="0 0 0"/>
           <geometry>
-            <mesh filename="package://kuroko_description/meshes/kuroko/obj/shin_r_rear_passive.obj"/>
+            <mesh filename="${MESH_DIR}/kuroko/obj/shin_r_rear_passive.obj"/>
           </geometry>
         </visual>
@@ -228,5 +228,5 @@
           <origin xyz="0.0335 0 0" rpy="0 0 0"/>
           <geometry>
-            <mesh filename="package://kuroko_description/meshes/kuroko/obj/knee_r_passive.obj"/>
+            <mesh filename="${MESH_DIR}/kuroko/obj/knee_r_passive.obj"/>
           </geometry>
         </visual>
@@ -278,5 +278,5 @@
           <origin xyz="0 0 0.1" rpy="0 0 0"/>
           <geometry>
-            <mesh filename="package://kuroko_description/meshes/kuroko/obj/thigh_r_rear_passive.obj"/>
+            <mesh filename="${MESH_DIR}/kuroko/obj/thigh_r_rear_passive.obj"/>
           </geometry>
         </visual>
@@ -306,5 +306,5 @@
           <origin xyz="0.0335 0 0" rpy="0 0 0"/>
           <geometry>
-            <mesh filename="package://kuroko_description/meshes/kuroko/obj/ankle_r_pitch_passive.obj"/>
+            <mesh filename="${MESH_DIR}/kuroko/obj/ankle_r_pitch_passive.obj"/>
           </geometry>
         </visual>
@@ -333,5 +333,5 @@
           <origin xyz="0 0 0" rpy="0 0 0"/>
           <geometry>
-            <mesh filename="package://kuroko_description/meshes/kuroko/obj/ankle_l_roll.obj"/>
+            <mesh filename="${MESH_DIR}/kuroko/obj/ankle_l_roll.obj"/>
           </geometry>
         </visual>
@@ -357,5 +357,5 @@
           <origin xyz="0 0 0" rpy="0 0 0"/>
           <geometry>
-            <mesh filename="package://kuroko_description/meshes/kuroko/obj/ankle_r_yaw.obj"/>
+            <mesh filename="${MESH_DIR}/kuroko/obj/ankle_r_yaw.obj"/>
           </geometry>
         </visual>

File: kuroko_description/xacro/kuroko/parts/leg_r.xacro (robot description, xacro)
@@ -16,5 +16,5 @@
           <origin xyz="0 0 0" rpy="0 0 0"/>
           <geometry>
-            <mesh filename="package://kuroko_description/meshes/kuroko/obj/hip_r_roll.obj"/>
+            <mesh filename="${MESH_DIR}/kuroko/obj/hip_r_roll.obj"/>
           </geometry>
         </visual>
@@ -40,5 +40,5 @@
           <origin xyz="0 0 0" rpy="0 0 0"/>
           <geometry>
-            <mesh filename="package://kuroko_description/meshes/kuroko/obj/hip_r_pitch.obj"/>
+            <mesh filename="${MESH_DIR}/kuroko/obj/hip_r_pitch.obj"/>
           </geometry>
         </visual>
@@ -64,5 +64,5 @@
           <origin xyz="0 0 0" rpy="0 0 0"/>
           <geometry>
-            <mesh filename="package://kuroko_description/meshes/kuroko/obj/shin_r_active.obj"/>
+            <mesh filename="${MESH_DIR}/kuroko/obj/shin_r_active.obj"/>
           </geometry>
         </visual>
@@ -88,5 +88,5 @@
           <origin xyz="0 0 0" rpy="0 0 0"/>
           <geometry>
-            <mesh filename="package://kuroko_description/meshes/kuroko/obj/thigh_r_active.obj"/>
+            <mesh filename="${MESH_DIR}/kuroko/obj/thigh_r_active.obj"/>
           </geometry>
         </visual>
@@ -134,5 +134,5 @@
           <origin xyz="0 0 0" rpy="0 0 0"/>
           <geometry>
-            <mesh filename="package://kuroko_description/meshes/kuroko/obj/shin_r_front_passive.obj"/>
+            <mesh filename="${MESH_DIR}/kuroko/obj/shin_r_front_passive.obj"/>
           </geometry>
         </visual>
@@ -158,5 +158,5 @@
           <origin xyz="0 0 0" rpy="0 0 0"/>
           <geometry>
-            <mesh filename="package://kuroko_description/meshes/kuroko/obj/thigh_r_middle_passive.obj"/>
+            <mesh filename="${MESH_DIR}/kuroko/obj/thigh_r_middle_passive.obj"/>
           </geometry>
         </visual>
@@ -204,5 +204,5 @@
           <origin xyz="0 0 0" rpy="0 0 0"/>
           <geometry>
-            <mesh filename="package://kuroko_description/meshes/kuroko/obj/shin_r_rear_passive.obj"/>
+            <mesh filename="${MESH_DIR}/kuroko/obj/shin_r_rear_passive.obj"/>
           </geometry>
         </visual>
@@ -228,5 +228,5 @@
           <origin xyz="0.0335 0 0" rpy="0 0 0"/>
           <geometry>
-            <mesh filename="package://kuroko_description/meshes/kuroko/obj/knee_r_passive.obj"/>
+            <mesh filename="${MESH_DIR}/kuroko/obj/knee_r_passive.obj"/>
           </geometry>
         </visual>
@@ -278,5 +278,5 @@
           <origin xyz="0 0 0.1" rpy="0 0 0"/>
           <geometry>
-            <mesh filename="package://kuroko_description/meshes/kuroko/obj/thigh_r_rear_passive.obj"/>
+            <mesh filename="${MESH_DIR}/kuroko/obj/thigh_r_rear_passive.obj"/>
           </geometry>
         </visual>
@@ -306,5 +306,5 @@
           <origin xyz="0.0335 0 0" rpy="0 0 0"/>
           <geometry>
-            <mesh filename="package://kuroko_description/meshes/kuroko/obj/ankle_r_pitch_passive.obj"/>
+            <mesh filename="${MESH_DIR}/kuroko/obj/ankle_r_pitch_passive.obj"/>
           </geometry>
         </visual>
@@ -334,5 +334,5 @@
           <origin xyz="0 0 0" rpy="0 0 0"/>
           <geometry>
-            <mesh filename="package://kuroko_description/meshes/kuroko/obj/ankle_r_roll.obj"/>
+            <mesh filename="${MESH_DIR}/kuroko/obj/ankle_r_roll.obj"/>
           </geometry>
         </visual>
@@ -358,5 +358,5 @@
           <origin xyz="0 0 0" rpy="0 0 0"/>
           <geometry>
-            <mesh filename="package://kuroko_description/meshes/kuroko/obj/ankle_r_yaw.obj"/>
+            <mesh filename="${MESH_DIR}/kuroko/obj/ankle_r_yaw.obj"/>
           </geometry>
         </visual>
