Commit message: Use range sensor

File: kuroko_description/xacro/sensors/range/tfluna_gazebo.xacro (robot description, xacro)
@@ -1,5 +1,5 @@
 <?xml version="1.0" encoding="UTF-8"?>
 <robot xmlns:xacro="http://www.ros.org/wiki/xacro">
-  <xacro:macro name="tfluna_gazebo" params="name ros_topic update_rate:=10 maxRange:=8.0 minRange:=0.2 fov:=0.03 ray_count:=5">
+  <xacro:macro name="tfluna_gazebo" params="name ros_topic update_rate:=10 maxRange:=8.0 minRange:=0.0 fov:=0.03 ray_count:=5">
     <gazebo reference="${name}_link">
       <sensor type="ray" name="${name}">
