Commit message: (WIP) Update damping

File: kuroko_description/xacro/export/kuroko.urdf (robot description, URDF)
Before this commit: robot kuroko, 42 links, 41 joints
Joints:
- joint chest: limit lower=-3.1 upper=3.1 effort=1000.0 velocity=10.0 -> lower=-3.1 upper=3.1 effort=3.1 velocity=6.5
- joint elbow_l_front: limit lower=-2.6180 upper=2.6180 effort=1000.0 velocity=10.0 -> lower=-2.6180 upper=2.6180 effort=3.1 velocity=6.5
- joint elbow_l_rear: limit lower=-2.6180 upper=2.6180 effort=1000.0 velocity=10.0 -> lower=-2.6180 upper=2.6180 effort=3.1 velocity=6.5
- joint elbow_r_front: limit lower=-2.6180 upper=2.6180 effort=1000.0 velocity=10.0 -> lower=-2.6180 upper=2.6180 effort=3.1 velocity=6.6
- joint elbow_r_rear: limit lower=-2.6180 upper=2.6180 effort=1000.0 velocity=10.0 -> lower=-2.6180 upper=2.6180 effort=3.1 velocity=6.5
- joint shoulder_l_pitch: limit lower=-3.1 upper=3.1 effort=1000.0 velocity=10.0 -> lower=-3.1 upper=3.1 effort=3.1 velocity=6.5
- joint shoulder_l_roll: limit lower=-3.1 upper=3.1 effort=1000.0 velocity=10.0 -> lower=-3.1 upper=3.1 effort=8.9 velocity=6.9
- joint shoulder_r_pitch: limit lower=-3.1 upper=3.1 effort=1000.0 velocity=10.0 -> lower=-3.1 upper=3.1 effort=3.1 velocity=6.5
- joint shoulder_r_roll: limit lower=-3.1 upper=3.1 effort=1000.0 velocity=10.0 -> lower=-3.1 upper=3.1 effort=8.9 velocity=6.9

File: kuroko_description/xacro/kuroko/parts/arm_l.xacro (robot description, xacro)
@@ -8,6 +8,6 @@
       <origin xyz="0 0.128 0.01275" rpy="0 0 0"/>
       <axis xyz="0 1 0"/>
-      <limit effort="1000.0" lower="-3.1" upper="3.1" velocity="10.0"/>
-      <dynamics damping="0.0" friction="0.0"/>
+      <limit effort="3.1" lower="-3.1" upper="3.1" velocity="6.5"/>
+      <dynamics damping="0.4769" friction="0.0"/>
     </joint>
     <link name="shoulder_l_pitch_link">
@@ -26,6 +26,6 @@
       <origin xyz="0 0.05425 0" rpy="1.5708 0 0"/>
       <axis xyz="1 0 0"/>
-      <limit effort="1000.0" lower="-3.1" upper="3.1" velocity="10.0"/>
-      <dynamics damping="0.0" friction="0.0"/>
+      <limit effort="8.9" lower="-3.1" upper="3.1" velocity="6.9"/>
+      <dynamics damping="1.290" friction="0.0"/>
     </joint>
     <link name="shoulder_l_roll_link">
@@ -44,6 +44,6 @@
       <origin xyz="0 -0.023 -0.036" rpy="0 0 0"/>
       <axis xyz="0 -1 0"/>
-      <limit effort="1000.0" lower="-2.6180" upper="2.6180" velocity="10.0"/>
-      <dynamics damping="0.0" friction="0.0"/>
+      <limit effort="3.1" lower="-2.6180" upper="2.6180" velocity="6.5"/>
+      <dynamics damping="0.4769" friction="0.0"/>
     </joint>
     <link name="elbow_l_front_link">
@@ -63,6 +63,6 @@
       <origin xyz="0 -0.024 -0.036" rpy="0 0 0"/>
       <axis xyz="0 1 0"/>
-      <limit effort="1000.0" lower="-2.6180" upper="2.6180" velocity="10.0"/>
-      <dynamics damping="0.0" friction="0.0"/>
+      <limit effort="3.1" lower="-2.6180" upper="2.6180" velocity="6.5"/>
+      <dynamics damping="0.4769" friction="0.0"/>
     </joint>
     <link name="elbow_l_rear_link">

File: kuroko_description/xacro/kuroko/parts/arm_r.xacro (robot description, xacro)
@@ -8,6 +8,6 @@
       <origin xyz="0 -0.128 0.01275" rpy="0 0 0"/>
       <axis xyz="0 -1 0"/>
-      <limit effort="1000.0" lower="-3.1" upper="3.1" velocity="10.0"/>
-      <dynamics damping="0.0" friction="0.0"/>
+      <limit effort="3.1" lower="-3.1" upper="3.1" velocity="6.5"/>
+      <dynamics damping="0.4769" friction="0.0"/>
     </joint>
     <link name="shoulder_r_pitch_link">
@@ -26,6 +26,6 @@
       <origin xyz="0 -0.05425 0" rpy="-1.5708 0 0"/>
       <axis xyz="1 0 0"/>
-      <limit effort="1000.0" lower="-3.1" upper="3.1" velocity="10.0"/>
-      <dynamics damping="0.0" friction="0.0"/>
+      <limit effort="8.9" lower="-3.1" upper="3.1" velocity="6.9"/>
+      <dynamics damping="1.290" friction="0.0"/>
     </joint>
     <link name="shoulder_r_roll_link">
@@ -44,6 +44,6 @@
       <origin xyz="0 0.023 -0.036" rpy="0 0 0"/>
       <axis xyz="0 1 0"/>
-      <limit effort="1000.0" lower="-2.6180" upper="2.6180" velocity="10.0"/>
-      <dynamics damping="0.0" friction="0.0"/>
+      <limit effort="3.1" lower="-2.6180" upper="2.6180" velocity="6.6"/>
+      <dynamics damping="0.4769" friction="0.0"/>
     </joint>
     <link name="elbow_r_front_link">
@@ -63,6 +63,6 @@
       <origin xyz="0 0.024 -0.036" rpy="0 0 0"/>
       <axis xyz="0 -1 0"/>
-      <limit effort="1000.0" lower="-2.6180" upper="2.6180" velocity="10.0"/>
-      <dynamics damping="0.0" friction="0.0"/>
+      <limit effort="3.1" lower="-2.6180" upper="2.6180" velocity="6.5"/>
+      <dynamics damping="0.4769" friction="0.0"/>
     </joint>
     <link name="elbow_r_rear_link">

File: kuroko_description/xacro/kuroko/parts/body.xacro (robot description, xacro)
@@ -19,6 +19,6 @@
       <origin xyz="0 0 0" rpy="0 0 0"/>
       <axis xyz="0 0 1"/>
-      <limit effort="1000.0" lower="-3.1" upper="3.1" velocity="10.0"/>
-      <dynamics damping="0.0" friction="0.0"/>
+      <limit effort="3.1" lower="-3.1" upper="3.1" velocity="6.5"/>
+      <dynamics damping="0.4769" friction="0.0"/>
     </joint>
     <!-- chest -->

File: kuroko_description/xacro/kuroko/parts/leg_l.xacro (robot description, xacro)
@@ -8,6 +8,6 @@
       <origin xyz="0 0 -0.08425" rpy="0 0 0"/>
       <axis xyz="-1 0 0"/>
-      <limit effort="1000.0" lower="-0.5550" upper="1.8640" velocity="10.0"/>
-      <dynamics damping="0.0" friction="0.0"/>
+      <limit effort="3.1" lower="-0.5550" upper="1.8640" velocity="6.5"/>
+      <dynamics damping="0.4796" friction="0.0"/>
     </joint>
     <link name="hip_l_roll_link">
@@ -27,6 +27,6 @@
       <origin xyz="0 0.027 0" rpy="0 0 0"/>
       <axis xyz="0 1 0"/>
-      <limit effort="1000.0" lower="-3.1" upper="3.1" velocity="10.0"/>
-      <dynamics damping="0.0" friction="0.0"/>
+      <limit effort="3.1" lower="-3.1" upper="3.1" velocity="6.9"/>
+      <dynamics damping="1.290" friction="0.0"/>
     </joint>
     <link name="hip_l_pitch_link">
@@ -46,6 +46,6 @@
       <origin xyz="0.015 0.02925 -0.0305" rpy="0 -0.785398163 0"/>
       <axis xyz="0 -1 0"/>
-      <limit effort="1000.0" lower="-1.8588" upper="0.4974" velocity="10.0"/>
-      <dynamics damping="0.0" friction="0.0"/>
+      <limit effort="8.9" lower="-1.8588" upper="0.4974" velocity="6.9"/>
+      <dynamics damping="1.290" friction="0.0"/>
     </joint>
     <link name="thigh_l_active_link">
@@ -64,6 +64,6 @@
       <origin xyz="-0.0185 0.02925 -0.0305" rpy="0 1.047197551 0"/>
       <axis xyz="0 -1 0"/>
-      <limit effort="1000.0" lower="-0.4974" upper="1.8588" velocity="10.0"/>
-      <dynamics damping="0.0" friction="0.0"/>
+      <limit effort="8.9" lower="-0.4974" upper="1.8588" velocity="6.9"/>
+      <dynamics damping="1.290" friction="0.0"/>
     </joint>
     <link name="shin_l_active_link">
@@ -83,5 +83,5 @@
       <origin xyz="-0.0185 0.02925 -0.0305" rpy="0 -0.785398163 0"/>
       <axis xyz="0 -1 0"/>
-      <limit effort="1000.0" lower="-3.1" upper="3.1" velocity="10.0"/>
+      <limit effort="0.0" lower="-3.1" upper="3.1" velocity="10.0"/>
       <dynamics damping="0.0" friction="0.0"/>
       <mimic joint="thigh_l_active" multiplier="1" offset="0"/>
@@ -107,5 +107,5 @@
         <origin xyz="0 0 -0.03" rpy="0 -1.832597551 0"/>
         <axis xyz="0 -1 0"/>
-        <limit effort="1000.0" lower="-3.1" upper="3.1" velocity="10.0"/>
+        <limit effort="0.0" lower="-3.1" upper="3.1" velocity="100.0"/>
         <dynamics damping="0.0" friction="0.0"/>
         <mimic joint="shin_l_active" multiplier="-1" offset="0"/>
@@ -117,5 +117,5 @@
         <origin xyz="0 0 0" rpy="0 0 0"/>
         <axis xyz="0 -1 0"/>
-        <limit effort="1000.0" lower="-3.1" upper="3.1" velocity="10.0"/>
+        <limit effort="0.0" lower="-3.1" upper="3.1" velocity="100.0"/>
         <dynamics damping="0.0" friction="0.0"/>
         <mimic joint="thigh_l_active" multiplier="1" offset="0"/>
@@ -128,5 +128,5 @@
         <origin xyz="0 0 -0.03" rpy="0 -1.832597551 0"/>
         <axis xyz="0 -1 0"/>
-        <limit effort="1000.0" lower="-1.5708" upper="0.9948" velocity="10.0"/>
+        <limit effort="0.0" lower="-1.5708" upper="0.9948" velocity="100.0"/>
         <dynamics damping="0.0" friction="0.0"/>
       </joint>
@@ -149,5 +149,5 @@
       <origin xyz="0 0 -0.1" rpy="0 0.785398163 0"/>
       <axis xyz="0 -1 0"/>
-      <limit effort="1000.0" lower="-0.4974" upper="1.8588" velocity="10.0"/>
+      <limit effort="0.0" lower="-0.4974" upper="1.8588" velocity="100.0"/>
       <dynamics damping="0.0" friction="0.0"/>
       <mimic joint="thigh_l_active" multiplier="-1" offset="0"/>
@@ -168,5 +168,5 @@
       <origin xyz="0 0 0" rpy="0 0.785398163 0"/>
       <axis xyz="0 -1 0"/>
-      <limit effort="1000.0" lower="-0.4974" upper="1.8588" velocity="10.0"/>
+      <limit effort="0.0" lower="-0.4974" upper="1.8588" velocity="100.0"/>
       <dynamics damping="0.0" friction="0.0"/>
       <mimic joint="shin_l_active" multiplier="1" offset="0"/>
@@ -187,5 +187,5 @@
       <origin xyz="-0.0335 0 0" rpy="0 0.785398163 0"/>
       <axis xyz="0 -1 0"/>
-      <limit effort="1000.0" lower="-0.4974" upper="1.8588" velocity="10.0"/>
+      <limit effort="0.0" lower="-0.4974" upper="1.8588" velocity="100.0"/>
       <dynamics damping="0.0" friction="0.0"/>
       <mimic joint="shin_l_active" multiplier="1" offset="0"/>
@@ -210,5 +210,5 @@
       <origin xyz="0 0 -0.1" rpy="0 -0.785398163 0"/>
       <axis xyz="0 -1 0"/>
-      <limit effort="1000.0" lower="-1.8588" upper="0.4974" velocity="10.0"/>
+      <limit effort="0.0" lower="-1.8588" upper="0.4974" velocity="100.0"/>
       <dynamics damping="0.0" friction="0.0"/>
       <mimic joint="shin_l_active" multiplier="-1" offset="0"/>
@@ -230,6 +230,6 @@
       <origin xyz="-0.015 0 -0.027" rpy="0 0 0"/>
       <axis xyz="1 0 0"/>
-      <limit effort="1000.0" lower="-1.5708" upper="0.3704" velocity="10.0"/>
-      <dynamics damping="0.0" friction="0.0"/>
+      <limit effort="3.1" lower="-1.5708" upper="0.3704" velocity="6.5"/>
+      <dynamics damping="0.4769" friction="0.0"/>
     </joint>
     <link name="ankle_l_roll_link">
@@ -249,6 +249,6 @@
       <origin xyz="0 0 -0.03825" rpy="0 0 0"/>
       <axis xyz="0 0 -1"/>
-      <limit effort="1000.0" lower="-3.1" upper="3.1" velocity="10.0"/>
-      <dynamics damping="0.0" friction="0.0"/>
+      <limit effort="3.1" lower="-3.1" upper="3.1" velocity="6.5"/>
+      <dynamics damping="0.4769" friction="0.0"/>
     </joint>
     <link name="ankle_l_yaw_link">

Commit message: WIP

File: kuroko_description/xacro/export/kuroko.urdf (robot description, URDF)
Before this commit: robot kuroko, 42 links, 41 joints
Links:
- removed link thigh_l_rear_passive_mimic_link
- removed link thigh_r_rear_passive_mimic_link
Joints:
- removed joint thigh_l_rear_passive_mimic
- removed joint thigh_r_rear_passive_mimic
- joint ankle_l_pitch_passive: limit lower=-1.8588 upper=0.4974 effort=1000.0 velocity=10.0 -> lower=-1.8588 upper=0.4974 effort=0.0 velocity=100.0
- joint ankle_l_roll: limit lower=-1.5708 upper=0.3704 effort=1000.0 velocity=10.0 -> lower=-1.5708 upper=0.3704 effort=3.1 velocity=6.5
- joint ankle_l_yaw: limit lower=-3.1 upper=3.1 effort=1000.0 velocity=10.0 -> lower=-3.1 upper=3.1 effort=3.1 velocity=6.5
- joint hip_l_pitch: limit lower=-3.1 upper=3.1 effort=1000.0 velocity=10.0 -> lower=-3.1 upper=3.1 effort=3.1 velocity=6.9
- joint hip_l_roll: limit lower=-0.5550 upper=1.8640 effort=1000.0 velocity=10.0 -> lower=-0.5550 upper=1.8640 effort=3.1 velocity=6.5
- joint knee_l_passive: limit lower=-0.4974 upper=1.8588 effort=1000.0 velocity=10.0 -> lower=-0.4974 upper=1.8588 effort=0.0 velocity=100.0
- joint shin_l_active: limit lower=-0.4974 upper=1.8588 effort=1000.0 velocity=10.0 -> lower=-0.4974 upper=1.8588 effort=8.9 velocity=6.9
- joint shin_l_front_passive: limit lower=-0.4974 upper=1.8588 effort=1000.0 velocity=10.0 -> lower=-0.4974 upper=1.8588 effort=0.0 velocity=100.0
- joint shin_l_rear_passive: limit lower=-0.4974 upper=1.8588 effort=1000.0 velocity=10.0 -> lower=-0.4974 upper=1.8588 effort=0.0 velocity=100.0
- joint thigh_l_active: limit lower=-1.8588 upper=0.4974 effort=1000.0 velocity=10.0 -> lower=-1.8588 upper=0.4974 effort=8.9 velocity=6.9
- joint thigh_l_middle_passive: limit lower=-3.1 upper=3.1 effort=1000.0 velocity=10.0 -> lower=-3.1 upper=3.1 effort=0.0 velocity=10.0
- joint thigh_l_rear_passive: limit lower=-3.1 upper=3.1 effort=1000.0 velocity=10.0 -> lower=-1.5708 upper=0.9948 effort=0.0 velocity=100.0; mimic joint=thigh_l_active multiplier=1 offset=0 -> (none); origin xyz=0 0 0 rpy=0 0 0 -> xyz=0 0 -0.03 rpy=0 -1.832597551 0; parent thigh_l_rear_passive_mimic_link -> shin_l_active_link
- joint thigh_r_rear_passive: limit lower=-3.1 upper=3.1 effort=1000.0 velocity=10.0 -> lower=-0.9948 upper=1.5708 effort=1000.0 velocity=10.0; mimic joint=thigh_r_active multiplier=1 offset=0 -> (none); origin xyz=0 0 0 rpy=0 0 0 -> xyz=0 0 -0.03 rpy=0 -1.832597551 0; parent thigh_r_rear_passive_mimic_link -> shin_r_active_link

File: kuroko_description/xacro/kuroko/parts/body.xacro (robot description, xacro)
@@ -20,5 +20,5 @@
       <axis xyz="0 0 1"/>
       <limit effort="3.1" lower="-3.1" upper="3.1" velocity="6.5"/>
-      <dynamics damping="0.4769" friction="0.0"/>
+      <dynamics damping="4769.0" friction="0.0"/>
     </joint>
     <!-- chest -->
