Commit message: (WIP) Move files

File: kuroko_description/xacro/kuroko.xacro (robot description, xacro)
@@ -4,5 +4,6 @@
   <xacro:arg name="gazebo_motor_model" default="dc"/>
   <xacro:arg name="gazebo_hw_interface" default="position"/>
-  <xacro:property name="XACRO_DIR" value="$(cwd)/${xacro.abs_filename('..')}" />
+  <xacro:property name="XACRO_DIR" value="$(cwd)" />
+  <xacro:property name="MESH_DIR" value="$(cwd)/meshes" />
   <xacro:include filename="${XACRO_DIR}/physics/box_physics.xacro"/>
   <xacro:include filename="${XACRO_DIR}/physics/gazebo_passive_joint.xacro"/>

File: kuroko_description/xacro/kuroko/parts/arm_l.xacro (robot description, xacro)
@@ -1,5 +1,4 @@
 <?xml version="1.0"?>
 <robot xmlns:xacro="http://www.ros.org/wiki/xacro">
-  <xacro:property name="MESH_DIR" value="$(cwd)/${xacro.abs_filename('../../../meshes')}" />
   <xacro:macro name="arm_l_xacro">
     <!-- Link conencts from body. Shoulder first. -->

File: kuroko_description/xacro/kuroko/parts/arm_r.xacro (robot description, xacro)
@@ -1,5 +1,4 @@
 <?xml version="1.0"?>
 <robot xmlns:xacro="http://www.ros.org/wiki/xacro">
-  <xacro:property name="MESH_DIR" value="$(cwd)/${xacro.abs_filename('../../../meshes')}" />
   <xacro:macro name="arm_r_xacro">
     <!-- Link conencts from body. Shoulder first. -->

File: kuroko_description/xacro/kuroko/parts/body.xacro (robot description, xacro)
@@ -1,5 +1,4 @@
 <?xml version="1.0"?>
 <robot xmlns:xacro="http://www.ros.org/wiki/xacro">
-  <xacro:property name="MESH_DIR" value="$(cwd)/${xacro.abs_filename('../../../meshes')}" />
   <xacro:macro name="body_xacro">
     <!-- waist -->

File: kuroko_description/xacro/kuroko/parts/leg_l.xacro (robot description, xacro)
@@ -1,5 +1,4 @@
 <?xml version="1.0"?>
 <robot xmlns:xacro="http://www.ros.org/wiki/xacro">
-  <xacro:property name="MESH_DIR" value="$(cwd)/${xacro.abs_filename('../../../meshes')}" />
   <xacro:macro name="leg_l_xacro" params="gazebo:=false">
     <!-- Link conencts from body. Hip first. -->

File: kuroko_description/xacro/kuroko/parts/leg_r.xacro (robot description, xacro)
@@ -1,5 +1,4 @@
 <?xml version="1.0"?>
 <robot xmlns:xacro="http://www.ros.org/wiki/xacro">
-  <xacro:property name="MESH_DIR" value="$(cwd)/${xacro.abs_filename('../../../meshes')}" />
   <xacro:macro name="leg_r_xacro" params="gazebo:=false">
     <!-- Link conencts from body. Hip first. -->

Commit message: WIP

File: kuroko_description/xacro/kuroko.xacro (robot description, xacro)
@@ -4,6 +4,6 @@
   <xacro:arg name="gazebo_motor_model" default="dc"/>
   <xacro:arg name="gazebo_hw_interface" default="position"/>
-  <xacro:property name="XACRO_DIR" value="$(cwd)" />
-  <xacro:property name="MESH_DIR" value="$(cwd)/meshes" />
+  <xacro:property name="XACRO_DIR" value="$(find kuroko_description)/xacro" />
+  <xacro:property name="MESH_DIR" value="$(find kuroko_description)/xacro/meshes" />
   <xacro:include filename="${XACRO_DIR}/physics/box_physics.xacro"/>
   <xacro:include filename="${XACRO_DIR}/physics/gazebo_passive_joint.xacro"/>
