Commit message: Generate files

File: kuroko_description/xacro/kuroko/isaac_sim/export/kuroko.urdf (robot description, URDF)
Before this commit: robot kuroko, 46 links, 45 joints
Links:
- removed link shin_l_front_mimic_link
- removed link shin_l_rear_mimic_link
- removed link shin_r_front_mimic_link
- removed link shin_r_rear_mimic_link
- removed link thigh_l_rear_mimic_link
- removed link thigh_r_rear_mimic_link
- link shin_l_front_passive_link: geometry collision box size=0.014 0.0385 0.114; visual mesh filename=/home/nyx/lib/isaaclab/kuroko_ros/kuroko_description/meshes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
Joints:
- removed joint shin_l_front_mimic
- removed joint shin_l_rear_mimic
- removed joint shin_r_front_mimic
- removed joint shin_r_rear_mimic
- removed joint thigh_l_rear_mimic
- removed joint thigh_r_rear_mimic
- joint ankle_l_roll: limit lower=-1.5708 upper=0.3704 effort=1000.0 velocity=10.0 -> lower=-1.5708 upper=0.3704 effort=3.1 velocity=6.5
- joint ankle_l_yaw: limit lower=-3.1 upper=3.1 effort=1000.0 velocity=10.0 -> lower=-3.1416 upper=3.1416 effort=3.1 velocity=6.5
- joint ankle_r_roll: limit lower=-0.3704 upper=1.5708 effort=1000.0 velocity=10.0 -> lower=-0.3704 upper=1.5708 effort=3.1 velocity=6.5
- joint ankle_r_yaw: limit lower=-3.1 upper=3.1 effort=1000.0 velocity=10.0 -> lower=-3.1 upper=3.1 effort=3.1 velocity=6.5
- joint hip_r_pitch: limit lower=-3.1 upper=3.1 effort=1000.0 velocity=10.0 -> lower=-3.1 upper=3.1 effort=3.1 velocity=6.5
- joint hip_r_roll: limit lower=-0.5550 upper=1.8640 effort=1000.0 velocity=10.0 -> lower=-0.5550 upper=1.8640 effort=3.1 velocity=6.5
- joint shin_l_front_passive: limit lower=-3.1416 upper=3.1416 effort=0 velocity=1000 -> lower=-1.570796327 upper=0.9948 effort=0 velocity=1000.0; mimic joint=shin_l_active multiplier=-1 offset=0 -> (none); origin xyz=0 0 0 rpy=0 0.785398163 0 -> xyz=0 0 -0.1 rpy=0 1.570796327 0; parent shin_l_front_mimic_link -> thigh_l_active_link
- joint shin_l_rear_passive: limit lower=-3.1416 upper=3.1416 effort=0 velocity=1000 -> lower=-1.570796327 upper=0.9948 effort=0 velocity=1000.0; mimic joint=shin_l_active multiplier=-1 offset=0 -> (none); origin xyz=0 0 0 rpy=0 0.785398163 0 -> xyz=0 0 -0.1 rpy=0 1.570796327 0; parent shin_l_rear_mimic_link -> thigh_l_middle_passive_link
- joint shin_r_front_passive: limit lower=-3.1416 upper=3.1416 effort=0 velocity=1000 -> lower=-1.570796327 upper=0.9948 effort=0 velocity=1000.0; mimic joint=shin_r_active multiplier=1 offset=0 -> (none); origin xyz=0 0 0 rpy=0 0.785398163 0 -> xyz=0 0 -0.1 rpy=0 1.570796327 0; parent shin_r_front_mimic_link -> thigh_r_active_link
- joint shin_r_rear_passive: limit lower=-3.1416 upper=3.1416 effort=0 velocity=1000 -> lower=-1.570796327 upper=0.9948 effort=0 velocity=1000.0; mimic joint=shin_r_active multiplier=1 offset=0 -> (none); origin xyz=0 0 0 rpy=0 0.785398163 0 -> xyz=0 0 -0.1 rpy=0 1.570796327 0; parent shin_r_rear_mimic_link -> thigh_r_middle_passive_link
- joint thigh_l_rear_passive: limit lower=-3.1416 upper=3.1416 effort=0 velocity=1000 -> lower=-0.9948 upper=1.570796327 effort=0 velocity=1000.0; mimic joint=shin_l_active multiplier=1 offset=0 -> (none); origin xyz=0 0 0 rpy=0 -0.785398163 0 -> xyz=-0.00776457 0 -0.0289778 rpy=0 -1.570796327 0; parent thigh_l_rear_mimic_link -> shin_l_rear_passive_link
- joint thigh_r_rear_passive: limit lower=-3.1416 upper=3.1416 effort=0 velocity=1000 -> lower=-0.9948 upper=1.570796327 effort=0 velocity=1000.0; mimic joint=shin_r_active multiplier=-1 offset=0 -> (none); origin xyz=0 0 0 rpy=0 -0.785398163 0 -> xyz=-0.00776457 0 -0.0289778 rpy=0 -1.570796327 0; parent thigh_r_rear_mimic_link -> shin_r_rear_passive_link
